Commit message: roll ankle joint is not a problem (RBDL just complain but it works)

File: kangaroo_description/robots/kangaroo.urdf (robot description, URDF)
Before this commit: robot kangaroo, 24 links, 23 joints
Joints:
- joint leg_left_5_joint: axis -1 0 0 -> -0.93969 0 0.34202
- joint leg_right_5_joint: axis -1. 0 0. -> -0.93969 0 0.34202
