Commit message: Update URDF with new meshes and zero at crouched position

File: kangaroo_description/robots/kangaroo.urdf.xacro (robot description, xacro)
@@ -21,7 +21,7 @@
   <link name="base_link">
     <inertial>
-      <origin xyz="-0.089859 0.0001101 -0.029078" rpy="0 0 0" />
+      <origin xyz="-0.089879 0.00011011 -0.029078" rpy="0 0 0" />
       <mass value="3.0844" />
-      <inertia ixx="0.0036879" ixy="-2.038E-06" ixz="3.8713E-05"
+      <inertia ixx="0.0036879" ixy="-2.0377E-06" ixz="3.8713E-05"
         iyy="0.0020689" iyz="-1.5142E-06" izz="0.0045246" />
     </inertial>
@@ -32,5 +32,5 @@
       </geometry>
       <material name="">
-        <color rgba="0.25098 0.25098 0.25098 1" />
+        <color rgba="0.75294 0.75294 0.75294 1" />
       </material>
     </visual>
@@ -43,13 +43,13 @@
   </link>
   <xacro:kangaroo_leg side="left" reflect="1" parent="base_link">
-    <origin xyz="-0.01602 0.08 -0.0585" rpy="0 0 ${-22.5 *deg_to_rad}" />
+    <origin xyz="-0.01602 0.08 -0.0585" rpy="0 0 0" />
   </xacro:kangaroo_leg>
   <xacro:property name="deg_to_rad"       value="0.01745329251994329577" />
   <xacro:kangaroo_leg side="right" reflect="-1" parent="base_link">
-    <origin xyz="-0.01602 -0.08 -0.0585" rpy="0 0 ${-22.5 *deg_to_rad}" />
+    <origin xyz="-0.01602 -0.08 -0.0585" rpy="0 0 0" />
   </xacro:kangaroo_leg>
   <!-- Generic simulator_gazebo plugins -->
   <!-- <xacro:include filename="$(find kangaroo_description)/gazebo/gazebo.urdf.xacro" /> -->
   <!-- Materials for visualization -->
-  <!-- <xacro:include filename="$(find kangaroo_description)/urdf/materials.urdf.xacro" /> -->ah
+  <!-- <xacro:include filename="$(find kangaroo_description)/urdf/materials.urdf.xacro" /> -->
 </robot>

File: kangaroo_description/urdf/leg/leg.urdf.xacro (robot description, xacro)
@@ -5,5 +5,5 @@
   <xacro:property name="eps_radians"      value="0.008" /> <!-- 0.45deg -->
   <xacro:property name="eps_meters"       value="0.005" />
-  <xacro:property name="leg_1_min_pos"   value="${15.0 *deg_to_rad}" />
+  <xacro:property name="leg_1_min_pos"   value="${-15.0 *deg_to_rad}" />
   <xacro:property name="leg_1_max_pos"   value="${40.0 *deg_to_rad}" />
   <xacro:property name="leg_2_min_pos"   value="${-42.5 *deg_to_rad}" />
@@ -22,8 +22,7 @@
     <link name="leg_${side}_1_link">
       <inertial>
-        <origin xyz="0.046108 -0.00082663 0.0089763" rpy="0 0 0" />
-        <mass value="2.4995" />
-        <inertia ixx="0.0015118" ixy="${reflect * 8.833E-06}" ixz="${reflect * 2.1775E-05}"
-          iyy="0.0015488" iyz="${reflect * -1.9445E-05}" izz="0.0013611" />
+        <origin xyz="0.0461079574284527 -0.000826631128234001 0.00897630312181676" rpy="0 0 0" />
+        <mass value="2.49954419149183" />
+        <inertia ixx="0.00151181747940305" ixy="${reflect * 8.83298140320242E-06}" ixz="${reflect * 2.17752660615735E-05}" iyy="0.00154876023440654" iyz="${reflect * -1.94449871986378E-05}" izz="0.00136106613590181" />
       </inertial>
       <visual>
@@ -33,5 +32,5 @@
         </geometry>
         <material name="">
-          <color rgba="0.75294 0.75294 0.75294 1" />
+          <color rgba="0.752941176470588 0.752941176470588 0.752941176470588 1" />
         </material>
       </visual>
@@ -45,5 +44,5 @@
     <joint name="leg_${side}_1_joint" type="revolute">
       <xacro:insert_block name="origin"/>
-      <parent link="base_link" />
+      <parent link="${parent}" />
       <child link="leg_${side}_1_link" />
       <axis xyz="0 0 1" />
@@ -52,8 +51,8 @@
     <link name="leg_${side}_2_link">
       <inertial>
-        <origin xyz="-0.00299642516878476 -0.000101293190038237 6.76272080002427E-10" rpy="0 0 0" />
+        <origin xyz="-0.00299642516878475 -0.000101293190038279 6.76277450706309E-10" rpy="0 0 0" />
         <mass value="0.0907287903783648" />
-        <inertia ixx="6.10402208807908E-06" ixy="${reflect * 3.54403077254808E-08}" ixz="${reflect * -3.09102931154027E-13}"
-          iyy="3.90470919341026E-05" iyz="${reflect * -1.14069181411126E-12}" izz="3.64238433670963E-05" />
+        <inertia ixx="6.10402208807908E-06" ixy="${reflect * 3.54403077254796E-08}" ixz="${reflect * -3.0910293306339E-13}"
+          iyy="3.90470919341026E-05" iyz="${reflect * -1.14069181428674E-12}" izz="3.64238433670963E-05" />
       </inertial>
       <visual>
@@ -82,8 +81,8 @@
     <link name="leg_${side}_3_link">
       <inertial>
-        <origin xyz="-0.0427914878682149 0.0477271416375379 -0.0411219974644161" rpy="0 0 0" />
-        <mass value="3.66987228133342" />
-        <inertia ixx="0.00226579366349613" ixy="${reflect * 0.000186528768977949}" ixz="${reflect * -9.44645206556725E-05}"
-          iyy="0.00347844172194194" iyz="${reflect * 4.48425081711929E-05}" izz="0.00335571078458133" />
+        <origin xyz="-0.042791492019428 0.0477271400490046 -0.0411219993940296" rpy="0 0 0" />
+        <mass value="3.66987205802361" />
+        <inertia ixx="0.00226579365890287" ixy="${reflect * 0.000186528466622377}" ixz="${reflect * -9.4464170720752E-05}"
+          iyy="0.00347844100338387" iyz="${reflect * 4.48424073671215E-05}" izz="0.00335571040406776" />
       </inertial>
       <visual>
@@ -112,8 +111,8 @@
     <link name="leg_${side}_4_link">
       <inertial>
-        <origin xyz="0.0531600041431671 0.000182667138322462 -0.148696920103582" rpy="0 0 0" />
-        <mass value="3.57413912348169" />
-        <inertia ixx="0.011509845839246" ixy="2.31593768751343E-05" ixz="0.00277647053237418"
-          iyy="0.0126050754047825" iyz="-1.96116832593457E-05" izz="0.00259389726745579" />
+        <origin xyz="0.114702002010089 0.000182856660852354 -0.0143986490691173" rpy="0 0 0" />
+        <mass value="3.57408268817521" />
+        <inertia ixx="0.00247170768644724" ixy="2.87874888621229E-05" ixz="0.00247469186737281"
+          iyy="0.0126050262407564" iyz="1.01404330133204E-05" izz="0.0116319632922522" />
       </inertial>
       <visual>
@@ -137,13 +136,13 @@
       <parent link="leg_${side}_3_link" />
       <child link="leg_${side}_4_link" />
-      <axis xyz="0 -1 0" />
+      <axis xyz="0 1 0" />
       <limit lower="${leg_4_min_pos}" upper="${leg_4_max_pos}" effort="0" velocity="0" />
     </joint>
     <link name="leg_${side}_5_link">
       <inertial>
-        <origin xyz="-0.0529041756836645 -8.15108495758055E-05 -0.137328569344222" rpy="0 0 0" />
-        <mass value="0.872279568157368" />
-        <inertia ixx="0.0021665932584343" ixy="-1.19083065331687E-07" ixz="-0.000583613527350316"
-          iyy="0.00242182628094296" iyz="8.06585633275114E-07" izz="0.000420858513123063" />
+        <origin xyz="-0.158662729273678 -8.28192764317226E-05 -0.0337468261967321" rpy="0 0 0" />
+        <mass value="0.87223211672797" />
+        <inertia ixx="0.000350603269949793" ixy="6.37793331536252E-07" ixz="-0.000461550351107159"
+          iyy="0.00242184402988972" iyz="5.09327556678297E-07" izz="0.0022368624903808" />
       </inertial>
       <visual>
@@ -164,16 +163,16 @@
     </link>
     <joint name="leg_${side}_5_joint" type="revolute">
-      <origin xyz="0.12996 0 -0.35709" rpy="0 0 0" />
+      <origin xyz="0.37413 0 -0.066509" rpy="0 0 0" />
       <parent link="leg_${side}_4_link" />
       <child link="leg_${side}_5_link" />
-      <axis xyz="0 1 0" />
+      <axis xyz="0 -1 0" />
       <limit lower="${leg_5_min_pos}" upper="${leg_5_max_pos}" effort="0" velocity="0" />
     </joint>
     <link name="leg_${side}_6_link">
       <inertial>
-        <origin xyz="-0.0071416033287726 4.83111717297646E-09 0.00259941265069108" rpy="0 0 0" />
-        <mass value="0.0905836559788969" />
-        <inertia ixx="7.07461991271068E-06" ixy="-1.86951000652729E-12" ixz="8.3028214389883E-06"
-          iyy="2.92762498059214E-05" iyz="1.82895645247132E-11" izz="2.68643074366888E-05" />
+        <origin xyz="-0.00714160332877733 4.8311277200952E-09 0.00259941265068991" rpy="0 0 0" />
+        <mass value="0.0905836559788966" />
+        <inertia ixx="7.07461991271062E-06" ixy="-1.86951004827933E-12" ixz="8.30282143898823E-06"
+          iyy="2.92762498059213E-05" iyz="1.82895645239997E-11" izz="2.68643074366886E-05" />
       </inertial>
       <visual>
@@ -194,5 +193,5 @@
     </link>
     <joint name="leg_${side}_6_joint" type="revolute">
-      <origin xyz="-0.12998 0 -0.35708" rpy="0 0 0" />
+      <origin xyz="-0.37432 0 -0.065464" rpy="0 0 0" />
       <parent link="leg_${side}_5_link" />
       <child link="leg_${side}_6_link" />
@@ -202,8 +201,8 @@
     <link name="leg_${side}_7_link">
       <inertial>
-        <origin xyz="0.0177425968295876 -3.68243086795172E-05 -0.0172694813829377" rpy="0 0 0" />
-        <mass value="0.394418123669799" />
-        <inertia ixx="0.000228382744880235" ixy="-2.56733548021984E-07" ixz="4.11795854076809E-05"
-          iyy="0.0010865368568379" iyz="7.8613236143388E-09" izz="0.00126437640745907" />
+        <origin xyz="0.0177425915954867 -3.67950153736807E-05 -0.0172694732454237" rpy="0 0 0" />
+        <mass value="0.394418327358563" />
+        <inertia ixx="0.000228382894016579" ixy="-2.56621760255351E-07" ixz="4.1179623691202E-05"
+          iyy="0.00108653696539759" iyz="7.85648127231571E-09" izz="0.0012643765698811" />
       </inertial>
       <visual>

Commit message: When enable crane option is parsed, use the world link rather than parsing up the crane model

File: kangaroo_description/robots/kangaroo.urdf.xacro (robot description, xacro)
@@ -8,7 +8,4 @@
         xmlns:controller="http://playerstage.sourceforge.net/gazebo/xmlschema/#controller"
         xmlns:interface="http://playerstage.sourceforge.net/gazebo/xmlschema/#interface">
-  <xacro:if value="$(arg enable_crane)">
-    <xacro:include filename="$(find kangaroo_description)/urdf/crane/crane.urdf.xacro" />
-  </xacro:if>
   <xacro:include filename="$(find kangaroo_description)/urdf/leg/leg.urdf.xacro" />
   <!--************************-->
@@ -39,5 +36,12 @@
   </link>
   <xacro:if value="$(arg enable_crane)">
-    <xacro:crane parent="base_link"/>
+    <!-- <xacro:include filename="$(find kangaroo_description)/urdf/crane/crane.urdf.xacro" /> -->
+    <!-- <xacro:crane parent="base_link"/> -->
+    <link name="world"/>
+    <joint name="world_base_link" type="fixed">
+      <origin xyz="0.0 0.0 1.2" rpy="0.0  0.0  0.0"/>
+      <parent link="world" />
+      <child link="base_link" />
+    </joint>
   </xacro:if>
   <xacro:kangaroo_leg side="left" reflect="1" parent="base_link">

Commit message: Use only one file for both leg type with conditionnal blocks

File: kangaroo_description/robots/kangaroo.urdf.xacro (robot description, xacro)
@@ -8,10 +8,4 @@
         xmlns:controller="http://playerstage.sourceforge.net/gazebo/xmlschema/#controller"
         xmlns:interface="http://playerstage.sourceforge.net/gazebo/xmlschema/#interface">
-  <xacro:if value="$(arg prismatic)">
-  	<xacro:include filename="$(find kangaroo_description)/urdf/leg/leg_prismatic.urdf.xacro" />
-  </xacro:if>
-  <xacro:unless value="$(arg prismatic)">
-  	<xacro:include filename="$(find kangaroo_description)/urdf/leg/leg.urdf.xacro" />
-  </xacro:unless>
   <!--************************-->
   <!--        BASE_LINK       -->
@@ -50,9 +44,16 @@
     </joint>
   </xacro:if>
-  <xacro:kangaroo_leg side="left" reflect="1" parent="base_link" simulation="$(arg simulation)">
+  <xacro:include filename="$(find kangaroo_description)/urdf/leg/leg.urdf.xacro" />
+	<xacro:if value="$(arg prismatic)">
+  	<xacro:property name="leg_type"       value="prismatic" />
+  </xacro:if>
+	<xacro:unless value="$(arg prismatic)">
+  	<xacro:property name="leg_type"       value="dynamic" />
+  </xacro:unless>
+  <xacro:kangaroo_leg side="left" reflect="1" parent="base_link" simulation="$(arg simulation)" type="${leg_type}">
     <origin xyz="-0.01602 0.08 -0.0585" rpy="0 0 0" />
   </xacro:kangaroo_leg>
   <xacro:property name="deg_to_rad"       value="0.01745329251994329577" />
-  <xacro:kangaroo_leg side="right" reflect="-1" parent="base_link" simulation="$(arg simulation)">
+  <xacro:kangaroo_leg side="right" reflect="-1" parent="base_link" simulation="$(arg simulation)" type="${leg_type}">
     <origin xyz="-0.01602 -0.08 -0.0585" rpy="0 0 0" />
   </xacro:kangaroo_leg>

File: kangaroo_description/urdf/leg/leg.urdf.xacro (robot description, xacro)
@@ -113,67 +113,133 @@
       <limit lower="${leg_3_min_pos}" upper="${leg_3_max_pos}" effort="100" velocity="3.87" />
     </joint>
-    <link name="leg_${side}_4_link">
-      <inertial>
-        <origin xyz="0.114702002010089 0.000182856660852354 -0.0143986490691173" rpy="0 0 0" />
-        <mass value="3.57408268817521" />
-        <inertia ixx="0.00247170768644724" ixy="2.87874888621229E-05" ixz="0.00247469186737281"
-          iyy="0.0126050262407564" iyz="1.01404330133204E-05" izz="0.0116319632922522" />
-      </inertial>
-      <visual>
-        <origin xyz="0 0 0" rpy="0 0 0" />
-        <geometry>
-          <mesh filename="package://kangaroo_description/meshes/leg_4_link.stl" />
-        </geometry>
-        <material name="">
-          <color rgba="0.752941176470588 0.752941176470588 0.752941176470588 1" />
-        </material>
-      </visual>
-      <collision>
-        <origin xyz="0 0 0" rpy="0 0 0" />
-        <geometry>
-          <mesh filename="package://kangaroo_description/meshes/leg_4_link.stl" />
-        </geometry>
-      </collision>
-    </link>
-    <joint name="leg_${side}_4_joint" type="revolute">
-      <origin xyz="0 ${reflect * 0.0669} -0.09" rpy="0 ${-10.0 * deg_to_rad} 0" />
-      <parent link="leg_${side}_3_link" />
-      <child link="leg_${side}_4_link" />
-      <axis xyz="0 1 0" />
-      <limit lower="${leg_4_min_pos}" upper="${leg_4_max_pos}" effort="100" velocity="3.87" />
-    </joint>
-    <link name="leg_${side}_5_link">
-      <inertial>
-        <origin xyz="-0.158662729273678 -8.28192764317226E-05 -0.0337468261967321" rpy="0 0 0" />
-        <mass value="0.87223211672797" />
-        <inertia ixx="0.000350603269949793" ixy="6.37793331536252E-07" ixz="-0.000461550351107159"
-          iyy="0.00242184402988972" iyz="5.09327556678297E-07" izz="0.0022368624903808" />
-      </inertial>
-      <visual>
-        <origin xyz="0 0 0" rpy="0 0 0" />
-        <geometry>
-          <mesh filename="package://kangaroo_description/meshes/leg_5_link.stl" />
-        </geometry>
-        <material name="">
-          <color rgba="0.752941176470588 0.752941176470588 0.752941176470588 1" />
-        </material>
-      </visual>
-      <collision>
-        <origin xyz="0 0 0" rpy="0 0 0" />
-        <geometry>
-          <mesh filename="package://kangaroo_description/meshes/leg_5_link.stl" />
-        </geometry>
-      </collision>
-    </link>
-    <joint name="leg_${side}_5_joint" type="revolute">
-      <origin xyz="0.37413 0 -0.066509" rpy="0 ${20.0 * deg_to_rad} 0" />
-      <parent link="leg_${side}_4_link" />
-      <child link="leg_${side}_5_link" />
-      <axis xyz="0 -1 0" />
-      <limit lower="${leg_5_min_pos}" upper="${leg_5_max_pos}" effort="100" velocity="3.87" />
-    </joint>
+    <xacro:unless value="${type=='prismatic'}" > <!-- load the model with both joints (hip and knee)-->
+		  <link name="leg_${side}_4_link">
+		    <inertial>
+		      <origin xyz="0.114702002010089 0.000182856660852354 -0.0143986490691173" rpy="0 0 0" />
+		      <mass value="3.57408268817521" />
+		      <inertia ixx="0.00247170768644724" ixy="2.87874888621229E-05" ixz="0.00247469186737281"
+		        iyy="0.0126050262407564" iyz="1.01404330133204E-05" izz="0.0116319632922522" />
+		    </inertial>
+		    <visual>
+		      <origin xyz="0 0 0" rpy="0 0 0" />
+		      <geometry>
+		        <mesh filename="package://kangaroo_description/meshes/leg_4_link.stl" />
+		      </geometry>
+		      <material name="">
+		        <color rgba="0.752941176470588 0.752941176470588 0.752941176470588 1" />
+		      </material>
+		    </visual>
+		    <collision>
+		      <origin xyz="0 0 0" rpy="0 0 0" />
+		      <geometry>
+		        <mesh filename="package://kangaroo_description/meshes/leg_4_link.stl" />
+		      </geometry>
+		    </collision>
+		  </link>
+		  <joint name="leg_${side}_4_joint" type="revolute">
+		    <origin xyz="0 ${reflect * 0.0669} -0.09" rpy="0 ${-10.0 * deg_to_rad} 0" />
+		    <parent link="leg_${side}_3_link" />
+		    <child link="leg_${side}_4_link" />
+		    <axis xyz="0 1 0" />
+		    <limit lower="${leg_4_min_pos}" upper="${leg_4_max_pos}" effort="100" velocity="3.87" />
+		  </joint>
+		  <link name="leg_${side}_5_link">
+		    <inertial>
+		      <origin xyz="-0.158662729273678 -8.28192764317226E-05 -0.0337468261967321" rpy="0 0 0" />
+		      <mass value="0.87223211672797" />
+		      <inertia ixx="0.000350603269949793" ixy="6.37793331536252E-07" ixz="-0.000461550351107159"
+		        iyy="0.00242184402988972" iyz="5.09327556678297E-07" izz="0.0022368624903808" />
+		    </inertial>
+		    <visual>
+		      <origin xyz="0 0 0" rpy="0 0 0" />
+		      <geometry>
+		        <mesh filename="package://kangaroo_description/meshes/leg_5_link.stl" />
+		      </geometry>
+		      <material name="">
+		        <color rgba="0.752941176470588 0.752941176470588 0.752941176470588 1" />
+		      </material>
+		    </visual>
+		    <collision>
+		      <origin xyz="0 0 0" rpy="0 0 0" />
+		      <geometry>
+		        <mesh filename="package://kangaroo_description/meshes/leg_5_link.stl" />
+		      </geometry>
+		    </collision>
+		  </link>
+		  <joint name="leg_${side}_5_joint" type="revolute">
+		    <origin xyz="0.37413 0 -0.066509" rpy="0 ${20.0 * deg_to_rad} 0" />
+		    <parent link="leg_${side}_4_link" />
+		    <child link="leg_${side}_5_link" />
+		    <axis xyz="0 -1 0" />
+		    <limit lower="${leg_5_min_pos}" upper="${leg_5_max_pos}" effort="100" velocity="3.87" />
+		  </joint>
+    </xacro:unless>
+    <xacro:if value="${type=='prismatic'}" > <!-- load the model with the leg lenght prismatic joint-->
+			 <link name="leg_${side}_4_link">
+		    <inertial>
+		      <origin rpy="0 0 0" xyz="0.0 0.0 ${leg_min_length/2.0}"/>
+					<!-- TODO: update inertia and mass -->
+		      <mass value="3.57408268817521" />
+		      <inertia ixx="0.00247170768644724" ixy="2.87874888621229E-05" ixz="0.00247469186737281"
+		        iyy="0.0126050262407564" iyz="1.01404330133204E-05" izz="0.0116319632922522" />
+		    </inertial>
+		    <visual>
+		      <origin rpy="0 0 0" xyz="0 0 ${leg_min_length/2.0}"/>
+		      <geometry>
+		        <cylinder length="${leg_min_length}" radius="0.02"/>
+		      </geometry>
+		      <material name="DarkGrey" />
+		    </visual>
+		    <collision>
+		      <origin rpy="0 0 0" xyz="0 0 ${leg_min_length/2.0}"/>
+		      <geometry>
+		        <cylinder length="${leg_min_length}" radius="0.02"/>
+		      </geometry>
+		    </collision>
+		  </link>
+		  <joint name="leg_${side}_length_fixed_joint" type="fixed">
+		    <origin xyz="0 ${reflect * 0.0669} -0.09" rpy="0 ${180 * deg_to_rad} 0" />
+		    <parent link="leg_${side}_3_link" />
+		    <child link="leg_${side}_4_link" />
+		    <axis xyz="0 0 1" />
+		  </joint>
+		  <link name="leg_${side}_5_link">
+		    <inertial>
+		      <origin rpy="0 0 0" xyz="0.0 0.0 ${-leg_min_length}"/>
+					<!-- TODO: update inertia and mass -->
+		      <mass value="0.87223211672797" />
+		      <inertia ixx="0.000350603269949793" ixy="6.37793331536252E-07" ixz="-0.000461550351107159"
+		        iyy="0.00242184402988972" iyz="5.09327556678297E-07" izz="0.0022368624903808" />
+		    </inertial>
+		    <visual>
+		      <origin rpy="0 0 0" xyz="0 0 ${(leg_min_length - leg_max_length)/2}"/>
+		      <geometry>
+		        <cylinder length="${(leg_max_length - leg_min_length)}" radius="0.02"/>
+		      </geometry>
+		      <material name="DarkGrey" />
+		    </visual>
+		    <!--<collision>
+		      <origin rpy="0 0 0" xyz="0 0 ${(leg_min_length - leg_max_length)/2}"/>
+		      <geometry>
+		        <cylinder length="${(leg_min_length - leg_max_length)}" radius="0.02"/>
+		      </geometry>
+		    </collision> -->
+		  </link>
+		  <joint name="leg_${side}_5_joint" type="prismatic">
+		   <origin xyz="0.0 0.0 ${leg_min_length}"  rpy="0.0 0.0 0.0"/>
+		    <parent link="leg_${side}_4_link" />
+		    <child link="leg_${side}_5_link" />
+		    <axis xyz="0 0 1" />
+		    <limit lower="0" upper="${leg_max_length - leg_min_length}" effort="100" velocity="10" /> <!-- TODO: update effort and velocity -->
+		  </joint>
+    </xacro:if>
     <xacro:if value="${type=='dynamic'}" >
       <xacro:kangaroo_ankle side="${side}" parent="leg_${side}_5_link" reflect="${reflect}" roll_joint="7" pitch_joint="6" read_actuator="leg_${side}_length_motor">
         <origin xyz="-0.37432 0 -0.065464" rpy="0 0 0" />
+      </xacro:kangaroo_ankle>
+    </xacro:if>
+    <xacro:if value="${type=='prismatic'}" >
+      <xacro:kangaroo_ankle side="${side}" parent="leg_${side}_5_link" reflect="${reflect}" roll_joint="7" pitch_joint="6" read_actuator="leg_${side}_length_motor">
+        <origin xyz="0. 0 -0." rpy="0 ${180 * deg_to_rad} 0" />
       </xacro:kangaroo_ankle>
     </xacro:if>
@@ -184,5 +250,5 @@
     </xacro:unless>
     <xacro:if value="${simulation}">
-      <xacro:kangaroo_lower_body_simple_simulation_transmission side="${side}"/>
+      <xacro:kangaroo_lower_body_simple_simulation_transmission side="${side}" prismatic="${type=='prismatic'}"/>
     </xacro:if>
    <gazebo reference="leg_${side}_1_link">
