Commit message: replace tabs by spaces in the files

File: kangaroo_description/robots/kangaroo.urdf.xacro (robot description, xacro)
@@ -47,9 +47,9 @@
   </xacro:if>
   <xacro:include filename="$(find kangaroo_description)/urdf/leg/leg.urdf.xacro" />
-	<xacro:if value="$(arg prismatic)">
-  	<xacro:property name="leg_type"       value="prismatic" />
+  <xacro:if value="$(arg prismatic)">
+    <xacro:property name="leg_type"       value="prismatic" />
   </xacro:if>
-	<xacro:unless value="$(arg prismatic)">
-  	<xacro:property name="leg_type"       value="dynamic" />
+  <xacro:unless value="$(arg prismatic)">
+    <xacro:property name="leg_type"       value="dynamic" />
   </xacro:unless>
   <xacro:kangaroo_leg side="left" reflect="1" parent="base_link" simulation="$(arg simulation)" type="${leg_type}">

File: kangaroo_description/urdf/leg/leg.urdf.xacro (robot description, xacro)
@@ -114,123 +114,123 @@
     </joint>
     <xacro:unless value="${type=='prismatic'}" > <!-- load the model with both joints (hip and knee)-->
-		  <link name="leg_${side}_4_link">
-		    <inertial>
-		      <origin xyz="0.114702002010089 0.000182856660852354 -0.0143986490691173" rpy="0 0 0" />
-		      <mass value="3.57408268817521" />
-		      <inertia ixx="0.00247170768644724" ixy="2.87874888621229E-05" ixz="0.00247469186737281"
-		        iyy="0.0126050262407564" iyz="1.01404330133204E-05" izz="0.0116319632922522" />
-		    </inertial>
-		    <visual>
-		      <origin xyz="0 0 0" rpy="0 0 0" />
-		      <geometry>
-		        <mesh filename="package://kangaroo_description/meshes/leg_4_link.stl" />
-		      </geometry>
-		      <material name="">
-		        <color rgba="0.752941176470588 0.752941176470588 0.752941176470588 1" />
-		      </material>
-		    </visual>
-		    <collision>
-		      <origin xyz="0 0 0" rpy="0 0 0" />
-		      <geometry>
-		        <mesh filename="package://kangaroo_description/meshes/leg_4_link.stl" />
-		      </geometry>
-		    </collision>
-		  </link>
-		  <joint name="leg_${side}_4_joint" type="revolute">
-		    <origin xyz="0 ${reflect * 0.0669} -0.09" rpy="0 ${-10.0 * deg_to_rad} 0" />
-		    <parent link="leg_${side}_3_link" />
-		    <child link="leg_${side}_4_link" />
-		    <axis xyz="0 1 0" />
-		    <limit lower="${leg_4_min_pos}" upper="${leg_4_max_pos}" effort="100" velocity="3.87" />
-		  </joint>
-		  <link name="leg_${side}_5_link">
-		    <inertial>
-		      <origin xyz="-0.158662729273678 -8.28192764317226E-05 -0.0337468261967321" rpy="0 0 0" />
-		      <mass value="0.87223211672797" />
-		      <inertia ixx="0.000350603269949793" ixy="6.37793331536252E-07" ixz="-0.000461550351107159"
-		        iyy="0.00242184402988972" iyz="5.09327556678297E-07" izz="0.0022368624903808" />
-		    </inertial>
-		    <visual>
-		      <origin xyz="0 0 0" rpy="0 0 0" />
-		      <geometry>
-		        <mesh filename="package://kangaroo_description/meshes/leg_5_link.stl" />
-		      </geometry>
-		      <material name="">
-		        <color rgba="0.752941176470588 0.752941176470588 0.752941176470588 1" />
-		      </material>
-		    </visual>
-		    <collision>
-		      <origin xyz="0 0 0" rpy="0 0 0" />
-		      <geometry>
-		        <mesh filename="package://kangaroo_description/meshes/leg_5_link.stl" />
-		      </geometry>
-		    </collision>
-		  </link>
-		  <joint name="leg_${side}_5_joint" type="revolute">
-		    <origin xyz="0.37413 0 -0.066509" rpy="0 ${20.0 * deg_to_rad} 0" />
-		    <parent link="leg_${side}_4_link" />
-		    <child link="leg_${side}_5_link" />
-		    <axis xyz="0 -1 0" />
-		    <limit lower="${leg_5_min_pos}" upper="${leg_5_max_pos}" effort="100" velocity="3.87" />
-		  </joint>
+      <link name="leg_${side}_4_link">
+        <inertial>
+          <origin xyz="0.114702002010089 0.000182856660852354 -0.0143986490691173" rpy="0 0 0" />
+          <mass value="3.57408268817521" />
+          <inertia ixx="0.00247170768644724" ixy="2.87874888621229E-05" ixz="0.00247469186737281"
+            iyy="0.0126050262407564" iyz="1.01404330133204E-05" izz="0.0116319632922522" />
+        </inertial>
+        <visual>
+          <origin xyz="0 0 0" rpy="0 0 0" />
+          <geometry>
+            <mesh filename="package://kangaroo_description/meshes/leg_4_link.stl" />
+          </geometry>
+          <material name="">
+            <color rgba="0.752941176470588 0.752941176470588 0.752941176470588 1" />
+          </material>
+        </visual>
+        <collision>
+          <origin xyz="0 0 0" rpy="0 0 0" />
+          <geometry>
+            <mesh filename="package://kangaroo_description/meshes/leg_4_link.stl" />
+          </geometry>
+        </collision>
+      </link>
+      <joint name="leg_${side}_4_joint" type="revolute">
+        <origin xyz="0 ${reflect * 0.0669} -0.09" rpy="0 ${-10.0 * deg_to_rad} 0" />
+        <parent link="leg_${side}_3_link" />
+        <child link="leg_${side}_4_link" />
+        <axis xyz="0 1 0" />
+        <limit lower="${leg_4_min_pos}" upper="${leg_4_max_pos}" effort="100" velocity="3.87" />
+      </joint>
+      <link name="leg_${side}_5_link">
+        <inertial>
+          <origin xyz="-0.158662729273678 -8.28192764317226E-05 -0.0337468261967321" rpy="0 0 0" />
+          <mass value="0.87223211672797" />
+          <inertia ixx="0.000350603269949793" ixy="6.37793331536252E-07" ixz="-0.000461550351107159"
+            iyy="0.00242184402988972" iyz="5.09327556678297E-07" izz="0.0022368624903808" />
+        </inertial>
+        <visual>
+          <origin xyz="0 0 0" rpy="0 0 0" />
+          <geometry>
+            <mesh filename="package://kangaroo_description/meshes/leg_5_link.stl" />
+          </geometry>
+          <material name="">
+            <color rgba="0.752941176470588 0.752941176470588 0.752941176470588 1" />
+          </material>
+        </visual>
+        <collision>
+          <origin xyz="0 0 0" rpy="0 0 0" />
+          <geometry>
+            <mesh filename="package://kangaroo_description/meshes/leg_5_link.stl" />
+          </geometry>
+        </collision>
+      </link>
+      <joint name="leg_${side}_5_joint" type="revolute">
+        <origin xyz="0.37413 0 -0.066509" rpy="0 ${20.0 * deg_to_rad} 0" />
+        <parent link="leg_${side}_4_link" />
+        <child link="leg_${side}_5_link" />
+        <axis xyz="0 -1 0" />
+        <limit lower="${leg_5_min_pos}" upper="${leg_5_max_pos}" effort="100" velocity="3.87" />
+      </joint>
     </xacro:unless>
     <xacro:if value="${type=='prismatic'}" > <!-- load the model with the leg length prismatic joint-->
-			 <link name="leg_${side}_length_fixed_link">
-		    <inertial>
-		      <origin rpy="0 0 0" xyz="0.0 0.0 ${-leg_min_length/2.0}"/>
-					<!-- TODO: update inertia and mass -->
-		      <mass value="3.57408268817521" />
-		      <inertia ixx="0.00247170768644724" ixy="2.87874888621229E-05" ixz="0.00247469186737281"
-		        iyy="0.0126050262407564" iyz="1.01404330133204E-05" izz="0.0116319632922522" />
-		    </inertial>
-		    <visual>
-		      <origin rpy="0 0 0" xyz="0 0 ${-leg_min_length/2.0}"/>
-		      <geometry>
-		        <cylinder length="${leg_min_length}" radius="0.02"/>
-		      </geometry>
-		      <material name="DarkGrey" />
-		    </visual>
-		    <collision>
-		      <origin rpy="0 0 0" xyz="0 0 ${-leg_min_length/2.0}"/>
-		      <geometry>
-		        <cylinder length="${leg_min_length}" radius="0.02"/>
-		      </geometry>
-		    </collision>
-		  </link>
-		  <joint name="leg_${side}_length_fixed_joint" type="fixed">
-		    <origin xyz="0 ${reflect * 0.0669} -0.09" rpy="0 0 0" />
-		    <parent link="leg_${side}_3_link" />
-		    <child link="leg_${side}_length_fixed_link" />
-		    <axis xyz="0 0 0" />
-		  </joint>
-		  <link name="leg_${side}_4_link">
-		    <inertial>
-		      <origin rpy="0 0 0" xyz="0.0 0.0 ${(leg_max_length - leg_min_length)/2}"/>
-					<!-- TODO: update inertia and mass -->
-		      <mass value="0.87223211672797" />
-		      <inertia ixx="0.000350603269949793" ixy="6.37793331536252E-07" ixz="-0.000461550351107159"
-		        iyy="0.00242184402988972" iyz="5.09327556678297E-07" izz="0.0022368624903808" />
-		    </inertial>
-		    <visual>
-		      <origin rpy="0 0 0" xyz="0 0 ${(leg_max_length - leg_min_length)/2}"/>
-		      <geometry>
-		        <cylinder length="${(leg_max_length - leg_min_length)}" radius="0.02"/>
-		      </geometry>
-		      <material name="DarkGrey" />
-		    </visual>
-		    <!--<collision>
-		      <origin rpy="0 0 0" xyz="0 0 ${(leg_min_length - leg_max_length)/2}"/>
-		      <geometry>
-		        <cylinder length="${(leg_min_length - leg_max_length)}" radius="0.02"/>
-		      </geometry>
-		    </collision> -->
-		  </link>
-		  <joint name="leg_${side}_4_joint" type="prismatic">
-		   <origin xyz="0.0 0.0 ${-leg_min_length}"  rpy="0.0 0.0 0.0"/>
-		    <parent link="leg_${side}_length_fixed_link" />
-		    <child link="leg_${side}_4_link" />
-		    <axis xyz="0 0 -1" />
-		    <limit lower="0" upper="${leg_max_length - leg_min_length}" effort="100" velocity="10" /> <!-- TODO: update effort and velocity -->
-		  </joint>
+       <link name="leg_${side}_length_fixed_link">
+        <inertial>
+          <origin rpy="0 0 0" xyz="0.0 0.0 ${-leg_min_length/2.0}"/>
+          <!-- TODO: update inertia and mass -->
+          <mass value="3.57408268817521" />
+          <inertia ixx="0.00247170768644724" ixy="2.87874888621229E-05" ixz="0.00247469186737281"
+            iyy="0.0126050262407564" iyz="1.01404330133204E-05" izz="0.0116319632922522" />
+        </inertial>
+        <visual>
+          <origin rpy="0 0 0" xyz="0 0 ${-leg_min_length/2.0}"/>
+          <geometry>
+            <cylinder length="${leg_min_length}" radius="0.02"/>
+          </geometry>
+          <material name="DarkGrey" />
+        </visual>
+        <collision>
+          <origin rpy="0 0 0" xyz="0 0 ${-leg_min_length/2.0}"/>
+          <geometry>
+            <cylinder length="${leg_min_length}" radius="0.02"/>
+          </geometry>
+        </collision>
+      </link>
+      <joint name="leg_${side}_length_fixed_joint" type="fixed">
+        <origin xyz="0 ${reflect * 0.0669} -0.09" rpy="0 0 0" />
+        <parent link="leg_${side}_3_link" />
+        <child link="leg_${side}_length_fixed_link" />
+        <axis xyz="0 0 0" />
+      </joint>
+      <link name="leg_${side}_4_link">
+        <inertial>
+          <origin rpy="0 0 0" xyz="0.0 0.0 ${(leg_max_length - leg_min_length)/2}"/>
+          <!-- TODO: update inertia and mass -->
+          <mass value="0.87223211672797" />
+          <inertia ixx="0.000350603269949793" ixy="6.37793331536252E-07" ixz="-0.000461550351107159"
+            iyy="0.00242184402988972" iyz="5.09327556678297E-07" izz="0.0022368624903808" />
+        </inertial>
+        <visual>
+          <origin rpy="0 0 0" xyz="0 0 ${(leg_max_length - leg_min_length)/2}"/>
+          <geometry>
+            <cylinder length="${(leg_max_length - leg_min_length)}" radius="0.02"/>
+          </geometry>
+          <material name="DarkGrey" />
+        </visual>
+        <!--<collision>
+          <origin rpy="0 0 0" xyz="0 0 ${(leg_min_length - leg_max_length)/2}"/>
+          <geometry>
+            <cylinder length="${(leg_min_length - leg_max_length)}" radius="0.02"/>
+          </geometry>
+        </collision> -->
+      </link>
+      <joint name="leg_${side}_4_joint" type="prismatic">
+       <origin xyz="0.0 0.0 ${-leg_min_length}"  rpy="0.0 0.0 0.0"/>
+        <parent link="leg_${side}_length_fixed_link" />
+        <child link="leg_${side}_4_link" />
+        <axis xyz="0 0 -1" />
+        <limit lower="0" upper="${leg_max_length - leg_min_length}" effort="100" velocity="10" /> <!-- TODO: update effort and velocity -->
+      </joint>
     </xacro:if>
     <xacro:if value="${type=='dynamic'}" >
@@ -265,8 +265,8 @@
    </gazebo>
    <xacro:if value="${type=='prismatic'}" >
-		 <gazebo reference="leg_${side}_length_fixed_link">
-		   <mu1>0.9</mu1>
-		   <mu2>0.9</mu2>
-		 </gazebo>
+     <gazebo reference="leg_${side}_length_fixed_link">
+       <mu1>0.9</mu1>
+       <mu2>0.9</mu2>
+     </gazebo>
    </xacro:if>
    <gazebo reference="leg_${side}_4_link">
@@ -275,8 +275,8 @@
    </gazebo>
    <xacro:unless value="${type=='prismatic'}" >
-		 <gazebo reference="leg_${side}_5_link">
-		   <mu1>0.9</mu1>
-		   <mu2>0.9</mu2>
-		 </gazebo>
+     <gazebo reference="leg_${side}_5_link">
+       <mu1>0.9</mu1>
+       <mu2>0.9</mu2>
+     </gazebo>
    </xacro:unless>
    <gazebo reference="leg_${side}_1_joint">
@@ -289,12 +289,12 @@
       <implicitSpringDamper>1</implicitSpringDamper>
    </gazebo>
-	 <gazebo reference="leg_${side}_4_joint">
-	    <implicitSpringDamper>1</implicitSpringDamper>
-	 </gazebo>
-	 <xacro:unless value="${type=='prismatic'}" >
-		 <gazebo reference="leg_${side}_5_joint">
-		    <implicitSpringDamper>1</implicitSpringDamper>
-		 </gazebo>
-	 </xacro:unless>
+   <gazebo reference="leg_${side}_4_joint">
+      <implicitSpringDamper>1</implicitSpringDamper>
+   </gazebo>
+   <xacro:unless value="${type=='prismatic'}" >
+     <gazebo reference="leg_${side}_5_joint">
+        <implicitSpringDamper>1</implicitSpringDamper>
+     </gazebo>
+   </xacro:unless>
   <gazebo reference="leg_${side}_1_link">
     <material>Gazebo/FlatWhite</material>

Commit message: Updated base_link information with torso meshes and data

File: kangaroo_description/robots/kangaroo.urdf.xacro (robot description, xacro)
@@ -13,8 +13,9 @@
   <link name="base_link">
     <inertial>
-      <origin xyz="-0.089879 0.00011011 -0.029078" rpy="0 0 0" />
-      <mass value="3.0844" />
-      <inertia ixx="0.0036879" ixy="-2.0377E-06" ixz="3.8713E-05"
-        iyy="0.0020689" iyz="-1.5142E-06" izz="0.0045246" />
+      <origin xyz="-0.078625 0.0016806 0.12164" rpy="0 0 0" />
+      <mass
+        value="8.3635" />
+      <inertia ixx="0.051463" ixy="-2.3239E-05" ixz="0.000993"
+        iyy="0.051275" iyz="7.7677E-05" izz="0.014591" />
     </inertial>
     <visual>
