Commit message: Update URDF to use the complex model (prismatic + dynamic model)

File: kangaroo_description/robots/kangaroo.urdf.xacro (robot description, xacro)
@@ -8,4 +8,5 @@
         xmlns:controller="http://playerstage.sourceforge.net/gazebo/xmlschema/#controller"
         xmlns:interface="http://playerstage.sourceforge.net/gazebo/xmlschema/#interface">
+  <xacro:property name="deg_to_rad"       value="0.01745329251994329577" />
   <!--************************-->
   <!--        BASE_LINK       -->
@@ -48,15 +49,8 @@
   </xacro:if>
   <xacro:include filename="$(find kangaroo_description)/urdf/leg/leg.urdf.xacro" />
-  <xacro:if value="$(arg prismatic)">
-    <xacro:property name="leg_type"       value="prismatic" />
-  </xacro:if>
-  <xacro:unless value="$(arg prismatic)">
-    <xacro:property name="leg_type"       value="dynamic" />
-  </xacro:unless>
-  <xacro:kangaroo_leg side="left" reflect="1" parent="base_link" simulation="$(arg simulation)" type="${leg_type}">
+  <xacro:kangaroo_leg side="left" reflect="1" parent="base_link" simulation="$(arg simulation)">
     <origin xyz="-0.01602 0.08 -0.0585" rpy="0 0 0" />
   </xacro:kangaroo_leg>
-  <xacro:property name="deg_to_rad"       value="0.01745329251994329577" />
-  <xacro:kangaroo_leg side="right" reflect="-1" parent="base_link" simulation="$(arg simulation)" type="${leg_type}">
+  <xacro:kangaroo_leg side="right" reflect="-1" parent="base_link" simulation="$(arg simulation)">
     <origin xyz="-0.01602 -0.08 -0.0585" rpy="0 0 0" />
   </xacro:kangaroo_leg>

File: kangaroo_description/urdf/leg/leg.transmission.xacro (robot description, xacro)
@@ -5,5 +5,5 @@
 -->
 <robot name="kangaroo" xmlns:xacro="http://ros.org/wiki/xacro">
-  <xacro:macro name="kangaroo_lower_body_simple_simulation_transmission" params="side prismatic">
+  <xacro:macro name="kangaroo_lower_body_simple_simulation_transmission" params="side">
     <transmission name="leg_${side}_1_transmission">
       <type>transmission_interface/SimpleTransmission</type>
@@ -62,20 +62,18 @@
       </joint>
     </transmission>
-    <xacro:unless value="$(arg prismatic)">
-      <transmission name="leg_${side}_5_transmission">
-        <type>transmission_interface/SimpleTransmission</type>
-        <actuator name="leg_${side}_5_motor" >
-          <hardwareInterface>hardware_interface/PositionJointInterface</hardwareInterface>
-          <hardwareInterface>hardware_interface/EffortJointInterface</hardwareInterface>
-          <hardwareInterface>hardware_interface/JointStateInterface</hardwareInterface>
-          <mechanicalReduction>1.0</mechanicalReduction>
-        </actuator>
-        <joint name="leg_${side}_5_joint">
-          <hardwareInterface>hardware_interface/PositionJointInterface</hardwareInterface>
-          <hardwareInterface>hardware_interface/EffortJointInterface</hardwareInterface>
-          <hardwareInterface>hardware_interface/JointStateInterface</hardwareInterface>
-        </joint>
-      </transmission>
-    </xacro:unless>
+    <transmission name="leg_${side}_5_transmission">
+      <type>transmission_interface/SimpleTransmission</type>
+      <actuator name="leg_${side}_5_motor" >
+        <hardwareInterface>hardware_interface/PositionJointInterface</hardwareInterface>
+        <hardwareInterface>hardware_interface/EffortJointInterface</hardwareInterface>
+        <hardwareInterface>hardware_interface/JointStateInterface</hardwareInterface>
+        <mechanicalReduction>1.0</mechanicalReduction>
+      </actuator>
+      <joint name="leg_${side}_5_joint">
+        <hardwareInterface>hardware_interface/PositionJointInterface</hardwareInterface>
+        <hardwareInterface>hardware_interface/EffortJointInterface</hardwareInterface>
+        <hardwareInterface>hardware_interface/JointStateInterface</hardwareInterface>
+      </joint>
+    </transmission>
   </xacro:macro>
   <xacro:macro name="kangaroo_leg_length_actuator_transmission" params="side number1 number2 params_ns:=/leg_params" >

File: kangaroo_description/urdf/leg/leg.urdf.xacro (robot description, xacro)
@@ -18,5 +18,5 @@
   <xacro:property name="leg_min_length"   value="0.131973" />
   <xacro:property name="leg_max_length"   value="0.71416639" />
-  <xacro:macro name="kangaroo_leg" params="side reflect parent *origin simulation:=false type:=dynamic">
+  <xacro:macro name="kangaroo_leg" params="side reflect parent *origin simulation:=false">
     <link name="leg_${side}_1_link">
       <inertial>
@@ -113,135 +113,125 @@
       <limit lower="${leg_3_min_pos}" upper="${leg_3_max_pos}" effort="100" velocity="3.87" />
     </joint>
-    <xacro:unless value="${type=='prismatic'}" > <!-- load the model with both joints (hip and knee)-->
-      <link name="leg_${side}_4_link">
-        <inertial>
-          <origin xyz="0.114702002010089 0.000182856660852354 -0.0143986490691173" rpy="0 0 0" />
-          <mass value="3.57408268817521" />
-          <inertia ixx="0.00247170768644724" ixy="2.87874888621229E-05" ixz="0.00247469186737281"
-            iyy="0.0126050262407564" iyz="1.01404330133204E-05" izz="0.0116319632922522" />
-        </inertial>
-        <visual>
-          <origin xyz="0 0 0" rpy="0 0 0" />
-          <geometry>
-            <mesh filename="package://kangaroo_description/meshes/leg_4_link.stl" />
-          </geometry>
-          <material name="">
-            <color rgba="0.752941176470588 0.752941176470588 0.752941176470588 1" />
-          </material>
-        </visual>
-        <collision>
-          <origin xyz="0 0 0" rpy="0 0 0" />
-          <geometry>
-            <mesh filename="package://kangaroo_description/meshes/leg_4_link.stl" />
-          </geometry>
-        </collision>
-      </link>
-      <joint name="leg_${side}_4_joint" type="revolute">
-        <origin xyz="0 ${reflect * 0.0669} -0.09" rpy="0 ${-10.0 * deg_to_rad} 0" />
-        <parent link="leg_${side}_3_link" />
-        <child link="leg_${side}_4_link" />
-        <axis xyz="0 1 0" />
-        <limit lower="${leg_4_min_pos}" upper="${leg_4_max_pos}" effort="100" velocity="3.87" />
-      </joint>
-      <link name="leg_${side}_5_link">
-        <inertial>
-          <origin xyz="-0.158662729273678 -8.28192764317226E-05 -0.0337468261967321" rpy="0 0 0" />
-          <mass value="0.87223211672797" />
-          <inertia ixx="0.000350603269949793" ixy="6.37793331536252E-07" ixz="-0.000461550351107159"
-            iyy="0.00242184402988972" iyz="5.09327556678297E-07" izz="0.0022368624903808" />
-        </inertial>
-        <visual>
-          <origin xyz="0 0 0" rpy="0 0 0" />
-          <geometry>
-            <mesh filename="package://kangaroo_description/meshes/leg_5_link.stl" />
-          </geometry>
-          <material name="">
-            <color rgba="0.752941176470588 0.752941176470588 0.752941176470588 1" />
-          </material>
-        </visual>
-        <collision>
-          <origin xyz="0 0 0" rpy="0 0 0" />
-          <geometry>
-            <mesh filename="package://kangaroo_description/meshes/leg_5_link.stl" />
-          </geometry>
-        </collision>
-      </link>
-      <joint name="leg_${side}_5_joint" type="revolute">
-        <origin xyz="0.37413 0 -0.066509" rpy="0 ${20.0 * deg_to_rad} 0" />
-        <parent link="leg_${side}_4_link" />
-        <child link="leg_${side}_5_link" />
-        <axis xyz="0 -1 0" />
-        <limit lower="${leg_5_min_pos}" upper="${leg_5_max_pos}" effort="100" velocity="3.87" />
-      </joint>
-    </xacro:unless>
-    <xacro:if value="${type=='prismatic'}" > <!-- load the model with the leg length prismatic joint-->
-       <link name="leg_${side}_length_fixed_link">
-        <inertial>
-          <origin rpy="0 0 0" xyz="0.0 0.0 ${-leg_min_length/2.0}"/>
-          <!-- TODO: update inertia and mass -->
-          <mass value="3.57408268817521" />
-          <inertia ixx="0.00247170768644724" ixy="2.87874888621229E-05" ixz="0.00247469186737281"
-            iyy="0.0126050262407564" iyz="1.01404330133204E-05" izz="0.0116319632922522" />
-        </inertial>
-        <visual>
-          <origin rpy="0 0 0" xyz="0 0 ${-leg_min_length/2.0}"/>
-          <geometry>
-            <cylinder length="${leg_min_length}" radius="0.02"/>
-          </geometry>
-          <material name="DarkGrey" />
-        </visual>
-        <!--<collision>
-          <origin rpy="0 0 0" xyz="0 0 ${-leg_min_length/2.0}"/>
-          <geometry>
-            <cylinder length="${leg_min_length}" radius="0.02"/>
-          </geometry>
-        </collision>-->
-      </link>
-      <joint name="leg_${side}_length_fixed_joint" type="fixed">
-        <origin xyz="0 ${reflect * 0.0669} -0.09" rpy="0 0 0" />
+    <link name="leg_${side}_4_link">
+      <inertial>
+        <origin xyz="0.114702002010089 0.000182856660852354 -0.0143986490691173" rpy="0 0 0" />
+        <mass value="3.57408268817521" />
+        <inertia ixx="0.00247170768644724" ixy="2.87874888621229E-05" ixz="0.00247469186737281"
+          iyy="0.0126050262407564" iyz="1.01404330133204E-05" izz="0.0116319632922522" />
+      </inertial>
+      <visual>
+        <origin xyz="0 0 0" rpy="0 0 0" />
+        <geometry>
+          <mesh filename="package://kangaroo_description/meshes/leg_4_link.stl" />
+        </geometry>
+        <material name="">
+          <color rgba="0.752941176470588 0.752941176470588 0.752941176470588 1" />
+        </material>
+      </visual>
+      <collision>
+        <origin xyz="0 0 0" rpy="0 0 0" />
+        <geometry>
+          <mesh filename="package://kangaroo_description/meshes/leg_4_link.stl" />
+        </geometry>
+      </collision>
+    </link>
+    <joint name="leg_${side}_4_joint" type="revolute">
+      <origin xyz="0 ${reflect * 0.0669} -0.09" rpy="0 ${-10.0 * deg_to_rad} 0" />
+      <parent link="leg_${side}_3_link" />
+      <child link="leg_${side}_4_link" />
+      <axis xyz="0 1 0" />
+      <limit lower="${leg_4_min_pos}" upper="${leg_4_max_pos}" effort="100" velocity="3.87" />
+    </joint>
+    <link name="leg_${side}_5_link">
+      <inertial>
+        <origin xyz="-0.158662729273678 -8.28192764317226E-05 -0.0337468261967321" rpy="0 0 0" />
+        <mass value="0.87223211672797" />
+        <inertia ixx="0.000350603269949793" ixy="6.37793331536252E-07" ixz="-0.000461550351107159"
+          iyy="0.00242184402988972" iyz="5.09327556678297E-07" izz="0.0022368624903808" />
+      </inertial>
+      <visual>
+        <origin xyz="0 0 0" rpy="0 0 0" />
+        <geometry>
+          <mesh filename="package://kangaroo_description/meshes/leg_5_link.stl" />
+        </geometry>
+        <material name="">
+          <color rgba="0.752941176470588 0.752941176470588 0.752941176470588 1" />
+        </material>
+      </visual>
+      <collision>
+        <origin xyz="0 0 0" rpy="0 0 0" />
+        <geometry>
+          <mesh filename="package://kangaroo_description/meshes/leg_5_link.stl" />
+        </geometry>
+      </collision>
+    </link>
+    <joint name="leg_${side}_5_joint" type="revolute">
+      <origin xyz="0.37413 0 -0.066509" rpy="0 ${20.0 * deg_to_rad} 0" />
+      <parent link="leg_${side}_4_link" />
+      <child link="leg_${side}_5_link" />
+      <axis xyz="0 -1 0" />
+      <limit lower="${leg_5_min_pos}" upper="${leg_5_max_pos}" effort="100" velocity="3.87" />
+    </joint>
+    <link name="leg_${side}_length_fixed_link">
+      <inertial>
+        <origin rpy="0 0 0" xyz="0.0 0.0 ${leg_min_length/2.0}"/>
+        <!-- TODO: update inertia and mass -->
+        <mass value="0.1"/>
+        <inertia ixx="0.04287677484" ixy="0.00043705397" ixz="0.00078292368"
+                iyy="0.03598906971" iyz="0.00037717694" izz="0.01364791564" />
+      </inertial>
+      <visual>
+        <origin rpy="0 0 0" xyz="0 0 ${leg_min_length/2.0}"/>
+        <geometry>
+          <cylinder length="${leg_min_length}" radius="0.00005"/>
+        </geometry>
+        <material name="DarkGrey" />
+      </visual>
+      <collision>
+        <origin rpy="0 0 0" xyz="0 0 ${leg_min_length/2.0}"/>
+        <geometry>
+          <cylinder length="${leg_min_length}" radius="0.00005"/>
+        </geometry>
+      </collision>
+    </link>
+    <joint name="leg_${side}_length_fixed_joint" type="fixed">
+        <origin xyz="0 ${reflect * 0.0669} -0.09" rpy="0 ${180.0 * deg_to_rad} 0" />
         <parent link="leg_${side}_3_link" />
         <child link="leg_${side}_length_fixed_link" />
         <axis xyz="0 0 0" />
-      </joint>
-      <link name="leg_${side}_4_link">
-        <inertial>
-          <origin rpy="0 0 0" xyz="0.0 0.0 ${(leg_max_length - leg_min_length)/2}"/>
-          <!-- TODO: update inertia and mass -->
-          <mass value="0.87223211672797" />
-          <inertia ixx="0.000350603269949793" ixy="6.37793331536252E-07" ixz="-0.000461550351107159"
-            iyy="0.00242184402988972" iyz="5.09327556678297E-07" izz="0.0022368624903808" />
-        </inertial>
-        <visual>
-          <origin rpy="0 0 0" xyz="0 0 ${(leg_max_length - leg_min_length)/2}"/>
-          <geometry>
-            <cylinder length="${(leg_max_length - leg_min_length)}" radius="0.02"/>
-          </geometry>
-          <material name="DarkGrey" />
-        </visual>
-        <!--<collision>
-          <origin rpy="0 0 0" xyz="0 0 ${(leg_min_length - leg_max_length)/2}"/>
-          <geometry>
-            <cylinder length="${(leg_min_length - leg_max_length)}" radius="0.02"/>
-          </geometry>
-        </collision> -->
-      </link>
-      <joint name="leg_${side}_4_joint" type="prismatic">
-       <origin xyz="0.0 0.0 ${-leg_min_length}"  rpy="0.0 0.0 0.0"/>
-        <parent link="leg_${side}_length_fixed_link" />
-        <child link="leg_${side}_4_link" />
-        <axis xyz="0 0 -1" />
-        <limit lower="0" upper="${leg_max_length - leg_min_length}" effort="500" velocity="10" /> <!-- TODO: update effort and velocity -->
-      </joint>
-    </xacro:if>
-    <xacro:if value="${type=='dynamic'}" >
-      <xacro:kangaroo_ankle side="${side}" parent="leg_${side}_5_link" reflect="${reflect}" roll_joint="7" pitch_joint="6" read_actuator="leg_${side}_length_motor">
-        <origin xyz="-0.37432 0 -0.065464" rpy="0 0 0" />
-      </xacro:kangaroo_ankle>
-    </xacro:if>
-    <xacro:if value="${type=='prismatic'}" >
-      <xacro:kangaroo_ankle side="${side}" parent="leg_${side}_4_link" reflect="${reflect}" roll_joint="6" pitch_joint="5" read_actuator="leg_${side}_length_motor">
-        <origin xyz="-0.02 0 0" rpy="0 0 0" />
-      </xacro:kangaroo_ankle>
-    </xacro:if>
+    </joint>
+    <link name="leg_${side}_length_link">
+      <inertial>
+        <origin rpy="0 0 0" xyz="0.0 0.0 ${(leg_max_length - leg_min_length)/2}"/>
+        <!-- TODO: update inertia and mass -->
+        <mass value="3.57408268817521" />
+        <inertia ixx="0.00247170768644724" ixy="2.87874888621229E-05" ixz="0.00247469186737281"
+          iyy="0.0126050262407564" iyz="1.01404330133204E-05" izz="0.0116319632922522" />
+      </inertial>
+      <visual>
+        <origin rpy="0 0 0" xyz="0 0 ${(leg_min_length - leg_max_length)/2}"/>
+        <geometry>
+          <cylinder length="${(leg_min_length - leg_max_length)}" radius="0.00005"/>
+        </geometry>
+        <material name="DarkGrey" />
+      </visual>
+      <collision>
+        <origin rpy="0 0 0" xyz="0 0 ${(leg_min_length - leg_max_length)/2}"/>
+        <geometry>
+          <cylinder length="${(leg_min_length - leg_max_length)}" radius="0.00005"/>
+        </geometry>
+      </collision>
+    </link>
+    <joint name="leg_${side}_length_joint" type="prismatic">
+     <origin xyz="0.0 0.0 ${leg_min_length}"  rpy="0.0 0.0 0.0"/>
+      <parent link="leg_${side}_length_fixed_link" />
+      <child link="leg_${side}_length_link" />
+      <axis xyz="0 0 1" />
+      <limit lower="0" upper="${leg_max_length - leg_min_length}" effort="500" velocity="10" /> <!-- TODO: update effort and velocity -->
+    </joint>
+    <xacro:kangaroo_ankle side="${side}" parent="leg_${side}_5_link" reflect="${reflect}" roll_joint="7" pitch_joint="6" read_actuator="leg_${side}_length_motor">
+      <origin xyz="-0.37432 0 -0.065464" rpy="0 0 0" />
+    </xacro:kangaroo_ankle>
+    <!-- Load corresponding transmission info -->
     <xacro:unless value="${simulation}">
       <xacro:hip_transmission_yaw side="${side}" number="1" reduction="1.0" />
@@ -250,5 +240,5 @@
     </xacro:unless>
     <xacro:if value="${simulation}">
-      <xacro:kangaroo_lower_body_simple_simulation_transmission side="${side}" prismatic="${type=='prismatic'}"/>
+      <xacro:kangaroo_lower_body_simple_simulation_transmission side="${side}"/>
     </xacro:if>
    <gazebo reference="leg_${side}_1_link">
@@ -264,20 +254,16 @@
      <mu2>0.9</mu2>
    </gazebo>
-   <xacro:if value="${type=='prismatic'}" >
-     <gazebo reference="leg_${side}_length_fixed_link">
-       <mu1>0.9</mu1>
-       <mu2>0.9</mu2>
-     </gazebo>
-   </xacro:if>
+   <gazebo reference="leg_${side}_length_link">
+     <mu1>0.9</mu1>
+     <mu2>0.9</mu2>
+   </gazebo>
    <gazebo reference="leg_${side}_4_link">
      <mu1>0.9</mu1>
      <mu2>0.9</mu2>
    </gazebo>
-   <xacro:unless value="${type=='prismatic'}" >
-     <gazebo reference="leg_${side}_5_link">
-       <mu1>0.9</mu1>
-       <mu2>0.9</mu2>
-     </gazebo>
-   </xacro:unless>
+   <gazebo reference="leg_${side}_5_link">
+     <mu1>0.9</mu1>
+     <mu2>0.9</mu2>
+   </gazebo>
    <gazebo reference="leg_${side}_1_joint">
       <implicitSpringDamper>1</implicitSpringDamper>
@@ -292,9 +278,10 @@
       <implicitSpringDamper>1</implicitSpringDamper>
    </gazebo>
-   <xacro:unless value="${type=='prismatic'}" >
-     <gazebo reference="leg_${side}_5_joint">
-        <implicitSpringDamper>1</implicitSpringDamper>
-     </gazebo>
-   </xacro:unless>
+   <gazebo reference="leg_${side}_5_joint">
+      <implicitSpringDamper>1</implicitSpringDamper>
+   </gazebo>
+   <gazebo reference="leg_${side}_length_link">
+      <implicitSpringDamper>1</implicitSpringDamper>
+   </gazebo>
   <gazebo reference="leg_${side}_1_link">
     <material>Gazebo/FlatWhite</material>
@@ -312,4 +299,7 @@
     <material>Gazebo/FlatBlack</material>
   </gazebo>
+  <gazebo reference="leg_${side}_length_link">
+    <material>Gazebo/FlatBlack</material>
+  </gazebo>
   </xacro:macro>
 </robot>

Commit message: Inertial modifcations for torso + base link

File: kangaroo_description/robots/kangaroo.urdf.xacro (robot description, xacro)
@@ -14,9 +14,8 @@
   <link name="base_link">
     <inertial>
-      <origin xyz="-0.078625 0.0016806 0.12164" rpy="0 0 0" />
-      <mass
-        value="8.3635" />
-      <inertia ixx="0.051463" ixy="-2.3239E-05" ixz="0.000993"
-        iyy="0.051275" iyz="7.7677E-05" izz="0.014591" />
+      <origin xyz="-0.060294 0.00050634 0.15428" rpy="0 0 0" />
+      <mass value="12.296" />
+      <inertia  ixx="0.084937" ixy="-4.4873E-05" ixz="0.0036119"
+        iyy="0.080587" iyz="0.0001781" izz="0.0247" />
     </inertial>
     <visual>

Commit message: Fix primatic model. Add IMU. Tune PIDS

File: kangaroo_description/robots/kangaroo.urdf.xacro (robot description, xacro)
@@ -9,4 +9,5 @@
         xmlns:interface="http://playerstage.sourceforge.net/gazebo/xmlschema/#interface">
   <xacro:property name="deg_to_rad"       value="0.01745329251994329577" />
+  <xacro:include filename="$(find kangaroo_description)/urdf/sensors/imu.urdf.xacro" />
   <!--************************-->
   <!--        BASE_LINK       -->
@@ -48,4 +49,7 @@
   </xacro:if>
   <xacro:include filename="$(find kangaroo_description)/urdf/leg/leg.urdf.xacro" />
+  <xacro:kangaroo_imu name="imu" parent="base_link" update_rate="100.0">
+    <origin xyz="0.0 0.0 0.0" rpy="${180.0*deg_to_rad} ${0.0*deg_to_rad} ${90.0*deg_to_rad}"/>
+  </xacro:kangaroo_imu>
   <xacro:kangaroo_leg side="left" reflect="1" parent="base_link" simulation="$(arg simulation)">
     <origin xyz="-0.01602 0.08 -0.0585" rpy="0 0 0" />

File: kangaroo_description/urdf/ankle/ankle.urdf.xacro (robot description, xacro)
@@ -63,4 +63,11 @@
       <limit lower="${roll_joint_min_pos}" upper="${roll_joint_max_pos}" effort="100" velocity="3.87" />
     </joint>
+    <link name="${side}_sole_link"/>
+    <joint name="${side}_sole_fix_joint" type="fixed">
+      <parent link="leg_${side}_${roll_joint}_link" />
+      <child link="${side}_sole_link" />
+      <origin xyz="0.0 0.0 -0.03" rpy="0 0 0" />
+      <axis xyz="1 0 0" />
+    </joint>
     <xacro:unless value="${simulation}">
       <xacro:kangaroo_ankle_transmission side="${side}" roll_joint="${roll_joint}" pitch_joint="${pitch_joint}" read_actuator="${read_actuator}" />

File: kangaroo_description/urdf/leg/leg.urdf.xacro (robot description, xacro)
@@ -166,5 +166,5 @@
         <origin rpy="0 0 0" xyz="0 0 ${(leg_min_length - leg_max_length)/2}"/>
         <geometry>
-          <cylinder length="${(leg_min_length - leg_max_length)}" radius="0.00005"/>
+          <cylinder length="${(leg_max_length - leg_min_length)}" radius="0.00005"/>
         </geometry>
         <material name="DarkGrey" />

File: kangaroo_description/urdf/sensors/imu.urdf.xacro (robot description, xacro)
@@ -7,8 +7,7 @@
   Creative Commons, 444 Castro Street, Suite 900, Mountain View, California, 94041, USA.
 -->
-<robot name="talos" xmlns:xacro="http://ros.org/wiki/xacro">
-  <xacro:macro name="talos_imu" params="name parent update_rate *origin">
+<robot name="kangaroo" xmlns:xacro="http://ros.org/wiki/xacro">
+  <xacro:macro name="kangaroo_imu" params="name parent update_rate *origin">
     <link name="${name}_link">
-      <xacro:call macro="${name}_link_inertial" />
       <visual>
         <origin rpy="0 0 0" xyz="0 0 0"/>

Commit message: Update imu transformation

File: kangaroo_description/robots/kangaroo.urdf.xacro (robot description, xacro)
@@ -50,5 +50,5 @@
   <xacro:include filename="$(find kangaroo_description)/urdf/leg/leg.urdf.xacro" />
   <xacro:kangaroo_imu name="imu" parent="base_link" update_rate="100.0">
-    <origin xyz="0.0 0.0 0.0" rpy="${180.0*deg_to_rad} ${0.0*deg_to_rad} ${90.0*deg_to_rad}"/>
+    <origin xyz="-0.07075 0.0 0.012" rpy="${0.0*deg_to_rad} ${180.0*deg_to_rad} ${0.0*deg_to_rad}"/>
   </xacro:kangaroo_imu>
   <xacro:kangaroo_leg side="left" reflect="1" parent="base_link" simulation="$(arg simulation)">
