Commit message: added use_mimic parameter to enable/disable mimic joints

File: kangaroo_description/robots/kangaroo.urdf.xacro (robot description, xacro)
@@ -52,9 +52,9 @@
     <origin xyz="-0.07075 0.0 0.012" rpy="${0.0*deg_to_rad} ${180.0*deg_to_rad} ${0.0*deg_to_rad}"/>
   </xacro:kangaroo_imu>
-  <xacro:kangaroo_leg side="left" reflect="1" parent="base_link" simulation="$(arg simulation)">
-    <origin xyz="-0.01602 0.08 -0.0585" rpy="0 0 0" />
+  <xacro:kangaroo_leg side="left" reflect="1" parent="base_link" simulation="$(arg simulation)" use_mimic="$(arg use_mimic)">
+    <origin xyz="-0.01602 0.08 -0.0585" rpy="0 0 0"/>
   </xacro:kangaroo_leg>
-  <xacro:kangaroo_leg side="right" reflect="-1" parent="base_link" simulation="$(arg simulation)">
-    <origin xyz="-0.01602 -0.08 -0.0585" rpy="0 0 0" />
+  <xacro:kangaroo_leg side="right" reflect="-1" parent="base_link" simulation="$(arg simulation)"  use_mimic="$(arg use_mimic)">
+    <origin xyz="-0.01602 -0.08 -0.0585" rpy="0 0 0"/>
   </xacro:kangaroo_leg>
   <!-- Generic simulator_gazebo plugins -->

File: kangaroo_description/urdf/leg/leg.urdf.xacro (robot description, xacro)
@@ -36,5 +36,5 @@
     </gazebo>
   </xacro:macro>
-  <xacro:macro name="kangaroo_leg" params="side reflect parent *origin simulation:=false">
+  <xacro:macro name="kangaroo_leg" params="side reflect parent *origin simulation:=false use_mimic:=true">
     <link name="leg_${side}_1_link">
       <inertial>
@@ -196,5 +196,7 @@
       <axis xyz="0 1 0" />
       <limit lower="${leg_femur_min_pos}" upper="${leg_femur_max_pos}" effort="100" velocity="3.87" />
-      <mimic joint="leg_${side}_length_joint" multiplier="1.69435" offset="-0.096145"/>
+      <xacro:if value="${use_mimic}">
+      	<mimic joint="leg_${side}_length_joint" multiplier="1.69435" offset="-0.096145"/>
+      </xacro:if>
     </joint>
     <joint name="leg_${side}_knee_joint" type="revolute">
@@ -204,5 +206,7 @@
       <axis xyz="0 -1 0" />
       <limit lower="${leg_knee_min_pos}" upper="${leg_knee_max_pos}" effort="100" velocity="3.87" />
-      <mimic joint="leg_${side}_length_joint" multiplier="3.38877" offset="-0.19229"/>
+      <xacro:if value="${use_mimic}">
+      	<mimic joint="leg_${side}_length_joint" multiplier="3.38877" offset="-0.19229"/>
+      </xacro:if>
     </joint>
     <!-- THIS FRAME NEEDS TO BE VALIDATED BY CAD!!! -->
@@ -285,6 +289,8 @@
      <material>Gazebo/FlatBlack</material>
    </gazebo>
-   <xacro:mimic_joint_plugin_gazebo name_prefix="" parent_joint="leg_${side}_length_joint" mimic_joint="leg_${side}_knee_joint" has_pid="false" multiplier="3.38877" offset="-0.19229" max_effort="100.0"/>
-   <xacro:mimic_joint_plugin_gazebo name_prefix="" parent_joint="leg_${side}_length_joint" mimic_joint="leg_${side}_femur_joint" has_pid="false" multiplier="1.69435" offset="-0.096145" max_effort="100.0"/>
+   <xacro:if value="${use_mimic}">
+   	<xacro:mimic_joint_plugin_gazebo name_prefix="" parent_joint="leg_${side}_length_joint" mimic_joint="leg_${side}_knee_joint" has_pid="false" multiplier="3.38877" offset="-0.19229" max_effort="100.0"/>
+   	<xacro:mimic_joint_plugin_gazebo name_prefix="" parent_joint="leg_${side}_length_joint" mimic_joint="leg_${side}_femur_joint" has_pid="false" multiplier="1.69435" offset="-0.096145" max_effort="100.0"/>
+   </xacro:if>
   </xacro:macro>
 </robot>

Commit message: Updated Kangaroo model with base_link with cage. Added possibility to use also old model without cage

File: kangaroo_description/robots/kangaroo.urdf.xacro (robot description, xacro)
@@ -13,27 +13,6 @@
   <!--        BASE_LINK       -->
   <!--************************-->
-  <link name="base_link">
-    <inertial>
-      <origin xyz="-0.060294 0.00050634 0.15428" rpy="0 0 0" />
-      <mass value="12.296" />
-      <inertia  ixx="0.084937" ixy="-4.4873E-05" ixz="0.0036119"
-        iyy="0.080587" iyz="0.0001781" izz="0.0247" />
-    </inertial>
-    <visual>
-      <origin xyz="0 0 0" rpy="0 0 0" />
-      <geometry>
-        <mesh filename="package://kangaroo_description/meshes/base_link.stl" />
-      </geometry>
-      <material name="">
-        <color rgba="0.75294 0.75294 0.75294 1" />
-      </material>
-    </visual>
-    <collision>
-      <origin xyz="0 0 0" rpy="0 0 0" />
-      <geometry>
-        <mesh filename="package://kangaroo_description/meshes/base_link.stl" />
-      </geometry>
-    </collision>
-  </link>
+  <xacro:include filename="$(find kangaroo_description)/urdf/base/base.urdf.xacro"/>
+  <xacro:base_link with_cage="true"/>
   <xacro:if value="$(arg enable_crane)">
     <xacro:include filename="$(find kangaroo_description)/urdf/crane/crane.urdf.xacro" />

Commit message: Fix IMU wrong orientation

File: kangaroo_description/robots/kangaroo.urdf.xacro (robot description, xacro)
@@ -29,5 +29,5 @@
   <xacro:include filename="$(find kangaroo_description)/urdf/leg/leg.urdf.xacro" />
   <xacro:kangaroo_imu name="imu" parent="base_link" update_rate="100.0">
-    <origin xyz="-0.07075 0.0 0.012" rpy="${0.0*deg_to_rad} ${180.0*deg_to_rad} ${0.0*deg_to_rad}"/>
+    <origin xyz="-0.07075 0.0 0.012" rpy="${180.0*deg_to_rad} ${0.0*deg_to_rad} ${0.0*deg_to_rad}"/>
   </xacro:kangaroo_imu>
   <xacro:kangaroo_leg side="left" reflect="1" parent="base_link" simulation="$(arg simulation)" use_mimic="$(arg use_mimic)">

Commit message: Argument to launch robot with F/T sensors or not

File: kangaroo_description/robots/kangaroo.urdf.xacro (robot description, xacro)
@@ -31,8 +31,8 @@
     <origin xyz="-0.07075 0.0 0.012" rpy="${180.0*deg_to_rad} ${0.0*deg_to_rad} ${0.0*deg_to_rad}"/>
   </xacro:kangaroo_imu>
-  <xacro:kangaroo_leg side="left" reflect="1" parent="base_link" simulation="$(arg simulation)" use_mimic="$(arg use_mimic)">
+  <xacro:kangaroo_leg side="left" reflect="1" parent="base_link" simulation="$(arg simulation)" use_mimic="$(arg use_mimic)" ft_sensors="$(arg ft_sensors)">
     <origin xyz="-0.01602 0.08 -0.0585" rpy="0 0 0"/>
   </xacro:kangaroo_leg>
-  <xacro:kangaroo_leg side="right" reflect="-1" parent="base_link" simulation="$(arg simulation)"  use_mimic="$(arg use_mimic)">
+  <xacro:kangaroo_leg side="right" reflect="-1" parent="base_link" simulation="$(arg simulation)"  use_mimic="$(arg use_mimic)" ft_sensors="$(arg ft_sensors)">
     <origin xyz="-0.01602 -0.08 -0.0585" rpy="0 0 0"/>
   </xacro:kangaroo_leg>

File: kangaroo_description/urdf/ankle/ankle.urdf.xacro (robot description, xacro)
@@ -9,5 +9,5 @@
   <xacro:property name="roll_joint_min_pos"   value="${-27.0 *deg_to_rad}" />
   <xacro:property name="roll_joint_max_pos"   value="${27.0 *deg_to_rad}" />
-  <xacro:macro name="kangaroo_ankle" params="side reflect parent *origin pitch_joint roll_joint read_actuator simulation:=false">
+  <xacro:macro name="kangaroo_ankle" params="side reflect parent *origin pitch_joint roll_joint read_actuator simulation:=false ft_sensors:=false">
     <link name="leg_${side}_${pitch_joint}_link">
       <inertial>
@@ -35,25 +35,48 @@
     </joint>
     <link name="leg_${side}_${roll_joint}_link">
-      <inertial>
-        <origin xyz="0.022056 -3.9166E-05 -0.0099049" rpy="0 0 0" />
-        <mass value="0.41343" />
-        <inertia ixx="0.00435" ixy="2.7E-07" ixz="0.000241"
-          iyy="0.0179" iyz="3.0E-07" izz="0.0185" />
-      </inertial>
-      <visual>
-        <origin xyz="0 0 0" rpy="0 0 0" />
-        <geometry>
-          <mesh filename="package://kangaroo_description/meshes/leg_7_link.stl" />
-        </geometry>
-        <material name="">
-          <color rgba="0.752941176470588 0.752941176470588 0.752941176470588 1" />
-        </material>
-      </visual>
-      <collision>
-        <origin xyz="0.035 0 -0.02" rpy="0 0 0" />
-        <geometry>
-          <box size="0.21 0.09 0.025"/>
-        </geometry>
-      </collision>
+      <xacro:unless value="${ft_sensors}">
+        <inertial>
+          <origin xyz="0.022056 -3.9166E-05 -0.0099049" rpy="0 0 0" />
+          <mass value="0.41343" />
+          <inertia ixx="0.00435" ixy="2.7E-07" ixz="0.000241" iyy="0.0179" iyz="3.0E-07" izz="0.0185" />
+        </inertial>
+        <visual>
+          <origin xyz="0 0 0" rpy="0 0 0" />
+          <geometry>
+            <mesh filename="package://kangaroo_description/meshes/leg_7_link.stl" />
+          </geometry>
+          <material name="">
+            <color rgba="0.752941176470588 0.752941176470588 0.752941176470588 1" />
+          </material>
+        </visual>
+        <collision>
+          <origin xyz="0.035 0 -0.02" rpy="0 0 0" />
+          <geometry>
+            <box size="0.21 0.09 0.025"/>
+          </geometry>
+        </collision>
+      </xacro:unless>
+      <xacro:if value="${ft_sensors}">
+        <inertial>
+          <origin xyz="0.022204 -8.11751E-06 -0.042186" rpy="0 0 0" />
+          <mass value="0.624725" />
+          <inertia ixx="0.0004094" ixy="2.2E-08" ixz="-0.000244" iyy="0.0009742" iyz="-1.25E-09" izz="0.0011036" />
+        </inertial>
+        <visual>
+          <origin xyz="0 0 0" rpy="0 0 0" />
+          <geometry>
+            <mesh filename="package://kangaroo_description/meshes/leg_7_link_ft.stl" />
+          </geometry>
+          <material name="">
+            <color rgba="0.752941176470588 0.752941176470588 0.752941176470588 1" />
+          </material>
+        </visual>
+        <collision>
+          <origin xyz="0 0 0" rpy="0 0 0" />
+          <geometry>
+            <mesh filename="package://kangaroo_description/meshes/leg_7_link_ft.stl" />
+          </geometry>
+        </collision>
+      </xacro:if>
     </link>
     <joint name="leg_${side}_${roll_joint}_joint" type="revolute">

File: kangaroo_description/urdf/leg/leg.urdf.xacro (robot description, xacro)
@@ -36,5 +36,5 @@
     </gazebo>
   </xacro:macro>
-  <xacro:macro name="kangaroo_leg" params="side reflect parent *origin simulation:=false use_mimic:=true">
+  <xacro:macro name="kangaroo_leg" params="side reflect parent *origin simulation:=false use_mimic:=true ft_sensors:=false">
     <link name="leg_${side}_1_link">
       <inertial>
@@ -248,5 +248,5 @@
     	<origin rpy="0 0 0" xyz="-0.38 0.0 0.0"/>
     </joint>
-    <xacro:kangaroo_ankle side="${side}" parent="leg_${side}_length_link" reflect="${reflect}" roll_joint="5" pitch_joint="4" read_actuator="leg_${side}_length_motor">
+    <xacro:kangaroo_ankle side="${side}" parent="leg_${side}_length_link" reflect="${reflect}" roll_joint="5" pitch_joint="4" read_actuator="leg_${side}_length_motor" ft_sensors="$(arg ft_sensors)">
       <origin xyz="0.0 0 0.0" rpy="0 ${180 *deg_to_rad} 0" />
     </xacro:kangaroo_ankle>

Commit message: Parameterize the version of Hip Z installed on the robot and update the parameters

File: kangaroo_description/robots/kangaroo.urdf.xacro (robot description, xacro)
@@ -9,4 +9,6 @@
         xmlns:interface="http://playerstage.sourceforge.net/gazebo/xmlschema/#interface">
   <xacro:property name="deg_to_rad"       value="0.01745329251994329577" />
+  <xacro:arg name="hipz_model" default="2023"/>
+  <xacro:property name="hipz_model" value="$(arg hipz_model)" />
   <xacro:include filename="$(find kangaroo_description)/urdf/sensors/imu.urdf.xacro" />
   <!--************************-->
@@ -31,8 +33,8 @@
     <origin xyz="-0.07075 0.0 0.012" rpy="${180.0*deg_to_rad} ${0.0*deg_to_rad} ${0.0*deg_to_rad}"/>
   </xacro:kangaroo_imu>
-  <xacro:kangaroo_leg side="left" reflect="1" parent="base_link" simulation="$(arg simulation)" use_mimic="$(arg use_mimic)" ft_sensors="$(arg ft_sensors)">
+  <xacro:kangaroo_leg side="left" reflect="1" parent="base_link" simulation="$(arg simulation)" use_mimic="$(arg use_mimic)" ft_sensors="$(arg ft_sensors)" hipz_model="$(arg hipz_model)">
     <origin xyz="-0.01602 0.08 -0.0585" rpy="0 0 0"/>
   </xacro:kangaroo_leg>
-  <xacro:kangaroo_leg side="right" reflect="-1" parent="base_link" simulation="$(arg simulation)"  use_mimic="$(arg use_mimic)" ft_sensors="$(arg ft_sensors)">
+  <xacro:kangaroo_leg side="right" reflect="-1" parent="base_link" simulation="$(arg simulation)"  use_mimic="$(arg use_mimic)" ft_sensors="$(arg ft_sensors)" hipz_model="$(arg hipz_model)">
     <origin xyz="-0.01602 -0.08 -0.0585" rpy="0 0 0"/>
   </xacro:kangaroo_leg>

File: kangaroo_description/urdf/leg/leg.urdf.xacro (robot description, xacro)
@@ -36,5 +36,5 @@
     </gazebo>
   </xacro:macro>
-  <xacro:macro name="kangaroo_leg" params="side reflect parent *origin simulation:=false use_mimic:=true ft_sensors:=false">
+  <xacro:macro name="kangaroo_leg" params="side reflect parent *origin hipz_model simulation:=false use_mimic:=true ft_sensors:=false">
     <link name="leg_${side}_1_link">
       <inertial>
@@ -253,5 +253,5 @@
     <!-- Load corresponding transmission info -->
     <xacro:unless value="${simulation}">
-      <xacro:hip_transmission_yaw side="${side}" params_ns="/${side}_hip_z_params" />
+      <xacro:hip_transmission_yaw side="${side}" params_ns="/${side}_hip_z_${hipz_model}_params" />
       <xacro:hip_transmission_roll_pitch side="${side}" roll_joint="3" pitch_joint="2" />
       <xacro:kangaroo_leg_length_actuator_transmission side="${side}" number1="4" number2="5" params_ns="/leg_params" />

Commit message: added version arg to the URDF and create different leg URDFs

File: kangaroo_description/robots/kangaroo.urdf.xacro (robot description, xacro)
@@ -10,5 +10,7 @@
   <xacro:property name="deg_to_rad"       value="0.01745329251994329577" />
   <xacro:arg name="hipz_model" default="2023"/>
+  <xacro:arg name="version" default="2023"/>
   <xacro:property name="hipz_model" value="$(arg hipz_model)" />
+  <xacro:property name="version" value="$(arg version)" />
   <xacro:include filename="$(find kangaroo_description)/urdf/sensors/imu.urdf.xacro" />
   <!--************************-->
@@ -29,5 +31,5 @@
     </joint>
   </xacro:if>
-  <xacro:include filename="$(find kangaroo_description)/urdf/leg/leg.urdf.xacro" />
+  <xacro:include filename="$(find kangaroo_description)/urdf/leg/leg_$(arg version).urdf.xacro" />
   <xacro:kangaroo_imu name="imu" parent="base_link" update_rate="100.0">
     <origin xyz="-0.07075 0.0 0.012" rpy="${180.0*deg_to_rad} ${0.0*deg_to_rad} ${0.0*deg_to_rad}"/>

Commit message: hardcode hipz model inside the leg urdf xacros

File: kangaroo_description/robots/kangaroo.urdf.xacro (robot description, xacro)
@@ -9,7 +9,5 @@
         xmlns:interface="http://playerstage.sourceforge.net/gazebo/xmlschema/#interface">
   <xacro:property name="deg_to_rad"       value="0.01745329251994329577" />
-  <xacro:arg name="hipz_model" default="2023"/>
   <xacro:arg name="version" default="2023"/>
-  <xacro:property name="hipz_model" value="$(arg hipz_model)" />
   <xacro:property name="version" value="$(arg version)" />
   <xacro:include filename="$(find kangaroo_description)/urdf/sensors/imu.urdf.xacro" />
@@ -35,8 +33,8 @@
     <origin xyz="-0.07075 0.0 0.012" rpy="${180.0*deg_to_rad} ${0.0*deg_to_rad} ${0.0*deg_to_rad}"/>
   </xacro:kangaroo_imu>
-  <xacro:kangaroo_leg side="left" reflect="1" parent="base_link" simulation="$(arg simulation)" use_mimic="$(arg use_mimic)" ft_sensors="$(arg ft_sensors)" hipz_model="$(arg hipz_model)">
+  <xacro:kangaroo_leg side="left" reflect="1" parent="base_link" simulation="$(arg simulation)" use_mimic="$(arg use_mimic)" ft_sensors="$(arg ft_sensors)">
     <origin xyz="-0.01602 0.08 -0.0585" rpy="0 0 0"/>
   </xacro:kangaroo_leg>
-  <xacro:kangaroo_leg side="right" reflect="-1" parent="base_link" simulation="$(arg simulation)"  use_mimic="$(arg use_mimic)" ft_sensors="$(arg ft_sensors)" hipz_model="$(arg hipz_model)">
+  <xacro:kangaroo_leg side="right" reflect="-1" parent="base_link" simulation="$(arg simulation)"  use_mimic="$(arg use_mimic)" ft_sensors="$(arg ft_sensors)">
     <origin xyz="-0.01602 -0.08 -0.0585" rpy="0 0 0"/>
   </xacro:kangaroo_leg>

File: kangaroo_description/urdf/leg/leg_2022.urdf.xacro (robot description, xacro)
@@ -36,5 +36,5 @@
     </gazebo>
   </xacro:macro>
-  <xacro:macro name="kangaroo_leg" params="side reflect parent *origin hipz_model simulation:=false use_mimic:=true ft_sensors:=false">
+  <xacro:macro name="kangaroo_leg" params="side reflect parent *origin hipz_model:=2022 simulation:=false use_mimic:=true ft_sensors:=false">
     <link name="leg_${side}_1_link">
       <inertial>

File: kangaroo_description/urdf/leg/leg_2023.urdf.xacro (robot description, xacro)
@@ -36,5 +36,5 @@
     </gazebo>
   </xacro:macro>
-  <xacro:macro name="kangaroo_leg" params="side reflect parent *origin hipz_model simulation:=false use_mimic:=true ft_sensors:=false">
+  <xacro:macro name="kangaroo_leg" params="side reflect parent *origin hipz_model:=2023 simulation:=false use_mimic:=true ft_sensors:=false">
     <link name="leg_${side}_1_link">
       <inertial>

Commit message: Added the kangaroo cameras

File: kangaroo_description/robots/kangaroo.urdf.xacro (robot description, xacro)
@@ -8,6 +8,32 @@
         xmlns:controller="http://playerstage.sourceforge.net/gazebo/xmlschema/#controller"
         xmlns:interface="http://playerstage.sourceforge.net/gazebo/xmlschema/#interface">
-  <xacro:property name="deg_to_rad"       value="0.01745329251994329577" />
+  <xacro:arg name="version" default="2023" />
+  <xacro:arg name="simulation" default="false" />
+  <xacro:arg name="torso_front_camera_model" default="realsense-D435i" />
+  <xacro:arg name="torso_back_camera_model" default="realsense-D435i" />
+  <xacro:arg name="wrist_front_camera_model" default="realsense-D435i" />
+  <xacro:arg name="wrist_back_camera_model" default="realsense-D435i" />
   <xacro:property name="version" value="$(arg version)" />
+  <xacro:property name="simulation" value="$(arg simulation)" />
+  <xacro:property name="torso_front_camera_model" value="$(arg torso_front_camera_model)" />
+  <xacro:property name="torso_back_camera_model" value="$(arg torso_back_camera_model)" />
+  <xacro:property name="wrist_front_camera_model" value="$(arg wrist_front_camera_model)" />
+  <xacro:property name="wrist_back_camera_model" value="$(arg wrist_back_camera_model)" />
+  <xacro:if value="${version not in ['2022','2023']}">
+    <xacro:wrong_version/>
+  </xacro:if>
+  <xacro:if value="${torso_front_camera_model not in ['realsense-D435i']}">
+    <xacro:wrong_torso_front_camera_model/>
+  </xacro:if>
+  <xacro:if value="${torso_back_camera_model not in ['realsense-D435i']}">
+    <xacro:wrong_torso_back_camera_model/>
+  </xacro:if>
+  <xacro:if value="${wrist_front_camera_model not in ['realsense-D435i']}">
+    <xacro:wrong_wrist_front_camera_model/>
+  </xacro:if>
+  <xacro:if value="${wrist_back_camera_model not in ['realsense-D435i']}">
+    <xacro:wrong_wrist_back_camera_model/>
+  </xacro:if>
+  <xacro:include filename="$(find kangaroo_description)/urdf/deg_to_rad.xacro" />
   <!--************************-->
   <!--        BASE_LINK       -->
@@ -35,6 +61,9 @@
   </xacro:kangaroo_leg>
   <!-- Generic simulator_gazebo plugins -->
-  <xacro:include filename="$(find kangaroo_description)/gazebo/gazebo.urdf.xacro" />
   <!-- Materials for visualization -->
   <xacro:include filename="$(find kangaroo_description)/urdf/materials.urdf.xacro" />
+  <xacro:include filename="$(find kangaroo_description)/urdf/torso/torso.urdf.xacro" />
+  <xacro:kangaroo_torso parent="base_link"/>
+  <xacro:include filename="$(find kangaroo_description)/urdf/wrist/wrist.urdf.xacro" />
+  <xacro:kangaroo_wrist parent="base_link"/>
 </robot>

File: kangaroo_description/urdf/base/base_2023.urdf.xacro (robot description, xacro)
@@ -26,36 +26,4 @@
     </collision>
   </link>
-  <link name="torso_link">
-    <inertial>
-      <origin xyz="-0.0085193 -0.00033267 0.22824" rpy="0 0 0" />
-      <mass value="13.843" />
-      <inertia ixx="0.087431" ixy="1.1038E-05" ixz="-9.0502E-06"
-        iyy="0.072736" iyz="2.6862E-05" izz="0.032695" />
-    </inertial>
-    <visual>
-      <origin xyz="0 0 0" rpy="0 0 0" />
-      <geometry>
-        <mesh filename="package://kangaroo_description/meshes/${version}/torso_link.stl" />
-      </geometry>
-      <material name="">
-        <color rgba="0.75294 0.75294 0.75294 1" />
-      </material>
-    </visual>
-    <collision>
-      <origin xyz="0 0 0" rpy="0 0 0" />
-      <geometry>
-        <mesh filename="package://kangaroo_description/meshes/${version}/torso_link_convex.stl" />
-      </geometry>
-    </collision>
-  </link>
-  <joint name="torso_link" type="fixed">
-    <origin xyz="-0.0918000000000001 0 0.0074999999999998" rpy="0 0 0" />
-    <parent link="base_link" />
-    <child link="torso_link" />
-    <axis xyz="0 0 0" />
-  </joint>
-  <xacro:kangaroo_imu name="imu" parent="torso_link" update_rate="100.0">
-    <origin xyz="0.071 -0.0014 0.02" rpy="${180.0*deg_to_rad} ${0.0*deg_to_rad} ${-90.0*deg_to_rad}"/>
-  </xacro:kangaroo_imu>
 </xacro:macro>
 </robot>

Commit message: Fix xacro macro urdf

File: kangaroo_description/robots/kangaroo.urdf.xacro (robot description, xacro)
@@ -20,5 +20,5 @@
   <xacro:property name="wrist_front_camera_model" value="$(arg wrist_front_camera_model)" />
   <xacro:property name="wrist_back_camera_model" value="$(arg wrist_back_camera_model)" />
-  <xacro:if value="${version not in ['2022','2023']}">
+  <xacro:if value="${version not in [2022,2023]}">
     <xacro:wrong_version/>
   </xacro:if>

File: kangaroo_description/urdf/torso/torso.urdf.xacro (robot description, xacro)
@@ -61,3 +61,4 @@
         rpy="0 -0.5236 ${180.0*deg_to_rad}"/>
     </xacro:sensor_d435>
+  </xacro:macro>
 </robot>
