Commit message: Change wrist to waist

File: kangaroo_description/robots/kangaroo.urdf.xacro (robot description, xacro)
@@ -12,12 +12,12 @@
   <xacro:arg name="torso_front_camera_model" default="realsense-D435i" />
   <xacro:arg name="torso_back_camera_model" default="realsense-D435i" />
-  <xacro:arg name="wrist_front_camera_model" default="realsense-D435i" />
-  <xacro:arg name="wrist_back_camera_model" default="realsense-D435i" />
+  <xacro:arg name="waist_front_camera_model" default="realsense-D435i" />
+  <xacro:arg name="waist_back_camera_model" default="realsense-D435i" />
   <xacro:property name="version" value="$(arg version)" />
   <xacro:property name="simulation" value="$(arg simulation)" />
   <xacro:property name="torso_front_camera_model" value="$(arg torso_front_camera_model)" />
   <xacro:property name="torso_back_camera_model" value="$(arg torso_back_camera_model)" />
-  <xacro:property name="wrist_front_camera_model" value="$(arg wrist_front_camera_model)" />
-  <xacro:property name="wrist_back_camera_model" value="$(arg wrist_back_camera_model)" />
+  <xacro:property name="waist_front_camera_model" value="$(arg waist_front_camera_model)" />
+  <xacro:property name="waist_back_camera_model" value="$(arg waist_back_camera_model)" />
   <xacro:if value="${version not in [2022,2023]}">
     <xacro:wrong_version/>
@@ -29,9 +29,9 @@
     <xacro:wrong_torso_back_camera_model/>
   </xacro:if>
-  <xacro:if value="${wrist_front_camera_model not in ['realsense-D435i']}">
-    <xacro:wrong_wrist_front_camera_model/>
+  <xacro:if value="${waist_front_camera_model not in ['realsense-D435i']}">
+    <xacro:wrong_waist_front_camera_model/>
   </xacro:if>
-  <xacro:if value="${wrist_back_camera_model not in ['realsense-D435i']}">
-    <xacro:wrong_wrist_back_camera_model/>
+  <xacro:if value="${waist_back_camera_model not in ['realsense-D435i']}">
+    <xacro:wrong_waist_back_camera_model/>
   </xacro:if>
   <xacro:include filename="$(find kangaroo_description)/urdf/deg_to_rad.xacro" />
@@ -65,5 +65,5 @@
   <xacro:include filename="$(find kangaroo_description)/urdf/torso/torso.urdf.xacro" />
   <xacro:kangaroo_torso parent="base_link"/>
-  <xacro:include filename="$(find kangaroo_description)/urdf/wrist/wrist.urdf.xacro" />
-  <xacro:kangaroo_wrist parent="base_link"/>
+  <xacro:include filename="$(find kangaroo_description)/urdf/waist/waist.urdf.xacro" />
+  <xacro:kangaroo_waist parent="base_link"/>
 </robot>

File: kangaroo_description/urdf/waist/waist.urdf.xacro (robot description, xacro)
@@ -11,10 +11,10 @@
   <xacro:include filename="$(find kangaroo_description)/urdf/deg_to_rad.xacro" />
   <xacro:include filename="$(find realsense2_description)/urdf/_d435.urdf.xacro" />
-  <xacro:macro name="kangaroo_wrist" params="parent">
-  <!-- Wrist front rgbd camera -->
+  <xacro:macro name="kangaroo_waist" params="parent">
+  <!-- Waist front rgbd camera -->
     <xacro:sensor_d435
-      name="wrist_front_rgbd_camera"
+      name="waist_front_rgbd_camera"
       parent="${parent}"
-      topics_ns="wrist_front_rgbd_camera"
+      topics_ns="waist_front_rgbd_camera"
       use_nominal_extrinsics="${simulation}">
       <origin
@@ -22,9 +22,9 @@
         rpy="0 1.0472 0"/>
     </xacro:sensor_d435>
-  <!-- Wrist back rgbd camera -->
+  <!-- Waist back rgbd camera -->
     <xacro:sensor_d435
-      name="wrist_back_rgbd_camera"
+      name="waist_back_rgbd_camera"
       parent="${parent}"
-      topics_ns="wrist_back_rgbd_camera"
+      topics_ns="waist_back_rgbd_camera"
       use_nominal_extrinsics="${simulation}">
       <origin
@@ -32,3 +32,4 @@
         rpy="0 -1.0472 ${180.0*deg_to_rad}"/>
     </xacro:sensor_d435>
+  </xacro:macro>
 </robot>

Commit message: Set the IMU definition for base version 2022

File: kangaroo_description/robots/kangaroo.urdf.xacro (robot description, xacro)
@@ -10,5 +10,4 @@
   <xacro:property name="deg_to_rad"       value="0.01745329251994329577" />
   <xacro:property name="version" value="$(arg version)" />
-  <xacro:include filename="$(find kangaroo_description)/urdf/sensors/imu.urdf.xacro" />
   <!--************************-->
   <!--        BASE_LINK       -->
@@ -29,7 +28,4 @@
   </xacro:if>
   <xacro:include filename="$(find kangaroo_description)/urdf/leg/leg_$(arg version).urdf.xacro" />
-  <xacro:kangaroo_imu name="imu" parent="base_link" update_rate="100.0">
-    <origin xyz="-0.07075 0.0 0.012" rpy="${180.0*deg_to_rad} ${0.0*deg_to_rad} ${0.0*deg_to_rad}"/>
-  </xacro:kangaroo_imu>
   <xacro:kangaroo_leg side="left" reflect="1" parent="base_link" simulation="$(arg simulation)" use_mimic="$(arg use_mimic)" ft_sensors="$(arg ft_sensors)">
     <origin xyz="-0.01602 0.08 -0.0585" rpy="0 0 0"/>

File: kangaroo_description/urdf/base/base_2022.urdf.xacro (robot description, xacro)
@@ -2,4 +2,5 @@
 <robot xmlns:xacro="http://ros.org/wiki/xacro" name="kangaroo">
 <xacro:macro name="base_link" params="with_cage:=true version:=2022">
+<xacro:include filename="$(find kangaroo_description)/urdf/sensors/imu.urdf.xacro"/>
 <xacro:if value="${with_cage}">
 <link name="base_link">
@@ -26,4 +27,7 @@
     </collision>
 </link>
+<xacro:kangaroo_imu name="imu" parent="base_link" update_rate="100.0">
+  <origin xyz="-0.07075 0.0 0.012" rpy="${180.0*deg_to_rad} ${0.0*deg_to_rad} ${0.0*deg_to_rad}"/>
+</xacro:kangaroo_imu>
 </xacro:if>
 <xacro:unless value="${with_cage}">
@@ -51,4 +55,7 @@
     </collision>
 </link>
+<xacro:kangaroo_imu name="imu" parent="base_link" update_rate="100.0">
+  <origin xyz="-0.07075 0.0 0.012" rpy="${180.0*deg_to_rad} ${0.0*deg_to_rad} ${0.0*deg_to_rad}"/>
+</xacro:kangaroo_imu>
 </xacro:unless>
 </xacro:macro>

Commit message: Add removed imu link and modify the placement of macros torso and waist

File: kangaroo_description/robots/kangaroo.urdf.xacro (robot description, xacro)
@@ -64,7 +64,3 @@
   <!-- Materials for visualization -->
   <xacro:include filename="$(find kangaroo_description)/urdf/materials.urdf.xacro" />
-  <xacro:include filename="$(find kangaroo_description)/urdf/torso/torso.urdf.xacro" />
-  <xacro:kangaroo_torso parent="base_link"/>
-  <xacro:include filename="$(find kangaroo_description)/urdf/waist/waist.urdf.xacro" />
-  <xacro:kangaroo_waist parent="base_link"/>
 </robot>

File: kangaroo_description/urdf/base/base_2023.urdf.xacro (robot description, xacro)
@@ -26,4 +26,11 @@
     </collision>
   </link>
+  <xacro:kangaroo_imu name="imu" parent="torso_link" update_rate="100.0">
+    <origin xyz="0.071 -0.0014 0.02" rpy="${180.0*deg_to_rad} ${0.0*deg_to_rad} ${-90.0*deg_to_rad}"/>
+  </xacro:kangaroo_imu>
+  <xacro:include filename="$(find kangaroo_description)/urdf/torso/torso.urdf.xacro" />
+  <xacro:kangaroo_torso parent="base_link"/>
+  <xacro:include filename="$(find kangaroo_description)/urdf/waist/waist.urdf.xacro" />
+  <xacro:kangaroo_waist parent="base_link"/>
 </xacro:macro>
 </robot>

Commit message: Update changes in Hip Z

File: kangaroo_description/robots/kangaroo.urdf.xacro (robot description, xacro)
@@ -55,8 +55,8 @@
   <xacro:include filename="$(find kangaroo_description)/urdf/leg/leg_$(arg version).urdf.xacro" />
   <xacro:kangaroo_leg side="left" reflect="1" parent="base_link" simulation="$(arg simulation)" use_mimic="$(arg use_mimic)" ft_sensors="$(arg ft_sensors)">
-    <origin xyz="-0.01602 0.08 -0.0585" rpy="0 0 0"/>
+    <origin xyz="-0.0150025976417119 0.08 -0.0585" rpy="0 0 0"/>
   </xacro:kangaroo_leg>
   <xacro:kangaroo_leg side="right" reflect="-1" parent="base_link" simulation="$(arg simulation)"  use_mimic="$(arg use_mimic)" ft_sensors="$(arg ft_sensors)">
-    <origin xyz="-0.01602 -0.08 -0.0585" rpy="0 0 0"/>
+    <origin xyz="-0.0150025976417119 -0.08 -0.0585" rpy="0 0 0"/>
   </xacro:kangaroo_leg>
   <!-- Generic simulator_gazebo plugins -->

File: kangaroo_description/urdf/leg/leg_2023.urdf.xacro (robot description, xacro)
@@ -39,8 +39,8 @@
     <link name="leg_${side}_1_link">
       <inertial>
-        <origin xyz="0.00643148180089947 ${reflect * 0.00470584363523306} -0.0104315706390075" rpy="0 0 0" />
-        <mass value="2.89547106393921" />
-        <inertia ixx="0.002373067757357" ixy="${reflect * 1.0458682341421E-05}" ixz="${reflect * 7.10544668703563E-05}"
-          iyy="0.00215576778669813" iyz="${reflect * -1.24262445397793E-05}" izz="0.00155640461041179" />
+        <origin xyz="0.0063167 ${reflect * 0.0045949} -0.0083828" rpy="0 0 0" />
+        <mass value="2.7478" />
+        <inertia ixx="0.0019336" ixy="${reflect * 8.5058E-06}" ixz="${reflect * 4.8385E-05}"
+          iyy="0.0018225" iyz="${reflect * -7.282E-06}" izz="0.001426" />
       </inertial>
       <visual>
@@ -75,5 +75,5 @@
       <inertial>
         <origin
-          xyz="-0.00292779640030026 -9.62074367728827E-05 1.0865936483917E-09"
+          xyz="-0.0029278 -9.6207E-05 1.0866E-09"
           rpy="0 0 0" />
         <mass value="0.0905312454913012" />
@@ -98,5 +98,5 @@
     </link>
     <joint name="leg_${side}_2_joint" type="revolute">
-      <origin xyz="0.015024 0 -0.0925" rpy="0 0 0" />
+      <origin xyz="0.015024 0 -0.1175" rpy="0 0 0" />
       <parent link="leg_${side}_1_link" />
       <child link="leg_${side}_2_link" />
@@ -106,8 +106,8 @@
     <link name="leg_${side}_3_link">
       <inertial>
-        <origin xyz="-0.0331126340475435 ${reflect * 0.0492000964734808} -0.0300270306298204" rpy="0 0 0" />
-        <mass value="3.45187520713338" />
-        <inertia ixx="0.0021995228245877" ixy="${reflect * 0.000142021792686858}" ixz="${reflect * -0.000114089540435782}"
-          iyy="0.00286983872145199" iyz="${reflect * 3.27704238559214E-05}" izz="0.00273461620254835" />
+        <origin xyz="-0.033949 ${reflect * 0.049989} -0.030543" rpy="0 0 0" />
+        <mass value="3.658" />
+        <inertia ixx="0.0025968" ixy="${reflect * 0.00018723}" ixz="${reflect * -0.00014976}"
+          iyy="0.0031521" iyz="${reflect * 3.7258E-05}" izz="0.0032376" />
       </inertial>
       <visual>

Commit message: Added torso and pelvis without params

File: kangaroo_description/robots/kangaroo.urdf.xacro (robot description, xacro)
@@ -60,4 +60,11 @@
     <origin xyz="-0.0150025976417119 -0.08 -0.0585" rpy="0 0 0"/>
   </xacro:kangaroo_leg>
+  <xacro:include filename="$(find kangaroo_description)/urdf/arm/arm.urdf.xacro" />
+  <xacro:kangaroo_arm name="arm" side="left" reflect="1" parent="torso_link" arm_1_offset="0" arm_2_offset="0" arm_3_offset="0" arm_4_offset="0">
+   <origin xyz="0 0.105954 0.384396" rpy="1.5708 0 0" />
+  </xacro:kangaroo_arm>
+  <xacro:kangaroo_arm name="arm" side="right" reflect="-1" parent="torso_link" arm_1_offset="0" arm_2_offset="0" arm_3_offset="0" arm_4_offset="0">
+   <origin xyz="0 -0.105954 0.384396" rpy="1.5708 0 3.14159" />
+  </xacro:kangaroo_arm>
   <!-- Generic simulator_gazebo plugins -->
   <xacro:include filename="$(find kangaroo_description)/gazebo/gazebo.urdf.xacro" />

File: kangaroo_description/urdf/base/base_2023.urdf.xacro (robot description, xacro)
@@ -2,4 +2,5 @@
 <robot xmlns:xacro="http://ros.org/wiki/xacro" name="kangaroo">
 <xacro:include filename="$(find kangaroo_description)/urdf/sensors/imu.urdf.xacro"/>
+<xacro:include filename="$(find kangaroo_description)/urdf/pelvis/pelvis.urdf.xacro" />
 <xacro:macro name="base_link" params="version:=2023 with_cage:=true">
   <link name="base_link">
@@ -29,6 +30,10 @@
     <origin xyz="0.071 -0.0014 0.02" rpy="${180.0*deg_to_rad} ${0.0*deg_to_rad} ${-90.0*deg_to_rad}"/>
   </xacro:kangaroo_imu>
+  <xacro:kangaroo_pelvis name="pelvis" parent="base_link" pelvis_1_offset="0" pelvis_2_offset="0">
+   <origin xyz="-0.0918000000000001 0 -0.0455" rpy="0 0 0" />
+  </xacro:kangaroo_pelvis>
   <xacro:include filename="$(find kangaroo_description)/urdf/torso/torso.urdf.xacro" />
-  <xacro:kangaroo_torso parent="base_link"/>
+  <xacro:kangaroo_torso parent="pelvis_2_link"/> <!-- base_link -->
+  <!-- waist cameras -->
   <xacro:include filename="$(find kangaroo_description)/urdf/waist/waist.urdf.xacro" />
   <xacro:kangaroo_waist parent="base_link"/>

File: kangaroo_description/urdf/torso/torso.urdf.xacro (robot description, xacro)
@@ -36,5 +36,6 @@
   </link>
   <joint name="torso_link" type="fixed">
-    <origin xyz="-0.0918000000000001 0 0.0075" rpy="0 0 0" />
+    <!--<origin xyz="-0.0918000000000001 0 0.0075" rpy="0 0 0" /> -->
+    <origin xyz="0 0 0.0061" rpy="0 0 0" />
     <parent link="${parent}" />
     <child link="torso_link" />
