Commit message: pelvis param and removed version 2022, default to 2023

File: kangaroo_description/robots/kangaroo.urdf.xacro (robot description, xacro)
@@ -8,5 +8,5 @@
         xmlns:controller="http://playerstage.sourceforge.net/gazebo/xmlschema/#controller"
         xmlns:interface="http://playerstage.sourceforge.net/gazebo/xmlschema/#interface">
-  <xacro:arg name="version" default="2023" />
+  <xacro:arg name="with_pelvis" default="false" />
   <xacro:arg name="simulation" default="false" />
   <xacro:arg name="torso_front_camera_model" default="realsense-D435i" />
@@ -14,5 +14,5 @@
   <xacro:arg name="waist_front_camera_model" default="realsense-D435i" />
   <xacro:arg name="waist_back_camera_model" default="realsense-D435i" />
-  <xacro:property name="version" value="$(arg version)" />
+  <xacro:property name="with_pelvis" value="$(arg with_pelvis)" />
   <xacro:property name="simulation" value="$(arg simulation)" />
   <xacro:property name="torso_front_camera_model" value="$(arg torso_front_camera_model)" />
@@ -20,7 +20,4 @@
   <xacro:property name="waist_front_camera_model" value="$(arg waist_front_camera_model)" />
   <xacro:property name="waist_back_camera_model" value="$(arg waist_back_camera_model)" />
-  <xacro:if value="${version not in [2022,2023]}">
-    <xacro:wrong_version/>
-  </xacro:if>
   <xacro:if value="${torso_front_camera_model not in ['realsense-D435i']}">
     <xacro:wrong_torso_front_camera_model/>
@@ -39,6 +36,6 @@
   <!--        BASE_LINK       -->
   <!--************************-->
-  <xacro:include filename="$(find kangaroo_description)/urdf/base/base_$(arg version).urdf.xacro"/>
-  <xacro:base_link with_cage="$(arg use_cage)"/>
+  <xacro:include filename="$(find kangaroo_description)/urdf/base/base.urdf.xacro"/>
+  <xacro:base_link with_pelvis="$(arg with_pelvis)"/>
   <xacro:if value="$(arg enable_crane)">
     <xacro:include filename="$(find kangaroo_description)/urdf/crane/crane.urdf.xacro" />
@@ -53,5 +50,5 @@
     </joint>
   </xacro:if>
-  <xacro:include filename="$(find kangaroo_description)/urdf/leg/leg_$(arg version).urdf.xacro" />
+  <xacro:include filename="$(find kangaroo_description)/urdf/leg/leg.urdf.xacro" />
   <xacro:kangaroo_leg side="left" reflect="1" parent="base_link" simulation="$(arg simulation)" use_mimic="$(arg use_mimic)" ft_sensors="$(arg ft_sensors)">
     <origin xyz="-0.0150025976417119 0.08 -0.0585" rpy="0 0 0"/>

File: kangaroo_description/urdf/ankle/ankle.urdf.xacro (robot description, xacro)
@@ -9,5 +9,5 @@
   <xacro:property name="roll_joint_min_pos"   value="${-27.0 *deg_to_rad}" />
   <xacro:property name="roll_joint_max_pos"   value="${27.0 *deg_to_rad}" />
-  <xacro:macro name="kangaroo_ankle" params="side reflect parent *origin pitch_joint roll_joint read_actuator simulation:=false ft_sensors:=false version:=2023">
+  <xacro:macro name="kangaroo_ankle" params="side reflect parent *origin pitch_joint roll_joint read_actuator simulation:=false ft_sensors:=false">
     <link name="leg_${side}_${pitch_joint}_link">
       <inertial>
@@ -51,5 +51,5 @@
           <origin xyz="0 0 0" rpy="0 0 0" />
           <geometry>
-            <mesh filename="package://kangaroo_description/meshes/${version}/leg_7_link.stl" />
+            <mesh filename="package://kangaroo_description/meshes/leg_7_link.stl" />
           </geometry>
           <material name="">
@@ -60,5 +60,5 @@
           <origin xyz="0 0 0" rpy="0 0 0" />
           <geometry>
-            <mesh filename="package://kangaroo_description/meshes/${version}/leg_7_link.stl" />
+            <mesh filename="package://kangaroo_description/meshes/leg_7_link.stl" />
           </geometry>
         </collision>
@@ -82,5 +82,5 @@
           <origin xyz="0 0 0" rpy="0 ${-20.0 * deg_to_rad} 0" />
           <geometry>
-            <mesh filename="package://kangaroo_description/meshes/${version}/leg_7_link_ft.stl" />
+            <mesh filename="package://kangaroo_description/meshes/leg_7_link_ft.stl" />
           </geometry>
           <material name="">
@@ -91,5 +91,5 @@
           <origin xyz="0 0 0" rpy="0 ${-20.0 * deg_to_rad} 0" />
           <geometry>
-            <mesh filename="package://kangaroo_description/meshes/${version}/leg_7_link_ft.stl" />
+            <mesh filename="package://kangaroo_description/meshes/leg_7_link_ft.stl" />
           </geometry>
         </collision>

File: kangaroo_description/urdf/base/base.urdf.xacro (robot description, xacro)
@@ -3,5 +3,5 @@
 <xacro:include filename="$(find kangaroo_description)/urdf/sensors/imu.urdf.xacro"/>
 <xacro:include filename="$(find kangaroo_description)/urdf/pelvis/pelvis.urdf.xacro" />
-<xacro:macro name="base_link" params="version:=2023 with_cage:=true">
+<xacro:macro name="base_link" params="with_pelvis:=false">
   <link name="base_link">
     <inertial>
@@ -14,5 +14,5 @@
       <origin xyz="0 0 0" rpy="0 0 0" />
       <geometry>
-        <mesh filename="package://kangaroo_description/meshes/${version}/base_link.stl" />
+        <mesh filename="package://kangaroo_description/meshes/base_link.stl" />
       </geometry>
       <material name="">
@@ -23,5 +23,5 @@
       <origin xyz="0 0 0" rpy="0 0 0" />
       <geometry>
-        <mesh filename="package://kangaroo_description/meshes/${version}/base_link_convex.stl" />
+        <mesh filename="package://kangaroo_description/meshes/base_link_convex.stl" />
       </geometry>
     </collision>
@@ -30,9 +30,20 @@
     <origin xyz="0.071 -0.0014 0.02" rpy="${180.0*deg_to_rad} ${0.0*deg_to_rad} ${-90.0*deg_to_rad}"/>
   </xacro:kangaroo_imu>
+    <!-- -->
+<xacro:if value="${with_pelvis}">
   <xacro:kangaroo_pelvis name="pelvis" parent="base_link" pelvis_1_offset="0" pelvis_2_offset="0">
    <origin xyz="-0.0918000000000001 0 -0.0455" rpy="0 0 0" />
   </xacro:kangaroo_pelvis>
   <xacro:include filename="$(find kangaroo_description)/urdf/torso/torso.urdf.xacro" />
-  <xacro:kangaroo_torso parent="pelvis_2_link"/> <!-- base_link -->
+  <xacro:kangaroo_torso parent="pelvis_2_link">
+    <origin xyz="0 0 0.0061" rpy="0 0 0" />
+  </xacro:kangaroo_torso> <!-- base_link -->
+</xacro:if>
+<xacro:unless value="${with_pelvis}">
+  <xacro:include filename="$(find kangaroo_description)/urdf/torso/torso.urdf.xacro" />
+  <xacro:kangaroo_torso parent="base_link">
+    <origin xyz="-0.0918000000000001 0 0.0075" rpy="0 0 0" />
+  </xacro:kangaroo_torso>
+</xacro:unless>
   <!-- waist cameras -->
   <xacro:include filename="$(find kangaroo_description)/urdf/waist/waist.urdf.xacro" />

File: kangaroo_description/urdf/leg/leg.urdf.xacro (robot description, xacro)
@@ -2,5 +2,5 @@
 <robot xmlns:xacro="http://ros.org/wiki/xacro" name="kangaroo">
   <xacro:include filename="$(find kangaroo_description)/urdf/leg/leg.transmission.xacro" />
-  <xacro:include filename="$(find kangaroo_description)/urdf/ankle/ankle_2022.urdf.xacro" />
+  <xacro:include filename="$(find kangaroo_description)/urdf/ankle/ankle.urdf.xacro" />
   <xacro:property name="deg_to_rad"       value="0.01745329251994329577" />
   <xacro:property name="eps_radians"      value="0.008" /> <!-- 0.45deg -->
@@ -9,5 +9,5 @@
   <xacro:property name="leg_1_max_pos"   value="${40.0 *deg_to_rad}" />
   <xacro:property name="leg_2_min_pos"   value="${-42.5 *deg_to_rad}" />
-  <xacro:property name="leg_2_max_pos"   value="${42.5 *deg_to_rad}" />
+  <xacro:property name="leg_2_max_pos"   value="${38.0 *deg_to_rad}" />
   <xacro:property name="leg_3_min_pos"   value="${-27.0 *deg_to_rad}" />
   <xacro:property name="leg_3_max_pos"   value="${27.0 *deg_to_rad}" />
@@ -36,15 +36,16 @@
     </gazebo>
   </xacro:macro>
-  <xacro:macro name="kangaroo_leg" params="side reflect parent *origin hipz_model:=2022 simulation:=false use_mimic:=true ft_sensors:=false">
+  <xacro:macro name="kangaroo_leg" params="side reflect parent *origin hipz_model:=2023 simulation:=false use_mimic:=true ft_sensors:=false">
     <link name="leg_${side}_1_link">
       <inertial>
-        <origin xyz="0.0461079574284527 ${reflect * -0.000826631128234001} 0.00897630312181676" rpy="0 0 0" />
-        <mass value="2.49954419149183" />
-        <inertia ixx="0.00151181747940305" ixy="${reflect * 8.83298140320242E-06}" ixz="${reflect * 2.17752660615735E-05}" iyy="0.00154876023440654" iyz="${reflect * -1.94449871986378E-05}" izz="0.00136106613590181" />
-      </inertial>
-      <visual>
-        <origin xyz="0 0 0" rpy="0 0 0" />
-        <geometry>
-          <mesh filename="package://kangaroo_description/meshes/2022/leg_1_link.stl" scale="1 ${reflect} 1"/>
+        <origin xyz="0.0063167 ${reflect * 0.0045949} -0.0083828" rpy="0 0 0" />
+        <mass value="2.7478" />
+        <inertia ixx="0.0019336" ixy="${reflect * 8.5058E-06}" ixz="${reflect * 4.8385E-05}"
+          iyy="0.0018225" iyz="${reflect * -7.282E-06}" izz="0.001426" />
+      </inertial>
+      <visual>
+        <origin xyz="0 0 0" rpy="0 0 0" />
+        <geometry>
+          <mesh filename="package://kangaroo_description/meshes/leg_1_link.stl" scale="1 ${reflect} 1"/>
         </geometry>
         <material name="">
@@ -55,5 +56,5 @@
         <origin xyz="0 0 0" rpy="0 0 0" />
         <geometry>
-          <mesh filename="package://kangaroo_description/meshes/2022/leg_1_link.stl" scale="1 ${reflect} 1"/>
+          <mesh filename="package://kangaroo_description/meshes/leg_1_link.stl"  scale="1 ${reflect} 1"/>
         </geometry>
       </collision>
@@ -65,16 +66,18 @@
       <axis xyz="0 0 1" />
       <xacro:if value="${reflect == 1}">
-        <limit lower="${leg_1_min_pos}" upper="${leg_1_max_pos}" effort="150" velocity="3.87" />
+        <limit lower="${leg_1_min_pos}" upper="${leg_1_max_pos}" effort="80" velocity="3.87" />
       </xacro:if>
       <xacro:if value="${reflect == -1}">
-        <limit lower="${reflect * leg_1_max_pos}" upper="${reflect * leg_1_min_pos}" effort="150" velocity="3.87" />
+        <limit lower="${reflect * leg_1_max_pos}" upper="${reflect * leg_1_min_pos}" effort="80" velocity="3.87" />
       </xacro:if>
     </joint>
     <link name="leg_${side}_2_link">
       <inertial>
-        <origin xyz="-0.00299642516878475 -0.000101293190038279 6.76277450706309E-10" rpy="0 0 0" />
-        <mass value="0.0907287903783648" />
-        <inertia ixx="6.10402208807908E-06" ixy="3.54403077254796E-08" ixz="-3.0910293306339E-13"
-          iyy="3.90470919341026E-05" iyz="-1.14069181428674E-12" izz="3.64238433670963E-05" />
+        <origin
+          xyz="-0.0029278 -9.6207E-05 1.0866E-09"
+          rpy="0 0 0" />
+        <mass value="0.0905312454913012" />
+        <inertia ixx="6.10166860944865E-06" ixy="4.64490555644666E-08" ixz="4.07017223451518E-13"
+          iyy="3.88541683636482E-05" iyz="-1.04538188015163E-12" izz="3.6228659424845E-05" />
       </inertial>
       <visual>
@@ -84,21 +87,27 @@
         </geometry>
         <material name="">
-          <color rgba="0.894117647058823 0.913725490196078 0.929411764705882 1" />
-        </material>
-      </visual>
+          <color rgba="0.894117647058823 0.913725490196078 0.929411764705882 1"/>
+        </material>
+      </visual>
+      <collision>
+        <origin xyz="0 0 0" rpy="0 0 0" />
+        <geometry>
+          <mesh filename="package://kangaroo_description/meshes/leg_2_link.stl" scale="1 ${reflect} 1"/>
+        </geometry>
+      </collision>
     </link>
     <joint name="leg_${side}_2_joint" type="revolute">
-      <origin xyz="0.016042 0 -0.0925" rpy="0 0 0" />
+      <origin xyz="0.015024 0 -0.1175" rpy="0 0 0" />
       <parent link="leg_${side}_1_link" />
       <child link="leg_${side}_2_link" />
       <axis xyz="0 1 0" />
-      <limit lower="${leg_2_min_pos}" upper="${leg_2_max_pos}" effort="150" velocity="3.87" />
+      <limit lower="${leg_2_min_pos}" upper="${leg_2_max_pos}" effort="230" velocity="3.87" />
     </joint>
     <link name="leg_${side}_3_link">
       <inertial>
-        <origin xyz="-0.042791492019428 ${reflect * 0.0477271400490046} -0.0411219993940296" rpy="0 0 0" />
-        <mass value="3.66987205802361" />
-        <inertia ixx="0.00226579365890287" ixy="${reflect * 0.000186528466622377}" ixz="${reflect * -9.4464170720752E-05}"
-          iyy="0.00347844100338387" iyz="${reflect * 4.48424073671215E-05}" izz="0.00335571040406776" />
+        <origin xyz="-0.033949 ${reflect * 0.049989} -0.030543" rpy="0 0 0" />
+        <mass value="3.658" />
+        <inertia ixx="0.0025968" ixy="${reflect * 0.00018723}" ixz="${reflect * -0.00014976}"
+          iyy="0.0031521" iyz="${reflect * 3.7258E-05}" izz="0.0032376" />
       </inertial>
       <visual>
@@ -123,23 +132,27 @@
       <child link="leg_${side}_3_link" />
       <axis xyz="1 0 0" />
-      <limit lower="${leg_3_min_pos}" upper="${leg_3_max_pos}" effort="150" velocity="3.87" />
+      <limit lower="${leg_3_min_pos}" upper="${leg_3_max_pos}" effort="139" velocity="3.87" />
     </joint>
     <link name="leg_${side}_femur_link">
-      <inertial>
-        <origin xyz="0.114702002010089 0.000182856660852354 -0.0143986490691173" rpy="0 0 0" />
-<xacro:if value="${use_mimic}">
-        <mass value="0.1" />
-        <inertia ixx="1.E-5" ixy="0.0" ixz="0.0" iyy="1.E-5" iyz="0.0" izz="1.E-5" />
-</xacro:if>
-<xacro:unless value="${use_mimic}">
-	<mass value="3.57408268817521" />
-        <inertia ixx="0.00247170768644724" ixy="2.87874888621229E-05" ixz="0.00247469186737281"
-          iyy="0.0126050262407564" iyz="1.01404330133204E-05" izz="0.0116319632922522" />
-</xacro:unless>
-      </inertial>
-      <visual>
-        <origin xyz="0 0 0" rpy="0 0 0" />
-        <geometry>
-          <mesh filename="package://kangaroo_description/meshes/leg_4_link.stl" />
+<!--       <xacro:if value="${use_mimic}">
+              <mass value="0.1" />
+              <inertia ixx="1.E-5" ixy="0.0" ixz="0.0" iyy="1.E-5" iyz="0.0" izz="1.E-5" />
+      </xacro:if>
+      <xacro:unless value="${use_mimic}">
+        <mass value="3.57408268817521" />
+              <inertia ixx="0.00247170768644724" ixy="2.87874888621229E-05" ixz="0.00247469186737281"
+                iyy="0.0126050262407564" iyz="1.01404330133204E-05" izz="0.0116319632922522" />
+      </xacro:unless> -->
+      <inertial>
+        <origin xyz="0.0527475093314697 0.000135688427874925 -0.146959283149568" rpy="0 0 0" />
+        <mass value="3.94567187082779" />
+        <inertia ixx="0.0111010751306264" ixy="2.24256967982894E-05" ixz="0.0025879993168672"
+          iyy="0.0121128398206334" iyz="-1.93362671261787E-05" izz="0.0025734913670898" />
+      </inertial>
+      <visual>
+        <origin xyz="0 0 0" rpy="0 0 0" />
+        <geometry>
+          <!-- The ballscrews are removed from the meshes for better visualization, but they are used for inertia computation etc -->
+          <mesh filename="package://kangaroo_description/meshes/leg_femur_link.stl" />
         </geometry>
         <material name="">
@@ -148,36 +161,40 @@
       </visual>
       <collision>
-        <origin xyz="0 0 0" rpy="0 0 0" />
-        <geometry>
-          <mesh filename="package://kangaroo_description/meshes/leg_4_link.stl"/>
+        <origin xyz="0 0 0" rpy="0 ${60.0 * deg_to_rad} 0" />
+        <geometry>
+          <!-- The ballscrews are removed from the meshes for better visualization, but they are used for inertia computation etc -->
+          <mesh filename="package://kangaroo_description/meshes/leg_4_collision_link.stl" />
         </geometry>
       </collision>
     </link>
     <link name="leg_${side}_knee_link">
-      <inertial>
-        <origin xyz="-0.158662729273678 -8.28192764317226E-05 -0.0337468261967321" rpy="0 0 0" />
-<xacro:if value="${use_mimic}">
-        <mass value="0.1" />
-        <inertia ixx="1.E-5" ixy="0.0" ixz="0.0" iyy="1.E-5" iyz="0.0" izz="1.E-5" />
-</xacro:if>
-<xacro:unless value="${use_mimic}">
-        <mass value="0.87223211672797" />
-        <inertia ixx="0.000350603269949793" ixy="6.37793331536252E-07" ixz="-0.000461550351107159"
-          iyy="0.00242184402988972" iyz="5.09327556678297E-07" izz="0.0022368624903808" />
-</xacro:unless>
-      </inertial>
-      <visual>
-        <origin xyz="0 0 0" rpy="0 0 0" />
+<!--       <xacro:if value="${use_mimic}">
+              <mass value="0.1" />
+              <inertia ixx="1.E-5" ixy="0.0" ixz="0.0" iyy="1.E-5" iyz="0.0" izz="1.E-5" />
+      </xacro:if>
+      <xacro:unless value="${use_mimic}">
+              <mass value="0.87223211672797" />
+              <inertia ixx="0.000350603269949793" ixy="6.37793331536252E-07" ixz="-0.000461550351107159"
+                iyy="0.00242184402988972" iyz="5.09327556678297E-07" izz="0.0022368624903808" />
+      </xacro:unless> -->
+      <inertial>
+        <origin xyz="-0.0569664873635563 -5.41309796184553E-05 -0.148820781933269" rpy="0 0 0" />
+        <mass value="1.02238189690276" />
+        <inertia ixx="0.00193955870555937" ixy="-7.22330237538467E-08" ixz="-0.000472475893337071"
+          iyy="0.00215347079183119" iyz="1.36520012214457E-06" izz="0.000391378760186175" />
+      </inertial>
+      <visual>
+        <origin xyz="0 0 0" rpy="0 0 0" />
+        <geometry>
+          <mesh filename="package://kangaroo_description/meshes/leg_tibia_link.stl" />
+        </geometry>
+        <material name="">
+          <color rgba="0.752941176470588 0.752941176470588 0.752941176470588 1" />
+        </material>
+      </visual>
+      <collision>
+        <origin xyz="0 0 0" rpy="0 ${-60.0 * deg_to_rad} 0" />
         <geometry>
           <mesh filename="package://kangaroo_description/meshes/leg_5_collision_link.stl" />
-        </geometry>
-        <material name="">
-          <color rgba="0.752941176470588 0.752941176470588 0.752941176470588 1" />
-        </material>
-      </visual>
-      <collision>
-        <origin xyz="0 0 0" rpy="0 0 0" />
-        <geometry>
-          <mesh filename="package://kangaroo_description/meshes/leg_5_collision_link.stl"/>
         </geometry>
       </collision>
@@ -214,8 +231,8 @@
       <child link="leg_${side}_length_link" />
       <axis xyz="0 0 1" />
-      <limit lower="${leg_min_length}" upper="${leg_max_length}" effort="1500" velocity="10" />
+      <limit lower="${leg_min_length}" upper="${leg_max_length}" effort="1100" velocity="10" />
     </joint>
     <joint name="leg_${side}_femur_joint" type="revolute">
-      <origin xyz="0 ${reflect * 0.0669} -0.09" rpy="0 ${-10.0 * deg_to_rad} 0" />
+      <origin xyz="0 ${reflect * 0.0669} -0.09" rpy="0 ${-70.0 * deg_to_rad} 0" />
       <parent link="leg_${side}_3_link" />
       <child link="leg_${side}_femur_link" />
@@ -227,5 +244,6 @@
     </joint>
     <joint name="leg_${side}_knee_joint" type="revolute">
-      <origin xyz="0.37413 0 -0.066509" rpy="0 ${20.0 * deg_to_rad} 0" />
+      <origin xyz="0.129944529468438 0 -0.357091611860635" rpy="0 ${140.0 * deg_to_rad} 0" />
+      <!-- <origin xyz="0.37413 0 -0.066509" rpy="0 ${-70.0 * deg_to_rad} 0" /> -->
       <parent link="leg_${side}_femur_link" />
       <child link="leg_${side}_knee_link" />
@@ -240,5 +258,5 @@
     	<parent link="leg_${side}_knee_link"/>
     	<child link="leg_${side}_knee_straight"/>
-    	<origin rpy="0 ${-10.0 * deg_to_rad} 0" xyz="0 0 0"/>
+    	<origin rpy="0 ${-70.0 * deg_to_rad} 0" xyz="0 0 0"/>
     </joint>
     <link name="leg_${side}_knee_lower_bearing"/>
@@ -249,5 +267,5 @@
     </joint>
     <xacro:kangaroo_ankle side="${side}" parent="leg_${side}_length_link" reflect="${reflect}" roll_joint="5" pitch_joint="4" read_actuator="leg_${side}_length_motor" ft_sensors="$(arg ft_sensors)">
-      <origin xyz="0.0 0 0.0" rpy="0 ${180 *deg_to_rad} 0" />
+      <origin xyz="0.0 0 0.0" rpy="0 ${200 *deg_to_rad} 0" />
     </xacro:kangaroo_ankle>
     <!-- Load corresponding transmission info -->

File: kangaroo_description/urdf/torso/torso.urdf.xacro (robot description, xacro)
@@ -11,5 +11,5 @@
   <xacro:include filename="$(find kangaroo_description)/urdf/deg_to_rad.xacro" />
   <xacro:include filename="$(find realsense2_description)/urdf/_d435.urdf.xacro" />
-  <xacro:macro name="kangaroo_torso" params="parent">
+  <xacro:macro name="kangaroo_torso" params="parent *origin">
   <link name="torso_link">
     <inertial>
@@ -22,5 +22,5 @@
       <origin xyz="0 0 0" rpy="0 0 0" />
       <geometry>
-        <mesh filename="package://kangaroo_description/meshes/2023/torso_link.stl" />
+        <mesh filename="package://kangaroo_description/meshes/torso_link.stl" />
       </geometry>
       <material name="">
@@ -31,11 +31,10 @@
       <origin xyz="0 0 0" rpy="0 0 0" />
       <geometry>
-        <mesh filename="package://kangaroo_description/meshes/2023/torso_link_convex.stl" />
+        <mesh filename="package://kangaroo_description/meshes/torso_link_convex.stl" />
       </geometry>
     </collision>
   </link>
   <joint name="torso_link" type="fixed">
-    <!--<origin xyz="-0.0918000000000001 0 0.0075" rpy="0 0 0" /> -->
-    <origin xyz="0 0 0.0061" rpy="0 0 0" />
+    <xacro:insert_block name="origin"/>
     <parent link="${parent}" />
     <child link="torso_link" />
