Commit message: Arms param and added pelvis transmission

File: kangaroo_description/robots/kangaroo.urdf.xacro (robot description, xacro)
@@ -9,4 +9,5 @@
         xmlns:interface="http://playerstage.sourceforge.net/gazebo/xmlschema/#interface">
   <xacro:arg name="with_pelvis" default="false" />
+  <xacro:arg name="with_arms" default="false" />
   <xacro:arg name="simulation" default="false" />
   <xacro:arg name="torso_front_camera_model" default="realsense-D435i" />
@@ -15,4 +16,5 @@
   <xacro:arg name="waist_back_camera_model" default="realsense-D435i" />
   <xacro:property name="with_pelvis" value="$(arg with_pelvis)" />
+  <xacro:property name="with_arms" value="$(arg with_arms)" />
   <xacro:property name="simulation" value="$(arg simulation)" />
   <xacro:property name="torso_front_camera_model" value="$(arg torso_front_camera_model)" />
@@ -50,4 +52,7 @@
     </joint>
   </xacro:if>
+  <!--************************-->
+  <!--           LEGS         -->
+  <!--************************-->
   <xacro:include filename="$(find kangaroo_description)/urdf/leg/leg.urdf.xacro" />
   <xacro:kangaroo_leg side="left" reflect="1" parent="base_link" simulation="$(arg simulation)" use_mimic="$(arg use_mimic)" ft_sensors="$(arg ft_sensors)">
@@ -57,11 +62,16 @@
     <origin xyz="-0.0150025976417119 -0.08 -0.0585" rpy="0 0 0"/>
   </xacro:kangaroo_leg>
-  <xacro:include filename="$(find kangaroo_description)/urdf/arm/arm.urdf.xacro" />
-  <xacro:kangaroo_arm name="arm" side="left" reflect="1" parent="torso_link" arm_1_offset="0" arm_2_offset="0" arm_3_offset="0" arm_4_offset="0">
-   <origin xyz="0 0.105954 0.384396" rpy="1.5708 0 0" />
-  </xacro:kangaroo_arm>
-  <xacro:kangaroo_arm name="arm" side="right" reflect="-1" parent="torso_link" arm_1_offset="0" arm_2_offset="0" arm_3_offset="0" arm_4_offset="0">
-   <origin xyz="0 -0.105954 0.384396" rpy="1.5708 0 3.14159" />
-  </xacro:kangaroo_arm>
+  <!--************************-->
+  <!--          ARMS          -->
+  <!--************************-->
+  <xacro:if value="$(arg with_arms)">
+    <xacro:include filename="$(find kangaroo_description)/urdf/arm/arm.urdf.xacro" />
+    <xacro:kangaroo_arm name="arm" side="left" reflect="1" parent="torso_link" arm_1_offset="0" arm_2_offset="0" arm_3_offset="0" arm_4_offset="0">
+      <origin xyz="0 0.105954 0.384396" rpy="1.5708 0 0" />
+    </xacro:kangaroo_arm>
+    <xacro:kangaroo_arm name="arm" side="right" reflect="-1" parent="torso_link" arm_1_offset="0" arm_2_offset="0" arm_3_offset="0" arm_4_offset="0">
+      <origin xyz="0 -0.105954 0.384396" rpy="1.5708 0 3.14159" />
+    </xacro:kangaroo_arm>
+  </xacro:if>
   <!-- Generic simulator_gazebo plugins -->
   <xacro:include filename="$(find kangaroo_description)/gazebo/gazebo.urdf.xacro" />

File: kangaroo_description/urdf/pelvis/pelvis.urdf.xacro (robot description, xacro)
@@ -1,168 +1,138 @@
 <?xml version="1.0" encoding="utf-8"?>
 <robot xmlns:xacro="http://ros.org/wiki/xacro" name="kangaroo">
-<xacro:macro name="kangaroo_pelvis" params="name parent *origin pelvis_1_offset pelvis_2_offset">
-  <xacro:property name="arm_eps"       value="${0.00 if no_safety_eps else 0.07}"/>
-  <link
-    name="${name}_base_link">
-    <inertial>
-      <origin
-        xyz="-0.020292 -0.000245 0.050005"
-        rpy="0 0 0" />
-      <mass
-        value="1.823847" />
-      <inertia
-        ixx="0.001676"
-        ixy="1.9E-05"
-        ixz="-0.000138"
-        iyy="0.007958"
-        iyz="-1.2E-05"
-        izz="0.00789" />
-    </inertial>
-    <visual>
-      <origin
-        xyz="0 0 0"
-        rpy="0 0 0" />
-      <geometry>
-        <mesh
-          filename="package://kangaroo_description/meshes/${name}_base_link.stl" />
-      </geometry>
-      <material
-        name="">
-        <color
-          rgba="0.75294 0.75294 0.75294 1" />
-      </material>
-    </visual>
-    <collision>
-      <origin
-        xyz="0 0 0"
-        rpy="0 0 0" />
-      <geometry>
-        <mesh
-          filename="package://kangaroo_description/meshes/${name}_base_link.stl" />
-      </geometry>
-    </collision>
-  </link>
-  <joint name="${name}_fixed_joint" type="fixed">
+  <xacro:include filename="$(find kangaroo_description)/urdf/pelvis/pelvis.transmission.xacro" />
+  <xacro:macro name="kangaroo_pelvis" params="name parent *origin pelvis_1_offset pelvis_2_offset">
+    <xacro:property name="arm_eps"       value="${0.00 if no_safety_eps else 0.07}"/>
+    <link name="${name}_base_link">
+      <inertial>
+        <origin xyz="-0.020292 -0.000245 0.050005" rpy="0 0 0" />
+        <mass value="1.823847" />
+        <inertia
+          ixx="0.001676"
+          ixy="1.9E-05"
+          ixz="-0.000138"
+          iyy="0.007958"
+          iyz="-1.2E-05"
+          izz="0.00789" />
+      </inertial>
+      <visual>
+        <origin xyz="0 0 0" rpy="0 0 0" />
+        <geometry>
+          <mesh filename="package://kangaroo_description/meshes/${name}_base_link.stl" />
+        </geometry>
+        <material name="">
+          <color rgba="0.75294 0.75294 0.75294 1" />
+        </material>
+      </visual>
+      <collision>
+        <origin xyz="0 0 0" rpy="0 0 0" />
+        <geometry>
+          <mesh filename="package://kangaroo_description/meshes/${name}_base_link.stl" />
+        </geometry>
+      </collision>
+    </link>
+    <joint name="${name}_fixed_joint" type="fixed">
       <xacro:insert_block name="origin"/>
       <parent link="${parent}" />
       <child link="${name}_base_link" />
-  </joint>
-  <link
-    name="${name}_1_link">
-    <inertial>
-      <origin
-        xyz="-0.02593 -1E-06 0.001466"
-        rpy="0 0 0" />
-      <mass
-        value="1.248563" />
-      <inertia
-        ixx="0.005394"
-        ixy="0"
-        ixz="7.7E-05"
-        iyy="0.004808"
-        iyz="0"
-        izz="0.003247" />
-    </inertial>
-    <visual>
-      <origin
-        xyz="0 0 0"
-        rpy="0 0 0" />
-      <geometry>
-        <mesh
-          filename="package://kangaroo_description/meshes/${name}_1_link.stl" />
-      </geometry>
-      <material
-        name="">
-        <color
-          rgba="0.75294 0.75294 0.75294 1" />
-      </material>
-    </visual>
-    <collision>
-      <origin
-        xyz="0 0 0"
-        rpy="0 0 0" />
-      <geometry>
-        <mesh
-          filename="package://kangaroo_description/meshes/${name}_1_link.stl" />
-      </geometry>
-    </collision>
-  </link>
-  <joint
-    name="${name}_1_joint"
-    type="revolute">
-    <origin
-      xyz="0 0 0.052"
-      rpy="0 1.5708 0" />
-    <parent
-      link="${name}_base_link" />
-    <child
-      link="${name}_1_link" />
-    <axis
-      xyz="0 0 -1" />
-    <limit
-      lower="-0.3490658504"
-      upper="0.3490658504"
-      effort="0"
-      velocity="0" />
-  </joint>
-  <link
-    name="${name}_2_link">
-    <inertial>
-      <origin
-        xyz="0 0 -0.011136"
-        rpy="0 0 0" />
-      <mass
-        value="0.435922" />
-      <inertia
-        ixx="0.000633"
-        ixy="-1.1E-05"
-        ixz="0"
-        iyy="0.000672"
-        iyz="0"
-        izz="0.001275" />
-    </inertial>
-    <visual>
-      <origin
-        xyz="0 0 0"
-        rpy="0 0 0" />
-      <geometry>
-        <mesh
-          filename="package://kangaroo_description/meshes/${name}_2_link.stl" />
-      </geometry>
-      <material
-        name="">
-        <color
-          rgba="0.75294 0.75294 0.75294 1" />
-      </material>
-    </visual>
-    <collision>
-      <origin
-        xyz="0 0 0"
-        rpy="0 0 0" />
-      <geometry>
-        <mesh
-          filename="package://kangaroo_description/meshes/${name}_2_link.stl" />
-      </geometry>
-    </collision>
-  </link>
-  <joint
-    name="${name}_2_joint"
-    type="revolute">
-    <origin
-      xyz="-0.0591 0 0"
-      rpy="0 -1.5708 0" />
-    <parent
-      link="${name}_1_link" />
-    <child
-      link="${name}_2_link" />
-    <axis
-      xyz="0 0 -1" />
-    <limit
-      lower="-1.308996939"
-      upper="1.308996939"
-      effort="0"
-      velocity="0" />
-  </joint>
-<!-- transmissions -->
-</xacro:macro>
+    </joint>
+    <link name="${name}_1_link">
+      <inertial>
+        <origin xyz="-0.02593 -1E-06 0.001466" rpy="0 0 0" />
+        <mass value="1.248563" />
+        <inertia
+          ixx="0.005394"
+          ixy="0"
+          ixz="7.7E-05"
+          iyy="0.004808"
+          iyz="0"
+          izz="0.003247" />
+      </inertial>
+      <visual>
+        <origin xyz="0 0 0" rpy="0 0 0" />
+        <geometry>
+          <mesh filename="package://kangaroo_description/meshes/${name}_1_link.stl" />
+        </geometry>
+        <material name="">
+          <color rgba="0.75294 0.75294 0.75294 1" />
+        </material>
+      </visual>
+      <collision>
+        <origin xyz="0 0 0" rpy="0 0 0" />
+        <geometry>
+          <mesh filename="package://kangaroo_description/meshes/${name}_1_link.stl" />
+        </geometry>
+      </collision>
+    </link>
+    <joint name="${name}_1_joint" type="revolute">
+      <origin xyz="0 0 0.052" rpy="0 1.5708 0" />
+      <parent link="${name}_base_link" />
+      <child link="${name}_1_link" />
+      <axis xyz="0 0 -1" />
+      <limit
+        lower="-0.3490658504"
+        upper="0.3490658504"
+        effort="0"
+        velocity="0" />
+    </joint>
+    <link name="${name}_2_link">
+      <inertial>
+        <origin xyz="0 0 -0.011136" rpy="0 0 0" />
+        <mass value="0.435922" />
+        <inertia
+          ixx="0.000633"
+          ixy="-1.1E-05"
+          ixz="0"
+          iyy="0.000672"
+          iyz="0"
+          izz="0.001275" />
+      </inertial>
+      <visual>
+        <origin xyz="0 0 0" rpy="0 0 0" />
+        <geometry>
+          <mesh filename="package://kangaroo_description/meshes/${name}_2_link.stl" />
+        </geometry>
+        <material name="">
+          <color rgba="0.75294 0.75294 0.75294 1" />
+        </material>
+      </visual>
+      <collision>
+        <origin xyz="0 0 0" rpy="0 0 0" />
+        <geometry>
+          <mesh filename="package://kangaroo_description/meshes/${name}_2_link.stl" />
+        </geometry>
+      </collision>
+    </link>
+    <joint name="${name}_2_joint" type="revolute">
+      <origin xyz="-0.0591 0 0" rpy="0 -1.5708 0" />
+      <parent link="${name}_1_link" />
+      <child  link="${name}_2_link" />
+      <axis xyz="0 0 -1" />
+      <limit
+        lower="-1.308996939"
+        upper="1.308996939"
+        effort="0"
+        velocity="0" />
+    </joint>
+    <!-- transmissions -->
+    <gazebo reference="${name}_1_link">
+      <mu1>0.9</mu1>
+      <mu2>0.9</mu2>
+    </gazebo>
+    <gazebo reference="${name}_2_link">
+      <mu1>0.9</mu1>
+      <mu2>0.9</mu2>
+    </gazebo>
+    <gazebo reference="${name}_1_joint">
+      <implicitSpringDamper>1</implicitSpringDamper>
+    </gazebo>
+    <gazebo reference="${name}_2_joint">
+      <implicitSpringDamper>1</implicitSpringDamper>
+      <provideFeedback>1</provideFeedback>
+    </gazebo>
+    <!-- extensions -->
+    <xacro:kangaroo_pelvis_differential_transmission name="${name}" number1="1" number2="2"
+                                                act_reduction1="1.0" act_reduction2="1.0"
+                                                jnt_reduction1="1.0" jnt_reduction2="1.0" />
+  </xacro:macro>
 </robot>

Commit message: Testing on the robot

File: kangaroo_description/robots/kangaroo.urdf.xacro (robot description, xacro)
@@ -68,8 +68,8 @@
     <xacro:include filename="$(find kangaroo_description)/urdf/arm/arm.urdf.xacro" />
     <xacro:kangaroo_arm name="arm" side="left" reflect="1" parent="torso_link" arm_1_offset="0" arm_2_offset="0" arm_3_offset="0" arm_4_offset="0">
-      <origin xyz="0 0.105954 0.384396" rpy="1.5708 0 0" />
+      <origin xyz="0 0.105954 0.384396" rpy="1.3963 0 0" />
     </xacro:kangaroo_arm>
     <xacro:kangaroo_arm name="arm" side="right" reflect="-1" parent="torso_link" arm_1_offset="0" arm_2_offset="0" arm_3_offset="0" arm_4_offset="0">
-      <origin xyz="0 -0.105954 0.384396" rpy="1.5708 0 3.14159" />
+      <origin xyz="0 -0.105954 0.384396" rpy="1.3963 0 3.14159" />
     </xacro:kangaroo_arm>
   </xacro:if>

Commit message: different base_link with and without pelvis, split torso from arm covers

File: kangaroo_description/robots/kangaroo.urdf.xacro (robot description, xacro)
@@ -39,5 +39,5 @@
   <!--************************-->
   <xacro:include filename="$(find kangaroo_description)/urdf/base/base.urdf.xacro"/>
-  <xacro:base_link with_pelvis="$(arg with_pelvis)"/>
+  <xacro:base_link with_pelvis="${with_pelvis}"/>
   <xacro:if value="$(arg enable_crane)">
     <xacro:include filename="$(find kangaroo_description)/urdf/crane/crane.urdf.xacro" />
@@ -65,5 +65,5 @@
   <!--          ARMS          -->
   <!--************************-->
-  <xacro:if value="$(arg with_arms)">
+  <xacro:if value="${with_arms}">
     <xacro:include filename="$(find kangaroo_description)/urdf/arm/arm.urdf.xacro" />
     <xacro:kangaroo_arm name="arm" side="left" reflect="1" parent="torso_link" arm_1_offset="0" arm_2_offset="0" arm_3_offset="0" arm_4_offset="0">
@@ -74,4 +74,16 @@
     </xacro:kangaroo_arm>
   </xacro:if>
+  <!--************************-->
+  <!--         WITHOUT ARMS   -->
+  <!--************************-->
+ <xacro:unless value="${with_arms}">
+   <xacro:include filename="$(find kangaroo_description)/urdf/arm/arm_cover.urdf.xacro" />
+   <xacro:kangaroo_arm_cover name="arm_cover" side="left" reflect="1" parent="torso_link">
+     <origin xyz="0 0.105954 0.384396" rpy="1.3963 0 0" />
+   </xacro:kangaroo_arm_cover>
+   <xacro:kangaroo_arm_cover name="arm_cover" side="right" reflect="-1" parent="torso_link">
+     <origin xyz="0 -0.105954 0.384396" rpy="1.3963 0 3.14159" />
+   </xacro:kangaroo_arm_cover>
+ </xacro:unless>
   <!-- Generic simulator_gazebo plugins -->
   <xacro:include filename="$(find kangaroo_description)/gazebo/gazebo.urdf.xacro" />

File: kangaroo_description/urdf/base/base.urdf.xacro (robot description, xacro)
@@ -4,27 +4,4 @@
 <xacro:include filename="$(find kangaroo_description)/urdf/pelvis/pelvis.urdf.xacro" />
 <xacro:macro name="base_link" params="with_pelvis:=false">
-  <link name="base_link">
-    <inertial>
-      <origin xyz="-0.051356 3.5728E-05 -0.029169" rpy="0 0 0" />
-      <mass value="2.6996" />
-      <inertia ixx="0.0058581" ixy="0.00011344" ixz="0.00017192"
-        iyy="0.008435" iyz="2.6065E-05" izz="0.012803" />
-    </inertial>
-    <visual>
-      <origin xyz="0 0 0" rpy="0 0 0" />
-      <geometry>
-        <mesh filename="package://kangaroo_description/meshes/base_link.stl" />
-      </geometry>
-      <material name="">
-        <color rgba="0.75294 0.75294 0.75294 1" />
-      </material>
-    </visual>
-    <collision>
-      <origin xyz="0 0 0" rpy="0 0 0" />
-      <geometry>
-        <mesh filename="package://kangaroo_description/meshes/base_link_convex.stl" />
-      </geometry>
-    </collision>
-  </link>
   <xacro:kangaroo_imu name="imu" parent="torso_link" update_rate="100.0">
     <origin xyz="0.071 -0.0014 0.02" rpy="${180.0*deg_to_rad} ${0.0*deg_to_rad} ${-90.0*deg_to_rad}"/>
@@ -32,4 +9,43 @@
 <!-- with pelvis DoF -->
 <xacro:if value="${with_pelvis}">
+  <link name="base_link">
+    <inertial>
+      <origin
+        xyz="-0.098278 0.0050886 -0.0322547"
+        rpy="0 0 0" />
+      <mass
+        value="2.6738" />
+      <inertia
+        ixx="0.022825"
+        ixy="-0.00038658"
+        ixz="0.00034009"
+        iyy="0.008341"
+        iyz="-4.4033E-05"
+        izz="0.027837" />
+    </inertial>
+    <visual>
+      <origin
+        xyz="0 0 0"
+        rpy="0 0 0" />
+      <geometry>
+        <mesh
+          filename="package://kangaroo_description/meshes/base_link_with_pelvis.stl" />
+      </geometry>
+      <material
+        name="">
+        <color
+          rgba="0.25098 0.25098 0.25098 1" />
+      </material>
+    </visual>
+    <collision>
+      <origin
+        xyz="0 0 0"
+        rpy="0 0 0" />
+      <geometry>
+        <mesh
+          filename="package://kangaroo_description/meshes/base_link_with_pelvis_collision.stl" />
+      </geometry>
+    </collision>
+  </link>
   <xacro:kangaroo_pelvis name="pelvis" parent="base_link" pelvis_1_offset="0" pelvis_2_offset="0">
    <origin xyz="-0.0918000000000001 0 -0.0455" rpy="0 0 0" />
@@ -41,13 +57,88 @@
 </xacro:if>
 <!-- without pelvis DoF -->
-<xacro:unless value="${with_pelvis}">
+  <xacro:unless value="${with_pelvis}">
+  <link name="base_link">
+    <inertial>
+      <origin
+        xyz="-0.0976652 0.0052196 -0.0319554"
+        rpy="0 0 0" />
+      <mass
+        value="2.5752" />
+      <inertia
+        ixx="0.022653"
+        ixy="-0.00037405"
+        ixz="0.00039289"
+        iyy="0.0079829"
+        iyz="-3.4044E-05"
+        izz="0.027412" />
+    </inertial>
+    <visual>
+      <origin xyz="0 0 0" rpy="0 0 0" />
+      <geometry>
+        <mesh filename="package://kangaroo_description/meshes/base_link.stl" />
+      </geometry>
+      <material name="">
+        <color rgba="0.25098 0.25098 0.25098 1" />
+      </material>
+    </visual>
+    <collision>
+      <origin xyz="0 0 0" rpy="0 0 0" />
+      <geometry>
+        <mesh filename="package://kangaroo_description/meshes/base_link_collision.stl" />
+      </geometry>
+    </collision>
+  </link>
+  <link name="waist_protector">
+     <inertial>
+      <origin
+        xyz="-0.06692 2E-05 -0.02479"
+        rpy="0 0 0" />
+      <mass
+        value="1.03458" />
+      <inertia
+        ixx="0.01972"
+        ixy="-1E-05"
+        ixz="-0.00037"
+        iyy="0.01996"
+        iyz="0"
+        izz="0.03879" />
+    </inertial>
+    <visual>
+      <origin
+        xyz="0 0 0"
+        rpy="0 0 0" />
+      <geometry>
+        <mesh
+          filename="package://kangaroo_description/meshes/waist_protector.stl" />
+      </geometry>
+      <material
+        name="">
+        <color
+           rgba="0.25098 0.25098 0.25098 1" />
+      </material>
+    </visual>
+    <collision>
+      <origin
+        xyz="0 0 0"
+        rpy="0 0 0" />
+      <geometry>
+        <mesh
+          filename="package://kangaroo_description/meshes/waist_protector_collision.stl" />
+      </geometry>
+    </collision>
+  </link>
+  <joint name="waist_protector_fixed_joint" type="fixed">
+      <origin xyz="0 0 0" rpy="0 0 0" />
+      <parent link="base_link" />
+      <child link="waist_protector" />
+  </joint>
   <xacro:include filename="$(find kangaroo_description)/urdf/torso/torso.urdf.xacro" />
   <xacro:kangaroo_torso parent="base_link">
     <origin xyz="-0.0918000000000001 0 0.0075" rpy="0 0 0" />
   </xacro:kangaroo_torso>
-</xacro:unless>
   <!-- waist cameras -->
   <xacro:include filename="$(find kangaroo_description)/urdf/waist/waist.urdf.xacro" />
   <xacro:kangaroo_waist parent="base_link"/>
+</xacro:unless>
 </xacro:macro>
 </robot>

File: kangaroo_description/urdf/pelvis/pelvis.urdf.xacro (robot description, xacro)
@@ -22,5 +22,5 @@
         </geometry>
         <material name="">
-          <color rgba="0.75294 0.75294 0.75294 1" />
+          <color rgba="0.25098 0.25098 0.25098 1" />
         </material>
       </visual>
@@ -28,5 +28,5 @@
         <origin xyz="0 0 0" rpy="0 0 0" />
         <geometry>
-          <mesh filename="package://kangaroo_description/meshes/${name}_base_link.stl" />
+          <mesh filename="package://kangaroo_description/meshes/${name}_base_link_collision.stl" />
         </geometry>
       </collision>
@@ -55,5 +55,5 @@
         </geometry>
         <material name="">
-          <color rgba="0.75294 0.75294 0.75294 1" />
+          <color rgba="0.25098 0.25098 0.25098 1" />
         </material>
       </visual>
@@ -61,5 +61,5 @@
         <origin xyz="0 0 0" rpy="0 0 0" />
         <geometry>
-          <mesh filename="package://kangaroo_description/meshes/${name}_1_link.stl" />
+          <mesh filename="package://kangaroo_description/meshes/${name}_1_link_collision.stl" />
         </geometry>
       </collision>
@@ -94,5 +94,5 @@
         </geometry>
         <material name="">
-          <color rgba="0.75294 0.75294 0.75294 1" />
+          <color rgba="0.25098 0.25098 0.25098 1" />
         </material>
       </visual>
@@ -100,5 +100,5 @@
         <origin xyz="0 0 0" rpy="0 0 0" />
         <geometry>
-          <mesh filename="package://kangaroo_description/meshes/${name}_2_link.stl" />
+          <mesh filename="package://kangaroo_description/meshes/${name}_2_link_collision.stl" />
         </geometry>
       </collision>

File: kangaroo_description/urdf/torso/torso.urdf.xacro (robot description, xacro)
@@ -14,8 +14,16 @@
   <link name="torso_link">
     <inertial>
-      <origin xyz="-0.0085193 -0.00033267 0.22824" rpy="0 0 0" />
-      <mass value="13.843" />
-      <inertia ixx="0.087431" ixy="1.1038E-05" ixz="-9.0502E-06"
-        iyy="0.072736" iyz="2.6862E-05" izz="0.032695" />
+      <origin
+        xyz="-0.01 -0.00074 0.22222"
+        rpy="0 0 0" />
+      <mass
+        value="13.33642" />
+      <inertia
+        ixx="0.28794"
+        ixy="-0.00047"
+        ixz="-0.00161"
+        iyy="0.26647"
+        iyz="0.00368"
+        izz="0.11215" />
     </inertial>
     <visual>
@@ -31,5 +39,5 @@
       <origin xyz="0 0 0" rpy="0 0 0" />
       <geometry>
-        <mesh filename="package://kangaroo_description/meshes/torso_link_convex.stl" />
+        <mesh filename="package://kangaroo_description/meshes/torso_link_collision.stl" />
       </geometry>
     </collision>
