Commit message: adding parameters for pelvis and legs

File: kangaroo_description/robots/kangaroo.urdf.xacro (robot description, xacro)
@@ -8,4 +8,5 @@
         xmlns:controller="http://playerstage.sourceforge.net/gazebo/xmlschema/#controller"
         xmlns:interface="http://playerstage.sourceforge.net/gazebo/xmlschema/#interface">
+  <xacro:arg name="with_legs" default="true" />
   <xacro:arg name="with_pelvis" default="false" />
   <xacro:arg name="with_arms" default="false" />
@@ -15,4 +16,5 @@
   <xacro:arg name="waist_front_camera_model" default="realsense-D435i" />
   <xacro:arg name="waist_back_camera_model" default="realsense-D435i" />
+  <xacro:property name="with_legs" value="$(arg with_legs)" />
   <xacro:property name="with_pelvis" value="$(arg with_pelvis)" />
   <xacro:property name="with_arms" value="$(arg with_arms)" />
@@ -55,11 +57,13 @@
   <!--           LEGS         -->
   <!--************************-->
-  <xacro:include filename="$(find kangaroo_description)/urdf/leg/leg.urdf.xacro" />
-  <xacro:kangaroo_leg side="left" reflect="1" parent="base_link" simulation="$(arg simulation)" use_mimic="$(arg use_mimic)" ft_sensors="$(arg ft_sensors)">
-    <origin xyz="-0.0150025976417119 0.08 -0.0585" rpy="0 0 0"/>
-  </xacro:kangaroo_leg>
-  <xacro:kangaroo_leg side="right" reflect="-1" parent="base_link" simulation="$(arg simulation)"  use_mimic="$(arg use_mimic)" ft_sensors="$(arg ft_sensors)">
-    <origin xyz="-0.0150025976417119 -0.08 -0.0585" rpy="0 0 0"/>
-  </xacro:kangaroo_leg>
+  <xacro:if value="${with_legs}">
+    <xacro:include filename="$(find kangaroo_description)/urdf/leg/leg.urdf.xacro" />
+    <xacro:kangaroo_leg side="left" reflect="1" parent="base_link" simulation="$(arg simulation)" use_mimic="$(arg use_mimic)" ft_sensors="$(arg ft_sensors)">
+      <origin xyz="-0.0150025976417119 0.08 -0.0585" rpy="0 0 0"/>
+    </xacro:kangaroo_leg>
+    <xacro:kangaroo_leg side="right" reflect="-1" parent="base_link" simulation="$(arg simulation)"  use_mimic="$(arg use_mimic)" ft_sensors="$(arg ft_sensors)">
+      <origin xyz="-0.0150025976417119 -0.08 -0.0585" rpy="0 0 0"/>
+    </xacro:kangaroo_leg>
+  </xacro:if>
   <!--************************-->
   <!--          ARMS          -->

Commit message: first draft

File: kangaroo_description/robots/kangaroo.urdf.xacro (robot description, xacro)
@@ -11,4 +11,6 @@
   <xacro:arg name="with_pelvis" default="false" />
   <xacro:arg name="with_arms" default="false" />
+  <xacro:arg name="with_belt" default="false" />
+  <xacro:arg name="torso_2024" default="false" />
   <xacro:arg name="simulation" default="false" />
   <xacro:arg name="torso_front_camera_model" default="realsense-D435i" />
@@ -19,4 +21,6 @@
   <xacro:property name="with_pelvis" value="$(arg with_pelvis)" />
   <xacro:property name="with_arms" value="$(arg with_arms)" />
+  <xacro:property name="with_belt" value="$(arg with_belt)" />
+  <xacro:property name="torso_2024" value="$(arg torso_2024)" />
   <xacro:property name="simulation" value="$(arg simulation)" />
   <xacro:property name="torso_front_camera_model" value="$(arg torso_front_camera_model)" />
@@ -41,5 +45,5 @@
   <!--************************-->
   <xacro:include filename="$(find kangaroo_description)/urdf/base/base.urdf.xacro"/>
-  <xacro:base_link with_pelvis="${with_pelvis}"/>
+  <xacro:base_link with_pelvis="${with_pelvis}" with_belt="${with_belt}" torso_2024="${torso_2024}"/>
   <xacro:if value="$(arg enable_crane)">
     <xacro:include filename="$(find kangaroo_description)/urdf/crane/crane.urdf.xacro" />

File: kangaroo_description/urdf/base/base.urdf.xacro (robot description, xacro)
@@ -3,5 +3,5 @@
 <xacro:include filename="$(find kangaroo_description)/urdf/sensors/imu.urdf.xacro"/>
 <xacro:include filename="$(find kangaroo_description)/urdf/pelvis/pelvis.urdf.xacro" />
-<xacro:macro name="base_link" params="with_pelvis:=false">
+<xacro:macro name="base_link" params="with_pelvis:=false with_belt:=false torso_2024:=false" >
   <xacro:kangaroo_imu name="imu" parent="torso_link" update_rate="100.0">
     <origin xyz="0.071 -0.0014 0.02" rpy="${180.0*deg_to_rad} ${0.0*deg_to_rad} ${-90.0*deg_to_rad}"/>
@@ -89,4 +89,11 @@
     </collision>
   </link>
+  <xacro:include filename="$(find kangaroo_description)/urdf/torso/torso.urdf.xacro" />
+  <xacro:kangaroo_torso parent="base_link">
+    <origin xyz="-0.0918000000000001 0 0.0075" rpy="0 0 0" />
+  </xacro:kangaroo_torso>
+  </xacro:unless>
+   <!-- belt waist protector and cameras-->
+  <xacro:if value="${with_belt}">
   <link name="waist_protector">
      <inertial>
@@ -133,12 +140,55 @@
       <child link="waist_protector" />
   </joint>
-  <xacro:include filename="$(find kangaroo_description)/urdf/torso/torso.urdf.xacro" />
-  <xacro:kangaroo_torso parent="base_link">
-    <origin xyz="-0.0918000000000001 0 0.0075" rpy="0 0 0" />
-  </xacro:kangaroo_torso>
   <!-- waist cameras -->
   <xacro:include filename="$(find kangaroo_description)/urdf/waist/waist.urdf.xacro" />
   <xacro:kangaroo_waist parent="base_link"/>
-</xacro:unless>
+</xacro:if>
+  <!-- with back handle -->
+  <xacro:unless value="${with_belt}">
+  <link name="back_handle">
+     <inertial>
+      <origin
+        xyz="-0.1 0 0.02479"
+        rpy="0 0 0" />
+      <mass
+        value="0.2" />
+      <inertia
+        ixx="0.01972"
+        ixy="-1E-05"
+        ixz="-0.00037"
+        iyy="0.01996"
+        iyz="0"
+        izz="0.03879" />
+    </inertial>
+    <visual>
+      <origin
+        xyz="0 0 0"
+        rpy="0 0 0" />
+      <geometry>
+        <mesh
+          filename="package://kangaroo_description/meshes/handle.stl" />
+      </geometry>
+      <material
+        name="">
+        <color
+           rgba="0.25098 0.25098 0.25098 1" />
+      </material>
+    </visual>
+    <collision>
+      <origin
+        xyz="0 0 0"
+        rpy="0 0 0" />
+      <geometry>
+        <mesh
+          filename="package://kangaroo_description/meshes/handle.stl" />
+      </geometry>
+    </collision>
+  </link>
+  <joint name="back_handle_fixed_joint" type="fixed">
+      <origin xyz="0 0 0" rpy="0 0 0" />
+      <parent link="base_link" />
+      <child link="back_handle" />
+  </joint>
+  </xacro:unless>
 </xacro:macro>
 </robot>

File: kangaroo_description/urdf/torso/torso.urdf.xacro (robot description, xacro)
@@ -30,5 +30,10 @@
       <origin xyz="0 0 0" rpy="0 0 0" />
       <geometry>
-        <mesh filename="package://kangaroo_description/meshes/torso_link.stl" />
+        <xacro:if value="${torso_2024}">
+          <mesh filename="package://kangaroo_description/meshes/torso_link_2024.stl" />
+        </xacro:if>
+        <xacro:unless value="${torso_2024}">
+          <mesh filename="package://kangaroo_description/meshes/torso_link.stl" />
+        </xacro:unless>
       </geometry>
       <material name="">
@@ -49,24 +54,46 @@
     <axis xyz="0 0 0" />
   </joint>
-  <!-- Torso front rgbd camera -->
+  <!-- Torso front upper rgbd camera -->
+  <xacro:sensor_d435
+    name="torso_front_rgbd_camera"
+    parent="torso_link"
+    topics_ns="torso_front_rgbd_camera"
+    use_nominal_extrinsics="${simulation}">
+    <origin
+      xyz="0.1056 0 0.40767"
+      rpy="0 0.5236 0"/>
+  </xacro:sensor_d435>
+  <!-- Torso back rgbd upper camera -->
+  <xacro:sensor_d435
+    name="torso_back_rgbd_camera"
+    parent="torso_link"
+    topics_ns="torso_back_rgbd_camera"
+    use_nominal_extrinsics="${simulation}">
+    <origin
+      xyz="-0.1056 0 0.40767"
+      rpy="0 0.5236 ${180.0*deg_to_rad}"/>
+  </xacro:sensor_d435>
+  <xacro:unless value="${torso_2024}">
+    <!-- Torso front lower rgbd camera -->
     <xacro:sensor_d435
-      name="torso_front_rgbd_camera"
+      name="waist_front_rgbd_camera"
       parent="torso_link"
-      topics_ns="torso_front_rgbd_camera"
+      topics_ns="waist_front_rgbd_camera"
       use_nominal_extrinsics="${simulation}">
       <origin
-        xyz="0.1056 0 0.40767"
-        rpy="0 0.5236 0"/>
+        xyz="0.09504 0 0.18649"
+        rpy="0 1.0472 0"/>
     </xacro:sensor_d435>
-  <!-- Torso back rgbd camera -->
+    <!-- Torso back lower rgbd camera -->
     <xacro:sensor_d435
-      name="torso_back_rgbd_camera"
+      name="waist_back_rgbd_camera"
       parent="torso_link"
-      topics_ns="torso_back_rgbd_camera"
+      topics_ns="waist_back_rgbd_camera"
       use_nominal_extrinsics="${simulation}">
       <origin
-        xyz="-0.1056 0 0.40767"
-        rpy="0 0.5236 ${180.0*deg_to_rad}"/>
+        xyz="-0.09504 0 0.18649"
+        rpy="0 1.0472 3.1416"/>
     </xacro:sensor_d435>
+  </xacro:unless>
   </xacro:macro>
 </robot>

Commit message: added 7dof arm

File: kangaroo_description/robots/kangaroo.urdf.xacro (robot description, xacro)
@@ -8,4 +8,6 @@
         xmlns:controller="http://playerstage.sourceforge.net/gazebo/xmlschema/#controller"
         xmlns:interface="http://playerstage.sourceforge.net/gazebo/xmlschema/#interface">
+  <!-- 4dof, 7dof -->
+  <xacro:arg name="arm_type" default="4dof" />
   <xacro:arg name="with_legs" default="true" />
   <xacro:arg name="with_pelvis" default="false" />
@@ -18,4 +20,5 @@
   <xacro:arg name="waist_front_camera_model" default="realsense-D435i" />
   <xacro:arg name="waist_back_camera_model" default="realsense-D435i" />
+  <xacro:property name="arm_type" value="$(arg arm_type)" />
   <xacro:property name="with_legs" value="$(arg with_legs)" />
   <xacro:property name="with_pelvis" value="$(arg with_pelvis)" />
@@ -75,10 +78,23 @@
   <xacro:if value="${with_arms}">
     <xacro:include filename="$(find kangaroo_description)/urdf/arm/arm.urdf.xacro" />
-    <xacro:kangaroo_arm name="arm" side="left" reflect="1" parent="torso_link" arm_1_offset="0" arm_2_offset="0" arm_3_offset="0" arm_4_offset="0">
-      <origin xyz="0 0.105954 0.384396" rpy="1.3963 0 0" />
+    <!-- Left Arm -->
+    <xacro:kangaroo_arm name="arm" type="${arm_type}" side="left" reflect="1" parent="torso_link" arm_1_offset="0" arm_2_offset="0" arm_3_offset="0" arm_4_offset="0">
+      <origin xyz="0 0.105954 0.384396" rpy="1.3963 3.14159 3.14159" />
     </xacro:kangaroo_arm>
-    <xacro:kangaroo_arm name="arm" side="right" reflect="-1" parent="torso_link" arm_1_offset="0" arm_2_offset="0" arm_3_offset="0" arm_4_offset="0">
-      <origin xyz="0 -0.105954 0.384396" rpy="1.3963 0 3.14159" />
+    <!-- Right Arm -->
+    <xacro:kangaroo_arm name="arm" type="${arm_type}" side="right" reflect="-1" parent="torso_link" arm_1_offset="0" arm_2_offset="0" arm_3_offset="0" arm_4_offset="0">
+      <origin xyz="0 -0.105954 0.384396" rpy="1.3963 3.14159 0" />
     </xacro:kangaroo_arm>
+    <xacro:if value="${arm_type=='4dof'}">
+      <xacro:include filename="$(find kangaroo_description)/urdf/end_effector/fake_forearm.urdf.xacro" />
+      <!-- Left Fake Forearm -->
+      <xacro:fake-forearm name="arm" side="left" reflect="1" parent="arm_left_3_link">
+        <origin xyz="-0.03711 -0.02 -0.17011" rpy="3.14159 1.5708 0" />
+      </xacro:fake-forearm>
+      <!-- Right Fake Forearm -->
+      <xacro:fake-forearm name="arm" side="right" reflect="-1" parent="arm_right_3_link">
+        <origin xyz="-0.03711 -0.02 -0.17011" rpy="3.14159 1.5708 0" />
+      </xacro:fake-forearm>
+    </xacro:if>
   </xacro:if>
   <!--************************-->
@@ -86,5 +102,5 @@
   <!--************************-->
  <xacro:unless value="${with_arms}">
-   <xacro:include filename="$(find kangaroo_description)/urdf/arm/arm_cover.urdf.xacro" />
+   <xacro:include filename="$(find kangaroo_description)/urdf/arm/arm_cover/arm_cover.urdf.xacro" />
    <xacro:kangaroo_arm_cover name="arm_cover" side="left" reflect="1" parent="torso_link">
      <origin xyz="0 0.105954 0.384396" rpy="1.3963 0 0" />

File: kangaroo_description/urdf/arm/arm.urdf.xacro (robot description, xacro)
@@ -1,281 +1,42 @@
 <?xml version="1.0" encoding="utf-8"?>
 <robot xmlns:xacro="http://ros.org/wiki/xacro" name="kangaroo">
-<xacro:include filename="$(find kangaroo_description)/urdf/arm/arm.transmission.xacro" />
-<xacro:property name="arm_friction"       value="1.0" />
-<xacro:property name="arm_damping"        value="1.0" />
-<xacro:property name="arm_1_max_velocity"      value="1.95" />
-<xacro:property name="arm_2_max_velocity"      value="1.95" />
-<xacro:property name="arm_3_max_velocity"      value="2.35" />
-<xacro:property name="arm_4_max_velocity"      value="2.35" />
-<xacro:property name="arm_1_max_effort"   value="43.0" />
-<xacro:property name="arm_2_max_effort"   value="43.0" />
-<xacro:property name="arm_3_max_effort"   value="43.0" />
-<xacro:property name="arm_4_max_effort"   value="43.0" />
-<xacro:macro name="kangaroo_arm" params="name side reflect parent *origin arm_1_offset arm_2_offset arm_3_offset arm_4_offset">
-  <xacro:property name="arm_eps"       value="${0.00 if no_safety_eps else 0.07}"/>
-  <link
-    name="${name}_${side}_base_link">
-    <inertial>
-      <origin
-        xyz="0 0 0"
-        rpy="0 0 0" />
-      <mass
-        value="0.1" />
-      <inertia
-        ixx="0.0000001"
-        ixy="0"
-        ixz="0"
-        iyy="0.0000001"
-        iyz="0"
-        izz="0.0000001" />
-    </inertial>
-    <visual>
-      <origin
-        xyz="0 0 0"
-        rpy="0 0 0" />
-      <geometry>
-        <mesh
-          filename="package://kangaroo_description/meshes/arm_base_link.stl" />
-      </geometry>
-      <material name="DarkGrey"/>
-    </visual>
-    <collision>
-      <origin
-        xyz="0 0 0"
-        rpy="0 0 0" />
-      <geometry>
-        <mesh
-          filename="package://kangaroo_description/meshes/arm_base_link.stl" />
-      </geometry>
-    </collision>
-  </link>
-  <joint name="${name}_${side}_fixed_joint" type="fixed">
-      <xacro:insert_block name="origin"/>
-      <parent link="${parent}" />
-      <child link="${name}_${side}_base_link" />
- </joint>
-  <!-- ARM 1 LINK -->
-  <link name="${name}_${side}_1_link">
-    <inertial>
-      <origin
-        xyz="-0.0065019 -0.002469 -0.040465" rpy="0 0 0" />
-      <mass
-        value="0.84824" />
-      <inertia
-        ixx="0.0023255"
-        ixy="5.09E-05"
-        ixz="0.0004503"
-        iyy="0.002368"
-        iyz="0.0001919"
-        izz="0.0008637" />
-    </inertial>
-    <visual>
-      <origin
-        xyz="0 0 0"
-        rpy="0 0 0" />
-      <geometry>
-        <mesh
-          filename="package://kangaroo_description/meshes/arm_1_link.stl" />
-      </geometry>
-      <material name="DarkGrey"/>
-    </visual>
-    <collision>
-      <origin
-        xyz="0 0 0"
-        rpy="0 0 0" />
-      <geometry>
-        <mesh
-          filename="package://kangaroo_description/meshes/arm_1_link.stl" />
-      </geometry>
-    </collision>
-  </link>
-  <joint name="${name}_${side}_1_joint" type="revolute">
-    <origin
-      xyz="0 0 -0.01511"
-      rpy="0 0 0" />
-    <parent
-      link="${name}_${side}_base_link" />
-    <child
-      link="${name}_${side}_1_link" />
-    <axis
-      xyz="0 0 -1" />
-    <limit
-      lower="-2.618"
-      upper="2.618"
-      effort="${arm_1_max_effort}"
-      velocity="${arm_1_max_velocity}" />
-  </joint>
-  <link
-    name="${name}_${side}_2_link">
-    <inertial>
-      <origin
-        xyz="-0.0295938 0.0049455 -0.024457"
-        rpy="0 0 0" />
-      <mass
-        value="0.9441753" />
-      <inertia
-        ixx="0.0010045"
-        ixy="-0.0004266"
-        ixz="-0.0001257"
-        iyy="0.0036599"
-        iyz="3.26E-05"
-        izz="0.0037326" />
-    </inertial>
-    <visual>
-      <origin
-        xyz="0 0 0"
-        rpy="0 0 0" />
-      <geometry>
-        <mesh
-          filename="package://kangaroo_description/meshes/arm_2_link.stl" />
-      </geometry>
-      <material name="DarkGrey"/>
-    </visual>
-    <collision>
-      <origin
-        xyz="0 0 0"
-        rpy="0 0 0" />
-      <geometry>
-        <mesh
-          filename="package://kangaroo_description/meshes/arm_2_link.stl" />
-      </geometry>
-    </collision>
-  </link>
-  <joint
-    name="${name}_${side}_2_joint" type="revolute">
-    <origin
-      xyz="-0.028337 -0.02 -0.155"
-      rpy="0 -1.5708 0" />
-    <parent
-      link="${name}_${side}_1_link" />
-    <child
-      link="${name}_${side}_2_link" />
-    <axis
-      xyz="0 0 1" />
-    <limit
-      lower="-1.1345"
-      upper="2.4435"
-      effort="${arm_2_max_effort}"
-      velocity="${arm_2_max_velocity}" />
-  </joint>
-  <link
-    name="${name}_${side}_3_link">
-    <inertial>
-      <origin
-        xyz="0.0055739 0.0021181 -0.0345099"
-        rpy="0 0 0" />
-      <mass
-        value="0.9891903" />
-      <inertia
-        ixx="0.0025603"
-        ixy="5.28E-05"
-        ixz="-0.0004831"
-        iyy="0.0026076"
-        iyz="-0.0002044"
-        izz="0.0010274" />
-    </inertial>
-    <visual>
-      <origin
-        xyz="0 0 0"
-        rpy="0 0 0" />
-      <geometry>
-        <mesh
-          filename="package://kangaroo_description/meshes/arm_3_link.stl" />
-      </geometry>
-      <material name="DarkGrey"/>
-    </visual>
-    <collision>
-      <origin
-        xyz="0 0 0"
-        rpy="0 0 0" />
-      <geometry>
-        <mesh
-          filename="package://kangaroo_description/meshes/arm_3_link.stl" />
-      </geometry>
-    </collision>
-  </link>
-  <joint
-    name="${name}_${side}_3_joint"
-    type="revolute">
-    <origin
-      xyz="-0.175 0.02 -0.028337"
-      rpy="0 1.5708 0" />
-    <parent
-      link="${name}_${side}_2_link" />
-    <child
-      link="${name}_${side}_3_link" />
-    <axis
-      xyz="0 0 -1" />
-    <limit
-      lower="-2.618"
-      upper="2.618"
-      effort="${arm_3_max_effort}"
-      velocity="${arm_3_max_velocity}" />
-  </joint>
-  <link
-    name="${name}_${side}_4_link">
-    <inertial>
-      <origin
-        xyz="0.0752641 -0.0079317 -0.023427"
-        rpy="0 0 0" />
-      <mass
-        value="1.4353488" />
-      <inertia
-        ixx="0.0012553"
-        ixy="-0.0012835"
-        ixz="9.49E-05"
-        iyy="0.0209442"
-        iyz="-1.1E-06"
-        izz="0.0210127" />
-    </inertial>
-    <visual>
-      <origin
-        xyz="0 0 0"
-        rpy="0 0 0" />
-      <geometry>
-        <mesh
-          filename="package://kangaroo_description/meshes/arm_${side}_4_link.stl" scale="1 1 1"/>
-      </geometry>
-      <material name="DarkGrey"/>
-    </visual>
-    <collision>
-      <origin
-        xyz="0 0 0"
-        rpy="0 0 0" />
-      <geometry>
-        <mesh
-          filename="package://kangaroo_description/meshes/arm_${side}_4_link.stl" scale="1 1 1"/>
-      </geometry>
-    </collision>
-  </link>
-  <joint
-    name="${name}_${side}_4_joint"
-    type="revolute">
-    <origin
-      xyz="0.0283 0.02 -0.155"
-      rpy="0 1.5708 0" />
-    <parent
-      link="${name}_${side}_3_link" />
-    <child
-      link="${name}_${side}_4_link" />
-    <axis
-      xyz="0 0 1" />
-    <limit
-      lower="-1.1345"
-      upper="2.4435"
-      effort="${arm_4_max_effort}"
-      velocity="${arm_4_max_velocity}" />
-  </joint>
-  <link name="ef_${side}_link"/>
-  <joint name="ef_${side}_joint" type="fixed">
-      <origin xyz="0.415 -0.015 ${-0.025 + reflect * 0.015}" rpy="0 0 0" />
-    <parent link="${name}_${side}_4_link" />
-    <child link="ef_${side}_link" />
+  <xacro:macro name="kangaroo_arm" params="name side type reflect parent *origin arm_1_offset:=0.0 arm_2_offset:=0.0 arm_3_offset:=0.0 arm_4_offset:=0.0">
+    <!-- 4DOF Arm -->
+    <xacro:if value="${type in ['4dof', '5dof', '7dof']}">
+      <xacro:include filename="$(find kangaroo_description)/urdf/arm/4dof/4dof_arm.urdf.xacro" />
+      <xacro:kangaroo_4dof_arm name="${name}" side="${side}" reflect="${reflect}" parent="${parent}">
+        <xacro:insert_block name="origin"/>
+      </xacro:kangaroo_4dof_arm>
+      <xacro:property name="tip_link" value="4" />
+      <xacro:property name="tool_link_xyz" value="0.35 -0.02 -0.0255" />
+      <xacro:property name="tool_link_rpy" value="0 0 0" />
+    </xacro:if>
+    <!-- 5DOF Arm -->
+    <xacro:if value="${type in ['5dof', '7dof']}">
+      <xacro:include filename="$(find kangaroo_description)/urdf/arm/5dof/5dof_arm.urdf.xacro" />
+      <xacro:kangaroo_5dof_arm name="${name}" side="${side}" reflect="${reflect}" parent="${name}_${side}_3_link">
+        <origin xyz="-0.03711 -0.02 -0.17011" rpy="0 -1.5708 0" />
+      </xacro:kangaroo_5dof_arm>
+      <xacro:property name="tip_link" value="5" />
+      <xacro:property name="tool_link_xyz" value="0 0 0.0303" />
+      <xacro:property name="tool_link_rpy" value="0 0 3.14159" />
+    </xacro:if>
+    <!-- 7DOF Arm -->
+    <xacro:if value="${type in ['7dof']}">
+      <xacro:include filename="$(find kangaroo_description)/urdf/arm/7dof/7dof_arm.urdf.xacro" />
+      <xacro:kangaroo_7dof_arm name="${name}" side="${side}" reflect="${reflect}" parent="${name}_${side}_4_link">
+        <origin xyz="-0.17011 0.02 -0.03711" rpy="0 -1.5708 0" />
+      </xacro:kangaroo_7dof_arm>
+      <xacro:property name="tip_link" value="7" />
+      <xacro:property name="tool_link_xyz" value="0 0 0.017" />
+      <xacro:property name="tool_link_rpy" value="0 0 0" />
+    </xacro:if>
+    <!-- Tool Link -->
+    <link name="${name}_${side}_tool_link" />
+    <joint name="${name}_${side}_tool_fixed_joint" type="fixed">
+      <origin xyz="${tool_link_xyz}" rpy="${tool_link_rpy}" />
+      <parent link="${name}_${side}_${tip_link}_link" />
+      <child link="${name}_${side}_tool_link" />
     </joint>
-<!-- TRANSMISSIONS -->
-    <xacro:arm_simple_transmission name="${name}_${side}" number="1" reduction="1.0" offset_value="${arm_1_offset}"/>
-    <xacro:arm_simple_transmission name="${name}_${side}" number="2" reduction="1.0" offset_value="${arm_2_offset}"/>
-    <xacro:arm_simple_transmission name="${name}_${side}" number="3" reduction="1.0" offset_value="${arm_3_offset}"/>
-    <xacro:arm_simple_transmission name="${name}_${side}" number="4" reduction="1.0" offset_value="${arm_4_offset}"/>
- </xacro:macro>
+  </xacro:macro>
 </robot>

File: kangaroo_description/urdf/materials.urdf.xacro (robot description, xacro)
@@ -23,4 +23,7 @@
    <color rgba="0.3 0.3 0.3 1.0"/>
  </material>
+ <material name="pal/DarkGrey">
+   <color rgba="0.3 0.3 0.3 1.0"/>
+ </material>
   <material name="Red">
     <color rgba="0.8 0.0 0.0 1.0"/>
