Commit message: added gripper configuration parameters

File: kangaroo_description/robots/kangaroo.urdf.xacro (robot description, xacro)
@@ -9,4 +9,5 @@
         xmlns:interface="http://playerstage.sourceforge.net/gazebo/xmlschema/#interface">
   <!-- 4dof, 7dof -->
+  <xacro:arg name="end_effector_type" default="fake-forearm" />
   <xacro:arg name="arm_type" default="4dof" />
   <xacro:arg name="with_legs" default="true" />
@@ -20,4 +21,5 @@
   <xacro:arg name="waist_front_camera_model" default="realsense-D435i" />
   <xacro:arg name="waist_back_camera_model" default="realsense-D435i" />
+  <xacro:property name="end_effector_type" default="$(arg end_effector_type)" />
   <xacro:property name="arm_type" value="$(arg arm_type)" />
   <xacro:property name="with_legs" value="$(arg with_legs)" />
@@ -31,4 +33,15 @@
   <xacro:property name="waist_front_camera_model" value="$(arg waist_front_camera_model)" />
   <xacro:property name="waist_back_camera_model" value="$(arg waist_back_camera_model)" />
+  <!-- Valid Combinations -->
+  <xacro:if value="${arm_type in ['4dof']}">
+    <xacro:if value="${end_effector_type not in ['fake-forearm']}">
+      <xacro:wrong_arm_end_effector_combination />
+    </xacro:if>
+  </xacro:if>
+  <xacro:if value="${arm_type in ['7dof']}">
+    <xacro:if value="${end_effector_type not in ['no-end-effector', 'gripper']}">
+      <xacro:wrong_arm_end_effector_combination />
+    </xacro:if>
+  </xacro:if>
   <xacro:if value="${torso_front_camera_model not in ['realsense-D435i']}">
     <xacro:wrong_torso_front_camera_model/>
@@ -86,4 +99,7 @@
       <origin xyz="0 -0.105954 0.384396" rpy="1.3963 3.14159 0" />
     </xacro:kangaroo_arm>
+    <!--************************-->
+    <!--      END EFFECTOR      -->
+    <!--************************-->
     <xacro:if value="${arm_type=='4dof'}">
       <xacro:include filename="$(find kangaroo_description)/urdf/end_effector/fake_forearm.urdf.xacro" />
@@ -96,4 +112,15 @@
         <origin xyz="-0.03711 -0.02 -0.17011" rpy="3.14159 1.5708 0" />
       </xacro:fake-forearm>
+    </xacro:if>
+    <xacro:if value="${arm_type=='7dof' and end_effector_type=='gripper'}">
+      <xacro:include filename="$(find kangaroo_description)/urdf/end_effector/gripper/gripper.urdf.xacro" />
+      <!-- Left Gripper -->
+      <xacro:pal_pro_gripper tool_changer="true" name="gripper_left" parent="arm_left_tool_link">
+        <origin xyz="0.0 0.0 0.0" rpy="0 0 -1.57" />
+      </xacro:pal_pro_gripper>
+      <!-- Right Gripper -->
+      <xacro:pal_pro_gripper tool_changer="true" name="gripper_right" parent="arm_right_tool_link">
+        <origin xyz="0.0 0.0 0.0" rpy="0 0 -1.57" />
+      </xacro:pal_pro_gripper>
     </xacro:if>
   </xacro:if>

Commit message: added free floating base joint by defauladded free floating base joint by default

File: kangaroo_description/robots/kangaroo.urdf.xacro (robot description, xacro)
@@ -234,14 +234,12 @@
     <xacro:include filename="$(find kangaroo_description)/mujoco/mj_tags.xacro" />
     <xacro:include filename="$(find pal_mujoco_scenes)/scenes/${world_name}.xacro" />
-    <xacro:if value="${sim_type == 'mujoco'}">
-    <!-- <xacro:if value="${fixation_type == 'floating' and sim_type == 'mujoco'}"> -->
-      <link name="origin">
-      </link>
-      <joint name="free_floating" type="floating">
-        <parent link="origin" />
-        <child link="base_link" />
-        <origin xyz="0.0 0.0 0.95" />
-      </joint>
-    </xacro:if>
+    <!-- Add free floating joint -->
+    <link name="origin">
+    </link>
+    <joint name="free_floating" type="floating">
+      <parent link="origin" />
+      <child link="base_link" />
+      <origin xyz="0.0 0.0 0.95" />
+    </joint>
     <mujoco_inputs>
       <!-- Mujoco environment -->

Commit message: handling floating base from launchfile

File: kangaroo_description/robots/kangaroo.urdf.xacro (robot description, xacro)
@@ -234,12 +234,4 @@
     <xacro:include filename="$(find kangaroo_description)/mujoco/mj_tags.xacro" />
     <xacro:include filename="$(find pal_mujoco_scenes)/scenes/${world_name}.xacro" />
-    <!-- Add free floating joint -->
-    <link name="origin">
-    </link>
-    <joint name="free_floating" type="floating">
-      <parent link="origin" />
-      <child link="base_link" />
-      <origin xyz="0.0 0.0 0.95" />
-    </joint>
     <mujoco_inputs>
       <!-- Mujoco environment -->
@@ -369,4 +361,5 @@
         <!-- <modify_element type="joint" name="joint1" frictionloss="1.0" damping="2.0"/>
         <modify_element type="body" name="forearm" gravcomp="1.0"/> -->
+        <modify_element type="body" name="base_link" pos="0 0 0.9" quat="1 0 0 0" />
       </processed_inputs>
     </mujoco_inputs>

Commit message: test to make inference work

File: kangaroo_description/robots/kangaroo.urdf.xacro (robot description, xacro)
@@ -225,4 +225,5 @@
       <!-- The contents of `raw_inputs` will be copied and pasted directly into the MJCF -->
       <raw_inputs>
+        <option timestep="0.001" />
         <!-- Default values -->
         <default>
@@ -279,5 +280,9 @@
         <!-- special pal_mujoco tag. This is the least invasive solution I found to add a site to a body  -->
         <!-- this tag won't work in a regular mjcf xml file -->
-        <!-- <site name="base_footprint_site" body_name="base_footprint"/> -->
+        <sensor>
+          <framequat name="imu_sensor_quat" objtype="site" objname="imu_link" />
+          <gyro name="imu_sensor_gyro" site="imu_link" />
+          <accelerometer name="imu_sensor_accel" site="imu_link" />
+        </sensor>
       </raw_inputs>
       <processed_inputs>

File: kangaroo_description/ros2_control/ros2_control.urdf.xacro (robot description, xacro)
@@ -39,6 +39,8 @@
           <plugin>mujoco_ros2_control/MujocoSystemInterface</plugin>
           <!-- Override the slowdown settings in the Simulate App and run at 1x speed -->
+          <param name="mujoco_model">/home/user/mujoco_ws/mjcf_data_4dof_fake-forearm/scene.xml</param>
           <param name="sim_speed_factor">1.0</param>
           <param name="pids_config_file">$(find kangaroo_mujoco)/config/pids.yaml</param>
+          <!-- <param name="pids_config_file">$(find kangaroo_mujoco)/config/rl_pids.yaml</param> -->
           <param name="initial_keyframe">home</param>
         </xacro:unless>
@@ -59,4 +61,25 @@
         <xacro:end_effector_ros2_control side="right" end_effector_type="${end_effector_type}"/>
       </xacro:if>
+      <sensor name="imu_sensor">
+        <param name="mujoco_type">imu</param>
+        <!-- There is no requirement for the mujoco_sensor_name to match the ros2_control sensor name -->
+        <param name="mujoco_sensor_name">imu_sensor</param>
+        <!-- Default value of orientation_mjcf_suffix is '_quat' -->
+        <param name="orientation_mjcf_suffix">_quat</param>
+        <!-- Default value of angular_velocity_mjcf_suffix is '_gyro' -->
+        <param name="angular_velocity_mjcf_suffix">_gyro</param>
+        <!-- Default value of linear_acceleration_mjcf_suffix is '_accel' -->
+        <param name="linear_acceleration_mjcf_suffix">_accel</param>
+        <state_interface name="orientation.x"/>
+        <state_interface name="orientation.y"/>
+        <state_interface name="orientation.z"/>
+        <state_interface name="orientation.w"/>
+        <state_interface name="angular_velocity.x"/>
+        <state_interface name="angular_velocity.y"/>
+        <state_interface name="angular_velocity.z"/>
+        <state_interface name="linear_acceleration.x"/>
+        <state_interface name="linear_acceleration.y"/>
+        <state_interface name="linear_acceleration.z"/>
+      </sensor>
     </ros2_control>
   </xacro:macro>

File: kangaroo_description/urdf/base/base.urdf.xacro (robot description, xacro)
@@ -14,11 +14,11 @@
   </xacro:unless>
   <!-- Sensors -->
-  <!-- <xacro:include filename="$(find kangaroo_description)/urdf/sensors/imu.urdf.xacro"/> -->
+  <xacro:include filename="$(find kangaroo_description)/urdf/sensors/imu.urdf.xacro"/>
   <!-- BASE LINK MACRO -->
   <xacro:macro name="base_link" params="has_pelvis:=false">
     <!-- IMU -->
-    <!-- <xacro:kangaroo_imu name="imu" parent="torso_link" update_rate="100.0">
+    <xacro:kangaroo_imu name="imu" parent="torso_link" >
       <origin xyz="0.071 -0.0014 0.02" rpy="${180.0*deg_to_rad} ${0.0*deg_to_rad} ${-90.0*deg_to_rad}"/>
-    </xacro:kangaroo_imu> -->
+    </xacro:kangaroo_imu>
     <!-- has pelvis DoF -->
     <xacro:if value="${has_pelvis}">

File: kangaroo_description/urdf/leg/leg.urdf.xacro (robot description, xacro)
@@ -168,5 +168,5 @@
           iyy="0.00215347079183119" iyz="1.36520012214457E-06" izz="0.000391378760186175" />
       </inertial>
-      <visual>
+      <!-- <visual>
         <origin xyz="0 0 0" rpy="0 0 0" />
         <geometry>
@@ -174,6 +174,6 @@
         </geometry>
         <material name="pal/DarkGrey" />
-      </visual>
-      <xacro:link_collision
+      </visual> -->
+      <!-- <xacro:link_collision
         mujoco="${sim_type in ['mujoco-ros2-control', 'mujoco']}"
         collision_type="${collision_type}"
@@ -186,5 +186,5 @@
             <xacro:origin xyz="-0.0569664873635563 ${reflect * 7.99553099622616e-06} -0.148820781933269" rpy="0 ${30.0 * deg_to_rad} 0" condition="${collision_type == 'capsule'}"/>
           </properties>
-      </xacro:link_collision>
+      </xacro:link_collision> -->
     </link>
     <!-- We approximate the virtual length link with a small cylinder mass and inertia -->

Commit message: update urdf and cleaning

File: kangaroo_description/robots/kangaroo.urdf.xacro (robot description, xacro)
@@ -34,11 +34,11 @@
   <xacro:arg name="use_mimic" default="False" />
   <!-- realsense-D435i -->
-  <xacro:arg name="torso_front_camera_model" default="realsense-D435i" />
+  <xacro:arg name="torso_front_up_camera_model" default="realsense-d435i" />
   <!-- realsense-D435i -->
-  <xacro:arg name="torso_back_camera_model" default="realsense-D435i" />
+  <xacro:arg name="torso_back_up_camera_model" default="realsense-d435i" />
   <!-- realsense-D435i -->
-  <xacro:arg name="waist_front_camera_model" default="realsense-D435i" />
+  <xacro:arg name="torso_front_down_camera_model" default="realsense-d435i" />
   <!-- realsense-D435i -->
-  <xacro:arg name="waist_back_camera_model" default="realsense-D435i" />
+  <xacro:arg name="torso_back_down_camera_model" default="realsense-d435i" />
   <!-- COMMON ARGS -->
   <!-- True, False -->
@@ -65,8 +65,11 @@
   <xacro:property name="world_name" value="$(arg world_name)" />
   <xacro:property name="use_mimic" value="$(arg use_mimic)" />
-  <xacro:property name="torso_front_camera_model" value="$(arg torso_front_camera_model)" />
-  <xacro:property name="torso_back_camera_model" value="$(arg torso_back_camera_model)" />
-  <xacro:property name="waist_front_camera_model" value="$(arg waist_front_camera_model)" />
-  <xacro:property name="waist_back_camera_model" value="$(arg waist_back_camera_model)" />
+  <xacro:property name="torso_front_up_camera_model" value="$(arg torso_front_up_camera_model)" />
+  <xacro:property name="torso_back_up_camera_model" value="$(arg torso_back_up_camera_model)" />
+  <xacro:property name="torso_front_down_camera_model" value="$(arg torso_front_down_camera_model)" />
+  <xacro:property name="torso_back_down_camera_model" value="$(arg torso_back_down_camera_model)" />
+  <!-- Camera properties -->
+  <xacro:property name="gazebo_version" value="classic"/>
+  <xacro:property name="namespace" value=""/>
   <!-- Properties check -->
   <xacro:if value="${sim_type not in ['mujoco-ros2-control', 'mujoco', 'no-simulation']}">
@@ -114,15 +117,15 @@
     <xacro:wrong_legs_type />
   </xacro:if>
-  <xacro:if value="${torso_front_camera_model not in ['realsense-D435i']}">
-    <xacro:wrong_torso_front_camera_model/>
-  </xacro:if>
-  <xacro:if value="${torso_back_camera_model not in ['realsense-D435i']}">
-    <xacro:wrong_torso_back_camera_model/>
-  </xacro:if>
-  <xacro:if value="${waist_front_camera_model not in ['realsense-D435i']}">
-    <xacro:wrong_waist_front_camera_model/>
-  </xacro:if>
-  <xacro:if value="${waist_back_camera_model not in ['realsense-D435i']}">
-    <xacro:wrong_waist_back_camera_model/>
+  <xacro:if value="${torso_front_up_camera_model not in ['realsense-d435i']}">
+    <xacro:wrong_torso_front_up_camera_model/>
+  </xacro:if>
+  <xacro:if value="${torso_back_up_camera_model not in ['realsense-d435i']}">
+    <xacro:wrong_torso_back_up_camera_model/>
+  </xacro:if>
+  <xacro:if value="${torso_front_down_camera_model not in ['realsense-d435i']}">
+    <xacro:wrong_torso_front_down_camera_model/>
+  </xacro:if>
+  <xacro:if value="${torso_back_down_camera_model not in ['realsense-d435i']}">
+    <xacro:wrong_torso_back_down_camera_model/>
   </xacro:if>
   <!-- INCLUDES -->

File: kangaroo_description/urdf/torso/torso.urdf.xacro (robot description, xacro)
@@ -9,10 +9,7 @@
 <robot xmlns:xacro="http://ros.org/wiki/xacro">
   <!--File includes-->
-  <!-- <xacro:include filename="$(find kangaroo_description)/urdf/deg_to_rad.xacro" />
-  <xacro:include filename="$(find kangaroo_description)/urdf/collision.xacro" /> -->
+  <!--<xacro:include filename="$(find kangaroo_description)/urdf/collision.xacro" /> -->
   <xacro:include filename="$(find pal_urdf_utils)/urdf/camera/realsense_d435i.urdf.xacro"/>
   <xacro:macro name="kangaroo_torso" params="parent *origin">
-  <xacro:property name="gazebo_version" value="classic"/>
-  <xacro:property name="namespace" value=""/>
   <link name="torso_link">
     <inertial>
@@ -55,16 +52,16 @@
     <child link="torso_link" />
   </joint>
-  <!-- Torso back cameras -->
-  <xacro:realsense_d435i name="torso_front_roof_rgbd_camera"  parent="torso_link" use_nominal_extrinsics="false">
+  <!-- Torso front cameras -->
+  <xacro:realsense_d435i name="torso_front_up_rgbd_camera"  parent="torso_link" use_nominal_extrinsics="${use_sim_time}">
       <origin xyz="0.1056 0 0.40767" rpy="0 0.5236 0"/>
   </xacro:realsense_d435i>
-  <xacro:realsense_d435i name="torso_front_base_rgbd_camera"  parent="torso_link" use_nominal_extrinsics="false">
+  <xacro:realsense_d435i name="torso_front_down_rgbd_camera"  parent="torso_link" use_nominal_extrinsics="${use_sim_time}">
     <origin xyz="0.095041 0 0.186487" rpy="0 1.0472 0"/>
   </xacro:realsense_d435i>
   <!-- Torso back cameras -->
-  <xacro:realsense_d435i name="torso_back_roof_rgbd_camera"  parent="torso_link" use_nominal_extrinsics="false">
+  <xacro:realsense_d435i name="torso_back_up_rgbd_camera"  parent="torso_link" use_nominal_extrinsics="${use_sim_time}">
     <origin xyz="-0.1056 0 0.40767" rpy="0 0.5236 3.14159"/>
   </xacro:realsense_d435i>
-  <xacro:realsense_d435i name="torso_back_base_rgbd_camera"  parent="torso_link" use_nominal_extrinsics="false">
+  <xacro:realsense_d435i name="torso_back_down_rgbd_camera"  parent="torso_link" use_nominal_extrinsics="${use_sim_time}">
     <origin xyz="-0.095041 0 0.186487" rpy="0 1.0472 3.14159"/>
   </xacro:realsense_d435i>

File: kangaroo_description/urdf/waist/waist.urdf.xacro (robot description, xacro)
@@ -9,28 +9,12 @@
 <robot xmlns:xacro="http://ros.org/wiki/xacro">
   <!--File includes-->
-  <!-- <xacro:include filename="$(find kangaroo_description)/urdf/deg_to_rad.xacro" /> -->
-  <!-- <xacro:include filename="$(find realsense2_description)/urdf/_d435.urdf.xacro" /> -->
+  <xacro:include filename="$(find pal_urdf_utils)/urdf/camera/realsense_d435i.urdf.xacro"/>
   <xacro:macro name="kangaroo_waist" params="parent">
-  <!-- Waist front rgbd camera -->
-    <!-- <xacro:sensor_d435
-      name="waist_front_rgbd_camera"
-      parent="${parent}"
-      topics_ns="waist_front_rgbd_camera"
-      use_nominal_extrinsics="${simulation}">
-      <origin
-        xyz="0.11998 0 -0.0085"
-        rpy="0 1.125 0"/>
-    </xacro:sensor_d435> -->
-  <!-- Waist back rgbd camera -->
-    <!-- <xacro:sensor_d435
-      name="waist_back_rgbd_camera"
-      parent="${parent}"
-      topics_ns="waist_back_rgbd_camera"
-      use_nominal_extrinsics="${simulation}">
-      <origin
-        xyz="-0.20238 0 -0.05049"
-        rpy="${180.0*deg_to_rad} 2.0944 0"/>
-    </xacro:sensor_d435>
-   -->
+  <xacro:realsense_d435i name="waist_front_rgbd_camera"  parent="${parent}" use_nominal_extrinsics="${use_sim_time}">
+    <origin xyz="0.11998 0 -0.0085" rpy="0 1.125 0"/>
+  </xacro:realsense_d435i>
+  <xacro:realsense_d435i name="waist_back_rgbd_camera"  parent="${parent}" use_nominal_extrinsics="${use_sim_time}">
+    <origin xyz="-0.20238 0 -0.05049" rpy="3.14159 2.0944 0"/>
+  </xacro:realsense_d435i>
   </xacro:macro>
 </robot>

Commit message: using rear instead of back

File: kangaroo_description/robots/kangaroo.urdf.xacro (robot description, xacro)
@@ -36,9 +36,9 @@
   <xacro:arg name="torso_front_up_camera_model" default="realsense-d435i" />
   <!-- realsense-D435i -->
-  <xacro:arg name="torso_back_up_camera_model" default="realsense-d435i" />
+  <xacro:arg name="torso_rear_up_camera_model" default="realsense-d435i" />
   <!-- realsense-D435i -->
   <xacro:arg name="torso_front_down_camera_model" default="realsense-d435i" />
   <!-- realsense-D435i -->
-  <xacro:arg name="torso_back_down_camera_model" default="realsense-d435i" />
+  <xacro:arg name="torso_rear_down_camera_model" default="realsense-d435i" />
   <!-- COMMON ARGS -->
   <!-- True, False -->
@@ -66,7 +66,7 @@
   <xacro:property name="use_mimic" value="$(arg use_mimic)" />
   <xacro:property name="torso_front_up_camera_model" value="$(arg torso_front_up_camera_model)" />
-  <xacro:property name="torso_back_up_camera_model" value="$(arg torso_back_up_camera_model)" />
+  <xacro:property name="torso_rear_up_camera_model" value="$(arg torso_rear_up_camera_model)" />
   <xacro:property name="torso_front_down_camera_model" value="$(arg torso_front_down_camera_model)" />
-  <xacro:property name="torso_back_down_camera_model" value="$(arg torso_back_down_camera_model)" />
+  <xacro:property name="torso_rear_down_camera_model" value="$(arg torso_rear_down_camera_model)" />
   <!-- Camera properties -->
   <xacro:property name="gazebo_version" value="classic"/>
@@ -120,12 +120,12 @@
     <xacro:wrong_torso_front_up_camera_model/>
   </xacro:if>
-  <xacro:if value="${torso_back_up_camera_model not in ['realsense-d435i']}">
-    <xacro:wrong_torso_back_up_camera_model/>
+  <xacro:if value="${torso_rear_up_camera_model not in ['realsense-d435i']}">
+    <xacro:wrong_torso_rear_up_camera_model/>
   </xacro:if>
   <xacro:if value="${torso_front_down_camera_model not in ['realsense-d435i']}">
     <xacro:wrong_torso_front_down_camera_model/>
   </xacro:if>
-  <xacro:if value="${torso_back_down_camera_model not in ['realsense-d435i']}">
-    <xacro:wrong_torso_back_down_camera_model/>
+  <xacro:if value="${torso_rear_down_camera_model not in ['realsense-d435i']}">
+    <xacro:wrong_torso_rear_down_camera_model/>
   </xacro:if>
   <!-- INCLUDES -->

File: kangaroo_description/urdf/torso/torso.urdf.xacro (robot description, xacro)
@@ -60,8 +60,8 @@
   </xacro:realsense_d435i>
   <!-- Torso back cameras -->
-  <xacro:realsense_d435i name="torso_back_up_rgbd_camera"  parent="torso_link" use_nominal_extrinsics="${use_sim_time}">
+  <xacro:realsense_d435i name="torso_rear_up_rgbd_camera"  parent="torso_link" use_nominal_extrinsics="${use_sim_time}">
     <origin xyz="-0.1056 0 0.40767" rpy="0 0.5236 3.14159"/>
   </xacro:realsense_d435i>
-  <xacro:realsense_d435i name="torso_back_down_rgbd_camera"  parent="torso_link" use_nominal_extrinsics="${use_sim_time}">
+  <xacro:realsense_d435i name="torso_rear_down_rgbd_camera"  parent="torso_link" use_nominal_extrinsics="${use_sim_time}">
     <origin xyz="-0.095041 0 0.186487" rpy="0 1.0472 3.14159"/>
   </xacro:realsense_d435i>
