Commit message: Split end effectors into sides

File: kangaroo_description/robots/kangaroo.urdf.xacro (robot description, xacro)
@@ -23,5 +23,6 @@
   <xacro:arg name="arm_type" default="4dof" />
   <!-- cover, no-end-effector, fake-forearm, gripper, RH8D -->
-  <xacro:arg name="end_effector_type" default="fake-forearm" />
+  <xacro:arg name="end_effector_right" default="fake-forearm" />
+  <xacro:arg name="end_effector_left" default="fake-forearm" />
   <!-- fixed, floating -->
   <xacro:arg name="fixation_type" default="floating" />
@@ -62,5 +63,6 @@
   <xacro:property name="legs_type" value="$(arg legs_type)" />
   <xacro:property name="fixation_type" value="$(arg fixation_type)" />
-  <xacro:property name="end_effector_type" value="$(arg end_effector_type)" />
+  <xacro:property name="end_effector_right" value="$(arg end_effector_right)" />
+  <xacro:property name="end_effector_left" value="$(arg end_effector_left)" />
   <xacro:property name="world_name" value="$(arg world_name)" />
   <xacro:property name="use_mimic" value="$(arg use_mimic)" />
@@ -89,25 +91,28 @@
   </xacro:if>
   <!-- (ft-gripper) not available -->
-  <xacro:if value="${end_effector_type not in ['cover', 'no-end-effector', 'fake-forearm', 'gripper', 'RH8D']}">
-    <xacro:wrong_end_effector_type />
+  <xacro:if value="${end_effector_right not in ['cover', 'no-end-effector', 'fake-forearm', 'gripper', 'RH8D']}">
+    <xacro:wrong_end_effector_right />
+  </xacro:if>
+  <xacro:if value="${end_effector_left not in ['cover', 'no-end-effector', 'fake-forearm', 'gripper', 'RH8D']}">
+    <xacro:wrong_end_effector_left />
   </xacro:if>
   <!-- Valid Combinations -->
   <xacro:if value="${arm_type in ['no-arm']}">
-    <xacro:if value="${end_effector_type not in ['cover']}">
+    <xacro:if value="${end_effector_right not in ['cover']}">
       <xacro:wrong_arm_end_effector_combination />
     </xacro:if>
   </xacro:if>
   <xacro:if value="${arm_type in ['4dof']}">
-    <xacro:if value="${end_effector_type not in ['fake-forearm']}">
+    <xacro:if value="${end_effector_right not in ['fake-forearm'] or end_effector_left not in ['fake-forearm']}">
       <xacro:wrong_arm_end_effector_combination />
     </xacro:if>
   </xacro:if>
   <xacro:if value="${arm_type in ['5dof']}">
-    <xacro:if value="${end_effector_type not in ['no-end-effector', 'RH8D']}">
+    <xacro:if value="${end_effector_right not in ['no-end-effector', 'RH8D'] or end_effector_left not in ['no-end-effector', 'RH8D']}">
       <xacro:wrong_arm_end_effector_combination />
     </xacro:if>
   </xacro:if>
   <xacro:if value="${arm_type in ['7dof']}">
-    <xacro:if value="${end_effector_type not in ['no-end-effector', 'gripper']}">
+    <xacro:if value="${end_effector_right not in ['no-end-effector', 'gripper'] or end_effector_left not in ['no-end-effector', 'gripper']}">
       <xacro:wrong_arm_end_effector_combination />
     </xacro:if>
@@ -131,6 +136,6 @@
   <!-- INCLUDES -->
   <!-- Tools -->
-  <xacro:include filename="$(find kangaroo_description)/urdf/materials.urdf.xacro" />
-  <xacro:include filename="$(find kangaroo_description)/urdf/deg_to_rad.xacro" />
+  <xacro:include filename="$(find pal_urdf_utils)/urdf/materials.urdf.xacro" />
+  <xacro:include filename="$(find pal_urdf_utils)/urdf/deg_to_rad.urdf.xacro" />
   <xacro:include filename="$(find kangaroo_description)/urdf/collision.xacro" />
   <!-- Base -->
@@ -140,18 +145,27 @@
   <!-- Arms -->
   <xacro:if value="${arm_type in ['4dof', '5dof', '7dof']}">
-    <xacro:include filename="$(find kangaroo_description)/urdf/arm/arm.urdf.xacro" />
+    <xacro:include filename="$(find pal_sea_arm_description)/urdf/arm/arm_properties/humanoid/arm.urdf.xacro" />
   </xacro:if>
   <xacro:unless value="${arm_type in ['4dof', '5dof', '7dof']}">
-    <xacro:include filename="$(find kangaroo_description)/urdf/arm/arm_cover/arm_cover.urdf.xacro" />
+    <xacro:include filename="$(find pal_sea_arm_description)/urdf/arm/humanoid/arm_cover.urdf.xacro" />
   </xacro:unless>
   <!-- End Effector -->
-  <xacro:if value="${end_effector_type in ['gripper']}">
-    <xacro:include filename="$(find kangaroo_description)/urdf/end_effector/pal_pro_gripper.urdf.xacro" />
-  </xacro:if>
-  <xacro:if value="${end_effector_type in ['RH8D']}">
-    <xacro:include filename="$(find kangaroo_description)/urdf/end_effector/rh8d_hand.urdf.xacro" />
-  </xacro:if>
-  <xacro:if value="${end_effector_type in ['fake-forearm']}">
-    <xacro:include filename="$(find kangaroo_description)/urdf/end_effector/fake_forearm.urdf.xacro" />
+  <xacro:if value="${end_effector_right in ['gripper']}">
+    <xacro:include filename="$(find pal_sea_arm_description)/urdf/end_effector/humanoid/pal_pro_gripper.urdf.xacro" />
+  </xacro:if>
+  <xacro:if value="${end_effector_right in ['RH8D']}">
+    <xacro:include filename="$(find pal_sea_arm_description)/urdf/end_effector/humanoid/rh8d_hand.urdf.xacro" />
+  </xacro:if>
+  <xacro:if value="${end_effector_right in ['fake-forearm']}">
+    <xacro:include filename="$(find pal_sea_arm_description)/urdf/end_effector/humanoid/fake_forearm.urdf.xacro" />
+  </xacro:if>
+  <xacro:if value="${end_effector_left in ['gripper']}">
+    <xacro:include filename="$(find pal_sea_arm_description)/urdf/end_effector/humanoid/pal_pro_gripper.urdf.xacro" />
+  </xacro:if>
+  <xacro:if value="${end_effector_left in ['RH8D']}">
+    <xacro:include filename="$(find pal_sea_arm_description)/urdf/end_effector/humanoid/rh8d_hand.urdf.xacro" />
+  </xacro:if>
+  <xacro:if value="${end_effector_left in ['fake-forearm']}">
+    <xacro:include filename="$(find pal_sea_arm_description)/urdf/end_effector/humanoid/fake_forearm.urdf.xacro" />
   </xacro:if>
   <!-- ROBOT DEFINITION -->
@@ -191,20 +205,26 @@
   </xacro:unless>
   <!-- END EFFECTOR -->
-  <xacro:if value="${end_effector_type in ['gripper']}">
+  <xacro:if value="${end_effector_right in ['gripper']}">
+    <xacro:gripper name="gripper_right" parent="arm_right_tool_link"/>
+  </xacro:if>
+  <xacro:if value="${end_effector_left in ['gripper']}">
     <xacro:gripper name="gripper_left" parent="arm_left_tool_link"/>
-    <xacro:gripper name="gripper_right" parent="arm_right_tool_link"/>
-  </xacro:if>
-  <xacro:if value="${end_effector_type in ['RH8D']}">
+  </xacro:if>
+  <xacro:if value="${end_effector_right in ['RH8D']}">
     <xacro:hand name="hand" side="left" parent="arm_left_tool_link" mimic="${use_mimic}">
       <origin xyz="0 0 0" rpy="0 0 1.5708"/>
     </xacro:hand>
+  </xacro:if>
+  <xacro:if value="${end_effector_left in ['RH8D']}">
     <xacro:hand name="hand" side="right" parent="arm_right_tool_link" mimic="${use_mimic}">
       <origin xyz="0 0 0" rpy="0 0 1.5708"/>
     </xacro:hand>
   </xacro:if>
-  <xacro:if value="${end_effector_type in ['fake-forearm']}">
+  <xacro:if value="${end_effector_right in ['fake-forearm']}">
     <xacro:fake-forearm name="arm" side="left" reflect="1" parent="arm_left_3_link">
       <origin xyz="-0.03711 -0.02 -0.17011" rpy="3.14159 1.5708 0" />
     </xacro:fake-forearm>
+  </xacro:if>
+  <xacro:if value="${end_effector_left in ['fake-forearm']}">
     <xacro:fake-forearm name="arm" side="right" reflect="-1" parent="arm_right_3_link">
       <origin xyz="-0.03711 -0.02 -0.17011" rpy="3.14159 1.5708 0" />
@@ -213,8 +233,8 @@
   <!-- MUJOCO   -->
   <xacro:if value="${sim_type == 'mujoco' or sim_type == 'mujoco-ros2-control'}">
-    <xacro:if value="${end_effector_type == 'gripper'}">
+    <xacro:if value="${end_effector_right == 'gripper'}">
       <xacro:include filename="$(find pal_pro_gripper_description)/mujoco/mj_tags.xacro" />
     </xacro:if>
-    <xacro:if value="${end_effector_type == 'RH8D'}">
+    <xacro:if value="${end_effector_right == 'RH8D'}">
       <xacro:include filename="$(find rh8d_description)/mujoco/mj_tags.xacro" />
     </xacro:if>
@@ -236,13 +256,17 @@
         <contact>
           <xacro:mj_robot_contacts />
-          <xacro:if value="${end_effector_type == 'gripper'}">
+          <xacro:if value="${end_effector_right == 'gripper'}">
+            <xacro:mj_gripper_contact name="gripper_right" />
+          </xacro:if>
+          <xacro:if value="${end_effector_left == 'gripper'}">
             <xacro:mj_gripper_contact name="gripper_left" />
-            <xacro:mj_gripper_contact name="gripper_right" />
-          </xacro:if>
-          <xacro:if value="${end_effector_type == 'RH8D'}">
+          </xacro:if>
+          <xacro:if value="${end_effector_right == 'RH8D'}">
+            <xacro:mj_hand_contact name="hand" side="right"/>
+            <exclude body1="hand_right_palm_link"  body2="arm_right_5_link"/>
+          </xacro:if>
+          <xacro:if value="${end_effector_left == 'RH8D'}">
             <xacro:mj_hand_contact name="hand" side="left"/>
-            <xacro:mj_hand_contact name="hand" side="right"/>
             <exclude body1="hand_left_palm_link"  body2="arm_left_5_link"/>
-            <exclude body1="hand_right_palm_link"  body2="arm_right_5_link"/>
           </xacro:if>
         </contact>
@@ -258,11 +282,15 @@
         <equality>
           <xacro:mj_robot_equality />
-          <xacro:if value="${end_effector_type == 'gripper'}">
+          <xacro:if value="${end_effector_right == 'gripper'}">
+            <xacro:mj_gripper_equality name="gripper_right" anchor_r="0.014 -0.0015 0" anchor_l="0.014 -0.001 0" />
+          </xacro:if>
+          <xacro:if value="${end_effector_left == 'gripper'}">
             <xacro:mj_gripper_equality name="gripper_left" anchor_r="0.01475 -0.001463 0.001" anchor_l="0.0145 -0.0015 0.001"/>
-            <xacro:mj_gripper_equality name="gripper_right" anchor_r="0.014 -0.0015 0" anchor_l="0.014 -0.001 0" />
-          </xacro:if>
-          <xacro:if value="${end_effector_type == 'RH8D'}">
+          </xacro:if>
+          <xacro:if value="${end_effector_right == 'RH8D'}">
+            <xacro:mj_hand_equality name="hand" side="right" />
+          </xacro:if>
+          <xacro:if value="${end_effector_left == 'RH8D'}">
             <xacro:mj_hand_equality name="hand" side="left" />
-            <xacro:mj_hand_equality name="hand" side="right" />
           </xacro:if>
         </equality>
@@ -270,11 +298,15 @@
         <actuator>
           <xacro:mj_robot_actuators/>
-          <xacro:if value="${end_effector_type == 'gripper'}">
+          <xacro:if value="${end_effector_right == 'gripper'}">
+            <xacro:mj_gripper_actuators name="gripper_right" />
+          </xacro:if>
+          <xacro:if value="${end_effector_left == 'gripper'}">
             <xacro:mj_gripper_actuators name="gripper_left" />
-            <xacro:mj_gripper_actuators name="gripper_right" />
-          </xacro:if>
-          <xacro:if value="${end_effector_type == 'RH8D'}">
+          </xacro:if>
+          <xacro:if value="${end_effector_right == 'RH8D'}">
+            <xacro:mj_hand_actuators name="hand" side="right" />
+          </xacro:if>
+          <xacro:if value="${end_effector_left == 'RH8D'}">
             <xacro:mj_hand_actuators name="hand" side="left" />
-            <xacro:mj_hand_actuators name="hand" side="right" />
           </xacro:if>
         </actuator>

File: kangaroo_description/ros2_control/ros2_control.urdf.xacro (robot description, xacro)
@@ -16,6 +16,6 @@
   <xacro:include filename="$(find kangaroo_description)/urdf/pelvis/ros2_control.urdf.xacro" />
   <xacro:include filename="$(find kangaroo_description)/urdf/leg/ros2_control.urdf.xacro" />
-  <xacro:include filename="$(find kangaroo_description)/urdf/arm/ros2_control.urdf.xacro" />
-  <xacro:include filename="$(find kangaroo_description)/urdf/end_effector/ros2_control.urdf.xacro" />
+  <xacro:include filename="$(find pal_sea_arm_description)/urdf/arm/arm_properties/humanoid/ros2_control.urdf.xacro" />
+  <xacro:include filename="$(find pal_sea_arm_description)/urdf/end_effector/humanoid/ros2_control.urdf.xacro" />
   <!-- calibration offsets -->
   <xacro:include filename="$(find kangaroo_description)/urdf/calibration_constants.urdf.xacro" />
@@ -55,7 +55,11 @@
         <xacro:arm_ros2_control side="right" arm_type="${arm_type}"/>
       </xacro:if>
-      <xacro:if value="${end_effector_type != 'no-end-effector'}">
-        <xacro:end_effector_ros2_control side="left" end_effector_type="${end_effector_type}"/>
-        <xacro:end_effector_ros2_control side="right" end_effector_type="${end_effector_type}"/>
+      <xacro:if value="${end_effector_right == 'pal-pro-gripper'}">
+        <!-- pal-pro-gripper right -->
+        <xacro:ros2_control_pal_pro_gripper name="gripper_right" reduction="1.0" />
+      </xacro:if>
+      <xacro:if value="${end_effector_left == 'pal-pro-gripper'}">
+        <!-- pal-pro-gripper left -->
+        <xacro:ros2_control_pal_pro_gripper name="gripper_left" reduction="1.0" />
       </xacro:if>
       <xacro:unless value="${sim_type == 'no-simulation'}">

Commit message: Add ft sensors

File: kangaroo_description/robots/kangaroo.urdf.xacro (robot description, xacro)
@@ -27,4 +27,6 @@
   <!-- fixed, floating -->
   <xacro:arg name="fixation_type" default="floating" />
+  <xacro:arg name="ft_sensor_left" default="no-ft-sensor" />
+  <xacro:arg name="ft_sensor_right" default="no-ft-sensor" />
   <!-- world name defined in pal_mujoco_scenes package -->
   <xacro:arg name="world_name" default="floor"/>
@@ -65,4 +67,6 @@
   <xacro:property name="end_effector_right" value="$(arg end_effector_right)" />
   <xacro:property name="end_effector_left" value="$(arg end_effector_left)" />
+  <xacro:property name="ft_sensor_left" value="$(arg ft_sensor_left)" />
+  <xacro:property name="ft_sensor_right" value="$(arg ft_sensor_right)" />
   <xacro:property name="world_name" value="$(arg world_name)" />
   <xacro:property name="use_mimic" value="$(arg use_mimic)" />
@@ -71,4 +75,8 @@
   <xacro:property name="torso_front_down_camera_model" value="$(arg torso_front_down_camera_model)" />
   <xacro:property name="torso_rear_down_camera_model" value="$(arg torso_rear_down_camera_model)" />
+  <xacro:property name="has_ft_sensor_left" value="${ft_sensor_left not in ['no-ft-sensor']}"/>
+  <xacro:property name="has_ft_sensor_right" value="${ft_sensor_right not in ['no-ft-sensor']}"/>
+  <xacro:property name="end_effector_right_link" value="${'wrist_right_ft_tool_link' if has_ft_sensor_right else 'arm_right_tool_link'}" />
+  <xacro:property name="end_effector_left_link" value="${'wrist_left_ft_tool_link' if has_ft_sensor_left else 'arm_left_tool_link'}" />
   <!-- Camera properties -->
   <xacro:property name="gazebo_version" value="classic"/>
@@ -90,5 +98,4 @@
     <xacro:wrong_arm_type />
   </xacro:if>
-  <!-- (ft-gripper) not available -->
   <xacro:if value="${end_effector_right not in ['cover', 'no-end-effector', 'fake-forearm', 'gripper', 'RH8D']}">
     <xacro:wrong_end_effector_right />
@@ -102,4 +109,11 @@
       <xacro:wrong_arm_end_effector_combination />
     </xacro:if>
+  </xacro:if>
+  <!-- FT SENSORS -->
+  <xacro:if value="${ft_sensor_left not in ['no-ft-sensor', 'ati']}">
+    <xacro:wrong_ft_sensor_left />
+  </xacro:if>
+  <xacro:if value="${ft_sensor_right not in ['no-ft-sensor', 'ati']}">
+    <xacro:wrong_ft_sensor_right />
   </xacro:if>
   <xacro:if value="${arm_type in ['4dof']}">
@@ -159,4 +173,9 @@
   <xacro:if value="${end_effector_right in ['fake-forearm'] or end_effector_left in ['fake-forearm']}">
     <xacro:include filename="$(find pal_sea_arm_description)/urdf/end_effector/humanoid/fake_forearm.urdf.xacro" />
+  </xacro:if>
+  <!-- FT Sensors  -->
+  <xacro:if value="${has_ft_sensor_right or has_ft_sensor_left}">
+    <xacro:include filename="$(find pal_urdf_utils)/urdf/ft_sensors/ft_sensor.urdf.xacro" />
+    <xacro:include filename="$(find pal_urdf_utils)/urdf/ft_sensors/ft_sensor.gazebo.xacro" />
   </xacro:if>
   <!-- ROBOT DEFINITION -->
@@ -197,8 +216,8 @@
   <!-- END EFFECTOR -->
   <xacro:if value="${end_effector_right in ['gripper']}">
-    <xacro:gripper name="gripper_right" parent="arm_right_tool_link"/>
+    <xacro:gripper name="gripper_right" parent="${end_effector_right_link}"/>
   </xacro:if>
   <xacro:if value="${end_effector_left in ['gripper']}">
-    <xacro:gripper name="gripper_left" parent="arm_left_tool_link"/>
+    <xacro:gripper name="gripper_left" parent="${end_effector_left_link}"/>
   </xacro:if>
   <xacro:if value="${end_effector_right in ['RH8D']}">
@@ -222,4 +241,11 @@
     </xacro:fake-forearm>
   </xacro:if>
+  <!-- FT SENSORS -->
+    <xacro:if value="${has_ft_sensor_left}">
+      <xacro:ft_sensor type="${ft_sensor_left}" name="wrist_left" parent="arm_left_tool_link"/>
+    </xacro:if>
+    <xacro:if value="${has_ft_sensor_right}">
+      <xacro:ft_sensor type="${ft_sensor_right}" name="wrist_right" parent="arm_right_tool_link"/>
+    </xacro:if>
   <!-- MUJOCO   -->
   <xacro:if value="${sim_type == 'mujoco' or sim_type == 'mujoco-ros2-control'}">
