Commit message: Remove cover as ee option and just check ee when has_arms is True

File: kangaroo_description/robots/kangaroo.urdf.xacro (robot description, xacro)
@@ -22,5 +22,5 @@
   <!-- no-arm, 4dof, 5dof, 7dof] -->
   <xacro:arg name="arm_type" default="4dof" />
-  <!-- cover, no-end-effector, fake-forearm, gripper, RH8D -->
+  <!-- no-end-effector, fake-forearm, gripper, RH8D -->
   <xacro:arg name="end_effector_right" default="no-end-effector" />
   <xacro:arg name="end_effector_left" default="no-end-effector" />
@@ -75,4 +75,5 @@
   <xacro:property name="torso_front_down_camera_model" value="$(arg torso_front_down_camera_model)" />
   <xacro:property name="torso_rear_down_camera_model" value="$(arg torso_rear_down_camera_model)" />
+  <xacro:property name="has_arms" value="${arm_type not in ['no-arm']}" />
   <xacro:property name="has_ft_sensor_left" value="${ft_sensor_left not in ['no-ft-sensor']}"/>
   <xacro:property name="has_ft_sensor_right" value="${ft_sensor_right not in ['no-ft-sensor']}"/>
@@ -98,15 +99,9 @@
     <xacro:wrong_arm_type />
   </xacro:if>
-  <xacro:if value="${end_effector_right not in ['cover', 'no-end-effector', 'fake-forearm', 'gripper', 'RH8D']}">
+  <xacro:if value="${end_effector_right not in ['no-end-effector', 'fake-forearm', 'gripper', 'RH8D']}">
     <xacro:wrong_end_effector_right />
   </xacro:if>
-  <xacro:if value="${end_effector_left not in ['cover', 'no-end-effector', 'fake-forearm', 'gripper', 'RH8D']}">
+  <xacro:if value="${end_effector_left not in ['no-end-effector', 'fake-forearm', 'gripper', 'RH8D']}">
     <xacro:wrong_end_effector_left />
-  </xacro:if>
-  <!-- Valid Combinations -->
-  <xacro:if value="${arm_type in ['no-arm']}">
-    <xacro:if value="${end_effector_right or end_effector_left not in ['cover'] or end_effector_left not in ['cover']}">
-      <xacro:wrong_arm_end_effector_combination />
-    </xacro:if>
   </xacro:if>
   <!-- FT SENSORS -->
@@ -158,25 +153,25 @@
   <xacro:include filename="$(find kangaroo_description)/urdf/leg/leg.urdf.xacro" />
   <!-- Arms -->
-  <xacro:if value="${arm_type in ['4dof', '5dof', '7dof']}">
+  <xacro:if value="${has_arms}">
     <xacro:include filename="$(find pal_sea_arm_description)/urdf/arm/arm_properties/humanoid/arm.urdf.xacro" />
-  </xacro:if>
-  <xacro:unless value="${arm_type in ['4dof', '5dof', '7dof']}">
-    <xacro:include filename="$(find pal_sea_arm_description)/urdf/arm/humanoid/arm_cover.urdf.xacro" />
+    <!-- End Effector -->
+    <xacro:if value="${end_effector_right in ['gripper'] or end_effector_left in ['gripper']}">
+      <xacro:include filename="$(find pal_sea_arm_description)/urdf/end_effector/humanoid/pal_pro_gripper.urdf.xacro" />
+    </xacro:if>
+    <xacro:if value="${end_effector_right in ['RH8D'] or end_effector_left in ['RH8D']}">
+      <xacro:include filename="$(find pal_sea_arm_description)/urdf/end_effector/humanoid/rh8d_hand.urdf.xacro" />
+    </xacro:if>
+    <xacro:if value="${end_effector_right in ['fake-forearm'] or end_effector_left in ['fake-forearm']}">
+      <xacro:include filename="$(find pal_sea_arm_description)/urdf/end_effector/humanoid/fake_forearm.urdf.xacro" />
+    </xacro:if>
+    <!-- FT Sensors  -->
+    <xacro:if value="${has_ft_sensor_right or has_ft_sensor_left}">
+      <xacro:include filename="$(find pal_urdf_utils)/urdf/ft_sensors/ft_sensor.urdf.xacro" />
+      <xacro:include filename="$(find pal_urdf_utils)/urdf/ft_sensors/ft_sensor.gazebo.xacro" />
+    </xacro:if>
+  </xacro:if>
+  <xacro:unless value="${has_arms}">
+    <xacro:include filename="$(find pal_sea_arm_description)/urdf/arm/arm_properties/humanoid/arm_cover.urdf.xacro" />
   </xacro:unless>
-  <!-- End Effector -->
-  <xacro:if value="${end_effector_right in ['gripper'] or end_effector_left in ['gripper']}">
-    <xacro:include filename="$(find pal_sea_arm_description)/urdf/end_effector/humanoid/pal_pro_gripper.urdf.xacro" />
-  </xacro:if>
-  <xacro:if value="${end_effector_right in ['RH8D'] or end_effector_left in ['RH8D']}">
-    <xacro:include filename="$(find pal_sea_arm_description)/urdf/end_effector/humanoid/rh8d_hand.urdf.xacro" />
-  </xacro:if>
-  <xacro:if value="${end_effector_right in ['fake-forearm'] or end_effector_left in ['fake-forearm']}">
-    <xacro:include filename="$(find pal_sea_arm_description)/urdf/end_effector/humanoid/fake_forearm.urdf.xacro" />
-  </xacro:if>
-  <!-- FT Sensors  -->
-  <xacro:if value="${has_ft_sensor_right or has_ft_sensor_left}">
-    <xacro:include filename="$(find pal_urdf_utils)/urdf/ft_sensors/ft_sensor.urdf.xacro" />
-    <xacro:include filename="$(find pal_urdf_utils)/urdf/ft_sensors/ft_sensor.gazebo.xacro" />
-  </xacro:if>
   <!-- ROBOT DEFINITION -->
   <!-- BASE, PELVIS, TORSO -->
@@ -194,5 +189,5 @@
   </xacro:if>
   <!-- ARMS -->
-  <xacro:if value="${arm_type in ['4dof', '5dof', '7dof']}">
+  <xacro:if value="${has_arms}">
     <!-- Left Arm -->
     <xacro:kangaroo_arm name="arm" side="left" type="${arm_type}" reflect="1" parent="torso_link" >
@@ -203,6 +198,40 @@
       <origin xyz="0 -0.105954 0.384396" rpy="1.3963 3.14159 0" />
     </xacro:kangaroo_arm>
-  </xacro:if>
-  <xacro:unless value="${arm_type in ['4dof', '5dof', '7dof']}">
+    <!-- END EFFECTOR -->
+    <xacro:if value="${end_effector_right in ['gripper']}">
+      <xacro:gripper name="gripper_right" parent="${end_effector_right_link}"/>
+    </xacro:if>
+    <xacro:if value="${end_effector_left in ['gripper']}">
+      <xacro:gripper name="gripper_left" parent="${end_effector_left_link}"/>
+    </xacro:if>
+    <xacro:if value="${end_effector_right in ['RH8D']}">
+      <xacro:hand name="hand" side="left" parent="arm_left_tool_link" mimic="${use_mimic}">
+        <origin xyz="0 0 0" rpy="0 0 1.5708"/>
+      </xacro:hand>
+    </xacro:if>
+    <xacro:if value="${end_effector_left in ['RH8D']}">
+      <xacro:hand name="hand" side="right" parent="arm_right_tool_link" mimic="${use_mimic}">
+        <origin xyz="0 0 0" rpy="0 0 1.5708"/>
+      </xacro:hand>
+    </xacro:if>
+    <xacro:if value="${end_effector_right in ['fake-forearm']}">
+      <xacro:fake-forearm name="arm" side="left" reflect="1" parent="arm_left_3_link">
+        <origin xyz="-0.03711 -0.02 -0.17011" rpy="3.14159 1.5708 0" />
+      </xacro:fake-forearm>
+    </xacro:if>
+    <xacro:if value="${end_effector_left in ['fake-forearm']}">
+      <xacro:fake-forearm name="arm" side="right" reflect="-1" parent="arm_right_3_link">
+        <origin xyz="-0.03711 -0.02 -0.17011" rpy="3.14159 1.5708 0" />
+      </xacro:fake-forearm>
+    </xacro:if>
+    <!-- FT SENSORS -->
+      <xacro:if value="${has_ft_sensor_left}">
+        <xacro:ft_sensor type="${ft_sensor_left}" name="wrist_left" parent="arm_left_tool_link"/>
+      </xacro:if>
+      <xacro:if value="${has_ft_sensor_right}">
+        <xacro:ft_sensor type="${ft_sensor_right}" name="wrist_right" parent="arm_right_tool_link"/>
+      </xacro:if>
+  </xacro:if>
+  <xacro:unless value="${has_arms}">
     <!-- Left Arm Cover -->
     <xacro:kangaroo_arm_cover name="arm_cover" side="left" reflect="1" parent="torso_link">
@@ -214,38 +243,4 @@
     </xacro:kangaroo_arm_cover>
   </xacro:unless>
-  <!-- END EFFECTOR -->
-  <xacro:if value="${end_effector_right in ['gripper']}">
-    <xacro:gripper name="gripper_right" parent="${end_effector_right_link}"/>
-  </xacro:if>
-  <xacro:if value="${end_effector_left in ['gripper']}">
-    <xacro:gripper name="gripper_left" parent="${end_effector_left_link}"/>
-  </xacro:if>
-  <xacro:if value="${end_effector_right in ['RH8D']}">
-    <xacro:hand name="hand" side="left" parent="arm_left_tool_link" mimic="${use_mimic}">
-      <origin xyz="0 0 0" rpy="0 0 1.5708"/>
-    </xacro:hand>
-  </xacro:if>
-  <xacro:if value="${end_effector_left in ['RH8D']}">
-    <xacro:hand name="hand" side="right" parent="arm_right_tool_link" mimic="${use_mimic}">
-      <origin xyz="0 0 0" rpy="0 0 1.5708"/>
-    </xacro:hand>
-  </xacro:if>
-  <xacro:if value="${end_effector_right in ['fake-forearm']}">
-    <xacro:fake-forearm name="arm" side="left" reflect="1" parent="arm_left_3_link">
-      <origin xyz="-0.03711 -0.02 -0.17011" rpy="3.14159 1.5708 0" />
-    </xacro:fake-forearm>
-  </xacro:if>
-  <xacro:if value="${end_effector_left in ['fake-forearm']}">
-    <xacro:fake-forearm name="arm" side="right" reflect="-1" parent="arm_right_3_link">
-      <origin xyz="-0.03711 -0.02 -0.17011" rpy="3.14159 1.5708 0" />
-    </xacro:fake-forearm>
-  </xacro:if>
-  <!-- FT SENSORS -->
-    <xacro:if value="${has_ft_sensor_left}">
-      <xacro:ft_sensor type="${ft_sensor_left}" name="wrist_left" parent="arm_left_tool_link"/>
-    </xacro:if>
-    <xacro:if value="${has_ft_sensor_right}">
-      <xacro:ft_sensor type="${ft_sensor_right}" name="wrist_right" parent="arm_right_tool_link"/>
-    </xacro:if>
   <!-- MUJOCO   -->
   <xacro:if value="${sim_type == 'mujoco' or sim_type == 'mujoco-ros2-control'}">

Commit message: Remove leg_type and add fett_type

File: kangaroo_description/robots/kangaroo.urdf.xacro (robot description, xacro)
@@ -18,6 +18,6 @@
   <!-- True, False -->
   <xacro:arg name="has_head" default="False" />
-  <!-- (ft-leg) not available, leg, no-leg -->
-  <xacro:arg name="legs_type" default="leg" />
+  <!-- fixed, detachable-->
+  <xacro:arg name="feet_type" default="fixed" />
   <!-- no-arm, 4dof, 5dof, 7dof] -->
   <xacro:arg name="arm_type" default="4dof" />
@@ -63,5 +63,5 @@
   <xacro:property name="has_head" value="$(arg has_head)" />
   <xacro:property name="arm_type" value="$(arg arm_type)" />
-  <xacro:property name="legs_type" value="$(arg legs_type)" />
+  <xacro:property name="feet_type" value="$(arg feet_type)" />
   <xacro:property name="fixation_type" value="$(arg fixation_type)" />
   <xacro:property name="end_effector_right" value="$(arg end_effector_right)" />
@@ -128,6 +128,6 @@
   </xacro:if>
   <!-- (ft-leg) not available -->
-  <xacro:if value="${legs_type not in ['leg', 'no-leg']}">
-    <xacro:wrong_legs_type />
+  <xacro:if value="${feet_type not in ['fixed', 'detachable']}">
+    <xacro:wrong_feet_type />
   </xacro:if>
   <xacro:if value="${torso_front_up_camera_model not in ['realsense-d435i']}">
@@ -178,11 +178,11 @@
   <xacro:base_link has_pelvis="${has_pelvis}"/>
   <!-- LEGS -->
-  <xacro:if value="${legs_type in ['leg', 'ft-leg']}">
+  <xacro:if value="${feet_type in ['fixed', 'detachable']}">
     <!-- Left Leg -->
-    <xacro:kangaroo_leg side="left" reflect="1" parent="base_link" leg_type="${legs_type}">
+    <xacro:kangaroo_leg side="left" reflect="1" parent="base_link" feet_type="${feet_type}">
       <origin xyz="-0.0150025976417119 0.08 -0.0585" rpy="0 0 0"/>
     </xacro:kangaroo_leg>
     <!-- Right Leg -->
-    <xacro:kangaroo_leg side="right" reflect="-1" parent="base_link" leg_type="${legs_type}">
+    <xacro:kangaroo_leg side="right" reflect="-1" parent="base_link" feet_type="${feet_type}">
       <origin xyz="-0.0150025976417119 -0.08 -0.0585" rpy="0 0 0"/>
     </xacro:kangaroo_leg>

File: kangaroo_description/ros2_control/ros2_control.urdf.xacro (robot description, xacro)
@@ -47,8 +47,6 @@
         <xacro:pelvis_ros2_control />
       </xacro:if>
-      <xacro:if value="${legs_type != 'no-leg'}">
-        <xacro:leg_ros2_control side="left"/>
-        <xacro:leg_ros2_control side="right"/>
-      </xacro:if>
+      <xacro:leg_ros2_control side="left"/>
+      <xacro:leg_ros2_control side="right"/>
       <xacro:if value="${arm_type != 'no-arm'}">
         <xacro:arm_ros2_control side="left" arm_type="${arm_type}"/>

Commit message: Add ros2 ft sensor for ankle

File: kangaroo_description/robots/kangaroo.urdf.xacro (robot description, xacro)
@@ -14,4 +14,7 @@
 <robot xmlns:xacro="http://ros.org/wiki/xacro" name="kangaroo" >
   <!-- ARGUMENTS -->
+  <!-- ati, no-ft-sensor -->
+  <xacro:arg name="ankle_ft_right" default="no-ft-sensor" />
+  <xacro:arg name="ankle_ft_left" default="no-ft-sensor" />
   <!-- True, False -->
   <xacro:arg name="has_pelvis" default="True" />
@@ -60,4 +63,6 @@
   <xacro:property name="torso_mesh" value="$(arg torso_mesh)"/>
   <!-- PROPERTIES -->
+  <xacro:property name="ankle_ft_right" value="$(arg ankle_ft_right)" />
+  <xacro:property name="ankle_ft_left" value="$(arg ankle_ft_left)" />
   <xacro:property name="has_pelvis" value="$(arg has_pelvis)" />
   <xacro:property name="has_head" value="$(arg has_head)" />
@@ -78,4 +83,6 @@
   <xacro:property name="has_ft_sensor_left" value="${ft_sensor_left not in ['no-ft-sensor']}"/>
   <xacro:property name="has_ft_sensor_right" value="${ft_sensor_right not in ['no-ft-sensor']}"/>
+  <xacro:property name="has_ankle_ft_sensor_left" value="${ankle_ft_left not in ['no-ft-sensor']}"/>
+  <xacro:property name="has_ankle_ft_sensor_right" value="${ankle_ft_right not in ['no-ft-sensor']}"/>
   <xacro:property name="end_effector_right_link" value="${'wrist_right_ft_tool_link' if has_ft_sensor_right else 'arm_right_tool_link'}" />
   <xacro:property name="end_effector_left_link" value="${'wrist_left_ft_tool_link' if has_ft_sensor_left else 'arm_left_tool_link'}" />
@@ -111,4 +118,10 @@
   <xacro:if value="${ft_sensor_right not in ['no-ft-sensor', 'ati']}">
     <xacro:wrong_ft_sensor_right />
+  </xacro:if>
+  <xacro:if value="${ankle_ft_left not in ['no-ft-sensor', 'ati']}">
+    <xacro:wrong_ankle_ft_sensor_left />
+  </xacro:if>
+  <xacro:if value="${ankle_ft_right not in ['no-ft-sensor', 'ati']}">
+    <xacro:wrong_ankle_ft_sensor_right />
   </xacro:if>
   <xacro:if value="${arm_type in ['4dof']}">
@@ -404,5 +417,5 @@
   <xacro:unless value="${sim_type == 'mujoco'}">
     <xacro:include filename="$(find kangaroo_description)/ros2_control/ros2_control.urdf.xacro" />
-    <xacro:kangaroo_ros2_control arm_type="${arm_type}"/>
+    <xacro:kangaroo_ros2_control arm_type="${arm_type}" has_ankle_ft_sensor_right="${has_ankle_ft_sensor_right}" has_ankle_ft_sensor_left="${has_ankle_ft_sensor_left}" />
   </xacro:unless>
 </robot>

File: kangaroo_description/ros2_control/ros2_control.urdf.xacro (robot description, xacro)
@@ -21,5 +21,5 @@
   <xacro:include filename="$(find kangaroo_description)/urdf/calibration_constants.urdf.xacro" />
   <!-- MACRO DEFINITION-->
-  <xacro:macro name="kangaroo_ros2_control" params="arm_type">
+  <xacro:macro name="kangaroo_ros2_control" params="arm_type has_ankle_ft_sensor_right has_ankle_ft_sensor_left">
     <ros2_control name="ros2_control_kangaroo_system" type="system" is_async="${'true' if sim_type == 'no-simulation' else 'false'}">
       <xacro:if value="${sim_type == 'no-simulation'}" >
@@ -47,17 +47,17 @@
         <xacro:pelvis_ros2_control />
       </xacro:if>
-      <xacro:leg_ros2_control side="left"/>
-      <xacro:leg_ros2_control side="right"/>
+      <xacro:leg_ros2_control side="left" has_ankle_ft_sensor="${has_ankle_ft_sensor_left}"/>
+      <xacro:leg_ros2_control side="right" has_ankle_ft_sensor="${has_ankle_ft_sensor_right}"/>
       <xacro:if value="${arm_type != 'no-arm'}">
         <xacro:arm_ros2_control side="left" arm_type="${arm_type}"/>
         <xacro:arm_ros2_control side="right" arm_type="${arm_type}"/>
-      </xacro:if>
-      <xacro:if value="${end_effector_right == 'pal-pro-gripper'}">
-        <!-- pal-pro-gripper right -->
-        <xacro:ros2_control_pal_pro_gripper name="gripper_right" reduction="1.0" />
-      </xacro:if>
-      <xacro:if value="${end_effector_left == 'pal-pro-gripper'}">
-        <!-- pal-pro-gripper left -->
-        <xacro:ros2_control_pal_pro_gripper name="gripper_left" reduction="1.0" />
+        <xacro:if value="${end_effector_right == 'pal-pro-gripper'}">
+          <!-- pal-pro-gripper right -->
+          <xacro:ros2_control_pal_pro_gripper name="gripper_right" reduction="1.0" />
+        </xacro:if>
+        <xacro:if value="${end_effector_left == 'pal-pro-gripper'}">
+          <!-- pal-pro-gripper left -->
+          <xacro:ros2_control_pal_pro_gripper name="gripper_left" reduction="1.0" />
+        </xacro:if>
       </xacro:if>
       <xacro:unless value="${sim_type == 'no-simulation'}">

File: kangaroo_description/urdf/leg/ros2_control.urdf.xacro (robot description, xacro)
@@ -20,5 +20,5 @@
   <xacro:include filename="$(find kangaroo_description)/urdf/ankle/ankle.transmission.xacro" />
   <!-- MACRO DEFINITION-->
-  <xacro:macro name="leg_ros2_control" params="side">
+  <xacro:macro name="leg_ros2_control" params="side" has_ankle_ft_sensor="false">
         <xacro:if value="${sim_type == 'no-simulation'}" >
           <xacro:hip_transmission_yaw side="${side}" offset="${leg_1_joint_offset}" initial_position="0.0" />
@@ -27,4 +27,8 @@
           <xacro:kangaroo_ankle_transmission side="${side}" roll_joint="5" pitch_joint="4" read_actuator="leg_${side}_length_actuator" />
         </xacro:if>
+        <xacro:if value="${has_ankle_ft_sensor}">
+           <xacro:include filename="$(find pal_urdf_utils)/urdf/ft_sensors/ftsensor.ros2_control.xacro"/>
+           <xacro:ros2_control_force_torque_sensor name="ankle_${side}_ft_sensor"/>
+        </xacro:if>
   </xacro:macro>
 </robot>
