Commit message: Add imus on the urdf

File: kangaroo_description/robots/kangaroo.urdf.xacro (robot description, xacro)
@@ -56,4 +56,7 @@
   <!-- mesh, capsule -->
   <xacro:arg name="collision_type" default="mesh" />
+  <!-- orientus, microstrain -->
+  <xacro:arg name="torso_imu_model" default="orientus" />
+  <xacro:arg name="base_imu_model" default="orientus" />
   <!-- GLOBAL PROPERTIES -->
   <xacro:property name="use_sim_time" value="$(arg use_sim_time)" />
@@ -87,4 +90,6 @@
   <xacro:property name="end_effector_right_link" value="${'wrist_right_ft_tool_link' if has_ft_sensor_right else 'arm_right_tool_link'}" />
   <xacro:property name="end_effector_left_link" value="${'wrist_left_ft_tool_link' if has_ft_sensor_left else 'arm_left_tool_link'}" />
+  <xacro:property name="torso_imu_model" value="$(arg torso_imu_model)" />
+  <xacro:property name="base_imu_model" value="$(arg base_imu_model)" />
   <!-- Camera properties -->
   <xacro:property name="gazebo_version" value="classic"/>
@@ -417,5 +422,5 @@
   <xacro:unless value="${sim_type == 'mujoco'}">
     <xacro:include filename="$(find kangaroo_description)/ros2_control/ros2_control.urdf.xacro" />
-    <xacro:kangaroo_ros2_control arm_type="${arm_type}" has_ankle_ft_sensor_right="${has_ankle_ft_sensor_right}" has_ankle_ft_sensor_left="${has_ankle_ft_sensor_left}" />
+    <xacro:kangaroo_ros2_control arm_type="${arm_type}" has_ankle_ft_sensor_right="${has_ankle_ft_sensor_right}" has_ankle_ft_sensor_left="${has_ankle_ft_sensor_left}" torso_imu_model="${torso_imu_model}" base_imu_model="${base_imu_model}" />
   </xacro:unless>
 </robot>

File: kangaroo_description/ros2_control/ros2_control.urdf.xacro (robot description, xacro)
@@ -21,5 +21,5 @@
   <xacro:include filename="$(find kangaroo_description)/urdf/calibration_constants.urdf.xacro" />
   <!-- MACRO DEFINITION-->
-  <xacro:macro name="kangaroo_ros2_control" params="arm_type has_ankle_ft_sensor_right has_ankle_ft_sensor_left">
+  <xacro:macro name="kangaroo_ros2_control" params="arm_type has_ankle_ft_sensor_right has_ankle_ft_sensor_left torso_imu_model base_imu_model">
     <ros2_control name="ros2_control_kangaroo_system" type="system" is_async="${'true' if sim_type == 'no-simulation' else 'false'}">
       <xacro:if value="${sim_type == 'no-simulation'}" >
@@ -62,8 +62,8 @@
       </xacro:if>
       <xacro:unless value="${sim_type == 'no-simulation'}">
-        <sensor name="imu_sensor">
+        <sensor name="torso_imu_sensor">
           <param name="mujoco_type">imu</param>
           <!-- There is no requirement for the mujoco_sensor_name to match the ros2_control sensor name -->
-          <param name="mujoco_sensor_name">imu_sensor</param>
+          <param name="mujoco_sensor_name">torso_imu_sensor</param>
           <!-- Default value of orientation_mjcf_suffix is '_quat' -->
           <param name="orientation_mjcf_suffix">_quat</param>
@@ -86,14 +86,44 @@
     </ros2_control>
     <xacro:if value="${sim_type == 'no-simulation'}">
-      <ros2_control name="ros2_control_orientus" type="sensor" rw_rate="1000" is_async="true">
-        <hardware>
-          <plugin>pal_orientus_sensor/OrientusSensor</plugin>
-          <param name="io_device">/dev/ttyUSB0</param>
-          <param name="sensor_name">imu_sensor</param>
-          <param name="orientation_to_enu_frame">3.14159, 0.0, 1.570796</param>
-          <!-- The following parameter is used to enable the ENU transformation for velocity and acceleration -->
-          <param name="enable_orientation_to_enu_frame">false</param>
-        </hardware>
-      </ros2_control>
+      <xacro:if value="${torso_imu_model == 'orientus'}">
+        <ros2_control name="ros2_control_orientus" type="sensor" rw_rate="1000" is_async="true">
+          <hardware>
+            <plugin>pal_orientus_sensor/OrientusSensor</plugin>
+            <param name="io_device">/dev/ttyUSB0</param>
+            <param name="sensor_name">torso_imu_sensor</param>
+            <param name="orientation_to_enu_frame">3.14159, 0.0, 1.570796</param>
+            <!-- The following parameter is used to enable the ENU transformation for velocity and acceleration -->
+            <param name="enable_orientation_to_enu_frame">false</param>
+          </hardware>
+        </ros2_control>
+      </xacro:if>
+      <xacro:if value="${torso_imu_model == 'microstrain'}">
+        <ros2_control name="ros2_control_microstrain" type="sensor" rw_rate="1000" is_async="true">
+          <hardware>
+            <plugin>pal_microstrain_sensor/MicrostrainSensor</plugin>
+            <param name="io_device">/dev/ttyACM0</param>
+            <param name="sensor_name">torso_imu_sensor</param>
+            <param name="orientation_to_enu_frame">3.14159, 0.0, 1.570796</param>
+            <!-- The following parameter is used to enable the ENU transformation for velocity and acceleration -->
+            <param name="enable_orientation_to_enu_frame">false</param>
+            <param name="baudrate">115200</param>
+            <param name="data_rate_hz">100</param>
+          </hardware>
+        </ros2_control>
+      </xacro:if>
+      <xacro:if value="${base_imu_model == 'microstrain'}">
+        <ros2_control name="ros2_control_microstrain_base" type="sensor" rw_rate="1000" is_async="true">
+          <hardware>
+            <plugin>pal_microstrain_sensor/MicrostrainSensor</plugin>
+            <param name="io_device">/dev/ttyACM0</param> <!--to be defined-->
+            <param name="sensor_name">base_imu_sensor</param>
+            <param name="orientation_to_enu_frame">3.14159, 0.0, 1.570796</param>
+            <!-- The following parameter is used to enable the ENU transformation for velocity and acceleration -->
+            <param name="enable_orientation_to_enu_frame">false</param>
+            <param name="baudrate">115200</param>
+            <param name="data_rate_hz">100</param>
+          </hardware>
+        </ros2_control>
+      </xacro:if>
     </xacro:if>
   </xacro:macro>

File: kangaroo_description/urdf/base/base.urdf.xacro (robot description, xacro)
@@ -18,5 +18,5 @@
   <xacro:macro name="base_link" params="has_pelvis:=false">
     <!-- IMU -->
-    <xacro:kangaroo_imu name="imu" parent="torso_link" >
+    <xacro:kangaroo_imu name="torso_imu" parent="torso_link" >
       <origin xyz="0.071 -0.0014 0.02" rpy="${180.0*deg_to_rad} ${0.0*deg_to_rad} ${-90.0*deg_to_rad}"/>
     </xacro:kangaroo_imu>
@@ -85,4 +85,10 @@
         <child link="back_handle" />
       </joint>
+      <!-- BASE IMU -->
+      <xacro:if value="${base_imu_model != 'no-imu'}">
+        <xacro:kangaroo_imu name="base_imu_sensor" parent="base_link" >
+          <origin xyz="0.05051 0 0.02055" rpy="${180.0*deg_to_rad} ${0.0*deg_to_rad} ${-90.0*deg_to_rad}"/>
+        </xacro:kangaroo_imu>
+      </xacro:if>
       <!-- PELVIS -->
       <xacro:kangaroo_pelvis name="pelvis" parent="base_link" pelvis_1_offset="0"

File: kangaroo_description/urdf/sensors/imu.urdf.xacro (robot description, xacro)
@@ -17,5 +17,5 @@
       </visual>
     </link>
-    <joint name="imu_joint" type="fixed">
+    <joint name="${name}_imu_joint" type="fixed">
       <xacro:insert_block name="origin"/>
       <parent link="${parent}"/>

Commit message: Add no imu option for torso imu

File: kangaroo_description/robots/kangaroo.urdf.xacro (robot description, xacro)
@@ -56,7 +56,7 @@
   <!-- mesh, capsule -->
   <xacro:arg name="collision_type" default="mesh" />
-  <!-- orientus, microstrain -->
+  <!-- orientus, microstrain, no-imu -->
   <xacro:arg name="torso_imu_model" default="orientus" />
-  <xacro:arg name="base_imu_model" default="orientus" />
+  <xacro:arg name="base_imu_model" default="no-imu" />
   <!-- GLOBAL PROPERTIES -->
   <xacro:property name="use_sim_time" value="$(arg use_sim_time)" />

File: kangaroo_description/urdf/base/base.urdf.xacro (robot description, xacro)
@@ -18,7 +18,9 @@
   <xacro:macro name="base_link" params="has_pelvis:=false">
     <!-- IMU -->
-    <xacro:kangaroo_imu name="torso_imu" parent="torso_link" >
-      <origin xyz="0.071 -0.0014 0.02" rpy="${180.0*deg_to_rad} ${0.0*deg_to_rad} ${-90.0*deg_to_rad}"/>
-    </xacro:kangaroo_imu>
+    <xacro:if value="${torso_imu_model != 'no-imu'}">
+      <xacro:kangaroo_imu name="torso_imu" parent="torso_link" >
+        <origin xyz="0.071 -0.0014 0.02" rpy="${180.0*deg_to_rad} ${0.0*deg_to_rad} ${-90.0*deg_to_rad}"/>
+      </xacro:kangaroo_imu>
+    </xacro:if>
     <!-- has pelvis DoF -->
     <xacro:if value="${has_pelvis}">

Commit message: Change fakeforearm to 4dof with no end effector

File: kangaroo_description/robots/kangaroo.urdf.xacro (robot description, xacro)
@@ -25,5 +25,5 @@
   <!-- no-arm, 4dof, 5dof, 7dof] -->
   <xacro:arg name="arm_type" default="4dof" />
-  <!-- no-end-effector, fake-forearm, gripper, RH8D -->
+  <!-- no-end-effector, gripper, RH8D -->
   <xacro:arg name="end_effector_right" default="no-end-effector" />
   <xacro:arg name="end_effector_left" default="no-end-effector" />
@@ -111,8 +111,8 @@
     <xacro:wrong_arm_type />
   </xacro:if>
-  <xacro:if value="${end_effector_right not in ['no-end-effector', 'fake-forearm', 'gripper', 'RH8D']}">
+  <xacro:if value="${end_effector_right not in ['no-end-effector', 'gripper', 'RH8D']}">
     <xacro:wrong_end_effector_right />
   </xacro:if>
-  <xacro:if value="${end_effector_left not in ['no-end-effector', 'fake-forearm', 'gripper', 'RH8D']}">
+  <xacro:if value="${end_effector_left not in ['no-end-effector', 'gripper', 'RH8D']}">
     <xacro:wrong_end_effector_left />
   </xacro:if>
@@ -131,5 +131,5 @@
   </xacro:if>
   <xacro:if value="${arm_type in ['4dof']}">
-    <xacro:if value="${end_effector_right not in ['fake-forearm'] or end_effector_left not in ['fake-forearm']}">
+    <xacro:if value="${end_effector_right not in ['no-end-effector'] or end_effector_left not in ['no-end-effector']}">
       <xacro:wrong_arm_end_effector_combination />
     </xacro:if>
@@ -179,7 +179,4 @@
     <xacro:if value="${end_effector_right in ['RH8D'] or end_effector_left in ['RH8D']}">
       <xacro:include filename="$(find pal_sea_arm_description)/urdf/end_effector/humanoid/rh8d_hand.urdf.xacro" />
-    </xacro:if>
-    <xacro:if value="${end_effector_right in ['fake-forearm'] or end_effector_left in ['fake-forearm']}">
-      <xacro:include filename="$(find pal_sea_arm_description)/urdf/end_effector/humanoid/fake_forearm.urdf.xacro" />
     </xacro:if>
     <!-- FT Sensors  -->
@@ -232,14 +229,4 @@
         <origin xyz="0 0 0" rpy="0 0 1.5708"/>
       </xacro:hand>
-    </xacro:if>
-    <xacro:if value="${end_effector_right in ['fake-forearm']}">
-      <xacro:fake-forearm name="arm" side="left" reflect="1" parent="arm_left_3_link">
-        <origin xyz="-0.03711 -0.02 -0.17011" rpy="3.14159 1.5708 0" />
-      </xacro:fake-forearm>
-    </xacro:if>
-    <xacro:if value="${end_effector_left in ['fake-forearm']}">
-      <xacro:fake-forearm name="arm" side="right" reflect="-1" parent="arm_right_3_link">
-        <origin xyz="-0.03711 -0.02 -0.17011" rpy="3.14159 1.5708 0" />
-      </xacro:fake-forearm>
     </xacro:if>
     <!-- FT SENSORS -->
