Commit message: added full model sim option that emits the transmissions

File: kangaroo_description/robots/kangaroo.urdf.xacro (robot description, xacro)
@@ -52,4 +52,6 @@
   <!-- mujoco-ros2-control, mujoco, no-simulation -->
   <xacro:arg name="sim_type" default="no-simulation" />
+  <!-- simple, full -->
+  <xacro:arg name="sim_model" default="simple" />
   <!-- false, position, motor -->
   <xacro:arg name="mj_control" default="position" />
@@ -62,4 +64,5 @@
   <xacro:property name="use_sim_time" value="$(arg use_sim_time)" />
   <xacro:property name="sim_type" value="$(arg sim_type)"/>
+  <xacro:property name="sim_model" value="$(arg sim_model)" />
   <xacro:property name="mj_control" value="$(arg mj_control)" />
   <xacro:property name="collision_type" value="$(arg collision_type)"/>
@@ -98,4 +101,7 @@
   <xacro:if value="${sim_type not in ['mujoco-ros2-control', 'mujoco', 'no-simulation']}">
     <xacro:wrong_sim_type />
+  </xacro:if>
+  <xacro:if value="${sim_model not in ['simple', 'full']}">
+    <xacro:wrong_sim_model />
   </xacro:if>
   <xacro:if value="${mj_control not in ['false', 'position', 'motor']}">
@@ -428,5 +434,11 @@
   <xacro:unless value="${sim_type == 'mujoco'}">
     <xacro:include filename="$(find kangaroo_description)/ros2_control/ros2_control.urdf.xacro" />
-    <xacro:kangaroo_ros2_control arm_type="${arm_type}" has_ankle_ft_sensor_right="${has_ankle_ft_sensor_right}" has_ankle_ft_sensor_left="${has_ankle_ft_sensor_left}" torso_imu_model="${torso_imu_model}" base_imu_model="${base_imu_model}" />
+    <xacro:kangaroo_ros2_control
+      arm_type="${arm_type}"
+      has_ankle_ft_sensor_right="${has_ankle_ft_sensor_right}"
+      has_ankle_ft_sensor_left="${has_ankle_ft_sensor_left}"
+      torso_imu_model="${torso_imu_model}"
+      base_imu_model="${base_imu_model}"
+      emit_transmissions="${sim_type == 'no-simulation' or sim_model == 'full'}" />
   </xacro:unless>
 </robot>

File: kangaroo_description/ros2_control/ros2_control.urdf.xacro (robot description, xacro)
@@ -45,5 +45,5 @@
   </xacro:macro>
   <!-- MACRO DEFINITION-->
-  <xacro:macro name="kangaroo_ros2_control" params="arm_type has_ankle_ft_sensor_right has_ankle_ft_sensor_left torso_imu_model base_imu_model">
+  <xacro:macro name="kangaroo_ros2_control" params="arm_type has_ankle_ft_sensor_right has_ankle_ft_sensor_left torso_imu_model base_imu_model emit_transmissions:=false">
     <ros2_control name="ros2_control_kangaroo_system" type="system" is_async="${'true' if sim_type == 'no-simulation' else 'false'}">
       <xacro:if value="${sim_type == 'no-simulation'}" >
@@ -71,6 +71,6 @@
         <xacro:pelvis_ros2_control />
       </xacro:if>
-      <xacro:leg_ros2_control side="left" has_ankle_ft_sensor="${has_ankle_ft_sensor_left}"/>
-      <xacro:leg_ros2_control side="right" has_ankle_ft_sensor="${has_ankle_ft_sensor_right}"/>
+      <xacro:leg_ros2_control side="left" has_ankle_ft_sensor="${has_ankle_ft_sensor_left}" emit_transmissions="${emit_transmissions}"/>
+      <xacro:leg_ros2_control side="right" has_ankle_ft_sensor="${has_ankle_ft_sensor_right}" emit_transmissions="${emit_transmissions}"/>
       <xacro:if value="${arm_type != 'no-arm'}">
         <xacro:arm_ros2_control side="left" arm_type="${arm_type}"/>

File: kangaroo_description/urdf/leg/ros2_control.urdf.xacro (robot description, xacro)
@@ -20,5 +20,5 @@
   <xacro:include filename="$(find kangaroo_description)/urdf/ankle/ankle.transmission.xacro" />
   <!-- MACRO DEFINITION-->
-  <xacro:macro name="leg_ros2_control" params="side has_ankle_ft_sensor:=false">
+  <xacro:macro name="leg_ros2_control" params="side has_ankle_ft_sensor:=false emit_transmissions:=false">
     <xacro:joint_ros2control name="leg_${side}_1" initial_position="0.0" />
     <xacro:joint_ros2control name="leg_${side}_2" initial_position="0.05" />
@@ -29,5 +29,5 @@
     <xacro:passive_joint_ros2control name="leg_${side}_femur" initial_position="0.9" />
     <xacro:passive_joint_ros2control name="leg_${side}_knee" initial_position="1.8" />
-    <xacro:if value="${sim_type == 'no-simulation'}" >
+    <xacro:if value="${emit_transmissions}">
       <xacro:hip_transmission_yaw side="${side}" offset="${leg_1_joint_offset}" initial_position="0.0" />
       <xacro:hip_transmission_roll_pitch side="${side}" roll_joint="3" pitch_joint="2" />
