Commit message: Updated the crane URDF to be similar to that of the TALOS

File: kangaroo_description/urdf/crane/crane.urdf.xacro (robot description, xacro)
@@ -1,70 +1,42 @@
 <?xml version="1.0"?>
 <!--
-  Copyright (c) 2020, PAL Robotics, S.L.
+  Copyright (c) 2016, PAL Robotics, S.L.
   All rights reserved.
+  This work is licensed under the Creative Commons Attribution-NonCommercial-NoDerivs 3.0 Unported License.
+  To view a copy of this license, visit http://creativecommons.org/licenses/by-nc-nd/3.0/ or send a letter to
+  Creative Commons, 444 Castro Street, Suite 900, Mountain View, California, 94041, USA.
 -->
 <robot xmlns:xacro="http://ros.org/wiki/xacro">
   <!--File includes-->
-  <xacro:include filename="$(find kangaroo_description)/urdf/deg_to_rad.xacro" />
+  <xacro:include filename="$(find talos_description)/urdf/deg_to_rad.xacro" />
   <xacro:macro name="crane" params="parent">
-    <link name="crane_link_1">
+    <link name="crane_link">
       <inertial>
-        <origin xyz="0.0 0.0 -0.5" rpy="0.0 0.0 0.0"/>
-        <mass value="10.0"/>
+        <origin xyz="0.0 0.0 0.25" rpy="0.0 0.0 0.0"/>
+        <mass value="0.0"/>
         <!-- [ m(3r^2 + h^2)/12     m(3r^2 + h^2)/12    mr^2/2] -->
-        <inertia ixx="0.011" ixy="0.0" ixz="0.0"
-                 iyy="0.011" iyz="0.0"
-                 izz="0.011"/>
+        <inertia ixx="0.0" ixy="0.0" ixz="0.0"
+                 iyy="0.0" iyz="0.0"
+                 izz="0.0"/>
       </inertial>
       <visual>
-        <origin xyz="0 0 -0.5" rpy="0 0 0" />
+        <origin xyz="0 0 0.25" rpy="0 0 0" />
         <geometry>
-          <box size="0.2 0.1 1.0"/>
+          <cylinder length="0.5" radius="0.3"/>
         </geometry>
         <material name="CraneMaterial" rgba="0.3 0.3 0.3 0.1"/>
       </visual>
       <collision>
-        <origin xyz="0 0 -0.5" rpy="0 0 0" />
+        <origin xyz="0 0 0.25" rpy="0 0 0" />
         <geometry>
-          <box size="0.2 0.1 1.0"/>
+          <cylinder length="0.5" radius="0.3"/>
         </geometry>
-          <material name="CraneMaterial"/>
+        <material name="CraneMaterial"/>
       </collision>
     </link>
-    <joint name="crane_joint_1" type="fixed">
+    <joint name="crane_joint" type="fixed">
       <parent link="${parent}" />
-      <child link="crane_link_1" />
-      <origin xyz="-0.25 0.0 0.0" rpy="0.0  0.0  0.0"/>
-      <limit lower="0.0" upper="0.0" effort="0.0" velocity="0.0" />
-      <dynamics friction="0.0" damping="0.0"/>
-    </joint>
-      <link name="crane_link_2">
-      <inertial>
-        <origin xyz="0.0 0.0 0.0" rpy="0.0 0.0 0.0"/>
-        <mass value="100.0"/>
-        <!-- [ m(3r^2 + h^2)/12     m(3r^2 + h^2)/12    mr^2/2] -->
-        <inertia ixx="0.011" ixy="0.0" ixz="0.0"
-                 iyy="0.011" iyz="0.0"
-                 izz="0.011"/>
-      </inertial>
-      <visual>
-        <origin xyz="0.0 0 0.0" rpy="0 0 0" />
-        <geometry>
-          <box size="0.8 0.8 0.05"/>
-        </geometry>
-        <material name="CraneMaterial" rgba="0.3 0.3 0.3 0.1"/>
-      </visual>
-      <collision>
-        <origin xyz="0.0 0 0.0" rpy="0 0 0" />
-        <geometry>
-          <box size="0.8 0.8 0.05"/>
-        </geometry>
-          <material name="CraneMaterial"/>
-      </collision>
-    </link>
-    <joint name="crane_joint_2" type="fixed">
-      <parent link="crane_link_1" />
-      <child link="crane_link_2" />
-      <origin xyz="0.0 0.0 -1.025" rpy="0.0  0.0  0.0"/>
+      <child link="crane_link" />
+      <origin xyz="0.003 0.0 0.4" rpy="0.0  0.0  0.0"/>
       <limit lower="0.0" upper="0.0" effort="0.0" velocity="0.0" />
       <dynamics friction="0.0" damping="0.0"/>
