Commit message: add version argument into the base link xacro

File: kangaroo_description/urdf/base/base_2022.urdf.xacro (robot description, xacro)
@@ -1,5 +1,5 @@
 <?xml version="1.0"?>
 <robot xmlns:xacro="http://ros.org/wiki/xacro" name="kangaroo">
-<xacro:macro name="base_link" params="with_cage:=true">
+<xacro:macro name="base_link" params="with_cage:=true version:=${version}">
 <xacro:if value="${with_cage}">
 <link name="base_link">
@@ -13,5 +13,5 @@
       <origin xyz="0 0 0" rpy="0 0 0" />
       <geometry>
-        <mesh filename="package://kangaroo_description/meshes/base_link_with_cage.stl" />
+        <mesh filename="package://kangaroo_description/meshes/${version}/base_link_with_cage.stl" />
       </geometry>
       <material name="">
@@ -22,5 +22,5 @@
       <origin xyz="0 0 0" rpy="0 0 0" />
       <geometry>
-        <mesh filename="package://kangaroo_description/meshes/base_link_convex_hull.stl" />
+        <mesh filename="package://kangaroo_description/meshes/${version}/base_link_convex_hull.stl" />
       </geometry>
     </collision>
@@ -38,5 +38,5 @@
       <origin xyz="0 0 0" rpy="0 0 0" />
       <geometry>
-        <mesh filename="package://kangaroo_description/meshes/base_link.stl" />
+        <mesh filename="package://kangaroo_description/meshes/${version}/base_link.stl" />
       </geometry>
       <material name="">
@@ -47,5 +47,5 @@
       <origin xyz="0 0 0" rpy="0 0 0" />
       <geometry>
-        <mesh filename="package://kangaroo_description/meshes/base_link.stl" />
+        <mesh filename="package://kangaroo_description/meshes/${version}/base_link.stl" />
       </geometry>
     </collision>

Commit message: fix the version hardcoded value of macro

File: kangaroo_description/urdf/base/base_2022.urdf.xacro (robot description, xacro)
@@ -1,5 +1,5 @@
 <?xml version="1.0"?>
 <robot xmlns:xacro="http://ros.org/wiki/xacro" name="kangaroo">
-<xacro:macro name="base_link" params="with_cage:=true version:=${version}">
+<xacro:macro name="base_link" params="with_cage:=true version:=2022">
 <xacro:if value="${with_cage}">
 <link name="base_link">
