Commit message: Set the proper IMU transform for the new model 2023

File: kangaroo_description/urdf/base/base_2023.urdf.xacro (robot description, xacro)
@@ -1,4 +1,5 @@
 <?xml version="1.0"?>
 <robot xmlns:xacro="http://ros.org/wiki/xacro" name="kangaroo">
+<xacro:include filename="$(find kangaroo_description)/urdf/sensors/imu.urdf.xacro"/>
 <xacro:macro name="base_link" params="version:=2023 with_cage:=true">
   <link name="base_link">
@@ -54,4 +55,7 @@
     <axis xyz="0 0 0" />
   </joint>
+  <xacro:kangaroo_imu name="imu" parent="torso_link" update_rate="100.0">
+    <origin xyz="0.071 -0.0014 0.02" rpy="${180.0*deg_to_rad} ${0.0*deg_to_rad} ${-90.0*deg_to_rad}"/>
+  </xacro:kangaroo_imu>
 </xacro:macro>
 </robot>
