Commit message: Changes to fix issues with tf

File: kangaroo_description/urdf/base/base.urdf.xacro (robot description, xacro)
@@ -22,5 +22,5 @@
       <origin xyz="0 0 0" rpy="0 0 0" />
       <geometry>
-        <mesh filename="package://kangaroo_description/meshes/base_link_with_cage.stl" />
+        <mesh filename="package://kangaroo_description/meshes/base_link_convex_hull.stl" />
       </geometry>
     </collision>

File: kangaroo_description/urdf/leg/leg.transmission.xacro (robot description, xacro)
@@ -59,4 +59,24 @@
         <hardwareInterface>hardware_interface/PositionJointInterface</hardwareInterface>
         <hardwareInterface>hardware_interface/EffortJointInterface</hardwareInterface>
+        <hardwareInterface>hardware_interface/JointStateInterface</hardwareInterface>
+      </joint>
+    </transmission>
+    <transmission name="leg_${side}_leg_knee_transmission">
+      <type>transmission_interface/SimpleTransmission</type>
+      <actuator name="leg_${side}_knee_motor" >
+        <hardwareInterface>hardware_interface/JointStateInterface</hardwareInterface>
+        <mechanicalReduction>1.0</mechanicalReduction>
+      </actuator>
+      <joint name="leg_${side}_knee_joint">
+        <hardwareInterface>hardware_interface/JointStateInterface</hardwareInterface>
+      </joint>
+    </transmission>
+    <transmission name="leg_${side}_femur_joint_transmission">
+      <type>transmission_interface/SimpleTransmission</type>
+      <actuator name="leg_${side}_femur_motor" >
+        <hardwareInterface>hardware_interface/JointStateInterface</hardwareInterface>
+        <mechanicalReduction>1.0</mechanicalReduction>
+      </actuator>
+      <joint name="leg_${side}_femur_joint">
         <hardwareInterface>hardware_interface/JointStateInterface</hardwareInterface>
       </joint>

Commit message: updated handle inertia

File: kangaroo_description/urdf/base/base.urdf.xacro (robot description, xacro)
@@ -147,17 +147,14 @@
   <xacro:unless value="${with_belt}">
   <link name="back_handle">
-     <inertial>
-      <origin
-        xyz="-0.1 0 0.02479"
-        rpy="0 0 0" />
-      <mass
-        value="0.2" />
+    <inertial>
+      <origin xyz="-0.1742 2.256E-05 -0.0026718" rpy="0 0 3.14159" />
+      <mass value="0.32489" />
       <inertia
-        ixx="0.01972"
-        ixy="-1E-05"
-        ixz="-0.00037"
-        iyy="0.01996"
-        iyz="0"
-        izz="0.03879" />
+        ixx="0.0054596"
+        ixy="-2.9277E-08"
+        ixz="-0.00058382"
+        iyy="0.0015135"
+        iyz="1.3465E-08"
+        izz="0.006106" />
     </inertial>
     <visual>

Commit message: Update base_link mass and inertial properties

File: kangaroo_description/urdf/base/base.urdf.xacro (robot description, xacro)
@@ -25,14 +25,8 @@
       <link name="base_link">
         <inertial>
-          <origin xyz="-0.098278 0.0050886 -0.0322547" rpy="0 0 0" />
-          <mass value="2.6738" />
-          <inertia
-            ixx="0.022825"
-            ixy="-0.00038658"
-            ixz="0.00034009"
-            iyy="0.008341"
-            iyz="-4.4033E-05"
-            izz="0.027837" />
-        </inertial>
+          <mass value="4.951914"/>
+          <origin xyz="-0.109747 -0.000051 -0.014501" rpy="0 0 0"/>
+          <inertia ixx="0.035976" ixy="-0.000021" ixz="0.001481"
+            iyy="0.025426" iyz="0.000014" izz="0.051135"/>
         <visual>
           <origin xyz="0 0 0" rpy="0 0 0" />
@@ -104,16 +98,8 @@
       <link name="base_link">
         <inertial>
-          <origin
-            xyz="-0.0976652 0.0052196 -0.0319554"
-            rpy="0 0 0" />
-          <mass
-            value="2.5752" />
-          <inertia
-            ixx="0.022653"
-            ixy="-0.00037405"
-            ixz="0.00039289"
-            iyy="0.0079829"
-            iyz="-3.4044E-05"
-            izz="0.027412" />
+          <mass value="4.951914"/>
+          <origin xyz="-0.109747 -0.000051 -0.014501" rpy="0 0 0"/>
+          <inertia ixx="0.035976" ixy="-0.000021" ixz="0.001481"
+            iyy="0.025426" iyz="0.000014" izz="0.051135"/>
         </inertial>
         <visual>

Commit message: Fix the missing inertial tag

File: kangaroo_description/urdf/base/base.urdf.xacro (robot description, xacro)
@@ -29,4 +29,5 @@
           <inertia ixx="0.035976" ixy="-0.000021" ixz="0.001481"
             iyy="0.025426" iyz="0.000014" izz="0.051135"/>
+        </inertial>
         <visual>
           <origin xyz="0 0 0" rpy="0 0 0" />
