Commit message: move the original ankle.urdf.xacro to be version 2022

File: kangaroo_description/urdf/ankle/ankle_2022.urdf.xacro (robot description, xacro)
@@ -9,11 +9,11 @@
   <xacro:property name="roll_joint_min_pos"   value="${-27.0 *deg_to_rad}" />
   <xacro:property name="roll_joint_max_pos"   value="${27.0 *deg_to_rad}" />
-  <xacro:macro name="kangaroo_ankle" params="side reflect parent *origin pitch_joint roll_joint read_actuator simulation:=false ft_sensors:=false">
+  <xacro:macro name="kangaroo_ankle" params="side reflect parent *origin pitch_joint roll_joint read_actuator simulation:=false ft_sensors:=false version:=2022">
     <link name="leg_${side}_${pitch_joint}_link">
       <inertial>
-        <origin xyz="-0.00759994843981759 -6.94997526196062E-09 5.88281323654627E-08" rpy="0 0 0" />
-        <mass value="0.0905838346535586" />
-        <inertia ixx="4.05264139412808E-06" ixy="-5.2860301956695E-12" ixz="4.99859544268276E-11"
-          iyy="2.92762581820543E-05" iyz="6.24254988575372E-12" izz="2.98863057177445E-05" />
+        <origin xyz="-0.00714160332877733 4.8311277200952E-09 0.00259941265068991" rpy="0 0 0" />
+        <mass value="0.0905836559788966" />
+        <inertia ixx="7.07461991271062E-06" ixy="-1.86951004827933E-12" ixz="8.30282143898823E-06"
+          iyy="2.92762498059213E-05" iyz="1.82895645239997E-11" izz="2.68643074366886E-05" />
       </inertial>
       <visual>
@@ -43,13 +43,12 @@
       <xacro:unless value="${ft_sensors}">
         <inertial>
-          <origin xyz="0.0056012722847415 -5.98528992629133E-06 -0.0297244079568318" rpy="0 0 0" />
-          <mass value="0.61562973648731" />
-          <inertia ixx="0.000511104633992357" ixy="2.29520535343244E-08" ixz="-0.000504403659563376"
-            iyy="0.00170802543470207" iyz="-1.88812897159487E-09" izz="0.00181438717200554" />
+          <origin xyz="0.022056 -3.9166E-05 -0.0099049" rpy="0 0 0" />
+          <mass value="0.41343" />
+          <inertia ixx="0.00435" ixy="2.7E-07" ixz="0.000241" iyy="0.0179" iyz="3.0E-07" izz="0.0185" />
         </inertial>
         <visual>
           <origin xyz="0 0 0" rpy="0 0 0" />
           <geometry>
-            <mesh filename="package://kangaroo_description/meshes/leg_7_link.stl" />
+            <mesh filename="package://kangaroo_description/meshes/${version}/leg_7_link.stl" />
           </geometry>
           <material name="">
@@ -66,13 +65,12 @@
       <xacro:if value="${ft_sensors}">
         <inertial>
-          <origin xyz="0.0056012722847415 -8.11751E-06 -0.062005508" rpy="0 0 0" />
-          <mass value="0.826924" />
-          <inertia ixx="0.000511104633992357" ixy="2.29520535343244E-08" ixz="-0.000504403659563376"
-            iyy="0.00170802543470207" iyz="-1.88812897159487E-09" izz="0.00181438717200554" />
+          <origin xyz="0.022204 -8.11751E-06 -0.042186" rpy="0 0 0" />
+          <mass value="0.624725" />
+          <inertia ixx="0.0004094" ixy="2.2E-08" ixz="-0.000244" iyy="0.0009742" iyz="-1.25E-09" izz="0.0011036" />
         </inertial>
         <visual>
           <origin xyz="0 0 0" rpy="0 0 0" />
           <geometry>
-            <mesh filename="package://kangaroo_description/meshes/leg_7_link_ft.stl" />
+            <mesh filename="package://kangaroo_description/meshes/${version}/leg_7_link_ft.stl" />
           </geometry>
           <material name="">
@@ -83,5 +81,5 @@
           <origin xyz="0 0 0" rpy="0 0 0" />
           <geometry>
-            <mesh filename="package://kangaroo_description/meshes/leg_7_link_ft.stl" />
+            <mesh filename="package://kangaroo_description/meshes/${version}/leg_7_link_ft.stl" />
           </geometry>
         </collision>

File: kangaroo_description/urdf/leg/leg_2022.urdf.xacro (robot description, xacro)
@@ -2,5 +2,5 @@
 <robot xmlns:xacro="http://ros.org/wiki/xacro" name="kangaroo">
   <xacro:include filename="$(find kangaroo_description)/urdf/leg/leg.transmission.xacro" />
-  <xacro:include filename="$(find kangaroo_description)/urdf/ankle/ankle.urdf.xacro" />
+  <xacro:include filename="$(find kangaroo_description)/urdf/ankle/ankle_2022.urdf.xacro" />
   <xacro:property name="deg_to_rad"       value="0.01745329251994329577" />
   <xacro:property name="eps_radians"      value="0.008" /> <!-- 0.45deg -->
