Commit message: reduce the range of the ankle

File: kangaroo_description/urdf/ankle/ankle_2023.urdf.xacro (robot description, xacro)
@@ -6,5 +6,5 @@
   <xacro:property name="eps_radians"      value="0.008" /> <!-- 0.45deg -->
   <xacro:property name="pitch_joint_min_pos"   value="${-42.5 *deg_to_rad}" />
-  <xacro:property name="pitch_joint_max_pos"   value="${42.5 *deg_to_rad}" />
+  <xacro:property name="pitch_joint_max_pos"   value="${38.0 *deg_to_rad}" />
   <xacro:property name="roll_joint_min_pos"   value="${-27.0 *deg_to_rad}" />
   <xacro:property name="roll_joint_max_pos"   value="${27.0 *deg_to_rad}" />

Commit message: apply angle with macro

File: kangaroo_description/urdf/ankle/ankle_2023.urdf.xacro (robot description, xacro)
@@ -49,5 +49,5 @@
         </inertial>
         <visual>
-          <origin xyz="0 0 0" rpy="0 0.349065850398867 0" />
+          <origin xyz="0 0 0" rpy="0 ${20.0 * deg_to_rad} 0" />
           <geometry>
             <mesh filename="package://kangaroo_description/meshes/${version}/leg_7_link.stl" />
@@ -58,5 +58,5 @@
         </visual>
         <collision>
-          <origin xyz="0 0 0" rpy="0 0.349065850398867 0" />
+          <origin xyz="0 0 0" rpy="0 ${20.0 * deg_to_rad} 0" />
           <geometry>
             <mesh filename="package://kangaroo_description/meshes/${version}/leg_7_link.stl" />
@@ -121,5 +121,5 @@
         <parent link="leg_${side}_${roll_joint}_aligned_link" />
         <child link="${side}_ft_sensor_link" />
-        <origin xyz="0.00855050358313864 0 -0.023492315519661" rpy="0 -0.349065850398857 0" />
+        <origin xyz="0.00855050358313864 0 -0.023492315519661" rpy="0 ${-20.0 * deg_to_rad} 0" />
       </joint>
     </xacro:if>

Commit message: Set the link 5 to the aligned one by default

File: kangaroo_description/urdf/ankle/ankle_2023.urdf.xacro (robot description, xacro)
@@ -49,5 +49,5 @@
         </inertial>
         <visual>
-          <origin xyz="0 0 0" rpy="0 ${20.0 * deg_to_rad} 0" />
+          <origin xyz="0 0 0" rpy="0 0 0" />
           <geometry>
             <mesh filename="package://kangaroo_description/meshes/${version}/leg_7_link.stl" />
@@ -58,5 +58,5 @@
         </visual>
         <collision>
-          <origin xyz="0 0 0" rpy="0 ${20.0 * deg_to_rad} 0" />
+          <origin xyz="0 0 0" rpy="0 0 0" />
           <geometry>
             <mesh filename="package://kangaroo_description/meshes/${version}/leg_7_link.stl" />
@@ -104,20 +104,20 @@
     </link>
     <joint name="leg_${side}_${roll_joint}_joint" type="revolute">
-      <origin xyz="0 0 0" rpy="0 0 0" />
+      <origin xyz="0 0 0" rpy="0 ${20.0 * deg_to_rad} 0" />
       <parent link="leg_${side}_${pitch_joint}_link" />
       <child link="leg_${side}_${roll_joint}_link" />
-      <axis xyz="-0.93969 0 0.34202" />
+      <axis xyz="-1 0 0" />
       <limit lower="${roll_joint_min_pos}" upper="${roll_joint_max_pos}" effort="100" velocity="3.87" />
     </joint>
     <link name="leg_${side}_${roll_joint}_aligned_link"/>
     <joint name="leg_${side}_${roll_joint}_aligned_joint" type="fixed">
-      <parent link="leg_${side}_${roll_joint}_link" />
+      <parent link="leg_${side}_${pitch_joint}_link" />
       <child link="leg_${side}_${roll_joint}_aligned_link" />
-      <origin xyz="0.0 0.0 0.0" rpy="0 ${20.0 * deg_to_rad} 0" />
+      <origin xyz="0 0 0" rpy="0 0 0" />
     </joint>
     <xacro:if value="${ft_sensors}">
       <link name="${side}_ft_sensor_link"/>
       <joint name="${side}_ft_sensor_joint" type="fixed">
-        <parent link="leg_${side}_${roll_joint}_aligned_link" />
+        <parent link="leg_${side}_${roll_joint}_link" />
         <child link="${side}_ft_sensor_link" />
         <origin xyz="0.00855050358313864 0 -0.023492315519661" rpy="0 ${-20.0 * deg_to_rad} 0" />
@@ -127,5 +127,5 @@
     <joint name="${side}_sole_joint" type="fixed">
       <xacro:unless value="${ft_sensors}">
-        <parent link="leg_${side}_${roll_joint}_link" />
+        <parent link="leg_${side}_${roll_joint}_aligned_link" />
         <child link="${side}_sole_link" />
         <origin xyz="0.028 0.0 -0.029" rpy="0 0 0" />

Commit message: Fix the collision link orientation

File: kangaroo_description/urdf/ankle/ankle_2023.urdf.xacro (robot description, xacro)
@@ -64,5 +64,5 @@
         </collision>
         <collision>
-          <origin xyz="0.0 0.0 -0.03" rpy="0 0 0" />
+          <origin xyz="0.0 0.0 -0.03" rpy="0 ${-20.0 * deg_to_rad} 0" />
           <geometry>
             <!-- The length of the sole is around 24cm, but with the attached rubber sole it would be 24.9cm -->

Commit message: Fix the ankle sole link position for the new soles

File: kangaroo_description/urdf/ankle/ankle_2023.urdf.xacro (robot description, xacro)
@@ -129,10 +129,10 @@
         <parent link="leg_${side}_${roll_joint}_aligned_link" />
         <child link="${side}_sole_link" />
-        <origin xyz="0.028 0.0 -0.029" rpy="0 0 0" />
+        <origin xyz="0.0 0.0 -0.029" rpy="0 0 0" />
       </xacro:unless>
       <xacro:if value="${ft_sensors}">
         <parent link="${side}_ft_sensor_link" />
         <child link="${side}_sole_link" />
-        <origin xyz="0.034889 0 -0.0495" rpy="0 0 0" />
+        <origin xyz="0.006889 0 -0.0495" rpy="0 0 0" />
       </xacro:if>
     </joint>

Commit message: Fix the leg sole link parent link

File: kangaroo_description/urdf/ankle/ankle_2023.urdf.xacro (robot description, xacro)
@@ -119,5 +119,5 @@
       <link name="${side}_ft_sensor_link"/>
       <joint name="${side}_ft_sensor_joint" type="fixed">
-        <parent link="leg_${side}_${roll_joint}_link" />
+        <parent link="leg_${side}_${roll_joint}_aligned_link" />
         <child link="${side}_ft_sensor_link" />
         <origin xyz="0.00855050358313864 0 -0.023492315519661" rpy="0 ${-20.0 * deg_to_rad} 0" />
@@ -127,7 +127,7 @@
     <joint name="${side}_sole_joint" type="fixed">
       <xacro:unless value="${ft_sensors}">
-        <parent link="leg_${side}_${roll_joint}_aligned_link" />
+        <parent link="leg_${side}_${roll_joint}_link" />
         <child link="${side}_sole_link" />
-        <origin xyz="0.0 0.0 -0.029" rpy="0 0 0" />
+        <origin xyz="0.0 0.0 -0.029" rpy="0 ${-20.0 * deg_to_rad} 0" />
       </xacro:unless>
       <xacro:if value="${ft_sensors}">

Commit message: change the ankle pitch joint to be aligned with the ankle roll link

File: kangaroo_description/urdf/ankle/ankle_2023.urdf.xacro (robot description, xacro)
@@ -18,5 +18,5 @@
       </inertial>
       <visual>
-        <origin xyz="0 0 0" rpy="0 0 0" />
+        <origin xyz="0 0 0" rpy="0 ${-20.0 * deg_to_rad} 0" />
         <geometry>
           <mesh filename="package://kangaroo_description/meshes/leg_6_link.stl" />
@@ -27,5 +27,5 @@
       </visual>
       <collision>
-        <origin xyz="0 0 0" rpy="0 0 0" />
+        <origin xyz="0 0 0" rpy="0 ${-20.0 * deg_to_rad} 0" />
         <geometry>
           <mesh filename="package://kangaroo_description/meshes/leg_6_link.stl" />
@@ -64,5 +64,5 @@
         </collision>
         <collision>
-          <origin xyz="0.0 0.0 -0.03" rpy="0 ${-20.0 * deg_to_rad} 0" />
+          <origin xyz="0.01 0.0 -0.0325" rpy="0 ${-20.0 * deg_to_rad} 0" />
           <geometry>
             <!-- The length of the sole is around 24cm, but with the attached rubber sole it would be 24.9cm -->
@@ -104,5 +104,5 @@
     </link>
     <joint name="leg_${side}_${roll_joint}_joint" type="revolute">
-      <origin xyz="0 0 0" rpy="0 ${20.0 * deg_to_rad} 0" />
+      <origin xyz="0 0 0" rpy="0 0 0" />
       <parent link="leg_${side}_${pitch_joint}_link" />
       <child link="leg_${side}_${roll_joint}_link" />
@@ -114,5 +114,5 @@
       <parent link="leg_${side}_${pitch_joint}_link" />
       <child link="leg_${side}_${roll_joint}_aligned_link" />
-      <origin xyz="0 0 0" rpy="0 0 0" />
+      <origin xyz="0 0 0" rpy="0 ${-20.0 * deg_to_rad} 0" />
     </joint>
     <xacro:if value="${ft_sensors}">
@@ -127,7 +127,7 @@
     <joint name="${side}_sole_joint" type="fixed">
       <xacro:unless value="${ft_sensors}">
-        <parent link="leg_${side}_${roll_joint}_link" />
+        <parent link="leg_${side}_${roll_joint}_aligned_link" />
         <child link="${side}_sole_link" />
-        <origin xyz="0.0 0.0 -0.029" rpy="0 ${-20.0 * deg_to_rad} 0" />
+        <origin xyz="0.0 0.0 -0.0425" rpy="0 0 0" />
       </xacro:unless>
       <xacro:if value="${ft_sensors}">

File: kangaroo_description/urdf/leg/leg_2023.urdf.xacro (robot description, xacro)
@@ -267,5 +267,5 @@
     </joint>
     <xacro:kangaroo_ankle side="${side}" parent="leg_${side}_length_link" reflect="${reflect}" roll_joint="5" pitch_joint="4" read_actuator="leg_${side}_length_motor" ft_sensors="$(arg ft_sensors)">
-      <origin xyz="0.0 0 0.0" rpy="0 ${180 *deg_to_rad} 0" />
+      <origin xyz="0.0 0 0.0" rpy="0 ${200 *deg_to_rad} 0" />
     </xacro:kangaroo_ankle>
     <!-- Load corresponding transmission info -->

Commit message: use the roll joint as the parent to the roll aligned joint

File: kangaroo_description/urdf/ankle/ankle_2023.urdf.xacro (robot description, xacro)
@@ -64,5 +64,5 @@
         </collision>
         <collision>
-          <origin xyz="0.01 0.0 -0.0325" rpy="0 ${-20.0 * deg_to_rad} 0" />
+          <origin xyz="0.01 0.0 -0.028" rpy="0 ${-20.0 * deg_to_rad} 0" />
           <geometry>
             <!-- The length of the sole is around 24cm, but with the attached rubber sole it would be 24.9cm -->
@@ -112,5 +112,5 @@
     <link name="leg_${side}_${roll_joint}_aligned_link"/>
     <joint name="leg_${side}_${roll_joint}_aligned_joint" type="fixed">
-      <parent link="leg_${side}_${pitch_joint}_link" />
+      <parent link="leg_${side}_${roll_joint}_link" />
       <child link="leg_${side}_${roll_joint}_aligned_link" />
       <origin xyz="0 0 0" rpy="0 ${-20.0 * deg_to_rad} 0" />

Commit message: Add 20 deg angle change to the old ankle model

File: kangaroo_description/urdf/ankle/ankle_2023.urdf.xacro (robot description, xacro)
@@ -80,5 +80,5 @@
         </inertial>
         <visual>
-          <origin xyz="0 0 0" rpy="0 0 0" />
+          <origin xyz="0 0 0" rpy="0 ${-20.0 * deg_to_rad} 0" />
           <geometry>
             <mesh filename="package://kangaroo_description/meshes/${version}/leg_7_link_ft.stl" />
@@ -89,5 +89,5 @@
         </visual>
         <collision>
-          <origin xyz="0 0 0" rpy="0 0 0" />
+          <origin xyz="0 0 0" rpy="0 ${-20.0 * deg_to_rad} 0" />
           <geometry>
             <mesh filename="package://kangaroo_description/meshes/${version}/leg_7_link_ft.stl" />
@@ -95,5 +95,5 @@
         </collision>
         <collision>
-          <origin xyz="0.0 0.0 -0.065" rpy="0 0 0" />
+          <origin xyz="0.0 0.0 -0.065" rpy="0 ${-20.0 * deg_to_rad} 0" />
           <geometry>
             <!-- The length of the sole is around 24cm, but with the attached rubber sole it would be 24.9cm -->

Commit message: Set correct effort joint limits

File: kangaroo_description/urdf/ankle/ankle_2023.urdf.xacro (robot description, xacro)
@@ -38,5 +38,5 @@
       <child link="leg_${side}_${pitch_joint}_link" />
       <axis xyz="0 1 0" />
-      <limit lower="${pitch_joint_min_pos}" upper="${pitch_joint_max_pos}" effort="100" velocity="3.87" />
+      <limit lower="${pitch_joint_min_pos}" upper="${pitch_joint_max_pos}" effort="140" velocity="3.87" />
     </joint>
     <link name="leg_${side}_${roll_joint}_link">
@@ -108,5 +108,5 @@
       <child link="leg_${side}_${roll_joint}_link" />
       <axis xyz="-1 0 0" />
-      <limit lower="${roll_joint_min_pos}" upper="${roll_joint_max_pos}" effort="100" velocity="3.87" />
+      <limit lower="${roll_joint_min_pos}" upper="${roll_joint_max_pos}" effort="82" velocity="3.87" />
     </joint>
     <link name="leg_${side}_${roll_joint}_aligned_link"/>

File: kangaroo_description/urdf/leg/leg_2023.urdf.xacro (robot description, xacro)
@@ -66,8 +66,8 @@
       <axis xyz="0 0 1" />
       <xacro:if value="${reflect == 1}">
-        <limit lower="${leg_1_min_pos}" upper="${leg_1_max_pos}" effort="150" velocity="3.87" />
+        <limit lower="${leg_1_min_pos}" upper="${leg_1_max_pos}" effort="80" velocity="3.87" />
       </xacro:if>
       <xacro:if value="${reflect == -1}">
-        <limit lower="${reflect * leg_1_max_pos}" upper="${reflect * leg_1_min_pos}" effort="150" velocity="3.87" />
+        <limit lower="${reflect * leg_1_max_pos}" upper="${reflect * leg_1_min_pos}" effort="80" velocity="3.87" />
       </xacro:if>
     </joint>
@@ -102,5 +102,5 @@
       <child link="leg_${side}_2_link" />
       <axis xyz="0 1 0" />
-      <limit lower="${leg_2_min_pos}" upper="${leg_2_max_pos}" effort="150" velocity="3.87" />
+      <limit lower="${leg_2_min_pos}" upper="${leg_2_max_pos}" effort="230" velocity="3.87" />
     </joint>
     <link name="leg_${side}_3_link">
@@ -132,5 +132,5 @@
       <child link="leg_${side}_3_link" />
       <axis xyz="1 0 0" />
-      <limit lower="${leg_3_min_pos}" upper="${leg_3_max_pos}" effort="150" velocity="3.87" />
+      <limit lower="${leg_3_min_pos}" upper="${leg_3_max_pos}" effort="139" velocity="3.87" />
     </joint>
     <link name="leg_${side}_femur_link">
@@ -231,5 +231,5 @@
       <child link="leg_${side}_length_link" />
       <axis xyz="0 0 1" />
-      <limit lower="${leg_min_length}" upper="${leg_max_length}" effort="1500" velocity="10" />
+      <limit lower="${leg_min_length}" upper="${leg_max_length}" effort="1100" velocity="10" />
     </joint>
     <joint name="leg_${side}_femur_joint" type="revolute">
