Commit message: Add both types of feet

File: kangaroo_description/urdf/ankle/foot_frames.urdf.xacro (robot description, xacro)
@@ -3,5 +3,5 @@
 <xacro:property name="foot_length"   value="0.21" />
 <xacro:property name="foot_width"   value="0.09" />
-<xacro:macro name="kangaroo_foot_frames" params="side parent offset_x:=0.0 offset_y:=0.0">
+<xacro:macro name="kangaroo_fixed_foot_frames" params="side parent offset_x:=0.0 offset_y:=0.0">
 	<link name="${side}_foot_upper_left"/>
 	<link name="${side}_foot_upper_right"/>

File: kangaroo_description/urdf/leg/leg.urdf.xacro (robot description, xacro)
@@ -19,7 +19,6 @@
   <!-- INCLUDES -->
   <!-- <xacro:include filename="$(find kangaroo_description)/urdf/leg/leg.transmission.xacro" /> -->
-  <xacro:include filename="$(find kangaroo_description)/urdf/ankle/ankle.urdf.xacro" />
   <xacro:macro name="kangaroo_leg"
-    params="side reflect parent *origin leg_type:=leg">
+    params="side reflect parent *origin feet_type">
     <link name="leg_${side}_1_link">
       <inertial>
@@ -244,8 +243,18 @@
       <origin rpy="0 0 0" xyz="-0.38 0.0 0.0" />
     </joint>
-    <xacro:kangaroo_ankle side="${side}" parent="leg_${side}_length_link" reflect="${reflect}"
-      roll_joint="5" pitch_joint="4" read_actuator="leg_${side}_length_motor">
-      <origin xyz="0.0 0 0.0" rpy="0 ${200 *deg_to_rad} 0" />
-    </xacro:kangaroo_ankle>
+    <xacro:if value ="${feet_type == 'fixed'}">
+      <xacro:include filename="$(find kangaroo_description)/urdf/ankle/fixed_ankle.urdf.xacro" />
+      <xacro:kangaroo_fixed_ankle side="${side}" parent="leg_${side}_length_link" reflect="${reflect}"
+        roll_joint="5" pitch_joint="4" read_actuator="leg_${side}_length_motor">
+        <origin xyz="0.0 0 0.0" rpy="0 ${200 *deg_to_rad} 0" />
+      </xacro:kangaroo_fixed_ankle>
+    </xacro:if>
+    <xacro:if value ="${feet_type == 'detachable'}">
+      <xacro:include filename="$(find kangaroo_description)/urdf/ankle/detachable_ankle.urdf.xacro" />
+      <xacro:kangaroo_detachable_ankle side="${side}" parent="leg_${side}_length_link" reflect="${reflect}"
+        roll_joint="5" pitch_joint="4" read_actuator="leg_${side}_length_motor">
+        <origin xyz="0.0 0 0.0" rpy="0 ${200 *deg_to_rad} 0" />
+      </xacro:kangaroo_detachable_ankle>
+    </xacro:if>
   </xacro:macro>
 </robot>
