Commit message: Change to prismatic model with mimic joints

File: kangaroo_description/urdf/ankle/ankle.urdf.xacro (robot description, xacro)
@@ -25,10 +25,4 @@
         </material>
       </visual>
-      <collision>
-        <origin xyz="0 0 0" rpy="0 0 0" />
-        <geometry>
-          <mesh filename="package://kangaroo_description/meshes/leg_6_link.stl" />
-        </geometry>
-      </collision>
     </link>
     <joint name="leg_${side}_${pitch_joint}_joint" type="revolute">
@@ -56,7 +50,7 @@
       </visual>
       <collision>
-        <origin xyz="0 0 0" rpy="0 0 0" />
+        <origin xyz="0.035 0 -0.02" rpy="0 0 0" />
         <geometry>
-          <mesh filename="package://kangaroo_description/meshes/leg_7_link.stl" />
+          <box size="0.21 0.09 0.025"/>
         </geometry>
       </collision>
@@ -78,29 +72,41 @@
      <mu1>0.9</mu1>
      <mu2>0.9</mu2>
+     <implicitSpringDamper>1</implicitSpringDamper>
+     <material>Gazebo/FlatWhite</material>
    </gazebo>
-  <!-- contact model for foot surface -->
-  <gazebo reference="leg_{side}_${roll_joint}_link">
-    <kp>1000000.0</kp>
-    <kd>100.0</kd>
-    <mu1>1.0</mu1>
-    <mu2>1.0</mu2>
-    <fdir1>1 0 0</fdir1>
-    <maxVel>1.0</maxVel>
-    <minDepth>0.00</minDepth>
-    <implicitSpringDamper>1</implicitSpringDamper>
-  </gazebo>
-   <gazebo reference="leg_${side}_${pitch_joint}_joint">
+   <!--
+   <gazebo reference="leg_${side}_${roll_joint}_link">
+     <mu1>0.9</mu1>
+     <mu2>0.9</mu2>
+     <implicitSpringDamper>1</implicitSpringDamper>
+     <material>Gazebo/FlatWhite</material>
+   </gazebo>  -->
+   <gazebo reference="leg_${side}_${roll_joint}_link">
+      <kp>1000000.0</kp> <!-- 1000000 -->
+      <kd>100.0</kd>
+      <mu1>1.0</mu1>
+      <mu2>1.0</mu2>
+      <fdir1>1 0 0</fdir1>
+      <maxVel>1.0</maxVel>
+      <minDepth>0.00</minDepth>
       <implicitSpringDamper>1</implicitSpringDamper>
-   </gazebo>
-   <gazebo reference="leg_${side}_${roll_joint}_joint">
       <provideFeedback>1</provideFeedback>
+      <material>Gazebo/FlatWhite</material>
+    </gazebo>
+    <!--
+    <gazebo reference="leg_{side}_${pitch_joint}_link">
+     <kp>1000.0</kp>
+      <kd>10.0</kd>
+      <mu1>1.0</mu1>
+      <mu2>1.0</mu2>
+      <fdir1>1 0 0</fdir1>
+      <fdir2>0 1 0</fdir2>
+      <maxVel>1.0</maxVel>
+      <minDepth>0.00</minDepth>
       <implicitSpringDamper>1</implicitSpringDamper>
-   </gazebo>
-  <gazebo reference="leg_${side}_${pitch_joint}_link">
-    <material>Gazebo/FlatWhite</material>
-  </gazebo>
-  <gazebo reference="leg_${side}_${roll_joint}_link">
-    <material>Gazebo/FlatWhite</material>
-  </gazebo>
+      <provideFeedback>1</provideFeedback>
+      <material>Gazebo/FlatWhite</material>
+    </gazebo>
+    -->
   </xacro:macro>
 </robot>

File: kangaroo_description/urdf/leg/leg.transmission.xacro (robot description, xacro)
@@ -48,5 +48,5 @@
       </joint>
     </transmission>
-    <transmission name="leg_${side}_4_transmission">
+    <!-- <transmission name="leg_${side}_4_transmission">
       <type>transmission_interface/SimpleTransmission</type>
       <actuator name="leg_${side}_4_motor" >
@@ -75,5 +75,5 @@
         <hardwareInterface>hardware_interface/JointStateInterface</hardwareInterface>
       </joint>
-    </transmission>
+    </transmission> -->
     <transmission name="leg_${side}_leg_length_transmission">
       <type>transmission_interface/SimpleTransmission</type>
@@ -91,5 +91,5 @@
     </transmission>
   </xacro:macro>
-  <xacro:macro name="kangaroo_leg_length_actuator_transmission" params="side number1 number2 params_ns:=/leg_params" >
+  <!-- <xacro:macro name="kangaroo_leg_length_actuator_transmission" params="side number1 number2 params_ns:=/leg_params" >
     <transmission name="leg_${side}_${number1}_trans">
       <type>pal_transmissions/LegCustomTransmission</type>
@@ -127,5 +127,5 @@
       </joint>
     </transmission>
-  </xacro:macro>
+  </xacro:macro> -->
   <xacro:macro name="hip_transmission_roll_pitch" params="side roll_joint pitch_joint">
     <transmission name="leg_${side}_transmission_roll_pitch">

File: kangaroo_description/urdf/leg/leg.urdf.xacro (robot description, xacro)
@@ -12,10 +12,28 @@
   <xacro:property name="leg_3_min_pos"   value="${-27.0 *deg_to_rad}" />
   <xacro:property name="leg_3_max_pos"   value="${27.0 *deg_to_rad}" />
-  <xacro:property name="leg_4_min_pos"   value="${10.0 *deg_to_rad}" />
-  <xacro:property name="leg_4_max_pos"   value="${70.0 *deg_to_rad}" />
-  <xacro:property name="leg_5_min_pos"   value="${20.0 *deg_to_rad}" />
-  <xacro:property name="leg_5_max_pos"   value="${140.0 *deg_to_rad}" />
+  <xacro:property name="leg_femur_min_pos"   value="${10.0 *deg_to_rad}" />
+  <xacro:property name="leg_femur_max_pos"   value="${70.0 *deg_to_rad}" />
+  <xacro:property name="leg_knee_min_pos"   value="${20.0 *deg_to_rad}" />
+  <xacro:property name="leg_knee_max_pos"   value="${140.0 *deg_to_rad}" />
   <xacro:property name="leg_min_length"   value="0.131973" />
   <xacro:property name="leg_max_length"   value="0.71416639" />
+  <xacro:macro name="mimic_joint_plugin_gazebo" params="name_prefix parent_joint mimic_joint has_pid:=false multiplier:=1.0 offset:=0 sensitiveness:=0.0 max_effort:=1.0 robot_namespace:=''">
+    <gazebo>
+      <plugin name="${name_prefix}mimic_joint_plugin" filename="libroboticsgroup_gazebo_mimic_joint_plugin.so">
+        <joint>${parent_joint}</joint>
+        <mimicJoint>${mimic_joint}</mimicJoint>
+        <xacro:if value="${has_pid}">                     <!-- if set to true, PID parameters from "/gazebo_ros_control/pid_gains/${mimic_joint}" are loaded -->
+          <hasPID />
+        </xacro:if>
+        <multiplier>${multiplier}</multiplier>
+        <offset>${offset}</offset>
+        <sensitiveness>${sensitiveness}</sensitiveness>   <!-- if absolute difference between setpoint and process value is below this threshold, do nothing; 0.0 = disable [rad] -->
+        <maxEffort>${max_effort}</maxEffort>              <!-- only taken into account if has_pid:=true [Nm] -->
+        <xacro:unless value="${robot_namespace == ''}">
+          <robotNamespace>${robot_namespace}</robotNamespace>
+        </xacro:unless>
+      </plugin>
+    </gazebo>
+  </xacro:macro>
   <xacro:macro name="kangaroo_leg" params="side reflect parent *origin simulation:=false">
     <link name="leg_${side}_1_link">
@@ -69,10 +87,4 @@
         </material>
       </visual>
-      <collision>
-        <origin xyz="0 0 0" rpy="0 0 0" />
-        <geometry>
-          <mesh filename="package://kangaroo_description/meshes/leg_2_link.stl" scale="1 ${reflect} 1"/>
-        </geometry>
-      </collision>
     </link>
     <joint name="leg_${side}_2_joint" type="revolute">
@@ -113,10 +125,9 @@
       <limit lower="${leg_3_min_pos}" upper="${leg_3_max_pos}" effort="100" velocity="3.87" />
     </joint>
-    <link name="leg_${side}_4_link">
+    <link name="leg_${side}_femur_link">
       <inertial>
         <origin xyz="0.114702002010089 0.000182856660852354 -0.0143986490691173" rpy="0 0 0" />
-        <mass value="3.57408268817521" />
-        <inertia ixx="0.00247170768644724" ixy="2.87874888621229E-05" ixz="0.00247469186737281"
-          iyy="0.0126050262407564" iyz="1.01404330133204E-05" izz="0.0116319632922522" />
+        <mass value="0.1" />
+        <inertia ixx="1.E-5" ixy="0.0" ixz="0.0" iyy="1.E-5" iyz="0.0" izz="1.E-5" />
       </inertial>
       <visual>
@@ -129,105 +140,60 @@
         </material>
       </visual>
-      <collision>
-        <origin xyz="0 0 0" rpy="0 0 0" />
-        <geometry>
-          <mesh filename="package://kangaroo_description/meshes/leg_4_link.stl" />
-        </geometry>
-      </collision>
-    </link>
-    <joint name="leg_${side}_4_joint" type="revolute">
+    </link>
+    <link name="leg_${side}_knee_link">
+      <inertial>
+        <origin xyz="-0.158662729273678 -8.28192764317226E-05 -0.0337468261967321" rpy="0 0 0" />
+        <mass value="0.1" />
+        <inertia ixx="1.E-5" ixy="0.0" ixz="0.0" iyy="1.E-5" iyz="0.0" izz="1.E-5" />
+      </inertial>
+      <visual>
+        <origin xyz="0 0 0" rpy="0 0 0" />
+        <geometry>
+          <mesh filename="package://kangaroo_description/meshes/leg_5_link.stl" />
+        </geometry>
+        <material name="">
+          <color rgba="0.752941176470588 0.752941176470588 0.752941176470588 1" />
+        </material>
+      </visual>
+    </link>
+    <link name="leg_${side}_length_link">
+      <inertial>
+        <origin rpy="0 0 0" xyz="0.0 0.0 -0.2"/>
+        <mass value="6.0" />
+        <inertia ixx="0.05" ixy="0.0" ixz="0.0" iyy="0.05" iyz="0.0" izz="0.016875" />
+      </inertial>
+      <visual>
+        <origin rpy="0 0 0" xyz="0 0 ${(leg_min_length - leg_max_length)/2}"/>
+        <geometry>
+          <cylinder length="${(leg_min_length - leg_max_length)}" radius="0.00005"/>
+        </geometry>
+        <material name="DarkGrey" />
+      </visual>
+    </link>
+    <joint name="leg_${side}_length_joint" type="prismatic">
+     <origin xyz="0 ${reflect * 0.0669} -0.09" rpy="0 ${180 * deg_to_rad} 0" />
+      <parent link="leg_${side}_3_link" />
+      <child link="leg_${side}_length_link" />
+      <axis xyz="0 0 1" />
+      <limit lower="${leg_min_length}" upper="${leg_max_length}" effort="500" velocity="10" />
+    </joint>
+    <joint name="leg_${side}_femur_joint" type="revolute">
       <origin xyz="0 ${reflect * 0.0669} -0.09" rpy="0 ${-10.0 * deg_to_rad} 0" />
       <parent link="leg_${side}_3_link" />
-      <child link="leg_${side}_4_link" />
+      <child link="leg_${side}_femur_link" />
       <axis xyz="0 1 0" />
-      <limit lower="${leg_4_min_pos}" upper="${leg_4_max_pos}" effort="100" velocity="3.87" />
-    </joint>
-    <link name="leg_${side}_5_link">
-      <inertial>
-        <origin xyz="-0.158662729273678 -8.28192764317226E-05 -0.0337468261967321" rpy="0 0 0" />
-        <mass value="0.87223211672797" />
-        <inertia ixx="0.000350603269949793" ixy="6.37793331536252E-07" ixz="-0.000461550351107159"
-          iyy="0.00242184402988972" iyz="5.09327556678297E-07" izz="0.0022368624903808" />
-      </inertial>
-      <visual>
-        <origin xyz="0 0 0" rpy="0 0 0" />
-        <geometry>
-          <mesh filename="package://kangaroo_description/meshes/leg_5_link.stl" />
-        </geometry>
-        <material name="">
-          <color rgba="0.752941176470588 0.752941176470588 0.752941176470588 1" />
-        </material>
-      </visual>
-      <collision>
-        <origin xyz="0 0 0" rpy="0 0 0" />
-        <geometry>
-          <mesh filename="package://kangaroo_description/meshes/leg_5_link.stl" />
-        </geometry>
-      </collision>
-    </link>
-    <joint name="leg_${side}_5_joint" type="revolute">
+      <limit lower="${leg_femur_min_pos}" upper="${leg_femur_max_pos}" effort="100" velocity="3.87" />
+      <mimic joint="leg_${side}_length_joint" multiplier="1.69435" offset="-0.096145"/>
+    </joint>
+    <joint name="leg_${side}_knee_joint" type="revolute">
       <origin xyz="0.37413 0 -0.066509" rpy="0 ${20.0 * deg_to_rad} 0" />
-      <parent link="leg_${side}_4_link" />
-      <child link="leg_${side}_5_link" />
+      <parent link="leg_${side}_femur_link" />
+      <child link="leg_${side}_knee_link" />
       <axis xyz="0 -1 0" />
-      <limit lower="${leg_5_min_pos}" upper="${leg_5_max_pos}" effort="100" velocity="3.87" />
-    </joint>
-    <link name="leg_${side}_length_fixed_link">
-      <inertial>
-        <origin rpy="0 0 0" xyz="0.0 0.0 ${leg_min_length/2.0}"/>
-        <!-- TODO: update inertia and mass -->
-        <mass value="1.E-3" />
-        <inertia ixx="1.0E-05" ixy="0.0" ixz="0.0" iyy="1.0E-05" iyz="0.0" izz="1.0E-05" />
-      </inertial>
-      <visual>
-        <origin rpy="0 0 0" xyz="0 0 ${leg_min_length/2.0}"/>
-        <geometry>
-          <cylinder length="${leg_min_length}" radius="0.00005"/>
-        </geometry>
-        <material name="DarkGrey" />
-      </visual>
-      <collision>
-        <origin rpy="0 0 0" xyz="0 0 ${leg_min_length/2.0}"/>
-        <geometry>
-          <cylinder length="${leg_min_length}" radius="0.00005"/>
-        </geometry>
-      </collision>
-    </link>
-    <joint name="leg_${side}_length_fixed_joint" type="fixed">
-        <origin xyz="0 ${reflect * 0.0669} -0.09" rpy="0 ${180.0 * deg_to_rad} 0" />
-        <parent link="leg_${side}_3_link" />
-        <child link="leg_${side}_length_fixed_link" />
-        <axis xyz="0 0 0" />
-    </joint>
-    <link name="leg_${side}_length_link">
-      <inertial>
-        <origin rpy="0 0 0" xyz="0.0 0.0 ${(leg_max_length - leg_min_length)/2}"/>
-        <!-- TODO: update inertia and mass -->
-        <mass value="1.E-3" />
-        <inertia ixx="1.0E-05" ixy="0.0" ixz="0.0" iyy="1.0E-05" iyz="0.0" izz="1.0E-05" />
-      </inertial>
-      <visual>
-        <origin rpy="0 0 0" xyz="0 0 ${(leg_min_length - leg_max_length)/2}"/>
-        <geometry>
-          <cylinder length="${(leg_min_length - leg_max_length)}" radius="0.00005"/>
-        </geometry>
-        <material name="DarkGrey" />
-      </visual>
-      <collision>
-        <origin rpy="0 0 0" xyz="0 0 ${(leg_min_length - leg_max_length)/2}"/>
-        <geometry>
-          <cylinder length="${(leg_min_length - leg_max_length)}" radius="0.00005"/>
-        </geometry>
-      </collision>
-    </link>
-    <joint name="leg_${side}_length_joint" type="prismatic">
-     <origin xyz="0.0 0.0 ${leg_min_length}"  rpy="0.0 0.0 0.0"/>
-      <parent link="leg_${side}_length_fixed_link" />
-      <child link="leg_${side}_length_link" />
-      <axis xyz="0 0 1" />
-      <limit lower="0" upper="${leg_max_length - leg_min_length}" effort="500" velocity="10" /> <!-- TODO: update effort and velocity -->
-    </joint>
-    <xacro:kangaroo_ankle side="${side}" parent="leg_${side}_5_link" reflect="${reflect}" roll_joint="7" pitch_joint="6" read_actuator="leg_${side}_length_motor">
-      <origin xyz="-0.37432 0 -0.065464" rpy="0 0 0" />
+      <limit lower="${leg_knee_min_pos}" upper="${leg_knee_max_pos}" effort="100" velocity="3.87" />
+      <mimic joint="leg_${side}_length_joint" multiplier="3.38877" offset="-0.19229"/>
+    </joint>
+    <xacro:kangaroo_ankle side="${side}" parent="leg_${side}_length_link" reflect="${reflect}" roll_joint="5" pitch_joint="4" read_actuator="leg_${side}_length_motor">
+      <origin xyz="0.0 0 0.0" rpy="0 ${180 *deg_to_rad} 0" />
     </xacro:kangaroo_ankle>
     <!-- Load corresponding transmission info -->
@@ -240,64 +206,66 @@
       <xacro:kangaroo_lower_body_simple_simulation_transmission side="${side}"/>
     </xacro:if>
+    <gazebo reference="leg_${side}_1_link">
+      <mu1>0.9</mu1>
+      <mu2>0.9</mu2>
+    </gazebo>
+    <gazebo reference="leg_${side}_2_link">
+      <mu1>0.9</mu1>
+      <mu2>0.9</mu2>
+    </gazebo>
+    <gazebo reference="leg_${side}_3_link">
+      <mu1>0.9</mu1>
+      <mu2>0.9</mu2>
+    </gazebo>
+    <gazebo reference="leg_${side}_length_link">
+      <mu1>0.9</mu1>
+      <mu2>0.9</mu2>
+    </gazebo>
+    <!-- <gazebo reference="leg_${side}_4_link">
+      <mu1>0.9</mu1>
+      <mu2>0.9</mu2>
+    </gazebo>
+    <gazebo reference="leg_${side}_5_link">
+      <mu1>0.9</mu1>
+      <mu2>0.9</mu2>
+    </gazebo> -->
+   <gazebo reference="leg_${side}_1_joint">
+      <implicitSpringDamper>1</implicitSpringDamper>
+   </gazebo>
+   <gazebo reference="leg_${side}_2_joint">
+      <implicitSpringDamper>1</implicitSpringDamper>
+   </gazebo>
+   <gazebo reference="leg_${side}_3_joint">
+      <implicitSpringDamper>1</implicitSpringDamper>
+   </gazebo>
+    <!-- <gazebo reference="leg_${side}_4_joint">
+      <implicitSpringDamper>1</implicitSpringDamper>
+   </gazebo>
+   <gazebo reference="leg_${side}_5_joint">
+      <implicitSpringDamper>1</implicitSpringDamper>
+   </gazebo> -->
+   <gazebo reference="leg_${side}_length_link">
+      <implicitSpringDamper>1</implicitSpringDamper>
+   </gazebo>
    <gazebo reference="leg_${side}_1_link">
-     <mu1>0.9</mu1>
-     <mu2>0.9</mu2>
+     <material>Gazebo/FlatWhite</material>
    </gazebo>
    <gazebo reference="leg_${side}_2_link">
-     <mu1>0.9</mu1>
-     <mu2>0.9</mu2>
+     <material>Gazebo/FlatWhite</material>
    </gazebo>
    <gazebo reference="leg_${side}_3_link">
-     <mu1>0.9</mu1>
-     <mu2>0.9</mu2>
-   </gazebo>
+     <material>Gazebo/FlatWhite</material>
+   </gazebo>
+   <!-- <gazebo reference="leg_${side}_4_link">
+     <material>Gazebo/FlatBlack</material>
+   </gazebo>
+   <gazebo reference="leg_${side}_5_link">
+     <material>Gazebo/FlatBlack</material>
+   </gazebo> -->
    <gazebo reference="leg_${side}_length_link">
-     <mu1>0.9</mu1>
-     <mu2>0.9</mu2>
-   </gazebo>
-   <gazebo reference="leg_${side}_4_link">
-     <mu1>0.9</mu1>
-     <mu2>0.9</mu2>
-   </gazebo>
-   <gazebo reference="leg_${side}_5_link">
-     <mu1>0.9</mu1>
-     <mu2>0.9</mu2>
-   </gazebo>
-   <gazebo reference="leg_${side}_1_joint">
-      <implicitSpringDamper>1</implicitSpringDamper>
-   </gazebo>
-   <gazebo reference="leg_${side}_2_joint">
-      <implicitSpringDamper>1</implicitSpringDamper>
-   </gazebo>
-   <gazebo reference="leg_${side}_3_joint">
-      <implicitSpringDamper>1</implicitSpringDamper>
-   </gazebo>
-   <gazebo reference="leg_${side}_4_joint">
-      <implicitSpringDamper>1</implicitSpringDamper>
-   </gazebo>
-   <gazebo reference="leg_${side}_5_joint">
-      <implicitSpringDamper>1</implicitSpringDamper>
-   </gazebo>
-   <gazebo reference="leg_${side}_length_link">
-      <implicitSpringDamper>1</implicitSpringDamper>
-   </gazebo>
-  <gazebo reference="leg_${side}_1_link">
-    <material>Gazebo/FlatWhite</material>
-  </gazebo>
-  <gazebo reference="leg_${side}_2_link">
-    <material>Gazebo/FlatWhite</material>
-  </gazebo>
-  <gazebo reference="leg_${side}_3_link">
-    <material>Gazebo/FlatWhite</material>
-  </gazebo>
-  <gazebo reference="leg_${side}_4_link">
-    <material>Gazebo/FlatBlack</material>
-  </gazebo>
-  <gazebo reference="leg_${side}_5_link">
-    <material>Gazebo/FlatBlack</material>
-  </gazebo>
-  <gazebo reference="leg_${side}_length_link">
-    <material>Gazebo/FlatBlack</material>
-  </gazebo>
+     <material>Gazebo/FlatBlack</material>
+   </gazebo>
+   <xacro:mimic_joint_plugin_gazebo name_prefix="" parent_joint="leg_${side}_length_joint" mimic_joint="leg_${side}_knee_joint" has_pid="false" multiplier="3.38877" offset="-0.19229" max_effort="100.0"/>
+   <xacro:mimic_joint_plugin_gazebo name_prefix="" parent_joint="leg_${side}_length_joint" mimic_joint="leg_${side}_femur_joint" has_pid="false" multiplier="1.69435" offset="-0.096145" max_effort="100.0"/>
   </xacro:macro>
 </robot>

Commit message: Add missing tag for F/T sensor

File: kangaroo_description/urdf/ankle/ankle.urdf.xacro (robot description, xacro)
@@ -76,10 +76,17 @@
       <xacro:kangaroo_ankle_simple_simulation_transmission side="${side}" roll_joint="${roll_joint}" pitch_joint="${pitch_joint}"/>
     </xacro:if>
-   <gazebo reference="leg_${side}_${pitch_joint}_link">
-     <mu1>0.9</mu1>
-     <mu2>0.9</mu2>
-     <implicitSpringDamper>1</implicitSpringDamper>
-     <material>Gazebo/FlatWhite</material>
-   </gazebo>
+    <gazebo reference="leg_${side}_${pitch_joint}_joint">
+      <implicitSpringDamper>1</implicitSpringDamper>
+    </gazebo>
+    <gazebo reference="leg_${side}_${roll_joint}_joint">
+      <implicitSpringDamper>1</implicitSpringDamper>
+      <provideFeedback>1</provideFeedback>
+     </gazebo>
+    <gazebo reference="leg_${side}_${pitch_joint}_link">
+      <mu1>0.9</mu1>
+      <mu2>0.9</mu2>
+      <implicitSpringDamper>1</implicitSpringDamper>
+      <material>Gazebo/FlatWhite</material>
+    </gazebo>
    <!--
    <gazebo reference="leg_${side}_${roll_joint}_link">

Commit message: Fix transformation of sole link

File: kangaroo_description/urdf/ankle/ankle.urdf.xacro (robot description, xacro)
@@ -67,5 +67,5 @@
       <parent link="leg_${side}_${roll_joint}_link" />
       <child link="${side}_sole_link" />
-      <origin xyz="0.0 0.0 -0.03" rpy="0 0 0" />
+      <origin xyz="0.028 0.0 -0.029" rpy="0 0 0" />
       <axis xyz="1 0 0" />
     </joint>

Commit message: small fix in ankles + added foot frames in the corners

File: kangaroo_description/urdf/ankle/ankle.urdf.xacro (robot description, xacro)
@@ -1,4 +1,5 @@
 <?xml version="1.0"?>
 <robot xmlns:xacro="http://ros.org/wiki/xacro" name="kangaroo">
+  <xacro:include filename="$(find kangaroo_description)/urdf/ankle/foot_frames.urdf.xacro" />
   <xacro:include filename="$(find kangaroo_description)/urdf/ankle/ankle.transmission.xacro" />
   <xacro:property name="deg_to_rad"       value="0.01745329251994329577" />
@@ -68,6 +69,6 @@
       <child link="${side}_sole_link" />
       <origin xyz="0.028 0.0 -0.029" rpy="0 0 0" />
-      <axis xyz="1 0 0" />
     </joint>
+    <xacro:kangaroo_foot_frames side="${side}" parent="${side}_sole_link" offset_x="0.01"/>
     <xacro:unless value="${simulation}">
       <xacro:kangaroo_ankle_transmission side="${side}" roll_joint="${roll_joint}" pitch_joint="${pitch_joint}" read_actuator="${read_actuator}" />
