Commit message: Tune torque control params

File: kangaroo_description/urdf/ankle/ankle.urdf.xacro (robot description, xacro)
@@ -124,4 +124,31 @@
     </gazebo>
     -->
+    <!--
+    <link name="${side}_pesa_link">
+      <inertial>
+        <origin xyz="0 0 0" rpy="0 0 0" />
+        <mass value="5.0" />
+        <inertia ixx="0.015291667" ixy="0.0" ixz="0.0"
+          iyy="0.015291667" iyz="0.0" izz="0.0302" />
+      </inertial>
+      <visual>
+        <origin xyz="0 0 0" rpy="0 0 0" />
+        <geometry>
+          <cylinder length="0.02" radius="0.11"/>
+        </geometry>
+      </visual>
+      <collision>
+        <origin xyz="0 0 0" rpy="0 0 0" />
+        <geometry>
+          <cylinder length="0.02" radius="0.11"/>
+        </geometry>
+      </collision>
+    </link>
+    <joint name="${side}_pesa_joint" type="fixed">
+      <parent link="${side}_sole_link" />
+      <child link="${side}_pesa_link" />
+      <origin xyz="0.0 0.0 -0.01" rpy="0 0 0" />
+    </joint>
+  -->
   </xacro:macro>
 </robot>

File: kangaroo_description/urdf/leg/leg.urdf.xacro (robot description, xacro)
@@ -65,5 +65,5 @@
       <axis xyz="0 0 1" />
       <xacro:if value="${reflect == 1}">
-        <limit lower="${leg_1_min_pos}" upper="${leg_1_max_pos}" effort="500" velocity="3.87" />
+        <limit lower="${leg_1_min_pos}" upper="${leg_1_max_pos}" effort="150" velocity="3.87" />
       </xacro:if>
       <xacro:if value="${reflect == -1}">
@@ -93,5 +93,5 @@
       <child link="leg_${side}_2_link" />
       <axis xyz="0 1 0" />
-      <limit lower="${leg_2_min_pos}" upper="${leg_2_max_pos}" effort="100" velocity="3.87" />
+      <limit lower="${leg_2_min_pos}" upper="${leg_2_max_pos}" effort="150" velocity="3.87" />
     </joint>
     <link name="leg_${side}_3_link">
@@ -123,5 +123,5 @@
       <child link="leg_${side}_3_link" />
       <axis xyz="1 0 0" />
-      <limit lower="${leg_3_min_pos}" upper="${leg_3_max_pos}" effort="100" velocity="3.87" />
+      <limit lower="${leg_3_min_pos}" upper="${leg_3_max_pos}" effort="150" velocity="3.87" />
     </joint>
     <link name="leg_${side}_femur_link">

Commit message: Added frame aligned to ankle joint_5 axis

File: kangaroo_description/urdf/ankle/ankle.urdf.xacro (robot description, xacro)
@@ -69,4 +69,10 @@
       <child link="${side}_sole_link" />
       <origin xyz="0.028 0.0 -0.029" rpy="0 0 0" />
+    </joint>
+    <link name="leg_${side}_${roll_joint}_aligned_link"/>
+    <joint name="leg_${side}_${roll_joint}_aligned_joint" type="fixed">
+      <parent link="leg_${side}_${roll_joint}_link" />
+      <child link="leg_${side}_${roll_joint}_aligned_link" />
+      <origin xyz="0.0 0.0 0.0" rpy="0 ${20.0 * deg_to_rad} 0" />
     </joint>
     <xacro:kangaroo_foot_frames side="${side}" parent="${side}_sole_link" offset_x="0.01"/>

Commit message: Increase foot inertia for MPC experiments

File: kangaroo_description/urdf/ankle/ankle.urdf.xacro (robot description, xacro)
@@ -36,8 +36,8 @@
     <link name="leg_${side}_${roll_joint}_link">
       <inertial>
-        <origin xyz="0.0177425915954867 -3.67950153736807E-05 -0.0172694732454237" rpy="0 0 0" />
-        <mass value="0.394418327358563" />
-        <inertia ixx="0.000228382894016579" ixy="-2.56621760255351E-07" ixz="4.1179623691202E-05"
-          iyy="0.00108653696539759" iyz="7.85648127231571E-09" izz="0.0012643765698811" />
+        <origin xyz="0.022056 -3.9166E-05 -0.0099049" rpy="0 0 0" />
+        <mass value="0.41343" />
+        <inertia ixx="0.00435" ixy="2.7E-07" ixz="0.000241"
+          iyy="0.0179" iyz="3.0E-07" izz="0.0185" />
       </inertial>
       <visual>

Commit message: Update homing and launch force_torque_sensor_controller when ft_sensors is true

File: kangaroo_description/urdf/ankle/ankle.urdf.xacro (robot description, xacro)
@@ -91,5 +91,10 @@
       <parent link="leg_${side}_${roll_joint}_link" />
       <child link="${side}_sole_link" />
-      <origin xyz="0.028 0.0 -0.029" rpy="0 0 0" />
+      <xacro:unless value="${ft_sensors}">
+        <origin xyz="0.028 0.0 -0.029" rpy="0 0 0" />
+      </xacro:unless>
+      <xacro:if value="${ft_sensors}">
+        <origin xyz="0.028 0.0 -0.074" rpy="0 0 0" />
+      </xacro:if>
     </joint>
     <link name="leg_${side}_${roll_joint}_aligned_link"/>

Commit message: Add sensor and sole link transformations

File: kangaroo_description/urdf/ankle/ankle.urdf.xacro (robot description, xacro)
@@ -87,15 +87,4 @@
       <limit lower="${roll_joint_min_pos}" upper="${roll_joint_max_pos}" effort="100" velocity="3.87" />
     </joint>
-    <link name="${side}_sole_link"/>
-    <joint name="${side}_sole_fix_joint" type="fixed">
-      <parent link="leg_${side}_${roll_joint}_link" />
-      <child link="${side}_sole_link" />
-      <xacro:unless value="${ft_sensors}">
-        <origin xyz="0.028 0.0 -0.029" rpy="0 0 0" />
-      </xacro:unless>
-      <xacro:if value="${ft_sensors}">
-        <origin xyz="0.028 0.0 -0.074" rpy="0 0 0" />
-      </xacro:if>
-    </joint>
     <link name="leg_${side}_${roll_joint}_aligned_link"/>
     <joint name="leg_${side}_${roll_joint}_aligned_joint" type="fixed">
@@ -103,4 +92,25 @@
       <child link="leg_${side}_${roll_joint}_aligned_link" />
       <origin xyz="0.0 0.0 0.0" rpy="0 ${20.0 * deg_to_rad} 0" />
+    </joint>
+    <xacro:if value="${ft_sensors}">
+      <link name="${side}_ft_sensor_link"/>
+      <joint name="${side}_ft_sensor_fix_joint" type="fixed">
+        <parent link="leg_${side}_${roll_joint}_aligned_link" />
+        <child link="${side}_ft_sensor_link" />
+        <origin xyz="0.0161604517721356 0 -0.0444004763321373" rpy="1.57079632679488 -0.349065850398857 0" />
+      </joint>
+    </xacro:if>
+    <link name="${side}_sole_link"/>
+    <joint name="${side}_sole_fix_joint" type="fixed">
+      <xacro:unless value="${ft_sensors}">
+        <parent link="leg_${side}_${roll_joint}_link" />
+        <child link="${side}_sole_link" />
+        <origin xyz="0.028 0.0 -0.029" rpy="0 0 0" />
+      </xacro:unless>
+      <xacro:if value="${ft_sensors}">
+        <parent link="${side}_ft_sensor_link" />
+        <child link="${side}_sole_link" />
+        <origin xyz="0.0345 -0.0272 0" rpy="0 0 0" />
+      </xacro:if>
     </joint>
     <xacro:kangaroo_foot_frames side="${side}" parent="${side}_sole_link" offset_x="0.01"/>

Commit message: Fix ft sensor transformations

File: kangaroo_description/urdf/ankle/ankle.urdf.xacro (robot description, xacro)
@@ -98,5 +98,5 @@
         <parent link="leg_${side}_${roll_joint}_aligned_link" />
         <child link="${side}_ft_sensor_link" />
-        <origin xyz="0.0161604517721356 0 -0.0444004763321373" rpy="1.57079632679488 -0.349065850398857 0" />
+        <origin xyz="0.0161604517721356 0 -0.0444004763321373" rpy="0 -0.34906 0" />
       </joint>
     </xacro:if>
@@ -111,5 +111,5 @@
         <parent link="${side}_ft_sensor_link" />
         <child link="${side}_sole_link" />
-        <origin xyz="0.0345 -0.0272 0" rpy="0 0 0" />
+        <origin xyz="0.03483 0 -0.02725" rpy="0 0 0" />
       </xacro:if>
     </joint>

Commit message: Remove fixed from sole & ft_sensor joints

File: kangaroo_description/urdf/ankle/ankle.urdf.xacro (robot description, xacro)
@@ -95,5 +95,5 @@
     <xacro:if value="${ft_sensors}">
       <link name="${side}_ft_sensor_link"/>
-      <joint name="${side}_ft_sensor_fix_joint" type="fixed">
+      <joint name="${side}_ft_sensor_joint" type="fixed">
         <parent link="leg_${side}_${roll_joint}_aligned_link" />
         <child link="${side}_ft_sensor_link" />
@@ -102,5 +102,5 @@
     </xacro:if>
     <link name="${side}_sole_link"/>
-    <joint name="${side}_sole_fix_joint" type="fixed">
+    <joint name="${side}_sole_joint" type="fixed">
       <xacro:unless value="${ft_sensors}">
         <parent link="leg_${side}_${roll_joint}_link" />

Commit message: fix the ft link frame as per the datasheet

File: kangaroo_description/urdf/ankle/ankle.urdf.xacro (robot description, xacro)
@@ -98,5 +98,5 @@
         <parent link="leg_${side}_${roll_joint}_aligned_link" />
         <child link="${side}_ft_sensor_link" />
-        <origin xyz="0.0161604517721356 0 -0.0444004763321373" rpy="0 -0.34906 0" />
+        <origin xyz="0.00855050358313864 0 -0.023492315519661" rpy="0 -0.349065850398857 0" />
       </joint>
     </xacro:if>
@@ -111,5 +111,5 @@
         <parent link="${side}_ft_sensor_link" />
         <child link="${side}_sole_link" />
-        <origin xyz="0.03483 0 -0.02725" rpy="0 0 0" />
+        <origin xyz="0.034889 0 -0.0495" rpy="0 0 0" />
       </xacro:if>
     </joint>

Commit message: update the ankle links mass, inertia and meshes

File: kangaroo_description/urdf/ankle/ankle.urdf.xacro (robot description, xacro)
@@ -12,8 +12,8 @@
     <link name="leg_${side}_${pitch_joint}_link">
       <inertial>
-        <origin xyz="-0.00714160332877733 4.8311277200952E-09 0.00259941265068991" rpy="0 0 0" />
-        <mass value="0.0905836559788966" />
-        <inertia ixx="7.07461991271062E-06" ixy="-1.86951004827933E-12" ixz="8.30282143898823E-06"
-          iyy="2.92762498059213E-05" iyz="1.82895645239997E-11" izz="2.68643074366886E-05" />
+        <origin xyz="-0.00759994843981759 -6.94997526196062E-09 5.88281323654627E-08" rpy="0 0 0" />
+        <mass value="0.0905838346535586" />
+        <inertia ixx="4.05264139412808E-06" ixy="-5.2860301956695E-12" ixz="4.99859544268276E-11"
+          iyy="2.92762581820543E-05" iyz="6.24254988575372E-12" izz="2.98863057177445E-05" />
       </inertial>
       <visual>
@@ -26,4 +26,10 @@
         </material>
       </visual>
+      <collision>
+        <origin xyz="0 0 0" rpy="0 0 0" />
+        <geometry>
+          <mesh filename="package://kangaroo_description/meshes/leg_6_link.stl" />
+        </geometry>
+      </collision>
     </link>
     <joint name="leg_${side}_${pitch_joint}_joint" type="revolute">
@@ -37,7 +43,8 @@
       <xacro:unless value="${ft_sensors}">
         <inertial>
-          <origin xyz="0.022056 -3.9166E-05 -0.0099049" rpy="0 0 0" />
-          <mass value="0.41343" />
-          <inertia ixx="0.00435" ixy="2.7E-07" ixz="0.000241" iyy="0.0179" iyz="3.0E-07" izz="0.0185" />
+          <origin xyz="0.0056012722847415 -5.98528992629133E-06 -0.0297244079568318" rpy="0 0 0" />
+          <mass value="0.61562973648731" />
+          <inertia ixx="0.000511104633992357" ixy="2.29520535343244E-08" ixz="-0.000504403659563376"
+            iyy="0.00170802543470207" iyz="-1.88812897159487E-09" izz="0.00181438717200554" />
         </inertial>
         <visual>
@@ -60,5 +67,5 @@
         <inertial>
           <origin xyz="0.022204 -8.11751E-06 -0.042186" rpy="0 0 0" />
-          <mass value="0.624725" />
+          <mass value="0.826924" />
           <inertia ixx="0.0004094" ixy="2.2E-08" ixz="-0.000244" iyy="0.0009742" iyz="-1.25E-09" izz="0.0011036" />
         </inertial>
@@ -76,4 +83,10 @@
           <geometry>
             <mesh filename="package://kangaroo_description/meshes/leg_7_link_ft.stl" />
+          </geometry>
+        </collision>
+        <collision>
+          <origin xyz="0.035 0 -0.06" rpy="0 0 0" />
+          <geometry>
+            <box size="0.21 0.09 0.025"/>
           </geometry>
         </collision>

Commit message: update the ankle inertia and collision info when considering the ft_sensor

File: kangaroo_description/urdf/ankle/ankle.urdf.xacro (robot description, xacro)
@@ -66,7 +66,8 @@
       <xacro:if value="${ft_sensors}">
         <inertial>
-          <origin xyz="0.022204 -8.11751E-06 -0.042186" rpy="0 0 0" />
+          <origin xyz="0.0056012722847415 -8.11751E-06 -0.062005508" rpy="0 0 0" />
           <mass value="0.826924" />
-          <inertia ixx="0.0004094" ixy="2.2E-08" ixz="-0.000244" iyy="0.0009742" iyz="-1.25E-09" izz="0.0011036" />
+          <inertia ixx="0.000511104633992357" ixy="2.29520535343244E-08" ixz="-0.000504403659563376"
+            iyy="0.00170802543470207" iyz="-1.88812897159487E-09" izz="0.00181438717200554" />
         </inertial>
         <visual>
@@ -86,5 +87,5 @@
         </collision>
         <collision>
-          <origin xyz="0.035 0 -0.06" rpy="0 0 0" />
+          <origin xyz="0.035 0 -0.065" rpy="0 0 0" />
           <geometry>
             <box size="0.21 0.09 0.025"/>

Commit message: Fix torso mesh and add material for better coloring in rviz

File: kangaroo_description/urdf/ankle/ankle.urdf.xacro (robot description, xacro)
@@ -22,7 +22,5 @@
           <mesh filename="package://kangaroo_description/meshes/leg_6_link.stl" />
         </geometry>
-        <material name="">
-          <color rgba="0.752941176470588 0.752941176470588 0.752941176470588 1" />
-        </material>
+        <material name="DarkGrey"/>
       </visual>
       <collision>
@@ -53,7 +51,5 @@
             <mesh filename="package://kangaroo_description/meshes/leg_7_link.stl" />
           </geometry>
-          <material name="">
-            <color rgba="0.752941176470588 0.752941176470588 0.752941176470588 1" />
-          </material>
+          <material name="DarkGrey"/>
         </visual>
         <collision>
@@ -84,7 +80,5 @@
             <mesh filename="package://kangaroo_description/meshes/leg_7_link_ft.stl" />
           </geometry>
-          <material name="">
-            <color rgba="0.752941176470588 0.752941176470588 0.752941176470588 1" />
-          </material>
+          <material name="DarkGrey"/>
         </visual>
         <collision>

File: kangaroo_description/urdf/arm/arm.urdf.xacro (robot description, xacro)
@@ -39,8 +39,5 @@
           filename="package://kangaroo_description/meshes/arm_base_link.stl" />
       </geometry>
-      <material
-        name="">
-        <color
-          rgba="0.75294 0.75294 0.75294 1" />
+      <material name="DarkGrey"/>
       </material>
     </visual>
@@ -83,9 +80,5 @@
           filename="package://kangaroo_description/meshes/arm_1_link.stl" />
       </geometry>
-      <material
-        name="">
-        <color
-          rgba="0.75294 0.75294 0.75294 1" />
-      </material>
+      <material name="DarkGrey"/>
     </visual>
     <collision>
@@ -139,9 +132,5 @@
           filename="package://kangaroo_description/meshes/arm_2_link.stl" />
       </geometry>
-      <material
-        name="">
-        <color
-          rgba="0.75294 0.75294 0.75294 1" />
-      </material>
+      <material name="DarkGrey"/>
     </visual>
     <collision>
@@ -196,9 +185,5 @@
           filename="package://kangaroo_description/meshes/arm_3_link.stl" />
       </geometry>
-      <material
-        name="">
-        <color
-          rgba="0.75294 0.75294 0.75294 1" />
-      </material>
+      <material name="DarkGrey"/>
     </visual>
     <collision>
@@ -254,9 +239,5 @@
           filename="package://kangaroo_description/meshes/arm_${side}_4_link.stl" scale="1 1 1"/>
       </geometry>
-      <material
-        name="">
-        <color
-          rgba="0.75294 0.75294 0.75294 1" />
-      </material>
+      <material name="DarkGrey"/>
     </visual>
     <collision>

File: kangaroo_description/urdf/arm/arm_cover.urdf.xacro (robot description, xacro)
@@ -26,9 +26,5 @@
           filename="package://kangaroo_description/meshes/arm_cover_link.stl" />
       </geometry>
-      <material
-        name="">
-        <color
-          rgba="0.75294 0.75294 0.75294 1" />
-      </material>
+      <material name="DarkGrey"/>
     </visual>
     <collision>

File: kangaroo_description/urdf/base/base.urdf.xacro (robot description, xacro)
@@ -170,8 +170,5 @@
       </geometry>
       <material
-        name="">
-        <color
-           rgba="0.25098 0.25098 0.25098 1" />
-      </material>
+        name="DarkGrey"/>
     </visual>
     <collision>

File: kangaroo_description/urdf/crane/crane.urdf.xacro (robot description, xacro)
@@ -44,5 +44,5 @@
   </xacro:macro>
     <material name="CraneMaterial">
-        <color rgba="0.2 0.2 0.2 0.5"/>
+        <color rgba="0.7 0.7 0.7 0.5"/>
     </material>
 </robot>

File: kangaroo_description/urdf/leg/leg.urdf.xacro (robot description, xacro)
@@ -49,7 +49,5 @@
           <mesh filename="package://kangaroo_description/meshes/leg_1_link.stl" scale="1 ${reflect} 1"/>
         </geometry>
-        <material name="">
-          <color rgba="0.752941176470588 0.752941176470588 0.752941176470588 1" />
-        </material>
+        <material name="DarkGrey"/>
       </visual>
       <collision>
@@ -86,7 +84,5 @@
           <mesh filename="package://kangaroo_description/meshes/leg_2_link.stl" scale="1 ${reflect} 1"/>
         </geometry>
-        <material name="">
-          <color rgba="0.894117647058823 0.913725490196078 0.929411764705882 1"/>
-        </material>
+        <material name="DarkGrey"/>
       </visual>
       <collision>
@@ -116,7 +112,5 @@
           <mesh filename="package://kangaroo_description/meshes/leg_3_link.stl" scale="1 ${reflect} 1"/>
         </geometry>
-        <material name="">
-          <color rgba="0.752941176470588 0.752941176470588 0.752941176470588 1" />
-        </material>
+        <material name="DarkGrey"/>
       </visual>
       <collision>
@@ -156,7 +150,5 @@
           <mesh filename="package://kangaroo_description/meshes/leg_femur_link.stl" />
         </geometry>
-        <material name="">
-          <color rgba="0.752941176470588 0.752941176470588 0.752941176470588 1" />
-        </material>
+        <material name="DarkGrey"/>
       </visual>
       <collision>
@@ -189,7 +181,5 @@
           <mesh filename="package://kangaroo_description/meshes/leg_tibia_link.stl" />
         </geometry>
-        <material name="">
-          <color rgba="0.752941176470588 0.752941176470588 0.752941176470588 1" />
-        </material>
+        <material name="DarkGrey"/>
       </visual>
       <collision>

File: kangaroo_description/urdf/materials.urdf.xacro (robot description, xacro)
@@ -21,5 +21,5 @@
   </material>
  <material name="DarkGrey">
-   <color rgba="0.2 0.2 0.2 1.0"/>
+   <color rgba="0.3 0.3 0.3 1.0"/>
  </material>
   <material name="Red">

File: kangaroo_description/urdf/pelvis/pelvis.urdf.xacro (robot description, xacro)
@@ -21,7 +21,5 @@
           <mesh filename="package://kangaroo_description/meshes/${name}_base_link.stl" />
         </geometry>
-        <material name="">
-          <color rgba="0.25098 0.25098 0.25098 1" />
-        </material>
+        <material name="DarkGrey"/>
       </visual>
       <collision>
@@ -54,7 +52,5 @@
           <mesh filename="package://kangaroo_description/meshes/${name}_1_link.stl" />
         </geometry>
-        <material name="">
-          <color rgba="0.25098 0.25098 0.25098 1" />
-        </material>
+        <material name="DarkGrey"/>
       </visual>
       <collision>
@@ -93,7 +89,5 @@
           <mesh filename="package://kangaroo_description/meshes/${name}_2_link.stl" />
         </geometry>
-        <material name="">
-          <color rgba="0.25098 0.25098 0.25098 1" />
-        </material>
+        <material name="DarkGrey"/>
       </visual>
       <collision>

File: kangaroo_description/urdf/torso/torso.urdf.xacro (robot description, xacro)
@@ -37,7 +37,5 @@
         </xacro:unless>
       </geometry>
-      <material name="">
-        <color rgba="0.75294 0.75294 0.75294 1" />
-      </material>
+      <material name="DarkGrey"/>
     </visual>
     <collision>

Commit message: removed unnecesary meshes

File: kangaroo_description/urdf/ankle/ankle.urdf.xacro (robot description, xacro)
@@ -66,11 +66,4 @@
             </properties>
         </xacro:link_collision>
-	      <collision>
-          <origin xyz="0.01 0.0 -0.028" rpy="0 ${-20.0 * deg_to_rad} 0" />
-          <geometry>
-            <!-- The length of the sole is around 24cm, but with the attached rubber sole it would be 24.9cm -->
-            <box size="0.249 0.10 0.025"/>
-          </geometry>
-        </collision>
       </xacro:unless>
       <!-- The FT sensors is still not available -->

File: kangaroo_description/urdf/leg/leg.urdf.xacro (robot description, xacro)
@@ -206,11 +206,4 @@
         </xacro:unless>
       </inertial>
-      <visual>
-        <origin rpy="0 0 0" xyz="0 0 ${(leg_min_length - leg_max_length)/2}"/>
-        <geometry>
-          <cylinder length="${(leg_max_length - leg_min_length)}" radius="0.00005"/>
-        </geometry>
-        <material name="pal/DarkGrey" />
-      </visual>
     </link>
     <joint name="leg_${side}_length_joint" type="prismatic">
