Commit message: Update the mass and the inertial elements of leg links

File: kangaroo_description/urdf/ankle/ankle.urdf.xacro (robot description, xacro)
@@ -11,8 +11,8 @@
     <link name="leg_${side}_${pitch_joint}_link">
       <inertial>
-        <origin xyz="-0.00759994843981759 -6.94997526196062E-09 5.88281323654627E-08" rpy="0 0 0" />
-        <mass value="0.0905838346535586" />
-        <inertia ixx="4.05264139412808E-06" ixy="-5.2860301956695E-12" ixz="4.99859544268276E-11"
-          iyy="2.92762581820543E-05" iyz="6.24254988575372E-12" izz="2.98863057177445E-05" />
+        <origin xyz="-0.007727 0 0" rpy="0 0 0" />
+        <mass value="0.086323" />
+        <inertia ixx="6e-06" ixy="0" ixz="0"
+          iyy="3.5e-05" iyz="0" izz="3.7e-05" />
       </inertial>
       <visual>

File: kangaroo_description/urdf/leg/leg.urdf.xacro (robot description, xacro)
@@ -24,8 +24,8 @@
     <link name="leg_${side}_1_link">
       <inertial>
-        <origin xyz="0.0063167 ${reflect * 0.0045949} -0.0083828" rpy="0 0 0" />
-        <mass value="2.7478" />
-        <inertia ixx="0.0019336" ixy="${reflect * 8.5058E-06}" ixz="${reflect * 4.8385E-05}"
-          iyy="0.0018225" iyz="${reflect * -7.282E-06}" izz="0.001426" />
+        <origin xyz="0.049076 ${reflect * 0.000248} -0.021744" rpy="0 0 0" />
+        <mass value="2.73393" />
+        <inertia ixx="0.007715" ixy="${reflect * -0.000015}" ixz="-0.000588"
+          iyy="0.005966" iyz="${reflect * -0.000019}" izz="0.005763"/>
       </inertial>
       <visual>
@@ -64,10 +64,8 @@
     <link name="leg_${side}_2_link">
       <inertial>
-        <origin
-          xyz="-0.0029278 -9.6207E-05 1.0866E-09"
-          rpy="0 0 0" />
-        <mass value="0.0905312454913012" />
-        <inertia ixx="6.10166860944865E-06" ixy="4.64490555644666E-08" ixz="4.07017223451518E-13"
-          iyy="3.88541683636482E-05" iyz="-1.04538188015163E-12" izz="3.6228659424845E-05" />
+        <origin xyz="-0.004242 -1.3e-05 9.1e-05" rpy="0 0 0" />
+        <mass value="0.105669" />
+        <inertia ixx="8e-06" ixy="0" ixz="0"
+          iyy="9.9e-05" iyz="0" izz="9.6e-05" />
       </inertial>
       <visual>
@@ -99,8 +97,8 @@
     <link name="leg_${side}_3_link">
       <inertial>
-        <origin xyz="-0.033949 ${reflect * 0.049989} -0.030543" rpy="0 0 0" />
-        <mass value="3.658" />
-        <inertia ixx="0.0025968" ixy="${reflect * 0.00018723}" ixz="${reflect * -0.00014976}"
-          iyy="0.0031521" iyz="${reflect * 3.7258E-05}" izz="0.0032376" />
+        <origin xyz="-0.048028 ${reflect * 0.057205} -0.037679" rpy="0 0 0" />
+        <mass value="3.646" />
+        <inertia ixx="0.013631" ixy="${reflect * 0.002527}" ixz="-0.000349"
+          iyy="0.013321" iyz="${reflect * 0.000445}" izz="0.020668"/>
       </inertial>
       <visual>
@@ -134,8 +132,8 @@
     <link name="leg_${side}_femur_link">
       <inertial>
-        <origin xyz="0.0527475093314697 0.000135688427874925 -0.146959283149568" rpy="0 0 0" />
-        <mass value="3.94567187082779" />
-        <inertia ixx="0.0111010751306264" ixy="2.24256967982894E-05" ixz="0.0025879993168672"
-          iyy="0.0121128398206334" iyz="-1.93362671261787E-05" izz="0.0025734913670898" />
+        <origin xyz="0.055462 0.000143 -0.149562" rpy="0 0 0" />
+        <mass value="4.94483" />
+        <inertia ixx="0.11136" ixy="-0.000012" ixz="0.02662"
+          iyy="0.120183" iyz="-0.000027" izz="0.015806"/>
       </inertial>
       <visual>
@@ -163,8 +161,8 @@
     <link name="leg_${side}_knee_link">
       <inertial>
-        <origin xyz="-0.0569664873635563 -5.41309796184553E-05 -0.148820781933269" rpy="0 0 0" />
-        <mass value="1.02238189690276" />
-        <inertia ixx="0.00193955870555937" ixy="-7.22330237538467E-08" ixz="-0.000472475893337071"
-          iyy="0.00215347079183119" iyz="1.36520012214457E-06" izz="0.000391378760186175" />
+        <origin xyz="-0.040771 -4.6e-05 -0.126665" rpy="0 0 0" />
+        <mass value="0.944388" />
+        <inertia ixx="0.012522" ixy="-0.000009" ixz="-0.005373"
+          iyy="0.015899" iyz="-0.000021" izz="0.004153"/>
       </inertial>
       <visual>
