Commit message: added changes of single URDF with leg length and dynamic model

File: kangaroo_description/urdf/ankle/ankle.transmission.xacro (robot description, xacro)
@@ -36,5 +36,33 @@
   </xacro:macro>
   <xacro:macro name="kangaroo_ankle_transmission" params="side roll_joint pitch_joint read_actuator">
-    <transmission name="leg_${side}_transmission">
+    <transmission name="leg_${side}_${pitch_joint}_transmission">
+      <type>transmission_interface/SimpleTransmission</type>
+      <actuator name="leg_${side}_${pitch_joint}_motor" >
+        <hardwareInterface>hardware_interface/PositionJointInterface</hardwareInterface>
+        <hardwareInterface>hardware_interface/EffortJointInterface</hardwareInterface>
+        <hardwareInterface>hardware_interface/JointStateInterface</hardwareInterface>
+        <mechanicalReduction>1.0</mechanicalReduction>
+      </actuator>
+      <joint name="leg_${side}_${pitch_joint}_joint">
+        <hardwareInterface>hardware_interface/PositionJointInterface</hardwareInterface>
+        <hardwareInterface>hardware_interface/EffortJointInterface</hardwareInterface>
+        <hardwareInterface>hardware_interface/JointStateInterface</hardwareInterface>
+      </joint>
+    </transmission>
+    <transmission name="leg_${side}_${roll_joint}_transmission">
+      <type>transmission_interface/SimpleTransmission</type>
+      <actuator name="leg_${side}_${roll_joint}_motor" >
+        <hardwareInterface>hardware_interface/PositionJointInterface</hardwareInterface>
+        <hardwareInterface>hardware_interface/EffortJointInterface</hardwareInterface>
+        <hardwareInterface>hardware_interface/JointStateInterface</hardwareInterface>
+        <mechanicalReduction>1.0</mechanicalReduction>
+      </actuator>
+      <joint name="leg_${side}_${roll_joint}_joint">
+        <hardwareInterface>hardware_interface/PositionJointInterface</hardwareInterface>
+        <hardwareInterface>hardware_interface/EffortJointInterface</hardwareInterface>
+        <hardwareInterface>hardware_interface/JointStateInterface</hardwareInterface>
+      </joint>
+    </transmission>
+<!--     <transmission name="leg_${side}_transmission">
       <type>pal_transmissions/AnkleCustomTransmission</type>
       <actuator name="leg_${side}_${roll_joint}_motor">
@@ -61,5 +89,5 @@
         <hardwareInterface>hardware_interface/EffortJointInterface</hardwareInterface>
       </joint>
-    </transmission>
+    </transmission> -->
   </xacro:macro>
 </robot>

File: kangaroo_description/urdf/leg/leg.transmission.xacro (robot description, xacro)
@@ -79,38 +79,35 @@
     </xacro:unless>
   </xacro:macro>
-  <xacro:macro name="kangaroo_leg_length_actuator_transmission" params="side number1 number2 leg_min_length leg_max_length femur intersection_crank_axis fbl11_long fbl11_short fbl21_fixed fbl21_long fbl21_short crank_slider_long crank_slider_short crank_slider_axis_angle shin_offset_angle connection_fbl_offset_angle shin_fbl11_offset_angle knee_angle_min knee_angle_max femur_angle_min femur_angle_max" >
-    <transmission name="leg_${side}_length_trans">
+  <xacro:macro name="kangaroo_leg_length_actuator_transmission" params="side number1 number2 params_ns:=/leg_params" >
+    <transmission name="leg_${side}_${number1}_trans">
       <type>pal_transmissions/LegCustomTransmission</type>
-      <actuator name="leg_${side}_length_motor">
-        <parameters>
-          <femur>${femur}</femur>
-          <fbl11_long>${fbl11_long}</fbl11_long>
-          <fbl11_short>${fbl11_short}</fbl11_short>
-          <intersection_crank_axis>${intersection_crank_axis}</intersection_crank_axis>
-          <fbl21_fixed>${fbl21_fixed}</fbl21_fixed>
-          <fbl21_long>${fbl21_long}</fbl21_long>
-          <fbl21_short>${fbl21_short}</fbl21_short>
-          <crank_slider_long>${crank_slider_long}</crank_slider_long>
-          <crank_slider_short>${crank_slider_short}</crank_slider_short>
-          <crank_slider_axis_angle>${crank_slider_axis_angle}</crank_slider_axis_angle>
-          <shin_offset_angle>${shin_offset_angle}</shin_offset_angle>
-          <connection_fbl_offset_angle>${connection_fbl_offset_angle} </connection_fbl_offset_angle>
-          <shin_fbl11_offset_angle>${shin_fbl11_offset_angle}</shin_fbl11_offset_angle>
-          <knee_angle_min>${knee_angle_min}</knee_angle_min>
-          <knee_angle_max>${knee_angle_max}</knee_angle_max>
-        </parameters>
-        <hardwareInterface>hardware_interface/PositionJointInterface</hardwareInterface>
-        <hardwareInterface>hardware_interface/EffortJointInterface</hardwareInterface>
-        <hardwareInterface>hardware_interface/JointStateInterface</hardwareInterface>
+      <actuator name="leg_${side}_leg_length_motor" >
+      </actuator>
+      <joint name="leg_${side}_${number1}_joint">
+        <joint_type> femur </joint_type>
+        <param_ns> ${params_ns} </param_ns>
+        <offset> 0.0 </offset>
+        <hardwareInterface>hardware_interface/JointStateInterface</hardwareInterface>
+      </joint>
+    </transmission>
+    <transmission name="leg_${side}_${number2}_trans">
+      <type>pal_transmissions/LegCustomTransmission</type>
+      <actuator name="leg_${side}_leg_length_motor" >
+      </actuator>
+      <joint name="leg_${side}_${number2}_joint">
+        <joint_type> knee </joint_type>
+        <param_ns> ${params_ns} </param_ns>
+        <offset> 0.0 </offset>
+        <hardwareInterface>hardware_interface/JointStateInterface</hardwareInterface>
+      </joint>
+    </transmission>
+    <transmission name="leg_${side}_leg_length_trans">
+      <type>pal_transmissions/LegCustomTransmission</type>
+      <actuator name="leg_${side}_leg_length_motor" >
       </actuator>
       <joint name="leg_${side}_length_joint">
-        <role> leg_length </role>
+        <joint_type> leg_length </joint_type>
+        <param_ns> ${params_ns} </param_ns>
         <offset> 0.0 </offset>
-        <limits>
-          <position>
-            <min> ${leg_min_length} </min>
-            <max> ${leg_max_length} </max>
-          </position>
-        </limits>
         <hardwareInterface>hardware_interface/PositionJointInterface</hardwareInterface>
         <hardwareInterface>hardware_interface/EffortJointInterface</hardwareInterface>

File: kangaroo_description/urdf/leg/leg.urdf.xacro (robot description, xacro)
@@ -247,5 +247,5 @@
       <xacro:hip_transmission_yaw side="${side}" number="1" reduction="1.0" />
       <xacro:hip_transmission_roll_pitch side="${side}" roll_joint="3" pitch_joint="2" />
-      <xacro:kangaroo_leg_length_actuator_transmission side="${side}" number1="4" number2="5" leg_min_length="${leg_min_length}" leg_max_length="${leg_max_length}" femur="0.380" intersection_crank_axis="0.155693813961639" fbl11_long="0.404273" fbl11_short="0.090" fbl21_fixed="0.115" fbl21_long="0.090" fbl21_short="0.040" crank_slider_long="0.215" crank_slider_short="0.090" crank_slider_axis_angle="${-15.65*deg_to_rad}" shin_offset_angle="${0.0*deg_to_rad}" connection_fbl_offset_angle="${-45.0*deg_to_rad}" shin_fbl11_offset_angle="${-15.00*deg_to_rad}" knee_angle_min ="${leg_5_min_pos - 5.0 *deg_to_rad}" knee_angle_max="${leg_5_max_pos + 5.0 *deg_to_rad}" femur_angle_min="${leg_4_min_pos}" femur_angle_max="${leg_4_max_pos}" />
+      <xacro:kangaroo_leg_length_actuator_transmission side="${side}" number1="4" number2="5" params_ns="/leg_params" />
     </xacro:unless>
     <xacro:if value="${simulation}">

Commit message: Changes to make work hipxy and leg length transmissions

File: kangaroo_description/urdf/ankle/ankle.transmission.xacro (robot description, xacro)
@@ -22,7 +22,7 @@
     <transmission name="leg_${side}_ankle_transmission">
       <plugin>kangaroo_transmissions/AnkleXYCustomTransmission</plugin>
-      <actuator name="leg_${side}_${roll_joint}_motor" role="actuator_right">
+      <actuator name="leg_${side}_${roll_joint}_actuator" role="actuator_right">
       </actuator>
-      <actuator name="leg_${side}_${pitch_joint}_motor" role="actuator_left">
+      <actuator name="leg_${side}_${pitch_joint}_actuator" role="actuator_left">
       </actuator>
       <actuator name="${read_actuator}" role="actuator_length">

File: kangaroo_description/urdf/leg/leg.transmission.xacro (robot description, xacro)
@@ -26,25 +26,28 @@
     <transmission name="leg_${side}_length_transmission">
       <plugin>kangaroo_transmissions/LegCustomTransmission</plugin>
-      <actuator name="leg_${side}_length_motor" role="actuator_main"/>
+      <actuator name="leg_${side}_length_actuator" role="actuator_main"/>
       <joint name="leg_${side}_length_joint" role="joint_main">
         <offset>0.0</offset>
       </joint>
       <param name="joint_type">leg_length</param>
+      <param name="leg_side">${side}</param>
     </transmission>
     <transmission name="leg_${side}_knee_joint_trans">
       <plugin>kangaroo_transmissions/LegCustomTransmission</plugin>
-      <actuator name="leg_${side}_length_motor" role="actuator_main"/>
+      <actuator name="leg_${side}_length_actuator" role="actuator_main"/>
       <joint name="leg_${side}_knee_joint" role="joint_aux">
         <offset>0.0</offset>
       </joint>
       <param name="joint_type">knee</param>
+      <param name="leg_side">${side}</param>
     </transmission>
     <transmission name="leg_${side}_femur_joint_trans">
       <plugin>kangaroo_transmissions/LegCustomTransmission</plugin>
-      <actuator name="leg_${side}_length_motor" role="actuator_main"/>
+      <actuator name="leg_${side}_length_actuator" role="actuator_main"/>
       <joint name="leg_${side}_femur_joint" role="joint_aux">
         <offset>0.0</offset>
       </joint>
       <param name="joint_type">femur</param>
+      <param name="leg_side">${side}</param>
     </transmission>
   </xacro:macro>
@@ -68,12 +71,12 @@
     <transmission name="leg_${side}_hip_transmission">
       <plugin>kangaroo_transmissions/HipXYCustomTransmission</plugin>
-      <actuator name="leg_${side}_${roll_joint}_motor" role="actuator_right">
+      <actuator name="leg_${side}_${pitch_joint}_actuator" role="actuator_left">
       </actuator>
-      <actuator name="leg_${side}_${pitch_joint}_motor" role="actuator_left">
+      <actuator name="leg_${side}_${roll_joint}_actuator" role="actuator_right">
       </actuator>
-      <joint name="leg_${side}_${roll_joint}_joint" role="roll">
+      <joint name="leg_${side}_${roll_joint}_joint" role="pitch">
         <offset>0.0</offset>
       </joint>
-      <joint name="leg_${side}_${pitch_joint}_joint" role="pitch">
+      <joint name="leg_${side}_${pitch_joint}_joint" role="roll">
         <offset>0.0</offset>
       </joint>

File: kangaroo_description/urdf/leg/ros2_control.urdf.xacro (robot description, xacro)
@@ -18,10 +18,11 @@
   <xacro:include filename="$(find kangaroo_description)/ros2_control/transmissions.urdf.xacro" />
   <xacro:include filename="$(find kangaroo_description)/urdf/leg/leg.transmission.xacro" />
+  <xacro:include filename="$(find kangaroo_description)/urdf/ankle/ankle.transmission.xacro" />
   <!-- MACRO DEFINITION-->
   <xacro:macro name="leg_ros2_control" params="side">
         <!-- <xacro:joint_ros2control name="leg_${side}_1" initial_position="0.0" /> -->
-        <xacro:joint_ros2control name="leg_${side}_2" initial_position="0.05" />
-        <xacro:joint_ros2control name="leg_${side}_3" initial_position="0.0" />
-        <xacro:joint_ros2control name="leg_${side}_length" initial_position="0.6" />
+        <!-- <xacro:joint_ros2control name="leg_${side}_2" initial_position="0.05" /> -->
+        <!-- <xacro:joint_ros2control name="leg_${side}_3" initial_position="0.0" /> -->
+        <!--xacro:joint_ros2control name="leg_${side}_length" initial_position="0.6" /-->
         <xacro:joint_ros2control name="leg_${side}_4" initial_position="-0.07" />
         <xacro:joint_ros2control name="leg_${side}_5" initial_position="0.0" />
@@ -31,7 +32,10 @@
           <!--xacro:simple_transmission name="leg_${side}_1" reduction="1.0" offset_value="${leg_1_joint_offset}" /-->
           <xacro:hip_transmission_yaw side="${side}" offset="${leg_1_joint_offset}" initial_position="0.0" />
-          <xacro:simple_transmission name="leg_${side}_2" reduction="1.0" offset_value="${leg_2_joint_offset}" />
-          <xacro:simple_transmission name="leg_${side}_3" reduction="1.0" offset_value="${leg_3_joint_offset}" />
-          <xacro:simple_transmission name="leg_${side}_length" reduction="1.0" offset_value="${leg_length_joint_offset}" />
+          <!-- xacro:simple_transmission name="leg_${side}_2" reduction="1.0" offset_value="${leg_2_joint_offset}" / -->
+          <xacro:hip_transmission_roll_pitch side="${side}" roll_joint="3" pitch_joint="2" />
+          <!-- <xacro:simple_transmission name="leg_${side}_3" reduction="1.0" offset_value="${leg_3_joint_offset}" /> -->
+          <xacro:kangaroo_leg_length_actuator_transmission side="${side}" />
+          <!--xacro:simple_transmission name="leg_${side}_length" reduction="1.0" offset_value="${leg_length_joint_offset}" /-->
+          <!--xacro:kangaroo_ankle_transmission side="${side}" roll_joint="4" pitch_joint="5" read_actuator="leg_${side}_length_actuator" /-->
           <xacro:simple_transmission name="leg_${side}_4" reduction="1.0" offset_value="${leg_4_joint_offset}" />
           <xacro:simple_transmission name="leg_${side}_5" reduction="1.0" offset_value="${leg_5_joint_offset}" />

Commit message: enable nl trans for all the joints

File: kangaroo_description/urdf/ankle/ankle.transmission.xacro (robot description, xacro)
@@ -28,8 +28,8 @@
       <actuator name="${read_actuator}" role="actuator_length">
       </actuator>
-      <joint name="leg_${side}_${roll_joint}_joint" role="roll">
+      <joint name="leg_${side}_${roll_joint}_joint" role="pitch">
         <offset>0.0</offset>
       </joint>
-      <joint name="leg_${side}_${pitch_joint}_joint" role="pitch">
+      <joint name="leg_${side}_${pitch_joint}_joint" role="roll">
         <offset>0.0</offset>
       </joint>

File: kangaroo_description/urdf/leg/ros2_control.urdf.xacro (robot description, xacro)
@@ -24,20 +24,20 @@
         <!-- <xacro:joint_ros2control name="leg_${side}_2" initial_position="0.05" /> -->
         <!-- <xacro:joint_ros2control name="leg_${side}_3" initial_position="0.0" /> -->
-        <!--xacro:joint_ros2control name="leg_${side}_length" initial_position="0.6" /-->
-        <xacro:joint_ros2control name="leg_${side}_4" initial_position="-0.07" />
-        <xacro:joint_ros2control name="leg_${side}_5" initial_position="0.0" />
-        <!--xacro:passive_joint_ros2control name="leg_${side}_femur" initial_position="0.9" />
-        <xacro:passive_joint_ros2control name="leg_${side}_knee" initial_position="1.8" /-->
+        <!-- <xacro:joint_ros2control name="leg_${side}_length" initial_position="0.6" /> -->
+        <!-- <xacro:joint_ros2control name="leg_${side}_4" initial_position="-0.07" /> -->
+        <!-- <xacro:joint_ros2control name="leg_${side}_5" initial_position="0.0" /> -->
+        <!-- <xacro:passive_joint_ros2control name="leg_${side}_femur" initial_position="0.9" /> -->
+        <!-- <xacro:passive_joint_ros2control name="leg_${side}_knee" initial_position="1.8" /> -->
         <xacro:if value="${sim_type == 'no-simulation'}" >
-          <!--xacro:simple_transmission name="leg_${side}_1" reduction="1.0" offset_value="${leg_1_joint_offset}" /-->
+          <!-- <xacro:simple_transmission name="leg_${side}_1" reduction="1.0" offset_value="${leg_1_joint_offset}" /> -->
+          <!-- <xacro:simple_transmission name="leg_${side}_2" reduction="1.0" offset_value="${leg_2_joint_offset}" /> -->
+          <!-- <xacro:simple_transmission name="leg_${side}_3" reduction="1.0" offset_value="${leg_3_joint_offset}" /> -->
+          <!-- <xacro:simple_transmission name="leg_${side}_length" reduction="1.0" offset_value="${leg_length_joint_offset}" /> -->
+          <!-- <xacro:simple_transmission name="leg_${side}_4" reduction="1.0" offset_value="${leg_4_joint_offset}" /> -->
+          <!-- <xacro:simple_transmission name="leg_${side}_5" reduction="1.0" offset_value="${leg_5_joint_offset}" /> -->
           <xacro:hip_transmission_yaw side="${side}" offset="${leg_1_joint_offset}" initial_position="0.0" />
-          <!-- xacro:simple_transmission name="leg_${side}_2" reduction="1.0" offset_value="${leg_2_joint_offset}" / -->
           <xacro:hip_transmission_roll_pitch side="${side}" roll_joint="3" pitch_joint="2" />
-          <!-- <xacro:simple_transmission name="leg_${side}_3" reduction="1.0" offset_value="${leg_3_joint_offset}" /> -->
           <xacro:kangaroo_leg_length_actuator_transmission side="${side}" />
-          <!--xacro:simple_transmission name="leg_${side}_length" reduction="1.0" offset_value="${leg_length_joint_offset}" /-->
-          <!--xacro:kangaroo_ankle_transmission side="${side}" roll_joint="4" pitch_joint="5" read_actuator="leg_${side}_length_actuator" /-->
-          <xacro:simple_transmission name="leg_${side}_4" reduction="1.0" offset_value="${leg_4_joint_offset}" />
-          <xacro:simple_transmission name="leg_${side}_5" reduction="1.0" offset_value="${leg_5_joint_offset}" />
+          <xacro:kangaroo_ankle_transmission side="${side}" roll_joint="5" pitch_joint="4" read_actuator="leg_${side}_length_actuator" />
         </xacro:if>
   </xacro:macro>

Commit message: Remove the duplicate interfaces information defined in the transmissions

File: kangaroo_description/urdf/ankle/ankle.transmission.xacro (robot description, xacro)
@@ -6,20 +6,4 @@
 <robot name="kangaroo" xmlns:xacro="http://ros.org/wiki/xacro">
   <xacro:macro name="kangaroo_ankle_transmission" params="side roll_joint pitch_joint read_actuator">
-    <joint name="leg_${side}_${roll_joint}_joint">
-      <command_interface name="position"/>
-      <command_interface name="velocity"/>
-      <command_interface name="effort"/>
-      <state_interface name="position"/>
-      <state_interface name="velocity"/>
-      <state_interface name="effort"/>
-    </joint>
-    <joint name="leg_${side}_${pitch_joint}_joint">
-      <command_interface name="position"/>
-      <command_interface name="velocity"/>
-      <command_interface name="effort"/>
-      <state_interface name="position"/>
-      <state_interface name="velocity"/>
-      <state_interface name="effort"/>
-    </joint>
     <transmission name="leg_${side}_ankle_transmission">
       <plugin>kangaroo_transmissions/AnkleXYCustomTransmission</plugin>

File: kangaroo_description/urdf/leg/leg.transmission.xacro (robot description, xacro)
@@ -6,22 +6,4 @@
 <robot name="kangaroo" xmlns:xacro="http://ros.org/wiki/xacro">
   <xacro:macro name="kangaroo_leg_length_actuator_transmission" params="side">
-    <joint name="leg_${side}_length_joint">
-      <command_interface name="position"/>
-      <command_interface name="velocity"/>
-      <command_interface name="effort"/>
-      <state_interface name="position"/>
-      <state_interface name="velocity"/>
-      <state_interface name="effort"/>
-    </joint>
-    <joint name="leg_${side}_knee_joint">
-      <state_interface name="position"/>
-      <state_interface name="velocity"/>
-      <state_interface name="effort"/>
-    </joint>
-    <joint name="leg_${side}_femur_joint">
-      <state_interface name="position"/>
-      <state_interface name="velocity"/>
-      <state_interface name="effort"/>
-    </joint>
     <transmission name="leg_${side}_length_transmission">
       <plugin>kangaroo_transmissions/LegCustomTransmission</plugin>
@@ -53,20 +35,4 @@
   </xacro:macro>
   <xacro:macro name="hip_transmission_roll_pitch" params="side roll_joint pitch_joint">
-    <joint name="leg_${side}_${roll_joint}_joint">
-      <command_interface name="position"/>
-      <command_interface name="velocity"/>
-      <command_interface name="effort"/>
-      <state_interface name="position"/>
-      <state_interface name="velocity"/>
-      <state_interface name="effort"/>
-    </joint>
-    <joint name="leg_${side}_${pitch_joint}_joint">
-      <command_interface name="position"/>
-      <command_interface name="velocity"/>
-      <command_interface name="effort"/>
-      <state_interface name="position"/>
-      <state_interface name="velocity"/>
-      <state_interface name="effort"/>
-    </joint>
     <transmission name="leg_${side}_hip_transmission">
       <plugin>kangaroo_transmissions/HipXYCustomTransmission</plugin>
@@ -83,14 +49,4 @@
   </xacro:macro>
   <xacro:macro name="hip_transmission_yaw" params="side offset initial_position:=0.0">
-    <joint name="leg_${side}_1_joint">
-      <command_interface name="position"/>
-      <command_interface name="velocity"/>
-      <command_interface name="effort"/>
-      <state_interface name="position">
-          <param name="initial_value">${initial_position}</param>
-      </state_interface>
-      <state_interface name="velocity"/>
-      <state_interface name="effort"/>
-    </joint>
     <transmission name="leg_${side}_yaw_transmission">
       <plugin>kangaroo_transmissions/HipZCustomTransmission</plugin>
