Commit message: Fix detachable feet joints

File: kangaroo_description/urdf/ankle/detachable_ankle.urdf.xacro (robot description, xacro)
@@ -38,5 +38,5 @@
       <parent link="${parent}" />
       <child link="leg_${side}_${pitch_joint}_link" />
-      <axis xyz="0 1 0" />
+      <axis xyz="0 -1 0" />
       <limit lower="${pitch_joint_min_pos}" upper="${pitch_joint_max_pos}" effort="140" velocity="3.87" />
     </joint>
@@ -98,5 +98,5 @@
       </collision>
     </link>
-    <joint name="leg_${side}_ankle_attach" type="continuous">
+    <joint name="leg_${side}_ankle_attach_joint" type="continuous">
       <origin xyz="0.013168 0 0.036178" rpy="0 0.34907 0" />
       <parent link="leg_${side}_${roll_joint}_link" />

Commit message: Set ankle attach joint to fixed

File: kangaroo_description/urdf/ankle/detachable_ankle.urdf.xacro (robot description, xacro)
@@ -98,5 +98,5 @@
       </collision>
     </link>
-    <joint name="leg_${side}_ankle_attach_joint" type="continuous">
+    <joint name="leg_${side}_ankle_attach_joint" type="fixed">
       <origin xyz="0.013168 0 0.036178" rpy="0 0.34907 0" />
       <parent link="leg_${side}_${roll_joint}_link" />

Commit message: Replace stl with covers and axis fixed

File: kangaroo_description/urdf/ankle/detachable_ankle.urdf.xacro (robot description, xacro)
@@ -10,9 +10,9 @@
     <link name="leg_${side}_${pitch_joint}_link">
       <inertial>
-          <origin xyz="-0.0027697 1.3528E-07 -3.7736E-05" rpy="0 0 0" />
-          <mass value="0.094024" />
-          <inertia ixx="5.8253E-06" ixy="-6.0567E-12" ixz="1.016E-07"
-                    iyy="1.4458E-05" iyz="-1.9404E-13"
-                    izz="1.5653E-05" />
+          <origin xyz="-0.002212 0.0 -0.000833" rpy="0 0 0" />
+          <mass value="0.132674" />
+          <inertia ixx="0.000017" ixy="0.0" ixz="0.000008"
+                    iyy="0.000031" iyz="0.0"
+                    izz="0.000036" />
       </inertial>
       <visual>
@@ -35,17 +35,17 @@
     </link>
     <joint name="leg_${side}_${pitch_joint}_joint" type="revolute">
-      <origin xyz="0 0 0" rpy="0 ${-20.0 * deg_to_rad} 3.1416" />
+      <xacro:insert_block name="origin"/>
       <parent link="${parent}" />
       <child link="leg_${side}_${pitch_joint}_link" />
-      <axis xyz="0 -1 0" />
+      <axis xyz="0 1 0" />
       <limit lower="${pitch_joint_min_pos}" upper="${pitch_joint_max_pos}" effort="140" velocity="3.87" />
     </joint>
     <link name="leg_${side}_${roll_joint}_link">
       <inertial>
-        <origin xyz="-0.014212 -3.1369E-05 0.015061" rpy="0 0 0" />
+        <origin xyz="-0.014212 0.000031 -0.015062" rpy="0 0 0" />
         <mass value="0.16804" />
-        <inertia ixx="4.3556E-05" ixy="-4.1754E-09" ixz="-7.0376E-06"
-                 iyy="0.00011001" iyz="2.2861E-09"
-                 izz="0.00012442" />
+        <inertia ixx="0.000051" ixy="0.0" ixz="0.000006"
+                 iyy="0.000135" iyz="0.0"
+                 izz="0.000152" />
       </inertial>
       <visual>
@@ -68,5 +68,5 @@
     </link>
     <joint name="leg_${side}_${roll_joint}_joint" type="revolute">
-      <origin xyz="0 0 0" rpy="0 0 0" />
+      <origin xyz="0 0 0" rpy="0 0.34907 0" />
       <parent link="leg_${side}_${pitch_joint}_link" />
       <child link="leg_${side}_${roll_joint}_link" />
@@ -76,9 +76,9 @@
     <link name="leg_${side}_ankle_attach">
       <inertial>
-        <origin xyz="0.0016478 -1.3433E-06 -0.0053101" rpy="0 0 0" />
+        <origin xyz="0.0016478 0.001648 0.0053101" rpy="0 0 0" />
         <mass value="0.088641" />
-        <inertia ixx="2.1418E-05" ixy="8.6637E-10" ixz="3.8778E-07"
-                 iyy="2.555E-05" iyz="6.1789E-10"
-                 izz="4.4373E-05" />
+        <inertia ixx="0.000022" ixy="0.0" ixz="-0.000001"
+                 iyy="0.000027" iyz="0.0"
+                 izz="0.000046" />
       </inertial>
       <visual>
@@ -90,7 +90,5 @@
       </visual>
       <collision>
-        <origin
-          xyz="0 0 0"
-          rpy="0 0 0" />
+        <origin xyz="0 0 0" rpy="0 0 0" />
         <geometry>
           <mesh filename="package://kangaroo_description/meshes/leg/leg_ankle_attach.stl" />
@@ -99,10 +97,10 @@
     </link>
     <joint name="leg_${side}_ankle_attach_joint" type="fixed">
-      <origin xyz="0.013168 0 0.036178" rpy="0 0.34907 0" />
+      <origin xyz="0.013168 0 -0.036178" rpy="0 -0.34907 0" />
       <parent link="leg_${side}_${roll_joint}_link" />
       <child link="leg_${side}_ankle_attach" />
       <axis xyz="1 0 0" />
     </joint>
-    <xacro:kangaroo_detachable_foot_frames side="${side}" parent="leg_${side}_ankle_attach" offset_x="0.0"/>
+    <xacro:kangaroo_detachable_foot_frames side="${side}" parent="leg_${side}_ankle_attach" />
   </xacro:macro>
 </robot>

File: kangaroo_description/urdf/ankle/detachable_foot_frames.urdf.xacro (robot description, xacro)
@@ -3,12 +3,12 @@
 <xacro:property name="foot_length"   value="0.21" />
 <xacro:property name="foot_width"   value="0.09" />
-    <xacro:macro name="kangaroo_detachable_foot_frames" params="side parent offset_x:=0.0 offset_y:=0.0">
+    <xacro:macro name="kangaroo_detachable_foot_frames" params="side parent">
         <link name="${side}_foot">
             <inertial>
-                <origin xyz="0.000132090232624911 -3.05273190426678E-05 0.00417401893266306" rpy="0 0 0" />
-                <mass value="0.126216116323818" />
-                <inertia ixx="5.05342139344645E-05" ixy="-1.21919910576268E-06" ixz="3.77129027963418E-08"
-                        iyy="3.0799641719044E-05" iyz="1.55920192749335E-08"
-                        izz="7.74873112907028E-05" />
+                <origin xyz="-0.000166 0.000023 -0.004617" rpy="0 0 0" />
+                <mass value="0.170698" />
+                <inertia ixx="0.00007" ixy="-0.000001" ixz="0.0"
+                        iyy="0.000065" iyz="0.0"
+                        izz="0.000125" />
             </inertial>
             <visual>
@@ -27,5 +27,5 @@
         </link>
         <joint name="${side}_foot_joint" type="fixed">
-            <origin xyz="${offset_x} ${offset_y} 0" rpy="0 0 0" />
+            <origin xyz="0 0 0" rpy="0 0 0" />
             <parent link="${parent}" />
             <child link="${side}_foot" />
@@ -35,8 +35,8 @@
             <inertial>
                 <origin xyz="-0.000443003666554599 0.000522074497974099 -0.0153068327087122" rpy="0 0 0" />
-                <mass value="0.00199617753343338" />
-                <inertia ixx="5.9973064680877E-07" ixy="2.01121334144999E-08" ixz="-8.68902393943816E-09"
-                        iyy="5.90181580371415E-07" iyz="1.10619053149078E-08"
-                        izz="8.97962347086075E-07" />
+                <mass value="0.345" />
+                <inertia ixx="0.000104" ixy="0.000003" ixz="-0.000002"
+                        iyy="0.000102" iyz="0.000002"
+                        izz="0.000155" />
             </inertial>
             <visual>
@@ -55,5 +55,5 @@
         </link>
         <joint name="${side}_foot_ft" type="fixed">
-            <origin xyz="0 0 0.014" rpy="0 3.1416 0" />
+            <origin xyz="0 0 -0.014" rpy="0 0 3.1416" />
             <parent link="${side}_foot" />
             <child link="${side}_foot_ft" />
@@ -62,9 +62,9 @@
         <link name="${side}_foot_sole">
             <inertial>
-                <origin xyz="0.000379366462454072 5.80159494661185E-05 -0.00336003668438848" rpy="0 0 0" />
-                <mass value="0.34359589794105" />
-                <inertia ixx="0.000243921537522367" ixy="-3.79473815942421E-07" ixz="1.12448005808514E-07"
-                        iyy="0.0015816516325665" iyz="5.17989402289206E-08"
-                        izz="0.00182204612839865" />
+                <origin xyz="-0.004657 -0.000039 0.022641" rpy="0 0 0" />
+                <mass value="1.081199" />
+                <inertia ixx="0.001267" ixy="0.0" ixz="0.000111"
+                        iyy="0.005705" iyz="0.0"
+                        izz="0.00652" />
             </inertial>
             <visual>
@@ -83,5 +83,5 @@
         </link>
         <joint name="${side}_foot_sole" type="fixed">
-            <origin xyz="0 0 -0.038472" rpy="0 3.1416 0" />
+            <origin xyz="0 0 -0.053972" rpy="0 0 -3.1416" />
             <parent link="${side}_foot_ft" />
             <child link="${side}_foot_sole" />

Commit message: Replace values to use deg_to_rad macro

File: kangaroo_description/urdf/ankle/detachable_ankle.urdf.xacro (robot description, xacro)
@@ -68,5 +68,5 @@
     </link>
     <joint name="leg_${side}_${roll_joint}_joint" type="revolute">
-      <origin xyz="0 0 0" rpy="0 0.34907 0" />
+      <origin xyz="0 0 0" rpy="0 ${20.0 * deg_to_rad} 0" />
       <parent link="leg_${side}_${pitch_joint}_link" />
       <child link="leg_${side}_${roll_joint}_link" />
@@ -97,5 +97,5 @@
     </link>
     <joint name="leg_${side}_ankle_attach_joint" type="fixed">
-      <origin xyz="0.013168 0 -0.036178" rpy="0 -0.34907 0" />
+      <origin xyz="0.013168 0 -0.036178" rpy="0 -${20 * deg_to_rad} 0" />
       <parent link="leg_${side}_${roll_joint}_link" />
       <child link="leg_${side}_ankle_attach" />

File: kangaroo_description/urdf/ankle/detachable_foot_frames.urdf.xacro (robot description, xacro)
@@ -55,5 +55,5 @@
         </link>
         <joint name="${side}_foot_ft" type="fixed">
-            <origin xyz="0 0 -0.014" rpy="0 0 3.1416" />
+            <origin xyz="0 0 -0.014" rpy="0 0 ${180 * deg_to_rad}" />
             <parent link="${side}_foot" />
             <child link="${side}_foot_ft" />
@@ -83,5 +83,5 @@
         </link>
         <joint name="${side}_foot_sole" type="fixed">
-            <origin xyz="0 0 -0.053972" rpy="0 0 -3.1416" />
+            <origin xyz="0 0 -0.053972" rpy="0 0 -${180 * deg_to_rad}" />
             <parent link="${side}_foot_ft" />
             <child link="${side}_foot_sole" />

Commit message: add cloesd loop frames to the foot conditionally

File: kangaroo_description/urdf/ankle/detachable_ankle.urdf.xacro (robot description, xacro)
@@ -7,5 +7,6 @@
   <xacro:property name="roll_joint_min_pos"   value="${-27.0 *deg_to_rad}" />
   <xacro:property name="roll_joint_max_pos"   value="${27.0 *deg_to_rad}" />
-  <xacro:macro name="kangaroo_detachable_ankle" params="side reflect parent *origin pitch_joint roll_joint read_actuator">
+  <xacro:macro name="kangaroo_detachable_ankle"
+    params="side reflect parent *origin pitch_joint roll_joint read_actuator full_model:='false'">
     <link name="leg_${side}_${pitch_joint}_link">
       <inertial>
@@ -96,4 +97,33 @@
       </collision>
     </link>
+    <!-- CLOSED LOOP CONNECTION FRAMES FOR THE ANKLE -->
+    <xacro:if value="${full_model == 'true'}">
+      <link name="${side}_ankle_tibia_bar_l_connect_b">
+        <inertial>
+          <origin xyz="1e-05 1e-05 1e-05" rpy="0 0 0" />
+          <mass value="1e-05" />
+          <inertia ixx="1e-05" ixy="0.0" ixz="0.0" iyy="1e-05" iyz="0.0" izz="1e-05" />
+        </inertial>
+      </link>
+      <joint name="${side}_ankle_tibia_bar_l_connect_b" type="fixed">
+        <origin xyz="-0.05638 -0.03390 0.0590" rpy="1.57079632679491 -0.34906585039887 3.14159265358978" />
+        <parent link="leg_${side}_ankle_attach" />
+        <child link="${side}_ankle_tibia_bar_l_connect_b" />
+        <axis xyz="0 0 0" />
+      </joint>
+      <link name="${side}_ankle_tibia_bar_r_connect_b">
+        <inertial>
+          <origin xyz="1e-05 1e-05 1e-05" rpy="0 0 0" />
+          <mass value="1e-05" />
+          <inertia ixx="1e-05" ixy="0.0" ixz="0.0" iyy="1e-05" iyz="0.0" izz="1e-05" />
+        </inertial>
+      </link>
+      <joint name="${side}_ankle_tibia_bar_r_connect_b" type="fixed">
+        <origin xyz="-0.05638 0.03390 0.0590" rpy="1.57079632679491 -0.34906585039887 3.14159265358978" />
+        <parent link="leg_${side}_ankle_attach" />
+        <child link="${side}_ankle_tibia_bar_r_connect_b" />
+        <axis xyz="0 0 0" />
+      </joint>
+    </xacro:if>
     <joint name="leg_${side}_ankle_attach_joint" type="fixed">
       <origin xyz="0.013168 0 -0.036178" rpy="0 -${20 * deg_to_rad} 0" />

File: kangaroo_description/urdf/ankle/fixed_ankle.urdf.xacro (robot description, xacro)
@@ -8,5 +8,6 @@
   <xacro:property name="roll_joint_min_pos"   value="${-27.0 *deg_to_rad}" />
   <xacro:property name="roll_joint_max_pos"   value="${27.0 *deg_to_rad}" />
-  <xacro:macro name="kangaroo_fixed_ankle" params="side reflect parent *origin pitch_joint roll_joint read_actuator">
+  <xacro:macro name="kangaroo_fixed_ankle"
+    params="side reflect parent *origin pitch_joint roll_joint read_actuator full_model:='false'">
     <link name="leg_${side}_${pitch_joint}_link">
       <inertial>
@@ -79,4 +80,33 @@
       <origin xyz="0 0 0" rpy="0 ${-20.0 * deg_to_rad} 0" />
     </joint>
+    <!-- CLOSED LOOP CONNECTION FRAMES FOR THE ANKLE -->
+    <xacro:if value="${full_model}">
+      <link name="${side}_ankle_tibia_bar_l_connect_b">
+        <inertial>
+          <origin xyz="1e-05 1e-05 1e-05" rpy="0 0 0" />
+          <mass value="1e-05" />
+          <inertia ixx="1e-05" ixy="0.0" ixz="0.0" iyy="1e-05" iyz="0.0" izz="1e-05" />
+        </inertial>
+      </link>
+      <joint name="${side}_ankle_tibia_bar_l_connect_b" type="fixed">
+        <origin xyz="-0.05638 -0.03390 0.0205" rpy="1.57079632679491 0.0 3.14159265358978" />
+        <parent link="leg_${side}_${roll_joint}_aligned_link" />
+        <child link="${side}_ankle_tibia_bar_l_connect_b" />
+        <axis xyz="0 0 0" />
+      </joint>
+      <link name="${side}_ankle_tibia_bar_r_connect_b">
+        <inertial>
+          <origin xyz="1e-05 1e-05 1e-05" rpy="0 0 0" />
+          <mass value="1e-05" />
+          <inertia ixx="1e-05" ixy="0.0" ixz="0.0" iyy="1e-05" iyz="0.0" izz="1e-05" />
+        </inertial>
+      </link>
+      <joint name="${side}_ankle_tibia_bar_r_connect_b" type="fixed">
+        <origin xyz="-0.05638 0.03390 0.0205" rpy="1.57079632679491 0.0 3.14159265358978" />
+        <parent link="leg_${side}_${roll_joint}_aligned_link" />
+        <child link="${side}_ankle_tibia_bar_r_connect_b" />
+        <axis xyz="0 0 0" />
+      </joint>
+    </xacro:if>
     <link name="${side}_sole_link"/>
     <joint name="${side}_sole_joint" type="fixed">
