Commit message: ankle bar frames were swapped, now they are correct

File: kangaroo_description/urdf/ankle/detachable_ankle.urdf.xacro (robot description, xacro)
@@ -107,5 +107,5 @@
       </link>
       <joint name="${side}_ankle_tibia_bar_l_connect_b" type="fixed">
-        <origin xyz="-0.05638 -0.03390 0.0590" rpy="1.57079632679491 -0.34906585039887 3.14159265358978" />
+        <origin xyz="-0.05638 0.03390 0.0590" rpy="1.57079632679491 -0.34906585039887 3.14159265358978" />
         <parent link="leg_${side}_ankle_attach" />
         <child link="${side}_ankle_tibia_bar_l_connect_b" />
@@ -120,5 +120,5 @@
       </link>
       <joint name="${side}_ankle_tibia_bar_r_connect_b" type="fixed">
-        <origin xyz="-0.05638 0.03390 0.0590" rpy="1.57079632679491 -0.34906585039887 3.14159265358978" />
+        <origin xyz="-0.05638 -0.03390 0.0590" rpy="1.57079632679491 -0.34906585039887 3.14159265358978" />
         <parent link="leg_${side}_ankle_attach" />
         <child link="${side}_ankle_tibia_bar_r_connect_b" />

File: kangaroo_description/urdf/ankle/fixed_ankle.urdf.xacro (robot description, xacro)
@@ -90,5 +90,5 @@
       </link>
       <joint name="${side}_ankle_tibia_bar_l_connect_b" type="fixed">
-        <origin xyz="-0.05638 -0.03390 0.0205" rpy="1.57079632679491 0.0 3.14159265358978" />
+        <origin xyz="-0.05638 0.03390 0.0205" rpy="1.57079632679491 0.0 3.14159265358978" />
         <parent link="leg_${side}_${roll_joint}_aligned_link" />
         <child link="${side}_ankle_tibia_bar_l_connect_b" />
@@ -103,5 +103,5 @@
       </link>
       <joint name="${side}_ankle_tibia_bar_r_connect_b" type="fixed">
-        <origin xyz="-0.05638 0.03390 0.0205" rpy="1.57079632679491 0.0 3.14159265358978" />
+        <origin xyz="-0.05638 -0.03390 0.0205" rpy="1.57079632679491 0.0 3.14159265358978" />
         <parent link="leg_${side}_${roll_joint}_aligned_link" />
         <child link="${side}_ankle_tibia_bar_r_connect_b" />
