Commit message: fixed name of the ft link so that it coherent with broadcaster config

File: kangaroo_description/urdf/ankle/detachable_foot_frames.urdf.xacro (robot description, xacro)
@@ -32,5 +32,5 @@
             <axis xyz="0 0 0" />
         </joint>
-        <link name="${side}_foot_ft">
+        <link name="ankle_${side}_ft_sensor_link">
             <inertial>
                 <origin xyz="-0.000443003666554599 0.000522074497974099 -0.0153068327087122" rpy="0 0 0" />
@@ -57,5 +57,5 @@
             <origin xyz="0 0 -0.014" rpy="0 0 ${180 * deg_to_rad}" />
             <parent link="${side}_foot" />
-            <child link="${side}_foot_ft" />
+            <child link="ankle_${side}_ft_sensor_link" />
             <axis xyz="0 0 0" />
         </joint>
@@ -84,5 +84,5 @@
         <joint name="${side}_foot_sole" type="fixed">
             <origin xyz="0 0 -0.053972" rpy="0 0 -${180 * deg_to_rad}" />
-            <parent link="${side}_foot_ft" />
+            <parent link="ankle_${side}_ft_sensor_link" />
             <child link="${side}_foot_sole" />
             <axis xyz="0 0 0" />

Commit message: Rename sole frame for detachable feet type so it has the same name as the fixed version

File: kangaroo_description/urdf/ankle/detachable_foot_frames.urdf.xacro (robot description, xacro)
@@ -60,5 +60,5 @@
             <axis xyz="0 0 0" />
         </joint>
-        <link name="${side}_foot_sole">
+        <link name="${side}_sole_link">
             <inertial>
                 <origin xyz="-0.004657 -0.000039 0.022641" rpy="0 0 0" />
@@ -85,5 +85,5 @@
             <origin xyz="0 0 -0.053972" rpy="0 0 -${180 * deg_to_rad}" />
             <parent link="ankle_${side}_ft_sensor_link" />
-            <child link="${side}_foot_sole" />
+            <child link="${side}_sole_link" />
             <axis xyz="0 0 0" />
         </joint>
