Commit message: Update transmission model info

File: kangaroo_description/urdf/leg/leg.transmission.xacro (robot description, xacro)
@@ -5,32 +5,41 @@
 -->
 <robot name="kangaroo" xmlns:xacro="http://ros.org/wiki/xacro">
-  <xacro:macro name="kangaroo_leg_length_actuator_transmission" params="side number1 number2 femur intersection_crank_axis fbl11_long fbl11_short fbl21_fixed fbl21_long fbl21_short crank_slider_long crank_slider_short crank_slider_axis_angle shin_offset_angle connection_fbl_offset_angle knee_angle_min knee_angle_max" >
-    <transmission name="leg_${side}_leg_length_trans">
-      <type>transmission_interface/LegLengthActuatorTransmission</type>
-      <actuator name="leg_${side}_leg_length_motor" >
-        <femur>${femur}</femur>
-        <fbl11_long>${fbl11_long}</fbl11_long>
-        <fbl11_short>${fbl11_short}</fbl11_short>
-        <intersection_crank_axis>${intersection_crank_axis}</intersection_crank_axis>
-        <fbl21_fixed>${fbl21_fixed}</fbl21_fixed>
-        <fbl21_long>${fbl21_long}</fbl21_long>
-        <fbl21_short>${fbl21_short}</fbl21_short>
-        <crank_slider_long>${crank_slider_long}</crank_slider_long>
-        <crank_slider_short>${crank_slider_short}</crank_slider_short>
-        <crank_slider_axis_angle>${crank_slider_axis_angle}</crank_slider_axis_angle>
-        <shin_offset_angle>${shin_offset_angle}</shin_offset_angle>
-        <connection_fbl_offset_angle>${connection_fbl_offset_angle} </connection_fbl_offset_angle>
-        <knee_angle_min>${knee_angle_min}</knee_angle_min>
-        <knee_angle_max>${knee_angle_max}</knee_angle_max>
+  <xacro:macro name="kangaroo_leg_length_actuator_transmission" params="side number1 number2 leg_min_length leg_max_length femur intersection_crank_axis fbl11_long fbl11_short fbl21_fixed fbl21_long fbl21_short crank_slider_long crank_slider_short crank_slider_axis_angle shin_offset_angle connection_fbl_offset_angle shin_fbl11_offset_angle knee_angle_min knee_angle_max femur_angle_min femur_angle_max" >
+    <transmission name="leg_${side}_length_trans">
+      <type>pal_transmissions/LegCustomTransmission</type>
+      <actuator name="leg_${side}_length_motor">
+        <parameters>
+          <femur>${femur}</femur>
+          <fbl11_long>${fbl11_long}</fbl11_long>
+          <fbl11_short>${fbl11_short}</fbl11_short>
+          <intersection_crank_axis>${intersection_crank_axis}</intersection_crank_axis>
+          <fbl21_fixed>${fbl21_fixed}</fbl21_fixed>
+          <fbl21_long>${fbl21_long}</fbl21_long>
+          <fbl21_short>${fbl21_short}</fbl21_short>
+          <crank_slider_long>${crank_slider_long}</crank_slider_long>
+          <crank_slider_short>${crank_slider_short}</crank_slider_short>
+          <crank_slider_axis_angle>${crank_slider_axis_angle}</crank_slider_axis_angle>
+          <shin_offset_angle>${shin_offset_angle}</shin_offset_angle>
+          <connection_fbl_offset_angle>${connection_fbl_offset_angle} </connection_fbl_offset_angle>
+          <shin_fbl11_offset_angle>${shin_fbl11_offset_angle}</shin_fbl11_offset_angle>
+          <knee_angle_min>${knee_angle_min}</knee_angle_min>
+          <knee_angle_max>${knee_angle_max}</knee_angle_max>
+        </parameters>
+        <hardwareInterface>hardware_interface/PositionJointInterface</hardwareInterface>
+        <hardwareInterface>hardware_interface/EffortJointInterface</hardwareInterface>
+        <hardwareInterface>hardware_interface/JointStateInterface</hardwareInterface>
       </actuator>
-      <joint name="leg_${side}_${number1}_joint">
+      <joint name="leg_${side}_length_joint">
+        <role> leg_length </role>
+        <offset> 0.0 </offset>
+        <limits>
+          <position>
+            <min> ${leg_min_length} </min>
+            <max> ${leg_max_length} </max>
+          </position>
+        </limits>
         <hardwareInterface>hardware_interface/PositionJointInterface</hardwareInterface>
-        <hardwareInterface>hardware_interface/VelocityJointInterface</hardwareInterface>
         <hardwareInterface>hardware_interface/EffortJointInterface</hardwareInterface>
-      </joint>
-       <joint name="leg_${side}_${number2}_joint">
-        <hardwareInterface>hardware_interface/PositionJointInterface</hardwareInterface>
-        <hardwareInterface>hardware_interface/VelocityJointInterface</hardwareInterface>
-        <hardwareInterface>hardware_interface/EffortJointInterface</hardwareInterface>
+        <hardwareInterface>hardware_interface/JointStateInterface</hardwareInterface>
       </joint>
     </transmission>

Commit message: use the simple transmission for the simulation

File: kangaroo_description/urdf/leg/leg.transmission.xacro (robot description, xacro)
@@ -5,4 +5,104 @@
 -->
 <robot name="kangaroo" xmlns:xacro="http://ros.org/wiki/xacro">
+  <xacro:macro name="kangaroo_lower_body_simple_simulation_transmission" params="side">
+    <transmission name="leg_${side}_1_transmission">
+      <type>transmission_interface/SimpleTransmission</type>
+      <actuator name="leg_${side}_1_motor" >
+        <hardwareInterface>hardware_interface/PositionJointInterface</hardwareInterface>
+        <hardwareInterface>hardware_interface/EffortJointInterface</hardwareInterface>
+        <hardwareInterface>hardware_interface/JointStateInterface</hardwareInterface>
+        <mechanicalReduction>1.0</mechanicalReduction>
+      </actuator>
+      <joint name="leg_${side}_1_joint">
+        <hardwareInterface>hardware_interface/PositionJointInterface</hardwareInterface>
+        <hardwareInterface>hardware_interface/EffortJointInterface</hardwareInterface>
+        <hardwareInterface>hardware_interface/JointStateInterface</hardwareInterface>
+      </joint>
+    </transmission>
+    <transmission name="leg_${side}_2_transmission">
+      <type>transmission_interface/SimpleTransmission</type>
+      <actuator name="leg_${side}_2_motor" >
+        <hardwareInterface>hardware_interface/PositionJointInterface</hardwareInterface>
+        <hardwareInterface>hardware_interface/EffortJointInterface</hardwareInterface>
+        <hardwareInterface>hardware_interface/JointStateInterface</hardwareInterface>
+        <mechanicalReduction>1.0</mechanicalReduction>
+      </actuator>
+      <joint name="leg_${side}_2_joint">
+        <hardwareInterface>hardware_interface/PositionJointInterface</hardwareInterface>
+        <hardwareInterface>hardware_interface/EffortJointInterface</hardwareInterface>
+        <hardwareInterface>hardware_interface/JointStateInterface</hardwareInterface>
+      </joint>
+    </transmission>
+    <transmission name="leg_${side}_3_transmission">
+      <type>transmission_interface/SimpleTransmission</type>
+      <actuator name="leg_${side}_3_motor" >
+        <hardwareInterface>hardware_interface/PositionJointInterface</hardwareInterface>
+        <hardwareInterface>hardware_interface/EffortJointInterface</hardwareInterface>
+        <hardwareInterface>hardware_interface/JointStateInterface</hardwareInterface>
+        <mechanicalReduction>1.0</mechanicalReduction>
+      </actuator>
+      <joint name="leg_${side}_3_joint">
+        <hardwareInterface>hardware_interface/PositionJointInterface</hardwareInterface>
+        <hardwareInterface>hardware_interface/EffortJointInterface</hardwareInterface>
+        <hardwareInterface>hardware_interface/JointStateInterface</hardwareInterface>
+      </joint>
+    </transmission>
+    <transmission name="leg_${side}_4_transmission">
+      <type>transmission_interface/SimpleTransmission</type>
+      <actuator name="leg_${side}_4_motor" >
+        <hardwareInterface>hardware_interface/PositionJointInterface</hardwareInterface>
+        <hardwareInterface>hardware_interface/EffortJointInterface</hardwareInterface>
+        <hardwareInterface>hardware_interface/JointStateInterface</hardwareInterface>
+        <mechanicalReduction>1.0</mechanicalReduction>
+      </actuator>
+      <joint name="leg_${side}_4_joint">
+        <hardwareInterface>hardware_interface/PositionJointInterface</hardwareInterface>
+        <hardwareInterface>hardware_interface/EffortJointInterface</hardwareInterface>
+        <hardwareInterface>hardware_interface/JointStateInterface</hardwareInterface>
+      </joint>
+    </transmission>
+    <transmission name="leg_${side}_5_transmission">
+      <type>transmission_interface/SimpleTransmission</type>
+      <actuator name="leg_${side}_5_motor" >
+        <hardwareInterface>hardware_interface/PositionJointInterface</hardwareInterface>
+        <hardwareInterface>hardware_interface/EffortJointInterface</hardwareInterface>
+        <hardwareInterface>hardware_interface/JointStateInterface</hardwareInterface>
+        <mechanicalReduction>1.0</mechanicalReduction>
+      </actuator>
+      <joint name="leg_${side}_5_joint">
+        <hardwareInterface>hardware_interface/PositionJointInterface</hardwareInterface>
+        <hardwareInterface>hardware_interface/EffortJointInterface</hardwareInterface>
+        <hardwareInterface>hardware_interface/JointStateInterface</hardwareInterface>
+      </joint>
+    </transmission>
+    <transmission name="leg_${side}_6_transmission">
+      <type>transmission_interface/SimpleTransmission</type>
+      <actuator name="leg_${side}_6_motor" >
+        <hardwareInterface>hardware_interface/PositionJointInterface</hardwareInterface>
+        <hardwareInterface>hardware_interface/EffortJointInterface</hardwareInterface>
+        <hardwareInterface>hardware_interface/JointStateInterface</hardwareInterface>
+        <mechanicalReduction>1.0</mechanicalReduction>
+      </actuator>
+      <joint name="leg_${side}_6_joint">
+        <hardwareInterface>hardware_interface/PositionJointInterface</hardwareInterface>
+        <hardwareInterface>hardware_interface/EffortJointInterface</hardwareInterface>
+        <hardwareInterface>hardware_interface/JointStateInterface</hardwareInterface>
+      </joint>
+    </transmission>
+    <transmission name="leg_${side}_7_transmission">
+      <type>transmission_interface/SimpleTransmission</type>
+      <actuator name="leg_${side}_7_motor" >
+        <hardwareInterface>hardware_interface/PositionJointInterface</hardwareInterface>
+        <hardwareInterface>hardware_interface/EffortJointInterface</hardwareInterface>
+        <hardwareInterface>hardware_interface/JointStateInterface</hardwareInterface>
+        <mechanicalReduction>1.0</mechanicalReduction>
+      </actuator>
+      <joint name="leg_${side}_7_joint">
+        <hardwareInterface>hardware_interface/PositionJointInterface</hardwareInterface>
+        <hardwareInterface>hardware_interface/EffortJointInterface</hardwareInterface>
+        <hardwareInterface>hardware_interface/JointStateInterface</hardwareInterface>
+      </joint>
+    </transmission>
+  </xacro:macro>
   <xacro:macro name="kangaroo_leg_length_actuator_transmission" params="side number1 number2 leg_min_length leg_max_length femur intersection_crank_axis fbl11_long fbl11_short fbl21_fixed fbl21_long fbl21_short crank_slider_long crank_slider_short crank_slider_axis_angle shin_offset_angle connection_fbl_offset_angle shin_fbl11_offset_angle knee_angle_min knee_angle_max femur_angle_min femur_angle_max" >
     <transmission name="leg_${side}_length_trans">

Commit message: added the rest the main transmission for rest of the joints

File: kangaroo_description/urdf/leg/leg.transmission.xacro (robot description, xacro)
@@ -145,3 +145,113 @@
     </transmission>
   </xacro:macro>
+  <xacro:macro name="hip_transmission_roll_pitch" params="side roll_joint pitch_joint">
+    <transmission name="leg_${side}_transmission_roll_pitch">
+      <type>pal_transmissions/HipCustomTransmission</type>
+      <actuator name="leg_${side}_${roll_joint}_motor">
+        <role>actuator1</role>
+        <virtual_linear_actuator>
+          <screw_lead> 0.005 </screw_lead>
+          <efficiency> 0.9 </efficiency>
+          <limits>
+            <position>
+              <min> 0.0 </min>
+              <max> 0.10 </max>
+            </position>
+            <velocity>
+              <min> -0.3 </min>
+              <max> 0.3 </max>
+            </velocity>
+          </limits>
+        </virtual_linear_actuator>
+        <mechanicalReduction>1.0</mechanicalReduction>
+      </actuator>
+      <actuator name="leg_${side}_${pitch_joint}_motor">
+        <role>actuator2</role>
+        <virtual_linear_actuator>
+          <screw_lead> 0.005 </screw_lead>
+          <efficiency> 0.9 </efficiency>
+          <limits>
+            <position>
+              <min> 0.0 </min>
+              <max> 0.10 </max>
+            </position>
+            <velocity>
+              <min> -0.3 </min>
+              <max> 0.3 </max>
+            </velocity>
+          </limits>
+        </virtual_linear_actuator>
+        <mechanicalReduction>1.0</mechanicalReduction>
+      </actuator>
+      <joint name="leg_${side}_${roll_joint}_joint">
+        <role>joint1</role>
+        <limits>
+          <position>
+            <min> ${ -27.0 * deg_to_rad} </min>
+            <max> ${ 27.0 * deg_to_rad} </max>
+          </position>
+        </limits>
+        <configuration>
+          <offset_x> 0.0035 </offset_x>
+          <offset_y> 0.0051 </offset_y>
+          <projected_distance> 0.17650 </projected_distance>
+          <dx> 0.0035 </dx>
+          <dy> 0.0060 </dy>
+        </configuration>
+        <hardwareInterface>hardware_interface/PositionJointInterface</hardwareInterface>
+        <hardwareInterface>hardware_interface/EffortJointInterface</hardwareInterface>
+      </joint>
+      <joint name="leg_${side}_${pitch_joint}_joint">
+        <role>joint2</role>
+        <limits>
+          <position>
+            <min> ${ -42.5 * deg_to_rad} </min>
+            <max> ${ 42.5 * deg_to_rad} </max>
+          </position>
+        </limits>
+        <hardwareInterface>hardware_interface/PositionJointInterface</hardwareInterface>
+        <hardwareInterface>hardware_interface/EffortJointInterface</hardwareInterface>
+      </joint>
+    </transmission>
+  </xacro:macro>
+  <xacro:macro name="hip_transmission_yaw" params="side number reduction">
+    <transmission name="leg_${side}_transmission_yaw">
+      <type>transmission_interface/SimpleTransmission</type>
+      <actuator name="leg_${side}_${number}_motor" >
+        <mechanicalReduction>${reduction}</mechanicalReduction>
+      </actuator>
+      <joint name="leg_${side}_${number}_joint">
+        <hardwareInterface>hardware_interface/PositionJointInterface</hardwareInterface>
+        <hardwareInterface>hardware_interface/EffortJointInterface</hardwareInterface>
+      </joint>
+    </transmission>
+  </xacro:macro>
+  <xacro:macro name="kangaroo_ankle_transmission" params="side roll_joint pitch_joint read_actuator">
+    <transmission name="leg_${side}_transmission">
+      <type>pal_transmissions/AnkleCustomTransmission</type>
+      <actuator name="leg_${side}_${roll_joint}_motor">
+        <role>right_actuator</role>
+        <param_ns>/ankle_params</param_ns>
+      </actuator>
+      <actuator name="leg_${side}_${pitch_joint}_motor">
+        <role>left_actuator</role>
+      </actuator>
+      <actuator name="${read_actuator}">
+        <role>leg_length</role>
+        <param_ns>/leg_params</param_ns>
+      </actuator>
+      <joint name="leg_${side}_${roll_joint}_joint">
+        <role>roll_joint</role>
+        <offset> 0.0 </offset>
+        <hardwareInterface>hardware_interface/PositionJointInterface</hardwareInterface>
+        <hardwareInterface>hardware_interface/EffortJointInterface</hardwareInterface>
+      </joint>
+      <joint name="leg_${side}_${pitch_joint}_joint">
+        <role>pitch_joint</role>
+        <offset> 0.0 </offset>
+        <hardwareInterface>hardware_interface/PositionJointInterface</hardwareInterface>
+        <hardwareInterface>hardware_interface/EffortJointInterface</hardwareInterface>
+      </joint>
+    </transmission>
+  </xacro:macro>
 </robot>
