Commit message: add the new ankle urdf macro to the leg

File: kangaroo_description/urdf/leg/leg.transmission.xacro (robot description, xacro)
@@ -71,32 +71,4 @@
       </actuator>
       <joint name="leg_${side}_5_joint">
-        <hardwareInterface>hardware_interface/PositionJointInterface</hardwareInterface>
-        <hardwareInterface>hardware_interface/EffortJointInterface</hardwareInterface>
-        <hardwareInterface>hardware_interface/JointStateInterface</hardwareInterface>
-      </joint>
-    </transmission>
-    <transmission name="leg_${side}_6_transmission">
-      <type>transmission_interface/SimpleTransmission</type>
-      <actuator name="leg_${side}_6_motor" >
-        <hardwareInterface>hardware_interface/PositionJointInterface</hardwareInterface>
-        <hardwareInterface>hardware_interface/EffortJointInterface</hardwareInterface>
-        <hardwareInterface>hardware_interface/JointStateInterface</hardwareInterface>
-        <mechanicalReduction>1.0</mechanicalReduction>
-      </actuator>
-      <joint name="leg_${side}_6_joint">
-        <hardwareInterface>hardware_interface/PositionJointInterface</hardwareInterface>
-        <hardwareInterface>hardware_interface/EffortJointInterface</hardwareInterface>
-        <hardwareInterface>hardware_interface/JointStateInterface</hardwareInterface>
-      </joint>
-    </transmission>
-    <transmission name="leg_${side}_7_transmission">
-      <type>transmission_interface/SimpleTransmission</type>
-      <actuator name="leg_${side}_7_motor" >
-        <hardwareInterface>hardware_interface/PositionJointInterface</hardwareInterface>
-        <hardwareInterface>hardware_interface/EffortJointInterface</hardwareInterface>
-        <hardwareInterface>hardware_interface/JointStateInterface</hardwareInterface>
-        <mechanicalReduction>1.0</mechanicalReduction>
-      </actuator>
-      <joint name="leg_${side}_7_joint">
         <hardwareInterface>hardware_interface/PositionJointInterface</hardwareInterface>
         <hardwareInterface>hardware_interface/EffortJointInterface</hardwareInterface>
@@ -227,31 +199,3 @@
     </transmission>
   </xacro:macro>
-  <xacro:macro name="kangaroo_ankle_transmission" params="side roll_joint pitch_joint read_actuator">
-    <transmission name="leg_${side}_transmission">
-      <type>pal_transmissions/AnkleCustomTransmission</type>
-      <actuator name="leg_${side}_${roll_joint}_motor">
-        <role>right_actuator</role>
-        <param_ns>/ankle_params</param_ns>
-      </actuator>
-      <actuator name="leg_${side}_${pitch_joint}_motor">
-        <role>left_actuator</role>
-      </actuator>
-      <actuator name="${read_actuator}">
-        <role>leg_length</role>
-        <param_ns>/leg_params</param_ns>
-      </actuator>
-      <joint name="leg_${side}_${roll_joint}_joint">
-        <role>roll_joint</role>
-        <offset> 0.0 </offset>
-        <hardwareInterface>hardware_interface/PositionJointInterface</hardwareInterface>
-        <hardwareInterface>hardware_interface/EffortJointInterface</hardwareInterface>
-      </joint>
-      <joint name="leg_${side}_${pitch_joint}_joint">
-        <role>pitch_joint</role>
-        <offset> 0.0 </offset>
-        <hardwareInterface>hardware_interface/PositionJointInterface</hardwareInterface>
-        <hardwareInterface>hardware_interface/EffortJointInterface</hardwareInterface>
-      </joint>
-    </transmission>
-  </xacro:macro>
 </robot>

File: kangaroo_description/urdf/leg/leg.urdf.xacro (robot description, xacro)
@@ -2,4 +2,5 @@
 <robot xmlns:xacro="http://ros.org/wiki/xacro" name="kangaroo">
   <xacro:include filename="$(find kangaroo_description)/urdf/leg/leg.transmission.xacro" />
+  <xacro:include filename="$(find kangaroo_description)/urdf/ankle/ankle.urdf.xacro" />
   <xacro:property name="deg_to_rad"       value="0.01745329251994329577" />
   <xacro:property name="eps_radians"      value="0.008" /> <!-- 0.45deg -->
@@ -15,11 +16,7 @@
   <xacro:property name="leg_5_min_pos"   value="${20.0 *deg_to_rad}" />
   <xacro:property name="leg_5_max_pos"   value="${140.0 *deg_to_rad}" />
-  <xacro:property name="leg_6_min_pos"   value="${-42.5 *deg_to_rad}" />
-  <xacro:property name="leg_6_max_pos"   value="${42.5 *deg_to_rad}" />
-  <xacro:property name="leg_7_min_pos"   value="${-27.0 *deg_to_rad}" />
-  <xacro:property name="leg_7_max_pos"   value="${27.0 *deg_to_rad}" />
   <xacro:property name="leg_min_length"   value="0.131973" />
   <xacro:property name="leg_max_length"   value="0.71416639" />
-  <xacro:macro name="kangaroo_leg" params="side reflect parent *origin simulation:=false">
+  <xacro:macro name="kangaroo_leg" params="side reflect parent *origin simulation:=false type:=dynamic">
     <link name="leg_${side}_1_link">
       <inertial>
@@ -176,69 +173,13 @@
       <limit lower="${leg_5_min_pos}" upper="${leg_5_max_pos}" effort="100" velocity="3.87" />
     </joint>
-    <link name="leg_${side}_6_link">
-      <inertial>
-        <origin xyz="-0.00714160332877733 4.8311277200952E-09 0.00259941265068991" rpy="0 0 0" />
-        <mass value="0.0905836559788966" />
-        <inertia ixx="7.07461991271062E-06" ixy="-1.86951004827933E-12" ixz="8.30282143898823E-06"
-          iyy="2.92762498059213E-05" iyz="1.82895645239997E-11" izz="2.68643074366886E-05" />
-      </inertial>
-      <visual>
-        <origin xyz="0 0 0" rpy="0 0 0" />
-        <geometry>
-          <mesh filename="package://kangaroo_description/meshes/leg_6_link.stl" />
-        </geometry>
-        <material name="">
-          <color rgba="0.752941176470588 0.752941176470588 0.752941176470588 1" />
-        </material>
-      </visual>
-      <collision>
-        <origin xyz="0 0 0" rpy="0 0 0" />
-        <geometry>
-          <mesh filename="package://kangaroo_description/meshes/leg_6_link.stl" />
-        </geometry>
-      </collision>
-    </link>
-    <joint name="leg_${side}_6_joint" type="revolute">
-      <origin xyz="-0.37432 0 -0.065464" rpy="0 0 0" />
-      <parent link="leg_${side}_5_link" />
-      <child link="leg_${side}_6_link" />
-      <axis xyz="0 1 0" />
-      <limit lower="${leg_6_min_pos}" upper="${leg_6_max_pos}" effort="100" velocity="3.87" />
-    </joint>
-    <link name="leg_${side}_7_link">
-      <inertial>
-        <origin xyz="0.0177425915954867 -3.67950153736807E-05 -0.0172694732454237" rpy="0 0 0" />
-        <mass value="0.394418327358563" />
-        <inertia ixx="0.000228382894016579" ixy="-2.56621760255351E-07" ixz="4.1179623691202E-05"
-          iyy="0.00108653696539759" iyz="7.85648127231571E-09" izz="0.0012643765698811" />
-      </inertial>
-      <visual>
-        <origin xyz="0 0 0" rpy="0 0 0" />
-        <geometry>
-          <mesh filename="package://kangaroo_description/meshes/leg_7_link.stl" />
-        </geometry>
-        <material name="">
-          <color rgba="0.752941176470588 0.752941176470588 0.752941176470588 1" />
-        </material>
-      </visual>
-      <collision>
-        <origin xyz="0 0 0" rpy="0 0 0" />
-        <geometry>
-          <mesh filename="package://kangaroo_description/meshes/leg_7_link.stl" />
-        </geometry>
-      </collision>
-    </link>
-    <joint name="leg_${side}_7_joint" type="revolute">
-      <origin xyz="0 0 0" rpy="0 0 0" />
-      <parent link="leg_${side}_6_link" />
-      <child link="leg_${side}_7_link" />
-      <axis xyz="-0.93969 0 0.34202" />
-      <limit lower="${leg_7_min_pos}" upper="${leg_7_max_pos}" effort="100" velocity="3.87" />
-    </joint>
+    <xacro:if value="${type=='dynamic'}" >
+      <xacro:kangaroo_ankle side="${side}" parent="leg_${side}_5_link" reflect="${reflect}" roll_joint="7" pitch_joint="6" read_actuator="leg_${side}_length_motor">
+        <origin xyz="-0.37432 0 -0.065464" rpy="0 0 0" />
+      </xacro:kangaroo_ankle>
+    </xacro:if>
     <xacro:unless value="${simulation}">
       <xacro:hip_transmission_yaw side="${side}" number="1" reduction="1.0" />
       <xacro:hip_transmission_roll_pitch side="${side}" roll_joint="3" pitch_joint="2" />
       <xacro:kangaroo_leg_length_actuator_transmission side="${side}" number1="4" number2="5" leg_min_length="${leg_min_length}" leg_max_length="${leg_max_length}" femur="0.380" intersection_crank_axis="0.155693813961639" fbl11_long="0.404273" fbl11_short="0.090" fbl21_fixed="0.115" fbl21_long="0.090" fbl21_short="0.040" crank_slider_long="0.215" crank_slider_short="0.090" crank_slider_axis_angle="${-15.65*deg_to_rad}" shin_offset_angle="${0.0*deg_to_rad}" connection_fbl_offset_angle="${-45.0*deg_to_rad}" shin_fbl11_offset_angle="${-15.00*deg_to_rad}" knee_angle_min ="${leg_5_min_pos - 5.0 *deg_to_rad}" knee_angle_max="${leg_5_max_pos + 5.0 *deg_to_rad}" femur_angle_min="${leg_4_min_pos}" femur_angle_max="${leg_4_max_pos}" />
-      <xacro:kangaroo_ankle_transmission side="${side}" roll_joint="7" pitch_joint="6" read_actuator="leg_${side}_length_motor" />
     </xacro:unless>
     <xacro:if value="${simulation}">
@@ -265,12 +206,4 @@
      <mu2>0.9</mu2>
    </gazebo>
-   <gazebo reference="leg_${side}_6_link">
-     <mu1>0.9</mu1>
-     <mu2>0.9</mu2>
-   </gazebo>
-   <gazebo reference="leg_${side}_7_link">
-     <mu1>0.9</mu1>
-     <mu2>0.9</mu2>
-   </gazebo>
    <gazebo reference="leg_${side}_1_joint">
       <implicitSpringDamper>1</implicitSpringDamper>
@@ -286,10 +219,4 @@
    </gazebo>
    <gazebo reference="leg_${side}_5_joint">
-      <implicitSpringDamper>1</implicitSpringDamper>
-   </gazebo>
-   <gazebo reference="leg_${side}_6_joint">
-      <implicitSpringDamper>1</implicitSpringDamper>
-   </gazebo>
-   <gazebo reference="leg_${side}_7_joint">
       <implicitSpringDamper>1</implicitSpringDamper>
    </gazebo>
@@ -309,10 +236,4 @@
     <material>Gazebo/FlatBlack</material>
   </gazebo>
-  <gazebo reference="leg_${side}_6_link">
-    <material>Gazebo/FlatWhite</material>
-  </gazebo>
-  <gazebo reference="leg_${side}_7_link">
-    <material>Gazebo/FlatWhite</material>
-  </gazebo>
   </xacro:macro>
 </robot>

Commit message: update leg_transmission.xacro to use the 'prismatic' parameter

File: kangaroo_description/urdf/leg/leg.transmission.xacro (robot description, xacro)
@@ -5,5 +5,5 @@
 -->
 <robot name="kangaroo" xmlns:xacro="http://ros.org/wiki/xacro">
-  <xacro:macro name="kangaroo_lower_body_simple_simulation_transmission" params="side">
+  <xacro:macro name="kangaroo_lower_body_simple_simulation_transmission" params="side prismatic">
     <transmission name="leg_${side}_1_transmission">
       <type>transmission_interface/SimpleTransmission</type>
@@ -48,18 +48,20 @@
       </joint>
     </transmission>
-    <transmission name="leg_${side}_4_transmission">
-      <type>transmission_interface/SimpleTransmission</type>
-      <actuator name="leg_${side}_4_motor" >
-        <hardwareInterface>hardware_interface/PositionJointInterface</hardwareInterface>
-        <hardwareInterface>hardware_interface/EffortJointInterface</hardwareInterface>
-        <hardwareInterface>hardware_interface/JointStateInterface</hardwareInterface>
-        <mechanicalReduction>1.0</mechanicalReduction>
-      </actuator>
-      <joint name="leg_${side}_4_joint">
-        <hardwareInterface>hardware_interface/PositionJointInterface</hardwareInterface>
-        <hardwareInterface>hardware_interface/EffortJointInterface</hardwareInterface>
-        <hardwareInterface>hardware_interface/JointStateInterface</hardwareInterface>
-      </joint>
-    </transmission>
+	  <xacro:unless value="$(arg prismatic)">
+		  <transmission name="leg_${side}_4_transmission">
+		    <type>transmission_interface/SimpleTransmission</type>
+		    <actuator name="leg_${side}_4_motor" >
+		      <hardwareInterface>hardware_interface/PositionJointInterface</hardwareInterface>
+		      <hardwareInterface>hardware_interface/EffortJointInterface</hardwareInterface>
+		      <hardwareInterface>hardware_interface/JointStateInterface</hardwareInterface>
+		      <mechanicalReduction>1.0</mechanicalReduction>
+		    </actuator>
+		    <joint name="leg_${side}_4_joint">
+		      <hardwareInterface>hardware_interface/PositionJointInterface</hardwareInterface>
+		      <hardwareInterface>hardware_interface/EffortJointInterface</hardwareInterface>
+		      <hardwareInterface>hardware_interface/JointStateInterface</hardwareInterface>
+		    </joint>
+		  </transmission>
+		</xacro:unless>
     <transmission name="leg_${side}_5_transmission">
       <type>transmission_interface/SimpleTransmission</type>

Commit message: minor fixes to maintain the naming sequence

File: kangaroo_description/urdf/leg/leg.transmission.xacro (robot description, xacro)
@@ -48,34 +48,34 @@
       </joint>
     </transmission>
-	  <xacro:unless value="$(arg prismatic)">
-		  <transmission name="leg_${side}_4_transmission">
-		    <type>transmission_interface/SimpleTransmission</type>
-		    <actuator name="leg_${side}_4_motor" >
-		      <hardwareInterface>hardware_interface/PositionJointInterface</hardwareInterface>
-		      <hardwareInterface>hardware_interface/EffortJointInterface</hardwareInterface>
-		      <hardwareInterface>hardware_interface/JointStateInterface</hardwareInterface>
-		      <mechanicalReduction>1.0</mechanicalReduction>
-		    </actuator>
-		    <joint name="leg_${side}_4_joint">
-		      <hardwareInterface>hardware_interface/PositionJointInterface</hardwareInterface>
-		      <hardwareInterface>hardware_interface/EffortJointInterface</hardwareInterface>
-		      <hardwareInterface>hardware_interface/JointStateInterface</hardwareInterface>
-		    </joint>
-		  </transmission>
-		</xacro:unless>
-    <transmission name="leg_${side}_5_transmission">
-      <type>transmission_interface/SimpleTransmission</type>
-      <actuator name="leg_${side}_5_motor" >
-        <hardwareInterface>hardware_interface/PositionJointInterface</hardwareInterface>
-        <hardwareInterface>hardware_interface/EffortJointInterface</hardwareInterface>
-        <hardwareInterface>hardware_interface/JointStateInterface</hardwareInterface>
-        <mechanicalReduction>1.0</mechanicalReduction>
-      </actuator>
-      <joint name="leg_${side}_5_joint">
-        <hardwareInterface>hardware_interface/PositionJointInterface</hardwareInterface>
-        <hardwareInterface>hardware_interface/EffortJointInterface</hardwareInterface>
-        <hardwareInterface>hardware_interface/JointStateInterface</hardwareInterface>
-      </joint>
-    </transmission>
+    <transmission name="leg_${side}_4_transmission">
+      <type>transmission_interface/SimpleTransmission</type>
+      <actuator name="leg_${side}_4_motor" >
+        <hardwareInterface>hardware_interface/PositionJointInterface</hardwareInterface>
+        <hardwareInterface>hardware_interface/EffortJointInterface</hardwareInterface>
+        <hardwareInterface>hardware_interface/JointStateInterface</hardwareInterface>
+        <mechanicalReduction>1.0</mechanicalReduction>
+      </actuator>
+      <joint name="leg_${side}_4_joint">
+        <hardwareInterface>hardware_interface/PositionJointInterface</hardwareInterface>
+        <hardwareInterface>hardware_interface/EffortJointInterface</hardwareInterface>
+        <hardwareInterface>hardware_interface/JointStateInterface</hardwareInterface>
+      </joint>
+    </transmission>
+    <xacro:unless value="$(arg prismatic)">
+      <transmission name="leg_${side}_5_transmission">
+        <type>transmission_interface/SimpleTransmission</type>
+        <actuator name="leg_${side}_5_motor" >
+          <hardwareInterface>hardware_interface/PositionJointInterface</hardwareInterface>
+          <hardwareInterface>hardware_interface/EffortJointInterface</hardwareInterface>
+          <hardwareInterface>hardware_interface/JointStateInterface</hardwareInterface>
+          <mechanicalReduction>1.0</mechanicalReduction>
+        </actuator>
+        <joint name="leg_${side}_5_joint">
+          <hardwareInterface>hardware_interface/PositionJointInterface</hardwareInterface>
+          <hardwareInterface>hardware_interface/EffortJointInterface</hardwareInterface>
+          <hardwareInterface>hardware_interface/JointStateInterface</hardwareInterface>
+        </joint>
+      </transmission>
+    </xacro:unless>
   </xacro:macro>
   <xacro:macro name="kangaroo_leg_length_actuator_transmission" params="side number1 number2 leg_min_length leg_max_length femur intersection_crank_axis fbl11_long fbl11_short fbl21_fixed fbl21_long fbl21_short crank_slider_long crank_slider_short crank_slider_axis_angle shin_offset_angle connection_fbl_offset_angle shin_fbl11_offset_angle knee_angle_min knee_angle_max femur_angle_min femur_angle_max" >

File: kangaroo_description/urdf/leg/leg.urdf.xacro (robot description, xacro)
@@ -175,6 +175,6 @@
 		  </joint>
     </xacro:unless>
-    <xacro:if value="${type=='prismatic'}" > <!-- load the model with the leg lenght prismatic joint-->
-			 <link name="leg_${side}_4_link">
+    <xacro:if value="${type=='prismatic'}" > <!-- load the model with the leg length prismatic joint-->
+			 <link name="leg_${side}_length_fixed_link">
 		    <inertial>
 		      <origin rpy="0 0 0" xyz="0.0 0.0 ${-leg_min_length/2.0}"/>
@@ -201,8 +201,8 @@
 		    <origin xyz="0 ${reflect * 0.0669} -0.09" rpy="0 0 0" />
 		    <parent link="leg_${side}_3_link" />
-		    <child link="leg_${side}_4_link" />
+		    <child link="leg_${side}_length_fixed_link" />
 		    <axis xyz="0 0 0" />
 		  </joint>
-		  <link name="leg_${side}_5_link">
+		  <link name="leg_${side}_4_link">
 		    <inertial>
 		      <origin rpy="0 0 0" xyz="0.0 0.0 ${(leg_max_length - leg_min_length)/2}"/>
@@ -226,8 +226,8 @@
 		    </collision> -->
 		  </link>
-		  <joint name="leg_${side}_5_joint" type="prismatic">
+		  <joint name="leg_${side}_4_joint" type="prismatic">
 		   <origin xyz="0.0 0.0 ${-leg_min_length}"  rpy="0.0 0.0 0.0"/>
-		    <parent link="leg_${side}_4_link" />
-		    <child link="leg_${side}_5_link" />
+		    <parent link="leg_${side}_length_fixed_link" />
+		    <child link="leg_${side}_4_link" />
 		    <axis xyz="0 0 -1" />
 		    <limit lower="0" upper="${leg_max_length - leg_min_length}" effort="100" velocity="10" /> <!-- TODO: update effort and velocity -->
@@ -240,6 +240,6 @@
     </xacro:if>
     <xacro:if value="${type=='prismatic'}" >
-      <xacro:kangaroo_ankle side="${side}" parent="leg_${side}_5_link" reflect="${reflect}" roll_joint="7" pitch_joint="6" read_actuator="leg_${side}_length_motor">
-        <origin xyz="0. 0 -0." rpy="0 0 0" />
+      <xacro:kangaroo_ankle side="${side}" parent="leg_${side}_4_link" reflect="${reflect}" roll_joint="6" pitch_joint="5" read_actuator="leg_${side}_length_motor">
+        <origin xyz="0 0 0" rpy="0 0 0" />
       </xacro:kangaroo_ankle>
     </xacro:if>

Commit message: added leg length simple transmission

File: kangaroo_description/urdf/leg/leg.transmission.xacro (robot description, xacro)
@@ -71,4 +71,18 @@
       </actuator>
       <joint name="leg_${side}_5_joint">
+        <hardwareInterface>hardware_interface/PositionJointInterface</hardwareInterface>
+        <hardwareInterface>hardware_interface/EffortJointInterface</hardwareInterface>
+        <hardwareInterface>hardware_interface/JointStateInterface</hardwareInterface>
+      </joint>
+    </transmission>
+    <transmission name="leg_${side}_leg_length_transmission">
+      <type>transmission_interface/SimpleTransmission</type>
+      <actuator name="leg_${side}_length_motor" >
+        <hardwareInterface>hardware_interface/PositionJointInterface</hardwareInterface>
+        <hardwareInterface>hardware_interface/EffortJointInterface</hardwareInterface>
+        <hardwareInterface>hardware_interface/JointStateInterface</hardwareInterface>
+        <mechanicalReduction>1.0</mechanicalReduction>
+      </actuator>
+      <joint name="leg_${side}_length_joint">
         <hardwareInterface>hardware_interface/PositionJointInterface</hardwareInterface>
         <hardwareInterface>hardware_interface/EffortJointInterface</hardwareInterface>
