Commit message: uncomment the kangaroo_leg_length_actuator_transmission in transmission xacro

File: kangaroo_description/urdf/leg/leg.transmission.xacro (robot description, xacro)
@@ -48,32 +48,4 @@
       </joint>
     </transmission>
-    <!-- <transmission name="leg_${side}_4_transmission">
-      <type>transmission_interface/SimpleTransmission</type>
-      <actuator name="leg_${side}_4_motor" >
-        <hardwareInterface>hardware_interface/PositionJointInterface</hardwareInterface>
-        <hardwareInterface>hardware_interface/EffortJointInterface</hardwareInterface>
-        <hardwareInterface>hardware_interface/JointStateInterface</hardwareInterface>
-        <mechanicalReduction>1.0</mechanicalReduction>
-      </actuator>
-      <joint name="leg_${side}_4_joint">
-        <hardwareInterface>hardware_interface/PositionJointInterface</hardwareInterface>
-        <hardwareInterface>hardware_interface/EffortJointInterface</hardwareInterface>
-        <hardwareInterface>hardware_interface/JointStateInterface</hardwareInterface>
-      </joint>
-    </transmission>
-    <transmission name="leg_${side}_5_transmission">
-      <type>transmission_interface/SimpleTransmission</type>
-      <actuator name="leg_${side}_5_motor" >
-        <hardwareInterface>hardware_interface/PositionJointInterface</hardwareInterface>
-        <hardwareInterface>hardware_interface/EffortJointInterface</hardwareInterface>
-        <hardwareInterface>hardware_interface/JointStateInterface</hardwareInterface>
-        <mechanicalReduction>1.0</mechanicalReduction>
-      </actuator>
-      <joint name="leg_${side}_5_joint">
-        <hardwareInterface>hardware_interface/PositionJointInterface</hardwareInterface>
-        <hardwareInterface>hardware_interface/EffortJointInterface</hardwareInterface>
-        <hardwareInterface>hardware_interface/JointStateInterface</hardwareInterface>
-      </joint>
-    </transmission> -->
     <transmission name="leg_${side}_leg_length_transmission">
       <type>transmission_interface/SimpleTransmission</type>
@@ -91,27 +63,5 @@
     </transmission>
   </xacro:macro>
-  <!-- <xacro:macro name="kangaroo_leg_length_actuator_transmission" params="side number1 number2 params_ns:=/leg_params" >
-    <transmission name="leg_${side}_${number1}_trans">
-      <type>pal_transmissions/LegCustomTransmission</type>
-      <actuator name="leg_${side}_length_motor" >
-      </actuator>
-      <joint name="leg_${side}_${number1}_joint">
-        <joint_type> femur </joint_type>
-        <param_ns> ${params_ns} </param_ns>
-        <offset> 0.0 </offset>
-        <hardwareInterface>hardware_interface/JointStateInterface</hardwareInterface>
-      </joint>
-    </transmission>
-    <transmission name="leg_${side}_${number2}_trans">
-      <type>pal_transmissions/LegCustomTransmission</type>
-      <actuator name="leg_${side}_length_motor" >
-      </actuator>
-      <joint name="leg_${side}_${number2}_joint">
-        <joint_type> knee </joint_type>
-        <param_ns> ${params_ns} </param_ns>
-        <offset> 0.0 </offset>
-        <hardwareInterface>hardware_interface/JointStateInterface</hardwareInterface>
-      </joint>
-    </transmission>
+  <xacro:macro name="kangaroo_leg_length_actuator_transmission" params="side number1 number2 params_ns:=/leg_params" >
     <transmission name="leg_${side}_leg_length_trans">
       <type>pal_transmissions/LegCustomTransmission</type>
@@ -127,5 +77,5 @@
       </joint>
     </transmission>
-  </xacro:macro> -->
+  </xacro:macro>
   <xacro:macro name="hip_transmission_roll_pitch" params="side roll_joint pitch_joint">
     <transmission name="leg_${side}_transmission_roll_pitch">

Commit message: Uncomment transmission for kangaroo pal_physics_simulator

File: kangaroo_description/urdf/leg/leg.transmission.xacro (robot description, xacro)
@@ -91,27 +91,5 @@
     </transmission>
   </xacro:macro>
-  <!-- <xacro:macro name="kangaroo_leg_length_actuator_transmission" params="side number1 number2 params_ns:=/leg_params" >
-    <transmission name="leg_${side}_${number1}_trans">
-      <type>pal_transmissions/LegCustomTransmission</type>
-      <actuator name="leg_${side}_length_motor" >
-      </actuator>
-      <joint name="leg_${side}_${number1}_joint">
-        <joint_type> femur </joint_type>
-        <param_ns> ${params_ns} </param_ns>
-        <offset> 0.0 </offset>
-        <hardwareInterface>hardware_interface/JointStateInterface</hardwareInterface>
-      </joint>
-    </transmission>
-    <transmission name="leg_${side}_${number2}_trans">
-      <type>pal_transmissions/LegCustomTransmission</type>
-      <actuator name="leg_${side}_length_motor" >
-      </actuator>
-      <joint name="leg_${side}_${number2}_joint">
-        <joint_type> knee </joint_type>
-        <param_ns> ${params_ns} </param_ns>
-        <offset> 0.0 </offset>
-        <hardwareInterface>hardware_interface/JointStateInterface</hardwareInterface>
-      </joint>
-    </transmission>
+  <xacro:macro name="kangaroo_leg_length_actuator_transmission" params="side number1 number2 params_ns:=/leg_params" >
     <transmission name="leg_${side}_leg_length_trans">
       <type>pal_transmissions/LegCustomTransmission</type>
@@ -127,5 +105,5 @@
       </joint>
     </transmission>
-  </xacro:macro> -->
+  </xacro:macro>
   <xacro:macro name="hip_transmission_roll_pitch" params="side roll_joint pitch_joint">
     <transmission name="leg_${side}_transmission_roll_pitch">

Commit message: Adding hip z custom transmission

File: kangaroo_description/urdf/leg/leg.transmission.xacro (robot description, xacro)
@@ -148,4 +148,20 @@
     </transmission>
   </xacro:macro>
+  <xacro:macro name="hip_transmission_yaw" params="side params_ns:=/hip_z_params" >
+    <transmission name="leg_${side}_transmission_yaw">
+      <type>kangaroo_transmissions/HipZCustomTransmission</type>
+      <actuator name="leg_${side}_1_motor" >
+      </actuator>
+      <joint name="leg_${side}_1_joint">
+        <side> ${side} </side>
+        <param_ns> ${params_ns} </param_ns>
+        <offset> 0.0 </offset>
+        <hardwareInterface>hardware_interface/PositionJointInterface</hardwareInterface>
+        <hardwareInterface>hardware_interface/EffortJointInterface</hardwareInterface>
+        <hardwareInterface>hardware_interface/JointStateInterface</hardwareInterface>
+      </joint>
+    </transmission>
+  </xacro:macro>
+<!--
   <xacro:macro name="hip_transmission_yaw" params="side number reduction">
     <transmission name="leg_${side}_transmission_yaw">
@@ -160,3 +176,4 @@
     </transmission>
   </xacro:macro>
+-->
 </robot>

File: kangaroo_description/urdf/leg/leg.urdf.xacro (robot description, xacro)
@@ -211,5 +211,5 @@
     <!-- Load corresponding transmission info -->
     <xacro:unless value="${simulation}">
-      <xacro:hip_transmission_yaw side="${side}" number="1" reduction="1.0" />
+      <xacro:hip_transmission_yaw side="${side}" params_ns="/hip_z_params" />
       <xacro:hip_transmission_roll_pitch side="${side}" roll_joint="3" pitch_joint="2" />
       <xacro:kangaroo_leg_length_actuator_transmission side="${side}" number1="4" number2="5" params_ns="/leg_params" />

Commit message: remove commented transmission

File: kangaroo_description/urdf/leg/leg.transmission.xacro (robot description, xacro)
@@ -163,17 +163,3 @@
     </transmission>
   </xacro:macro>
-<!--
-  <xacro:macro name="hip_transmission_yaw" params="side number reduction">
-    <transmission name="leg_${side}_transmission_yaw">
-      <type>transmission_interface/SimpleTransmission</type>
-      <actuator name="leg_${side}_${number}_motor" >
-        <mechanicalReduction>${reduction}</mechanicalReduction>
-      </actuator>
-      <joint name="leg_${side}_${number}_joint">
-        <hardwareInterface>hardware_interface/PositionJointInterface</hardwareInterface>
-        <hardwareInterface>hardware_interface/EffortJointInterface</hardwareInterface>
-      </joint>
-    </transmission>
-  </xacro:macro>
--->
 </robot>

Commit message: added the leg state transmission

File: kangaroo_description/urdf/leg/leg.transmission.xacro (robot description, xacro)
@@ -94,4 +94,19 @@
         <hardwareInterface>hardware_interface/PositionJointInterface</hardwareInterface>
         <hardwareInterface>hardware_interface/EffortJointInterface</hardwareInterface>
+        <hardwareInterface>hardware_interface/JointStateInterface</hardwareInterface>
+      </joint>
+    </transmission>
+    <transmission name="leg_${side}_leg_state_trans">
+      <type>kangaroo_transmissions/LegStateCustomTransmission</type>
+      <actuator name="leg_${side}_length_motor" >
+      </actuator>
+      <joint name="leg_${side}_knee_joint">
+        <joint_type> knee </joint_type>
+        <param_ns> ${params_ns} </param_ns>
+        <hardwareInterface>hardware_interface/JointStateInterface</hardwareInterface>
+      </joint>
+      <joint name="leg_${side}_femur_joint">
+        <joint_type> femur </joint_type>
+        <param_ns> ${params_ns} </param_ns>
         <hardwareInterface>hardware_interface/JointStateInterface</hardwareInterface>
       </joint>

Commit message: Test hip-z on actual robot

File: kangaroo_description/urdf/leg/leg.transmission.xacro (robot description, xacro)
@@ -81,10 +81,12 @@
     </transmission>
   </xacro:macro>
-  <xacro:macro name="hip_transmission_yaw" params="side">
+  <xacro:macro name="hip_transmission_yaw" params="side offset initial_position:=0.0">
     <joint name="leg_${side}_1_joint">
       <command_interface name="position"/>
       <command_interface name="velocity"/>
       <command_interface name="effort"/>
-      <state_interface name="position"/>
+      <state_interface name="position">
+          <param name="initial_value">${initial_position}</param>
+      </state_interface>
       <state_interface name="velocity"/>
       <state_interface name="effort"/>
@@ -92,7 +94,7 @@
     <transmission name="leg_${side}_yaw_transmission">
       <plugin>kangaroo_transmissions/HipZCustomTransmission</plugin>
-      <actuator name="leg_${side}_1_motor" role="actuator_yaw"/>
+      <actuator name="leg_${side}_1_actuator" role="actuator_yaw"/>
       <joint name="leg_${side}_1_joint" role="joint_yaw">
-        <offset>0.0</offset>
+        <offset>${offset}</offset>
       </joint>
       <param name="leg_side">${side}</param>

File: kangaroo_description/urdf/leg/ros2_control.urdf.xacro (robot description, xacro)
@@ -17,8 +17,8 @@
   <xacro:include filename="$(find kangaroo_description)/ros2_control/passive_joint.ros2_control.xacro" />
   <xacro:include filename="$(find kangaroo_description)/ros2_control/transmissions.urdf.xacro" />
-  <xacro:include filename="$(find kangaroo_description)/urdf/leg/leg.transmissions.xacro" />
+  <xacro:include filename="$(find kangaroo_description)/urdf/leg/leg.transmission.xacro" />
   <!-- MACRO DEFINITION-->
   <xacro:macro name="leg_ros2_control" params="side">
-        <xacro:joint_ros2control name="leg_${side}_1" initial_position="0.0" />
+        <!-- <xacro:joint_ros2control name="leg_${side}_1" initial_position="0.0" /> -->
         <xacro:joint_ros2control name="leg_${side}_2" initial_position="0.05" />
         <xacro:joint_ros2control name="leg_${side}_3" initial_position="0.0" />
@@ -26,9 +26,9 @@
         <xacro:joint_ros2control name="leg_${side}_4" initial_position="-0.07" />
         <xacro:joint_ros2control name="leg_${side}_5" initial_position="0.0" />
-        <xacro:passive_joint_ros2control name="leg_${side}_femur" initial_position="0.9" />
-        <xacro:passive_joint_ros2control name="leg_${side}_knee" initial_position="1.8" />
+        <!--xacro:passive_joint_ros2control name="leg_${side}_femur" initial_position="0.9" />
+        <xacro:passive_joint_ros2control name="leg_${side}_knee" initial_position="1.8" /-->
         <xacro:if value="${sim_type == 'no-simulation'}" >
           <!--xacro:simple_transmission name="leg_${side}_1" reduction="1.0" offset_value="${leg_1_joint_offset}" /-->
-          <xacro:hip_transmission_yaw side="${side}" />
+          <xacro:hip_transmission_yaw side="${side}" offset="${leg_1_joint_offset}" initial_position="0.0" />
           <xacro:simple_transmission name="leg_${side}_2" reduction="1.0" offset_value="${leg_2_joint_offset}" />
           <xacro:simple_transmission name="leg_${side}_3" reduction="1.0" offset_value="${leg_3_joint_offset}" />
