Commit message: Update the URDF configuration with limits w.r.t to kangaroo_leg_specifics

File: kangaroo_description/urdf/leg/leg.urdf.xacro (robot description, xacro)
@@ -11,8 +11,8 @@
   <xacro:property name="leg_3_min_pos"   value="${27.0 *deg_to_rad}" />
   <xacro:property name="leg_3_max_pos"   value="${-27.0 *deg_to_rad}" />
-  <xacro:property name="leg_4_min_pos"   value="${0.0 *deg_to_rad}" />
-  <xacro:property name="leg_4_max_pos"   value="${60.0 *deg_to_rad}" />
-  <xacro:property name="leg_5_min_pos"   value="${0.0 *deg_to_rad}" />
-  <xacro:property name="leg_5_max_pos"   value="${120.0 *deg_to_rad}" />
+  <xacro:property name="leg_4_min_pos"   value="${10.0 *deg_to_rad}" />
+  <xacro:property name="leg_4_max_pos"   value="${70.0 *deg_to_rad}" />
+  <xacro:property name="leg_5_min_pos"   value="${20.0 *deg_to_rad}" />
+  <xacro:property name="leg_5_max_pos"   value="${140.0 *deg_to_rad}" />
   <xacro:property name="leg_6_min_pos"   value="${-42.5 *deg_to_rad}" />
   <xacro:property name="leg_6_max_pos"   value="${42.5 *deg_to_rad}" />
@@ -133,5 +133,5 @@
     </link>
     <joint name="leg_${side}_4_joint" type="revolute">
-      <origin xyz="0 ${reflect * 0.0669} -0.09" rpy="0 0 0" />
+      <origin xyz="0 ${reflect * 0.0669} -0.09" rpy="0 ${-10.0 * deg_to_rad} 0" />
       <parent link="leg_${side}_3_link" />
       <child link="leg_${side}_4_link" />
@@ -163,5 +163,5 @@
     </link>
     <joint name="leg_${side}_5_joint" type="revolute">
-      <origin xyz="0.37413 0 -0.066509" rpy="0 0 0" />
+      <origin xyz="0.37413 0 -0.066509" rpy="0 ${20.0 * deg_to_rad} 0" />
       <parent link="leg_${side}_4_link" />
       <child link="leg_${side}_5_link" />

Commit message: Invert the min and max joint values of the leg_3 joint

File: kangaroo_description/urdf/leg/leg.urdf.xacro (robot description, xacro)
@@ -9,6 +9,6 @@
   <xacro:property name="leg_2_min_pos"   value="${-42.5 *deg_to_rad}" />
   <xacro:property name="leg_2_max_pos"   value="${42.5 *deg_to_rad}" />
-  <xacro:property name="leg_3_min_pos"   value="${27.0 *deg_to_rad}" />
-  <xacro:property name="leg_3_max_pos"   value="${-27.0 *deg_to_rad}" />
+  <xacro:property name="leg_3_min_pos"   value="${-27.0 *deg_to_rad}" />
+  <xacro:property name="leg_3_max_pos"   value="${27.0 *deg_to_rad}" />
   <xacro:property name="leg_4_min_pos"   value="${10.0 *deg_to_rad}" />
   <xacro:property name="leg_4_max_pos"   value="${70.0 *deg_to_rad}" />
@@ -106,5 +106,5 @@
       <parent link="leg_${side}_2_link" />
       <child link="leg_${side}_3_link" />
-      <axis xyz="1 0 0" />
+      <axis xyz="-1 0 0" />
       <limit lower="${leg_3_min_pos}" upper="${leg_3_max_pos}" effort="0" velocity="0" />
     </joint>

Commit message: add the pending gazebo reference info

File: kangaroo_description/urdf/leg/leg.urdf.xacro (robot description, xacro)
@@ -240,4 +240,24 @@
      <mu2>0.9</mu2>
    </gazebo>
+   <gazebo reference="leg_${side}_3_link">
+     <mu1>0.9</mu1>
+     <mu2>0.9</mu2>
+   </gazebo>
+   <gazebo reference="leg_${side}_4_link">
+     <mu1>0.9</mu1>
+     <mu2>0.9</mu2>
+   </gazebo>
+   <gazebo reference="leg_${side}_5_link">
+     <mu1>0.9</mu1>
+     <mu2>0.9</mu2>
+   </gazebo>
+   <gazebo reference="leg_${side}_6_link">
+     <mu1>0.9</mu1>
+     <mu2>0.9</mu2>
+   </gazebo>
+   <gazebo reference="leg_${side}_7_link">
+     <mu1>0.9</mu1>
+     <mu2>0.9</mu2>
+   </gazebo>
    <gazebo reference="leg_${side}_1_joint">
       <implicitSpringDamper>1</implicitSpringDamper>
@@ -246,9 +266,39 @@
       <implicitSpringDamper>1</implicitSpringDamper>
    </gazebo>
+   <gazebo reference="leg_${side}_3_joint">
+      <implicitSpringDamper>1</implicitSpringDamper>
+   </gazebo>
+   <gazebo reference="leg_${side}_4_joint">
+      <implicitSpringDamper>1</implicitSpringDamper>
+   </gazebo>
+   <gazebo reference="leg_${side}_5_joint">
+      <implicitSpringDamper>1</implicitSpringDamper>
+   </gazebo>
+   <gazebo reference="leg_${side}_6_joint">
+      <implicitSpringDamper>1</implicitSpringDamper>
+   </gazebo>
+   <gazebo reference="leg_${side}_7_joint">
+      <implicitSpringDamper>1</implicitSpringDamper>
+   </gazebo>
   <gazebo reference="leg_${side}_1_link">
+    <material>Gazebo/FlatWhite</material>
+  </gazebo>
+  <gazebo reference="leg_${side}_2_link">
+    <material>Gazebo/FlatWhite</material>
+  </gazebo>
+  <gazebo reference="leg_${side}_3_link">
+    <material>Gazebo/FlatWhite</material>
+  </gazebo>
+  <gazebo reference="leg_${side}_4_link">
     <material>Gazebo/FlatBlack</material>
   </gazebo>
-  <gazebo reference="leg_${side}_2_link">
+  <gazebo reference="leg_${side}_5_link">
     <material>Gazebo/FlatBlack</material>
+  </gazebo>
+  <gazebo reference="leg_${side}_6_link">
+    <material>Gazebo/FlatWhite</material>
+  </gazebo>
+  <gazebo reference="leg_${side}_7_link">
+    <material>Gazebo/FlatWhite</material>
   </gazebo>
   </xacro:macro>

Commit message: added the missing info of the effort and velocity limits in the URDF

File: kangaroo_description/urdf/leg/leg.urdf.xacro (robot description, xacro)
@@ -47,5 +47,5 @@
       <child link="leg_${side}_1_link" />
       <axis xyz="0 0 1" />
-      <limit lower="${leg_1_min_pos}" upper="${leg_1_max_pos}" effort="0" velocity="0" />
+      <limit lower="${leg_1_min_pos}" upper="${leg_1_max_pos}" effort="100" velocity="3.87" />
     </joint>
     <link name="leg_${side}_2_link">
@@ -77,5 +77,5 @@
       <child link="leg_${side}_2_link" />
       <axis xyz="0 1 0" />
-      <limit lower="${leg_2_min_pos}" upper="${leg_2_max_pos}" effort="0" velocity="0" />
+      <limit lower="${leg_2_min_pos}" upper="${leg_2_max_pos}" effort="100" velocity="3.87" />
     </joint>
     <link name="leg_${side}_3_link">
@@ -107,5 +107,5 @@
       <child link="leg_${side}_3_link" />
       <axis xyz="-1 0 0" />
-      <limit lower="${leg_3_min_pos}" upper="${leg_3_max_pos}" effort="0" velocity="0" />
+      <limit lower="${leg_3_min_pos}" upper="${leg_3_max_pos}" effort="100" velocity="3.87" />
     </joint>
     <link name="leg_${side}_4_link">
@@ -137,5 +137,5 @@
       <child link="leg_${side}_4_link" />
       <axis xyz="0 1 0" />
-      <limit lower="${leg_4_min_pos}" upper="${leg_4_max_pos}" effort="0" velocity="0" />
+      <limit lower="${leg_4_min_pos}" upper="${leg_4_max_pos}" effort="100" velocity="3.87" />
     </joint>
     <link name="leg_${side}_5_link">
@@ -167,5 +167,5 @@
       <child link="leg_${side}_5_link" />
       <axis xyz="0 -1 0" />
-      <limit lower="${leg_5_min_pos}" upper="${leg_5_max_pos}" effort="0" velocity="0" />
+      <limit lower="${leg_5_min_pos}" upper="${leg_5_max_pos}" effort="100" velocity="3.87" />
     </joint>
     <link name="leg_${side}_6_link">
@@ -197,5 +197,5 @@
       <child link="leg_${side}_6_link" />
       <axis xyz="0 1 0" />
-      <limit lower="${leg_6_min_pos}" upper="${leg_6_max_pos}" effort="0" velocity="0" />
+      <limit lower="${leg_6_min_pos}" upper="${leg_6_max_pos}" effort="100" velocity="3.87" />
     </joint>
     <link name="leg_${side}_7_link">
@@ -227,5 +227,5 @@
       <child link="leg_${side}_7_link" />
       <axis xyz="-0.93969 0 0.34202" />
-      <limit lower="${leg_7_min_pos}" upper="${leg_7_max_pos}" effort="0" velocity="0" />
+      <limit lower="${leg_7_min_pos}" upper="${leg_7_max_pos}" effort="100" velocity="3.87" />
     </joint>
 <!--

Commit message: change the limits of the joints of hip yaw

File: kangaroo_description/urdf/leg/leg.urdf.xacro (robot description, xacro)
@@ -47,5 +47,10 @@
       <child link="leg_${side}_1_link" />
       <axis xyz="0 0 1" />
-      <limit lower="${leg_1_min_pos}" upper="${leg_1_max_pos}" effort="100" velocity="3.87" />
+      <xacro:if value="${reflect == 1}">
+        <limit lower="${leg_1_min_pos}" upper="${leg_1_max_pos}" effort="100" velocity="3.87" />
+      </xacro:if>
+      <xacro:if value="${reflect == -1}">
+        <limit lower="${reflect * leg_1_max_pos}" upper="${reflect * leg_1_min_pos}" effort="100" velocity="3.87" />
+      </xacro:if>
     </joint>
     <link name="leg_${side}_2_link">

Commit message: Updated the leg xacro to use the transmission according to the arg simulation

File: kangaroo_description/urdf/leg/leg.urdf.xacro (robot description, xacro)
@@ -19,5 +19,7 @@
   <xacro:property name="leg_7_min_pos"   value="${-27.0 *deg_to_rad}" />
   <xacro:property name="leg_7_max_pos"   value="${27.0 *deg_to_rad}" />
-  <xacro:macro name="kangaroo_leg" params="side reflect parent *origin">
+  <xacro:property name="leg_min_length"   value="0.131973" />
+  <xacro:property name="leg_max_length"   value="0.71416639" />
+  <xacro:macro name="kangaroo_leg" params="side reflect parent *origin simulation:=false">
     <link name="leg_${side}_1_link">
       <inertial>
@@ -234,8 +236,13 @@
       <limit lower="${leg_7_min_pos}" upper="${leg_7_max_pos}" effort="100" velocity="3.87" />
     </joint>
-<!--
-    <xacro:kangaroo_leg_length_actuator_transmission side="${side}" number1="1" number2="2" femur="0.380" intersection_crank_axis="${0.360*5.8/9.2}" fbl11_long="0.360" fbl11_short="0.095" fbl21_fixed="0.1265" fbl21_long="0.099" fbl21_short="${0.1265/2.875}" crank_slider_long="0.120" crank_slider_short="0.090" crank_slider_axis_angle="{-5.0*deg_to_rad}" shin_offset_angle="{-5.0*deg_to_rad}" connection_fbl_offset_angle="{5.0*deg_to_rad}" knee_angle_min ="{40*deg_to_rad}" knee_angle_max="{160*deg_to_rad}" />
-    -->
-    <xacro:kangaroo_lower_body_simple_simulation_transmission side="${side}"/>
+    <xacro:unless value="${simulation}">
+      <xacro:hip_transmission_yaw side="${side}" number="1" reduction="1.0" />
+      <xacro:hip_transmission_roll_pitch side="${side}" roll_joint="3" pitch_joint="2" />
+      <xacro:kangaroo_leg_length_actuator_transmission side="${side}" number1="4" number2="5" leg_min_length="${leg_min_length}" leg_max_length="${leg_max_length}" femur="0.380" intersection_crank_axis="0.155693813961639" fbl11_long="0.404273" fbl11_short="0.090" fbl21_fixed="0.115" fbl21_long="0.090" fbl21_short="0.040" crank_slider_long="0.215" crank_slider_short="0.090" crank_slider_axis_angle="${-15.65*deg_to_rad}" shin_offset_angle="${0.0*deg_to_rad}" connection_fbl_offset_angle="${-45.0*deg_to_rad}" shin_fbl11_offset_angle="${-15.00*deg_to_rad}" knee_angle_min ="${leg_5_min_pos - 5.0 *deg_to_rad}" knee_angle_max="${leg_5_max_pos + 5.0 *deg_to_rad}" femur_angle_min="${leg_4_min_pos}" femur_angle_max="${leg_4_max_pos}" />
+      <xacro:kangaroo_ankle_transmission side="${side}" roll_joint="7" pitch_joint="6" read_actuator="leg_${side}_length_motor" />
+    </xacro:unless>
+    <xacro:if value="${simulation}">
+      <xacro:kangaroo_lower_body_simple_simulation_transmission side="${side}"/>
+    </xacro:if>
    <gazebo reference="leg_${side}_1_link">
      <mu1>0.9</mu1>

Commit message: Update prismatic leg model to avoid change rotation of the joint frame

File: kangaroo_description/urdf/leg/leg.urdf.xacro (robot description, xacro)
@@ -178,5 +178,5 @@
 			 <link name="leg_${side}_4_link">
 		    <inertial>
-		      <origin rpy="0 0 0" xyz="0.0 0.0 ${leg_min_length/2.0}"/>
+		      <origin rpy="0 0 0" xyz="0.0 0.0 ${-leg_min_length/2.0}"/>
 					<!-- TODO: update inertia and mass -->
 		      <mass value="3.57408268817521" />
@@ -185,5 +185,5 @@
 		    </inertial>
 		    <visual>
-		      <origin rpy="0 0 0" xyz="0 0 ${leg_min_length/2.0}"/>
+		      <origin rpy="0 0 0" xyz="0 0 ${-leg_min_length/2.0}"/>
 		      <geometry>
 		        <cylinder length="${leg_min_length}" radius="0.02"/>
@@ -192,5 +192,5 @@
 		    </visual>
 		    <collision>
-		      <origin rpy="0 0 0" xyz="0 0 ${leg_min_length/2.0}"/>
+		      <origin rpy="0 0 0" xyz="0 0 ${-leg_min_length/2.0}"/>
 		      <geometry>
 		        <cylinder length="${leg_min_length}" radius="0.02"/>
@@ -199,12 +199,12 @@
 		  </link>
 		  <joint name="leg_${side}_length_fixed_joint" type="fixed">
-		    <origin xyz="0 ${reflect * 0.0669} -0.09" rpy="0 ${180 * deg_to_rad} 0" />
+		    <origin xyz="0 ${reflect * 0.0669} -0.09" rpy="0 0 0" />
 		    <parent link="leg_${side}_3_link" />
 		    <child link="leg_${side}_4_link" />
-		    <axis xyz="0 0 1" />
+		    <axis xyz="0 0 0" />
 		  </joint>
 		  <link name="leg_${side}_5_link">
 		    <inertial>
-		      <origin rpy="0 0 0" xyz="0.0 0.0 ${-leg_min_length}"/>
+		      <origin rpy="0 0 0" xyz="0.0 0.0 ${(leg_max_length - leg_min_length)/2}"/>
 					<!-- TODO: update inertia and mass -->
 		      <mass value="0.87223211672797" />
@@ -213,5 +213,5 @@
 		    </inertial>
 		    <visual>
-		      <origin rpy="0 0 0" xyz="0 0 ${(leg_min_length - leg_max_length)/2}"/>
+		      <origin rpy="0 0 0" xyz="0 0 ${(leg_max_length - leg_min_length)/2}"/>
 		      <geometry>
 		        <cylinder length="${(leg_max_length - leg_min_length)}" radius="0.02"/>
@@ -227,8 +227,8 @@
 		  </link>
 		  <joint name="leg_${side}_5_joint" type="prismatic">
-		   <origin xyz="0.0 0.0 ${leg_min_length}"  rpy="0.0 0.0 0.0"/>
+		   <origin xyz="0.0 0.0 ${-leg_min_length}"  rpy="0.0 0.0 0.0"/>
 		    <parent link="leg_${side}_4_link" />
 		    <child link="leg_${side}_5_link" />
-		    <axis xyz="0 0 1" />
+		    <axis xyz="0 0 -1" />
 		    <limit lower="0" upper="${leg_max_length - leg_min_length}" effort="100" velocity="10" /> <!-- TODO: update effort and velocity -->
 		  </joint>
@@ -241,5 +241,5 @@
     <xacro:if value="${type=='prismatic'}" >
       <xacro:kangaroo_ankle side="${side}" parent="leg_${side}_5_link" reflect="${reflect}" roll_joint="7" pitch_joint="6" read_actuator="leg_${side}_length_motor">
-        <origin xyz="0. 0 -0." rpy="0 ${180 * deg_to_rad} 0" />
+        <origin xyz="0. 0 -0." rpy="0 0 0" />
       </xacro:kangaroo_ankle>
     </xacro:if>
@@ -281,7 +281,9 @@
       <implicitSpringDamper>1</implicitSpringDamper>
    </gazebo>
-   <gazebo reference="leg_${side}_4_joint">
-      <implicitSpringDamper>1</implicitSpringDamper>
-   </gazebo>
+	 <xacro:unless value="${type=='prismatic'}" >
+		 <gazebo reference="leg_${side}_4_joint">
+		    <implicitSpringDamper>1</implicitSpringDamper>
+		 </gazebo>
+	 </xacro:unless>
    <gazebo reference="leg_${side}_5_joint">
       <implicitSpringDamper>1</implicitSpringDamper>

Commit message: update effort and velocity limit for primsatic model

File: kangaroo_description/urdf/leg/leg.urdf.xacro (robot description, xacro)
@@ -231,5 +231,5 @@
         <child link="leg_${side}_4_link" />
         <axis xyz="0 0 -1" />
-        <limit lower="0" upper="${leg_max_length - leg_min_length}" effort="100" velocity="10" /> <!-- TODO: update effort and velocity -->
+        <limit lower="0" upper="${leg_max_length - leg_min_length}" effort="500" velocity="10" /> <!-- TODO: update effort and velocity -->
       </joint>
     </xacro:if>

Commit message: Remove collision shape of primsatic moving part

File: kangaroo_description/urdf/leg/leg.urdf.xacro (robot description, xacro)
@@ -176,4 +176,5 @@
     </xacro:unless>
     <xacro:if value="${type=='prismatic'}" > <!-- load the model with the leg length prismatic joint-->
+<<<<<<< HEAD
        <link name="leg_${side}_length_fixed_link">
         <inertial>
@@ -191,10 +192,10 @@
           <material name="DarkGrey" />
         </visual>
-        <collision>
+        <!--<collision>
           <origin rpy="0 0 0" xyz="0 0 ${-leg_min_length/2.0}"/>
           <geometry>
             <cylinder length="${leg_min_length}" radius="0.02"/>
           </geometry>
-        </collision>
+        </collision>-->
       </link>
       <joint name="leg_${side}_length_fixed_joint" type="fixed">

Commit message: Fix ankle position with respect to the leg lenght

File: kangaroo_description/urdf/leg/leg.urdf.xacro (robot description, xacro)
@@ -242,5 +242,5 @@
     <xacro:if value="${type=='prismatic'}" >
       <xacro:kangaroo_ankle side="${side}" parent="leg_${side}_4_link" reflect="${reflect}" roll_joint="6" pitch_joint="5" read_actuator="leg_${side}_length_motor">
-        <origin xyz="0 0 0" rpy="0 0 0" />
+        <origin xyz="-0.02 0 0" rpy="0 0 0" />
       </xacro:kangaroo_ankle>
     </xacro:if>

Commit message: Change masses and inertias for prismatic joint

File: kangaroo_description/urdf/leg/leg.urdf.xacro (robot description, xacro)
@@ -177,7 +177,6 @@
         <origin rpy="0 0 0" xyz="0.0 0.0 ${leg_min_length/2.0}"/>
         <!-- TODO: update inertia and mass -->
-        <mass value="0.1"/>
-        <inertia ixx="0.04287677484" ixy="0.00043705397" ixz="0.00078292368"
-                iyy="0.03598906971" iyz="0.00037717694" izz="0.01364791564" />
+        <mass value="1.E-3" />
+        <inertia ixx="1.0E-05" ixy="0.0" ixz="0.0" iyy="1.0E-05" iyz="0.0" izz="1.0E-05" />
       </inertial>
       <visual>
@@ -205,7 +204,6 @@
         <origin rpy="0 0 0" xyz="0.0 0.0 ${(leg_max_length - leg_min_length)/2}"/>
         <!-- TODO: update inertia and mass -->
-        <mass value="3.57408268817521" />
-        <inertia ixx="0.00247170768644724" ixy="2.87874888621229E-05" ixz="0.00247469186737281"
-          iyy="0.0126050262407564" iyz="1.01404330133204E-05" izz="0.0116319632922522" />
+        <mass value="1.E-3" />
+        <inertia ixx="1.0E-05" ixy="0.0" ixz="0.0" iyy="1.0E-05" iyz="0.0" izz="1.0E-05" />
       </inertial>
       <visual>

Commit message: fix COM displaced in y axis

File: kangaroo_description/urdf/leg/leg.urdf.xacro (robot description, xacro)
@@ -21,5 +21,5 @@
     <link name="leg_${side}_1_link">
       <inertial>
-        <origin xyz="0.0461079574284527 -0.000826631128234001 0.00897630312181676" rpy="0 0 0" />
+        <origin xyz="0.0461079574284527 ${reflect * -0.000826631128234001} 0.00897630312181676" rpy="0 0 0" />
         <mass value="2.49954419149183" />
         <inertia ixx="0.00151181747940305" ixy="${reflect * 8.83298140320242E-06}" ixz="${reflect * 2.17752660615735E-05}" iyy="0.00154876023440654" iyz="${reflect * -1.94449871986378E-05}" izz="0.00136106613590181" />
@@ -57,6 +57,6 @@
         <origin xyz="-0.00299642516878475 -0.000101293190038279 6.76277450706309E-10" rpy="0 0 0" />
         <mass value="0.0907287903783648" />
-        <inertia ixx="6.10402208807908E-06" ixy="${reflect * 3.54403077254796E-08}" ixz="${reflect * -3.0910293306339E-13}"
-          iyy="3.90470919341026E-05" iyz="${reflect * -1.14069181428674E-12}" izz="3.64238433670963E-05" />
+        <inertia ixx="6.10402208807908E-06" ixy="3.54403077254796E-08" ixz="-3.0910293306339E-13"
+          iyy="3.90470919341026E-05" iyz="-1.14069181428674E-12" izz="3.64238433670963E-05" />
       </inertial>
       <visual>
@@ -85,5 +85,5 @@
     <link name="leg_${side}_3_link">
       <inertial>
-        <origin xyz="-0.042791492019428 0.0477271400490046 -0.0411219993940296" rpy="0 0 0" />
+        <origin xyz="-0.042791492019428 ${reflect * 0.0477271400490046} -0.0411219993940296" rpy="0 0 0" />
         <mass value="3.66987205802361" />
         <inertia ixx="0.00226579365890287" ixy="${reflect * 0.000186528466622377}" ixz="${reflect * -9.4464170720752E-05}"

Commit message: Add collision meshes for knee_link and femur_link

File: kangaroo_description/urdf/leg/leg.urdf.xacro (robot description, xacro)
@@ -140,4 +140,10 @@
         </material>
       </visual>
+      <collision>
+        <origin xyz="0 0 0" rpy="0 0 0" />
+        <geometry>
+          <mesh filename="package://kangaroo_description/meshes/leg_4_link.stl"/>
+        </geometry>
+      </collision>
     </link>
     <link name="leg_${side}_knee_link">
@@ -156,4 +162,10 @@
         </material>
       </visual>
+      <collision>
+        <origin xyz="0 0 0" rpy="0 0 0" />
+        <geometry>
+          <mesh filename="package://kangaroo_description/meshes/leg_5_collision_link.stl"/>
+        </geometry>
+      </collision>
     </link>
     <link name="leg_${side}_length_link">

Commit message: Remove tibia link nad mimic joint

File: kangaroo_description/urdf/leg/leg.urdf.xacro (robot description, xacro)
@@ -147,5 +147,5 @@
       </collision>
     </link>
-    <link name="leg_${side}_knee_link">
+    <!-- <link name="leg_${side}_knee_link">
       <inertial>
         <origin xyz="-0.158662729273678 -8.28192764317226E-05 -0.0337468261967321" rpy="0 0 0" />
@@ -168,5 +168,5 @@
         </geometry>
       </collision>
-    </link>
+    </link> -->
     <link name="leg_${side}_length_link">
       <inertial>
@@ -198,5 +198,5 @@
       <mimic joint="leg_${side}_length_joint" multiplier="1.69435" offset="-0.096145"/>
     </joint>
-    <joint name="leg_${side}_knee_joint" type="revolute">
+    <!-- <joint name="leg_${side}_knee_joint" type="revolute">
       <origin xyz="0.37413 0 -0.066509" rpy="0 ${20.0 * deg_to_rad} 0" />
       <parent link="leg_${side}_femur_link" />
@@ -205,5 +205,5 @@
       <limit lower="${leg_knee_min_pos}" upper="${leg_knee_max_pos}" effort="100" velocity="3.87" />
       <mimic joint="leg_${side}_length_joint" multiplier="3.38877" offset="-0.19229"/>
-    </joint>
+    </joint> -->
     <xacro:kangaroo_ankle side="${side}" parent="leg_${side}_length_link" reflect="${reflect}" roll_joint="5" pitch_joint="4" read_actuator="leg_${side}_length_motor">
       <origin xyz="0.0 0 0.0" rpy="0 ${180 *deg_to_rad} 0" />

Commit message: Change negative axis of rotation

File: kangaroo_description/urdf/leg/leg.urdf.xacro (robot description, xacro)
@@ -122,5 +122,5 @@
       <parent link="leg_${side}_2_link" />
       <child link="leg_${side}_3_link" />
-      <axis xyz="-1 0 0" />
+      <axis xyz="1 0 0" />
       <limit lower="${leg_3_min_pos}" upper="${leg_3_max_pos}" effort="100" velocity="3.87" />
     </joint>

Commit message: Uncomment femur meshes for visualization

File: kangaroo_description/urdf/leg/leg.urdf.xacro (robot description, xacro)
@@ -147,5 +147,5 @@
       </collision>
     </link>
-    <!-- <link name="leg_${side}_knee_link">
+    <link name="leg_${side}_knee_link">
       <inertial>
         <origin xyz="-0.158662729273678 -8.28192764317226E-05 -0.0337468261967321" rpy="0 0 0" />
@@ -168,5 +168,5 @@
         </geometry>
       </collision>
-    </link> -->
+    </link>
     <link name="leg_${side}_length_link">
       <inertial>
@@ -198,5 +198,5 @@
       <mimic joint="leg_${side}_length_joint" multiplier="1.69435" offset="-0.096145"/>
     </joint>
-    <!-- <joint name="leg_${side}_knee_joint" type="revolute">
+    <joint name="leg_${side}_knee_joint" type="revolute">
       <origin xyz="0.37413 0 -0.066509" rpy="0 ${20.0 * deg_to_rad} 0" />
       <parent link="leg_${side}_femur_link" />
@@ -205,5 +205,5 @@
       <limit lower="${leg_knee_min_pos}" upper="${leg_knee_max_pos}" effort="100" velocity="3.87" />
       <mimic joint="leg_${side}_length_joint" multiplier="3.38877" offset="-0.19229"/>
-    </joint> -->
+    </joint>
     <xacro:kangaroo_ankle side="${side}" parent="leg_${side}_length_link" reflect="${reflect}" roll_joint="5" pitch_joint="4" read_actuator="leg_${side}_length_motor">
       <origin xyz="0.0 0 0.0" rpy="0 ${180 *deg_to_rad} 0" />
