Commit message: Added frame located at the tip of the knee link. Needs to be validated against CAD!

File: kangaroo_description/urdf/leg/leg.urdf.xacro (robot description, xacro)
@@ -206,4 +206,11 @@
       <mimic joint="leg_${side}_length_joint" multiplier="3.38877" offset="-0.19229"/>
     </joint>
+    <!-- THIS FRAME NEEDS TO BE VALIDATED BY CAD!!! -->
+    <link name="leg_${side}_knee_lower_bearing"/>
+    <joint name="leg_${side}_knee_lower_bearing_joint" type="fixed">
+    	<parent link="leg_${side}_knee_link"/>
+    	<child link="leg_${side}_knee_lower_bearing"/>
+    	<origin rpy="0 0 0" xyz="-0.375 0.0 -0.067"/>
+    </joint>
     <xacro:kangaroo_ankle side="${side}" parent="leg_${side}_length_link" reflect="${reflect}" roll_joint="5" pitch_joint="4" read_actuator="leg_${side}_length_motor">
       <origin xyz="0.0 0 0.0" rpy="0 ${180 *deg_to_rad} 0" />

Commit message: updated frames according to data sent to Pau

File: kangaroo_description/urdf/leg/leg.urdf.xacro (robot description, xacro)
@@ -211,9 +211,15 @@
     </joint>
     <!-- THIS FRAME NEEDS TO BE VALIDATED BY CAD!!! -->
+    <link name="leg_${side}_knee_straight"/>
+    <joint name="leg_${side}_knee_straight_joint" type="fixed">
+    	<parent link="leg_${side}_knee_link"/>
+    	<child link="leg_${side}_knee_straight"/>
+    	<origin rpy="0 ${-10.0 * deg_to_rad} 0" xyz="0 0 0"/>
+    </joint>
     <link name="leg_${side}_knee_lower_bearing"/>
     <joint name="leg_${side}_knee_lower_bearing_joint" type="fixed">
-    	<parent link="leg_${side}_knee_link"/>
+    	<parent link="leg_${side}_knee_straight"/>
     	<child link="leg_${side}_knee_lower_bearing"/>
-    	<origin rpy="0 0 0" xyz="-0.375 0.0 -0.067"/>
+    	<origin rpy="0 0 0" xyz="-0.38 0.0 0.0"/>
     </joint>
     <xacro:kangaroo_ankle side="${side}" parent="leg_${side}_length_link" reflect="${reflect}" roll_joint="5" pitch_joint="4" read_actuator="leg_${side}_length_motor">

Commit message: added clenaed leg_5_link mesh

File: kangaroo_description/urdf/leg/leg.urdf.xacro (robot description, xacro)
@@ -156,5 +156,5 @@
         <origin xyz="0 0 0" rpy="0 0 0" />
         <geometry>
-          <mesh filename="package://kangaroo_description/meshes/leg_5_link.stl" />
+          <mesh filename="package://kangaroo_description/meshes/leg_5_link_v2.stl" />
         </geometry>
         <material name="">

Commit message: using link5 collision mesh for visualization

File: kangaroo_description/urdf/leg/leg.urdf.xacro (robot description, xacro)
@@ -156,5 +156,5 @@
         <origin xyz="0 0 0" rpy="0 0 0" />
         <geometry>
-          <mesh filename="package://kangaroo_description/meshes/leg_5_link_v2.stl" />
+          <mesh filename="package://kangaroo_description/meshes/leg_5_collision_link.stl" />
         </geometry>
         <material name="">

Commit message: added closed kinematic chain joint for gazebo when use_mimic is false

File: kangaroo_description/urdf/leg/leg.urdf.xacro (robot description, xacro)
@@ -299,4 +299,16 @@
    	<xacro:mimic_joint_plugin_gazebo name_prefix="" parent_joint="leg_${side}_length_joint" mimic_joint="leg_${side}_femur_joint" has_pid="false" multiplier="1.69435" offset="-0.096145" max_effort="100.0"/>
    </xacro:if>
+   <xacro:unless value="${use_mimic}">
+	   <gazebo reference="">
+		<joint type="revolute" name="leg_${side}_closed_kin_joint">
+	              <pose>0 0 0 0 0 0</pose>
+		      <parent>leg_${side}_knee_link</parent>
+		      <child>leg_${side}_length_link</child>
+		      <axis>
+			<xyz>0 1 0</xyz>
+		      </axis>
+    		</joint>
+	   </gazebo>
+   </xacro:unless>
   </xacro:macro>
 </robot>

Commit message: when using use_mimic true the old masses and inertias are now used

File: kangaroo_description/urdf/leg/leg.urdf.xacro (robot description, xacro)
@@ -128,6 +128,13 @@
       <inertial>
         <origin xyz="0.114702002010089 0.000182856660852354 -0.0143986490691173" rpy="0 0 0" />
+<xacro:if value="${use_mimic}">
         <mass value="0.1" />
         <inertia ixx="1.E-5" ixy="0.0" ixz="0.0" iyy="1.E-5" iyz="0.0" izz="1.E-5" />
+</xacro:if>
+<xacro:unless value="${use_mimic}">
+	<mass value="3.57408268817521" />
+        <inertia ixx="0.00247170768644724" ixy="2.87874888621229E-05" ixz="0.00247469186737281"
+          iyy="0.0126050262407564" iyz="1.01404330133204E-05" izz="0.0116319632922522" />
+</xacro:unless>
       </inertial>
       <visual>
@@ -150,6 +157,13 @@
       <inertial>
         <origin xyz="-0.158662729273678 -8.28192764317226E-05 -0.0337468261967321" rpy="0 0 0" />
+<xacro:if value="${use_mimic}">
         <mass value="0.1" />
         <inertia ixx="1.E-5" ixy="0.0" ixz="0.0" iyy="1.E-5" iyz="0.0" izz="1.E-5" />
+</xacro:if>
+<xacro:unless value="${use_mimic}">
+        <mass value="0.87223211672797" />
+        <inertia ixx="0.000350603269949793" ixy="6.37793331536252E-07" ixz="-0.000461550351107159"
+          iyy="0.00242184402988972" iyz="5.09327556678297E-07" izz="0.0022368624903808" />
+</xacro:unless>
       </inertial>
       <visual>
@@ -169,9 +183,21 @@
       </collision>
     </link>
+    <!-- We approximate the virtual length link with a small cylinder mass and inertia -->
+    <xacro:property name="m"   value="0.1" /> <!-- mass -->
+    <xacro:property name="r"   value="0.01" /> <!-- radius -->
+    <xacro:property name="h"   value="0.1" /> <!-- height -->
     <link name="leg_${side}_length_link">
       <inertial>
+<xacro:if value="${use_mimic}">
         <origin rpy="0 0 0" xyz="0.0 0.0 -0.2"/>
         <mass value="6.0" />
         <inertia ixx="0.05" ixy="0.0" ixz="0.0" iyy="0.05" iyz="0.0" izz="0.016875" />
+</xacro:if>
+<xacro:unless value="${use_mimic}">
+        <origin rpy="0 0 0" xyz="0.0 0.0 0.0"/>
+        <mass value="${m}" />
+        <inertia ixx="${(1./12.)*m*(3.*r*r + h*h)}" ixy="0.0" ixz="0.0" iyy="${(1./12.)*m*(3.*r*r + h*h)}"
+		iyz="0.0" izz="${(1./2.)*m*r*r}" />
+</xacro:unless>
       </inertial>
       <visual>

Commit message: Increase max effort

File: kangaroo_description/urdf/leg/leg.urdf.xacro (robot description, xacro)
@@ -65,8 +65,8 @@
       <axis xyz="0 0 1" />
       <xacro:if value="${reflect == 1}">
-        <limit lower="${leg_1_min_pos}" upper="${leg_1_max_pos}" effort="100" velocity="3.87" />
+        <limit lower="${leg_1_min_pos}" upper="${leg_1_max_pos}" effort="500" velocity="3.87" />
       </xacro:if>
       <xacro:if value="${reflect == -1}">
-        <limit lower="${reflect * leg_1_max_pos}" upper="${reflect * leg_1_min_pos}" effort="100" velocity="3.87" />
+        <limit lower="${reflect * leg_1_max_pos}" upper="${reflect * leg_1_min_pos}" effort="500" velocity="3.87" />
       </xacro:if>
     </joint>
@@ -214,5 +214,5 @@
       <child link="leg_${side}_length_link" />
       <axis xyz="0 0 1" />
-      <limit lower="${leg_min_length}" upper="${leg_max_length}" effort="500" velocity="10" />
+      <limit lower="${leg_min_length}" upper="${leg_max_length}" effort="1000" velocity="10" />
     </joint>
     <joint name="leg_${side}_femur_joint" type="revolute">

Commit message: Increase leg length effort limits

File: kangaroo_description/urdf/leg/leg.urdf.xacro (robot description, xacro)
@@ -214,5 +214,5 @@
       <child link="leg_${side}_length_link" />
       <axis xyz="0 0 1" />
-      <limit lower="${leg_min_length}" upper="${leg_max_length}" effort="1000" velocity="10" />
+      <limit lower="${leg_min_length}" upper="${leg_max_length}" effort="1500" velocity="10" />
     </joint>
     <joint name="leg_${side}_femur_joint" type="revolute">

Commit message: reduce broadcaster update rate and uncomment the meshes

File: kangaroo_description/urdf/leg/leg.urdf.xacro (robot description, xacro)
@@ -140,9 +140,9 @@
       </inertial>
       <visual>
-        <origin xyz="0 0 0" rpy="0 0 0" />
+        <origin xyz="0 0 0" rpy="0 ${60.0 * deg_to_rad} 0" />
         <geometry>
           <!-- The ballscrews are removed from the meshes for better visualization, but they are
         used for inertia computation etc -->
-          <mesh filename="package://kangaroo_description/meshes/leg/leg_femur_link.stl" />
+          <mesh filename="package://kangaroo_description/meshes/leg/leg_4_collision_link.stl" />
         </geometry>
         <material name="pal/DarkGrey" />
@@ -168,5 +168,5 @@
           iyy="0.00215347079183119" iyz="1.36520012214457E-06" izz="0.000391378760186175" />
       </inertial>
-      <!-- <visual>
+      <visual>
         <origin xyz="0 0 0" rpy="0 0 0" />
         <geometry>
@@ -174,6 +174,6 @@
         </geometry>
         <material name="pal/DarkGrey" />
-      </visual> -->
-      <!-- <xacro:link_collision
+      </visual>
+      <xacro:link_collision
         mujoco="${sim_type in ['mujoco-ros2-control', 'mujoco']}"
         collision_type="${collision_type}"
@@ -186,5 +186,5 @@
             <xacro:origin xyz="-0.0569664873635563 ${reflect * 7.99553099622616e-06} -0.148820781933269" rpy="0 ${30.0 * deg_to_rad} 0" condition="${collision_type == 'capsule'}"/>
           </properties>
-      </xacro:link_collision> -->
+      </xacro:link_collision>
     </link>
     <!-- We approximate the virtual length link with a small cylinder mass and inertia -->

Commit message: Change feet angle

File: kangaroo_description/urdf/leg/leg.urdf.xacro (robot description, xacro)
@@ -254,5 +254,5 @@
       <xacro:kangaroo_detachable_ankle side="${side}" parent="leg_${side}_length_link" reflect="${reflect}"
         roll_joint="5" pitch_joint="4" read_actuator="leg_${side}_length_motor">
-        <origin xyz="0.0 0 0.0" rpy="0 ${200 *deg_to_rad} 0" />
+        <origin xyz="0.0 0 0.0" rpy="0 ${180 *deg_to_rad} 0" />
       </xacro:kangaroo_detachable_ankle>
     </xacro:if>
