Commit message: fix urdf for arm mesh and inertia

File: kangaroo_description/urdf/arm/arm.urdf.xacro (robot description, xacro)
@@ -4,4 +4,5 @@
 <xacro:property name="arm_friction"       value="1.0" />
 <xacro:property name="arm_damping"        value="1.0" />
+s
 <xacro:property name="arm_1_max_velocity"      value="1.95" />
 <xacro:property name="arm_2_max_velocity"      value="1.95" />
@@ -21,34 +22,34 @@
         rpy="0 0 0" />
       <mass
-        value="0" />
-      <inertia
-        ixx="0"
+        value="0.1" />
+      <inertia
+        ixx="0.0000001"
         ixy="0"
         ixz="0"
-        iyy="0"
+        iyy="0.0000001"
         iyz="0"
-        izz="0" />
-    </inertial>
-    <visual>
-      <origin
-        xyz="0 0 0"
-        rpy="0 0 0" />
-      <geometry>
-        <mesh
-          filename="package://kangaroo_arm/meshes/base_link.STL" />
-      </geometry>
-      <material
-        name="">
-        <color
-          rgba="0.75294 0.75294 0.75294 1" />
-      </material>
-    </visual>
-    <collision>
-      <origin
-        xyz="0 0 0"
-        rpy="0 0 0" />
-      <geometry>
-        <mesh
-          filename="package://kangaroo_arm/meshes/base_link.STL" />
+        izz="0.0000001" />
+    </inertial>
+    <visual>
+      <origin
+        xyz="0 0 0"
+        rpy="0 0 0" />
+      <geometry>
+        <mesh
+          filename="package://kangaroo_description/meshes/arm_base_link.stl" />
+      </geometry>
+      <material
+        name="">
+        <color
+          rgba="0.75294 0.75294 0.75294 1" />
+      </material>
+    </visual>
+    <collision>
+      <origin
+        xyz="0 0 0"
+        rpy="0 0 0" />
+      <geometry>
+        <mesh
+          filename="package://kangaroo_description/meshes/arm_base_link.stl" />
       </geometry>
     </collision>

File: kangaroo_description/urdf/base/base.urdf.xacro (robot description, xacro)
@@ -30,5 +30,5 @@
     <origin xyz="0.071 -0.0014 0.02" rpy="${180.0*deg_to_rad} ${0.0*deg_to_rad} ${-90.0*deg_to_rad}"/>
   </xacro:kangaroo_imu>
-    <!-- -->
+<!-- with pelvis DoF -->
 <xacro:if value="${with_pelvis}">
   <xacro:kangaroo_pelvis name="pelvis" parent="base_link" pelvis_1_offset="0" pelvis_2_offset="0">
@@ -38,6 +38,7 @@
   <xacro:kangaroo_torso parent="pelvis_2_link">
     <origin xyz="0 0 0.0061" rpy="0 0 0" />
-  </xacro:kangaroo_torso> <!-- base_link -->
+  </xacro:kangaroo_torso>
 </xacro:if>
+<!-- without pelvis DoF -->
 <xacro:unless value="${with_pelvis}">
   <xacro:include filename="$(find kangaroo_description)/urdf/torso/torso.urdf.xacro" />

Commit message: tested motions on the robot for standing up from ground

File: kangaroo_description/urdf/arm/arm.urdf.xacro (robot description, xacro)
@@ -11,6 +11,6 @@
 <xacro:property name="arm_1_max_effort"   value="43.0" />
 <xacro:property name="arm_2_max_effort"   value="43.0" />
-<xacro:property name="arm_3_max_effort"   value="26" />
-<xacro:property name="arm_4_max_effort"   value="26" />
+<xacro:property name="arm_3_max_effort"   value="43.0" />
+<xacro:property name="arm_4_max_effort"   value="43.0" />
 <xacro:macro name="kangaroo_arm" params="name side reflect parent *origin arm_1_offset arm_2_offset arm_3_offset arm_4_offset">
   <xacro:property name="arm_eps"       value="${0.00 if no_safety_eps else 0.07}"/>

Commit message: Add ef frames for the WBC

File: kangaroo_description/urdf/arm/arm.urdf.xacro (robot description, xacro)
@@ -267,4 +267,10 @@
       velocity="${arm_4_max_velocity}" />
   </joint>
+  <link name="ef_${side}_link"/>
+  <joint name="ef_${side}_joint" type="fixed">
+    <origin xyz="0.45 -0.05 -0.03" rpy="0 0 0" />
+    <parent link="${name}_${side}_4_link" />
+    <child link="ef_${side}_link" />
+  </joint>
 <!-- TRANSMISSIONS -->
     <xacro:arm_simple_transmission name="${name}_${side}" number="1" reduction="1.0" offset_value="${arm_1_offset}"/>

Commit message: Small typo fix

File: kangaroo_description/urdf/arm/arm.urdf.xacro (robot description, xacro)
@@ -4,5 +4,4 @@
 <xacro:property name="arm_friction"       value="1.0" />
 <xacro:property name="arm_damping"        value="1.0" />
-s
 <xacro:property name="arm_1_max_velocity"      value="1.95" />
 <xacro:property name="arm_2_max_velocity"      value="1.95" />
@@ -40,5 +39,4 @@
       </geometry>
       <material name="DarkGrey"/>
-      </material>
     </visual>
     <collision>

Commit message: Setting properly ef frames (hardcoded way prior fix on parent tfs)

File: kangaroo_description/urdf/arm/arm.urdf.xacro (robot description, xacro)
@@ -269,8 +269,13 @@
   <link name="ef_${side}_link"/>
   <joint name="ef_${side}_joint" type="fixed">
-    <origin xyz="0.45 -0.05 -0.03" rpy="0 0 0" />
+      <xacro:if value="${side == 'left'}">
+        <origin xyz="0.415 -0.02 -0.015" rpy="0 0 0"/>
+      </xacro:if>
+      <xacro:if value="${side == 'right'}">
+       <origin xyz="0.415 -0.015 -0.039" rpy="0 0 0"/>
+      </xacro:if>
     <parent link="${name}_${side}_4_link" />
     <child link="ef_${side}_link" />
-  </joint>
+    </joint>
 <!-- TRANSMISSIONS -->
     <xacro:arm_simple_transmission name="${name}_${side}" number="1" reduction="1.0" offset_value="${arm_1_offset}"/>

Commit message: Cleaner way to set ef_frames

File: kangaroo_description/urdf/arm/arm.urdf.xacro (robot description, xacro)
@@ -269,10 +269,5 @@
   <link name="ef_${side}_link"/>
   <joint name="ef_${side}_joint" type="fixed">
-      <xacro:if value="${side == 'left'}">
-        <origin xyz="0.415 -0.02 -0.015" rpy="0 0 0"/>
-      </xacro:if>
-      <xacro:if value="${side == 'right'}">
-       <origin xyz="0.415 -0.015 -0.039" rpy="0 0 0"/>
-      </xacro:if>
+      <origin xyz="0.415 -0.015 ${-0.025 + reflect * 0.015}" rpy="0 0 0" />
     <parent link="${name}_${side}_4_link" />
     <child link="ef_${side}_link" />
