Commit message: updated transmission tags for gripper

File: kangaroo_description/urdf/end_effector/gripper/gripper.transmission.xacro (robot description, xacro)
@@ -14,5 +14,5 @@
 <robot xmlns:xacro="http://ros.org/wiki/xacro">
   <xacro:macro name="pal_pro_gripper_transmission" params="name">
-    <transmission name="${name}_trans">
+    <!-- <transmission name="${name}_trans">
         <plugin>transmission_interface/SimpleTransmission</plugin>
         <actuator name="${name}_actuator" role="actuator1"/>
@@ -20,4 +20,16 @@
             <mechanical_reduction>1</mechanical_reduction>
         </joint>
+    </transmission> -->
+    <transmission name="${name}_trans">
+      <type>transmission_interface/SimpleTransmission</type>
+      <actuator name="${name}_motor" >
+        <mechanicalReduction>1</mechanicalReduction>
+      </actuator>
+      <joint name="${name}_joint">
+        <hardwareInterface>hardware_interface/PositionJointInterface</hardwareInterface>
+        <hardwareInterface>hardware_interface/VelocityJointInterface</hardwareInterface>
+        <hardwareInterface>hardware_interface/EffortJointInterface</hardwareInterface>
+        <hardwareInterface>hardware_interface/JointStateInterface</hardwareInterface>
+      </joint>
     </transmission>
   </xacro:macro>

File: kangaroo_description/urdf/end_effector/gripper/gripper.urdf.xacro (robot description, xacro)
@@ -174,4 +174,6 @@
       <provideFeedback>1</provideFeedback>
     </gazebo>
+    <xacro:include filename="$(find kangaroo_description)/urdf/end_effector/gripper/gripper.ros_control.xacro" />
+    <xacro:ros_control_pal_pro_gripper name="${name}" reduction="1.0" />
   </xacro:macro>
 </robot>
