Commit message: fixed joint limits and directions

File: kangaroo_description/urdf/arm/7dof/7dof_arm.urdf.xacro (robot description, xacro)
@@ -39,9 +39,9 @@
       <parent link="${parent}" />
       <child link="${name}_${side}_5_link" />
-      <axis xyz="0 0 -1" />
-      <xacro:if value="${side == 'left'}">
+      <axis xyz="0 0 1" />
+      <xacro:if value="${side == 'right'}">
         <limit lower="${deg_to_rad * -210}" upper="${deg_to_rad * 90}" effort="${arm_5_max_effort}" velocity="${arm_5_max_velocity}" />
       </xacro:if>
-      <xacro:if value="${side == 'right'}">
+      <xacro:if value="${side == 'left'}">
         <limit lower="${deg_to_rad * -90}" upper="${deg_to_rad * 210}" effort="${arm_5_max_effort}" velocity="${arm_5_max_velocity}" />
       </xacro:if>
@@ -112,5 +112,5 @@
       <parent link="${name}_${side}_6_link" />
       <child link="${name}_${side}_7_link" />
-      <axis xyz="0 0 -1" />
+      <axis xyz="0 0 1" />
       <limit lower="${deg_to_rad * -150}" upper="${deg_to_rad * 150}" effort="${arm_7_max_effort}" velocity="${arm_7_max_velocity}" />
     </joint>

Commit message: updated arm 5 joint limits

File: kangaroo_description/urdf/arm/7dof/7dof_arm.urdf.xacro (robot description, xacro)
@@ -40,10 +40,11 @@
       <child link="${name}_${side}_5_link" />
       <axis xyz="0 0 1" />
-      <xacro:if value="${side == 'right'}">
+      <limit lower="${deg_to_rad * -150}" upper="${deg_to_rad * 150}" effort="${arm_5_max_effort}" velocity="${arm_5_max_velocity}" />
+      <!-- <xacro:if value="${side == 'right'}">
         <limit lower="${deg_to_rad * -210}" upper="${deg_to_rad * 90}" effort="${arm_5_max_effort}" velocity="${arm_5_max_velocity}" />
       </xacro:if>
       <xacro:if value="${side == 'left'}">
         <limit lower="${deg_to_rad * -90}" upper="${deg_to_rad * 210}" effort="${arm_5_max_effort}" velocity="${arm_5_max_velocity}" />
-      </xacro:if>
+      </xacro:if> -->
     </joint>
     <!-- ARM 6 LINK -->

Commit message: Remove comment arm 5 reflection

File: kangaroo_description/urdf/arm/7dof/7dof_arm.urdf.xacro (robot description, xacro)
@@ -41,10 +41,4 @@
       <axis xyz="0 0 1" />
       <limit lower="${deg_to_rad * -150}" upper="${deg_to_rad * 150}" effort="${arm_5_max_effort}" velocity="${arm_5_max_velocity}" />
-      <!-- <xacro:if value="${side == 'right'}">
-        <limit lower="${deg_to_rad * -210}" upper="${deg_to_rad * 90}" effort="${arm_5_max_effort}" velocity="${arm_5_max_velocity}" />
-      </xacro:if>
-      <xacro:if value="${side == 'left'}">
-        <limit lower="${deg_to_rad * -90}" upper="${deg_to_rad * 210}" effort="${arm_5_max_effort}" velocity="${arm_5_max_velocity}" />
-      </xacro:if> -->
     </joint>
     <!-- ARM 6 LINK -->
