Commit message: updated ros2control tags

File: kangaroo_description/ros2_control/joint.ros2_control.xacro (robot description, xacro)
@@ -1,5 +1,5 @@
 <?xml version="1.0" encoding="utf-8"?>
 <robot xmlns:xacro="http://ros.org/wiki/xacro" name="kangaroo">
-    <xacro:macro name="kangaroo_joint_ros2control"
+    <xacro:macro name="joint_ros2control"
         params="name initial_position:=0.0">
         <joint name="${name}_joint">

File: kangaroo_description/ros2_control/passive_joint.ros2_control.xacro (robot description, xacro)
@@ -13,5 +13,5 @@
 -->
 <robot xmlns:xacro="http://ros.org/wiki/xacro">
-  <xacro:macro name="mimic_joint_ros2control" params="name initial_position:=0.0">
+  <xacro:macro name="passive_joint_ros2control" params="name initial_position:=0.0">
     <joint name="${name}_joint">
         <state_interface name="position">

File: kangaroo_description/ros2_control/ros2_control.urdf.xacro (robot description, xacro)
@@ -14,4 +14,5 @@
 <robot xmlns:xacro="http://ros.org/wiki/xacro" name="kangaroo">
   <!-- INCLUDES -->
+  <xacro:include filename="$(find kangaroo_description)/urdf/pelvis/ros2_control.urdf.xacro" />
   <xacro:include filename="$(find kangaroo_description)/urdf/leg/ros2_control.urdf.xacro" />
   <xacro:include filename="$(find kangaroo_description)/urdf/arm/ros2_control.urdf.xacro" />
@@ -26,6 +27,5 @@
       </hardware>
       <xacro:if value="${has_pelvis}">
-        <xacro:kangaroo_joint_ros2control name="pelvis_1" />
-        <xacro:kangaroo_joint_ros2control name="pelvis_2" />
+        <xacro:pelvis_ros2_control />
       </xacro:if>
       <xacro:if value="${legs_type != 'no-leg'}">

File: kangaroo_description/urdf/arm/ros2_control.urdf.xacro (robot description, xacro)
@@ -18,15 +18,15 @@
   <xacro:macro name="arm_ros2_control" params="side arm_type">
       <xacro:if value="${arm_type in ['4dof', '5dof', '7dof']}">
-        <xacro:kangaroo_joint_ros2control name="arm_${side}_1" initial_position="${(-1 if side == 'right' else 1) * 0.24}" />
-        <xacro:kangaroo_joint_ros2control name="arm_${side}_2" initial_position="1.32" />
-        <xacro:kangaroo_joint_ros2control name="arm_${side}_3" initial_position="${(-1 if side == 'right' else 1) * 1.57}" />
-        <xacro:kangaroo_joint_ros2control name="arm_${side}_4" initial_position="0.8" />
+        <xacro:joint_ros2control name="arm_${side}_1" initial_position="${(-1 if side == 'right' else 1) * 0.24}" />
+        <xacro:joint_ros2control name="arm_${side}_2" initial_position="1.32" />
+        <xacro:joint_ros2control name="arm_${side}_3" initial_position="${(-1 if side == 'right' else 1) * 1.57}" />
+        <xacro:joint_ros2control name="arm_${side}_4" initial_position="0.8" />
       </xacro:if>
       <xacro:if value="${arm_type in ['5dof', '7dof']}">
-        <xacro:kangaroo_joint_ros2control name="arm_${side}_5" initial_position="0.0" />
+        <xacro:joint_ros2control name="arm_${side}_5" initial_position="0.0" />
       </xacro:if>
       <xacro:if value="${arm_type in ['7dof']}">
-        <xacro:kangaroo_joint_ros2control name="arm_${side}_6" initial_position="0.0" />
-        <xacro:kangaroo_joint_ros2control name="arm_${side}_7" initial_position="0.0" />
+        <xacro:joint_ros2control name="arm_${side}_6" initial_position="0.0" />
+        <xacro:joint_ros2control name="arm_${side}_7" initial_position="0.0" />
       </xacro:if>
   </xacro:macro>

File: kangaroo_description/urdf/pelvis/ros2_control.urdf.xacro (robot description, xacro)
@@ -15,15 +15,8 @@
   <!-- INCLUDES -->
   <xacro:include filename="$(find kangaroo_description)/ros2_control/joint.ros2_control.xacro" />
-  <xacro:include filename="$(find kangaroo_description)/ros2_control/passive_joint.ros2_control.xacro" />
   <!-- MACRO DEFINITION-->
-  <xacro:macro name="leg_ros2_control" params="side">
-        <xacro:joint_ros2control name="leg_${side}_1" initial_position="0.0" />
-        <xacro:joint_ros2control name="leg_${side}_2" initial_position="0.05" />
-        <xacro:joint_ros2control name="leg_${side}_3" initial_position="0.0" />
-        <xacro:joint_ros2control name="leg_${side}_length" initial_position="0.6" />
-        <xacro:joint_ros2control name="leg_${side}_4" initial_position="-0.07" />
-        <xacro:joint_ros2control name="leg_${side}_5" initial_position="0.0" />
-        <xacro:passive_joint_ros2control name="leg_${side}_femur" initial_position="0.9" />
-        <xacro:passive_joint_ros2control name="leg_${side}_knee" initial_position="1.8" />
+  <xacro:macro name="pelvis_ros2_control" params="">
+        <xacro:joint_ros2control name="pelvis_1" />
+        <xacro:joint_ros2control name="pelvis_2" />
   </xacro:macro>
 </robot>
