Commit message: fixes mismatch

File: kangaroo_description/urdf/end_effector/fake_forearm.urdf.xacro (robot description, xacro)
@@ -27,5 +27,5 @@
       <origin  xyz="0 0 0" rpy="0 0 0" />
         <geometry>
-          <mesh filename="package://kangaroo_description/meshes/arm/arm3_link.STL" />
+          <mesh filename="package://kangaroo_description/meshes/arm/fake_forearm_${side}_link.stl" scale="1 1 1"/>
         </geometry>
       </collision>
