Commit message: improved fixed base logic

File: kangaroo_description/mujoco/mj_tags.xacro (robot description, xacro)
@@ -17,17 +17,45 @@
       <xacro:if value="${legs_type != 'no-leg'}">
         <xacro:if value="${has_pelvis}">
-          <exclude body1="base_link" body2="pelvis_1_link" />
-          <exclude body1="base_link" body2="pelvis_2_link" />
-          <exclude body1="leg_right_1_link" body2="pelvis_2_link" />
-          <exclude body1="leg_left_1_link" body2="pelvis_2_link" />
-          <exclude body1="leg_right_1_link" body2="pelvis_1_link" />
-          <exclude body1="leg_left_1_link" body2="pelvis_1_link" />
-        </xacro:if>
+          <exclude body1="pelvis_base_link" body2="base_link" />
+          <exclude body1="pelvis_base_link" body2="back_handle" />
+          <exclude body1="pelvis_base_link" body2="leg_left_1_link" />
+          <exclude body1="pelvis_base_link" body2="leg_left_2_link" />
+          <exclude body1="pelvis_base_link" body2="leg_right_1_link" />
+          <exclude body1="pelvis_base_link" body2="leg_right_2_link" />
+          <exclude body1="pelvis_1_link" body2="base_link" />
+          <exclude body1="pelvis_1_link" body2="back_handle" />
+          <exclude body1="pelvis_1_link" body2="pelvis_base_link" />
+          <exclude body1="pelvis_1_link" body2="leg_left_1_link" />
+          <exclude body1="pelvis_1_link" body2="leg_left_2_link" />
+          <exclude body1="pelvis_1_link" body2="leg_right_1_link" />
+          <exclude body1="pelvis_1_link" body2="leg_right_2_link" />
+          <exclude body1="pelvis_2_link" body2="base_link" />
+          <exclude body1="pelvis_2_link" body2="back_handle" />
+          <exclude body1="pelvis_2_link" body2="pelvis_base_link" />
+          <exclude body1="pelvis_2_link" body2="pelvis_1_link" />
+          <exclude body1="pelvis_2_link" body2="leg_left_1_link" />
+          <exclude body1="pelvis_2_link" body2="leg_left_2_link" />
+          <exclude body1="pelvis_2_link" body2="leg_right_1_link" />
+          <exclude body1="pelvis_2_link" body2="leg_right_2_link" />
+        </xacro:if>
+        <exclude body1="base_link" body2="back_handle" />
+        <exclude body1="base_link" body2="torso_link" />
         <exclude body1="base_link" body2="leg_left_1_link" />
         <exclude body1="base_link" body2="leg_left_2_link" />
         <exclude body1="base_link" body2="leg_left_3_link" />
+        <exclude body1="base_link" body2="leg_right_1_link" />
+        <exclude body1="base_link" body2="leg_right_2_link" />
+        <exclude body1="base_link" body2="leg_right_3_link" />
+        <exclude body1="base_link" body2="leg_right_femur_link" />
+        <exclude body1="base_link" body2="leg_left_femur_link" />
+        <exclude body1="back_handle" body2="leg_left_1_link"/>
+        <exclude body1="back_handle" body2="leg_left_2_link"/>
+        <exclude body1="back_handle" body2="leg_right_1_link"/>
+        <exclude body1="back_handle" body2="leg_right_2_link"/>
+        <exclude body1="torso_link" body2="leg_left_1_link"/>
+        <exclude body1="torso_link" body2="leg_left_2_link"/>
+        <exclude body1="torso_link" body2="leg_right_1_link"/>
+        <exclude body1="torso_link" body2="leg_right_2_link"/>
         <exclude body1="leg_left_1_link" body2="leg_right_1_link" />
-        <exclude body1="leg_right_femur_link" body2="base_link" />
-        <exclude body1="leg_left_femur_link" body2="base_link" />
         <exclude body1="leg_left_1_link" body2="leg_left_3_link" />
         <exclude body1="leg_left_2_link" body2="leg_left_3_link" />
@@ -44,7 +72,4 @@
         <exclude body1="leg_left_knee_link" body2="leg_left_5_link" />
         <exclude body1="leg_left_4_link" body2="leg_left_5_link" />
-        <exclude body1="base_link" body2="leg_right_1_link" />
-        <exclude body1="base_link" body2="leg_right_2_link" />
-        <exclude body1="base_link" body2="leg_right_3_link" />
         <exclude body1="leg_right_1_link" body2="leg_right_3_link" />
         <exclude body1="leg_right_2_link" body2="leg_right_3_link" />

File: kangaroo_description/robots/kangaroo.urdf.xacro (robot description, xacro)
@@ -24,5 +24,5 @@
   <!-- cover, no-end-effector, fake-forearm, (ft-gripper) not available, gripper, RH8D -->
   <xacro:arg name="end_effector_type" default="fake-forearm" />
-  <!-- crane, fixed, floating -->
+  <!-- fixed, floating -->
   <xacro:arg name="fixation_type" default="floating" />
   <!-- world name defined in pal_mujoco_scenes package -->
@@ -76,4 +76,7 @@
     <xacro:wrong_mj_control />
   </xacro:if>
+  <xacro:if value="${fixation_type not in ['fixed', 'floating']}">
+    <xacro:wrong_fixation_type />
+  </xacro:if>
   <xacro:if value="${collision_type not in ['mesh', 'capsule']}">
     <xacro:wrong_collision_type />
@@ -130,8 +133,4 @@
   <!-- Base -->
   <xacro:include filename="$(find kangaroo_description)/urdf/base/base.urdf.xacro"/>
-  <!-- Crane -->
-  <xacro:if value="${fixation_type == 'crane'}">
-    <xacro:include filename="$(find kangaroo_description)/urdf/crane/crane.urdf.xacro" />
-  </xacro:if>
   <!-- Legs -->
   <xacro:include filename="$(find kangaroo_description)/urdf/leg/leg.urdf.xacro" />
@@ -156,19 +155,4 @@
   <!-- BASE, PELVIS, TORSO -->
   <xacro:base_link has_pelvis="${has_pelvis}"/>
-  <!-- Fixed Base Link crane, fixed, floating -->
-   <!-- <xacro:if value="${fixation_type == 'fixed'}">
-    <link name="world"/>
-    <joint name="world_base_link" type="fixed">
-      <origin xyz="0.0 0.0 1.2" rpy="0.0  0.0  0.0"/>
-      <parent link="world" />
-      <child link="base_link" />
-    </joint>
-  </xacro:if> -->
-  <xacro:unless value="${fixation_type == 'fixed'}">
-    <xacro:if value="${fixation_type == 'crane'}">
-      <!-- Crane -->
-      <xacro:crane parent="base_link"/>
-    </xacro:if>
-  </xacro:unless>
   <!-- LEGS -->
   <xacro:if value="${legs_type in ['leg', 'ft-leg']}">
@@ -359,4 +343,7 @@
         <!-- <modify_element type="joint" name="joint1" frictionloss="1.0" damping="2.0"/>
         <modify_element type="body" name="forearm" gravcomp="1.0"/> -->
+        <xacro:if value="${fixation_type == 'fixed'}">
+          <modify_element type="body" name="base_link" pos="0 0 1.2" quat="1 0 0 0" />
+        </xacro:if>
       </processed_inputs>
     </mujoco_inputs>

Commit message: Remove legs_type

File: kangaroo_description/mujoco/mj_tags.xacro (robot description, xacro)
@@ -8,83 +8,79 @@
     <!-- Equality -->
     <xacro:macro name="mj_robot_equality">
-      <xacro:if value="${legs_type != 'no-leg'}">
-        <connect anchor="0.0 0.0 0.0" body1="leg_left_4_link" body2="leg_left_knee_link" name="leg_left_closed_kin_joint" solref="0.002 1" />
-        <connect anchor="0.0 0.0 0.0" body1="leg_right_4_link" body2="leg_right_knee_link" name="leg_right_closed_kin_joint" solref="0.002 1" />
-      </xacro:if>
+      <connect anchor="0.0 0.0 0.0" body1="leg_left_4_link" body2="leg_left_knee_link" name="leg_left_closed_kin_joint" solref="0.002 1" />
+      <connect anchor="0.0 0.0 0.0" body1="leg_right_4_link" body2="leg_right_knee_link" name="leg_right_closed_kin_joint" solref="0.002 1" />
     </xacro:macro>
     <!-- Contacts -->
     <xacro:macro name="mj_robot_contacts">
-      <xacro:if value="${legs_type != 'no-leg'}">
-        <xacro:if value="${has_pelvis}">
-          <exclude body1="pelvis_base_link" body2="base_link" />
-          <exclude body1="pelvis_base_link" body2="back_handle" />
-          <exclude body1="pelvis_base_link" body2="leg_left_1_link" />
-          <exclude body1="pelvis_base_link" body2="leg_left_2_link" />
-          <exclude body1="pelvis_base_link" body2="leg_right_1_link" />
-          <exclude body1="pelvis_base_link" body2="leg_right_2_link" />
-          <exclude body1="pelvis_1_link" body2="base_link" />
-          <exclude body1="pelvis_1_link" body2="back_handle" />
-          <exclude body1="pelvis_1_link" body2="pelvis_base_link" />
-          <exclude body1="pelvis_1_link" body2="leg_left_1_link" />
-          <exclude body1="pelvis_1_link" body2="leg_left_2_link" />
-          <exclude body1="pelvis_1_link" body2="leg_right_1_link" />
-          <exclude body1="pelvis_1_link" body2="leg_right_2_link" />
-          <exclude body1="pelvis_2_link" body2="base_link" />
-          <exclude body1="pelvis_2_link" body2="back_handle" />
-          <exclude body1="pelvis_2_link" body2="pelvis_base_link" />
-          <exclude body1="pelvis_2_link" body2="pelvis_1_link" />
-          <exclude body1="pelvis_2_link" body2="leg_left_1_link" />
-          <exclude body1="pelvis_2_link" body2="leg_left_2_link" />
-          <exclude body1="pelvis_2_link" body2="leg_right_1_link" />
-          <exclude body1="pelvis_2_link" body2="leg_right_2_link" />
-        </xacro:if>
-        <exclude body1="base_link" body2="back_handle" />
-        <exclude body1="base_link" body2="torso_link" />
-        <exclude body1="base_link" body2="leg_left_1_link" />
-        <exclude body1="base_link" body2="leg_left_2_link" />
-        <exclude body1="base_link" body2="leg_left_3_link" />
-        <exclude body1="base_link" body2="leg_right_1_link" />
-        <exclude body1="base_link" body2="leg_right_2_link" />
-        <exclude body1="base_link" body2="leg_right_3_link" />
-        <exclude body1="base_link" body2="leg_right_femur_link" />
-        <exclude body1="base_link" body2="leg_left_femur_link" />
-        <exclude body1="back_handle" body2="leg_left_1_link"/>
-        <exclude body1="back_handle" body2="leg_left_2_link"/>
-        <exclude body1="back_handle" body2="leg_right_1_link"/>
-        <exclude body1="back_handle" body2="leg_right_2_link"/>
-        <exclude body1="torso_link" body2="leg_left_1_link"/>
-        <exclude body1="torso_link" body2="leg_left_2_link"/>
-        <exclude body1="torso_link" body2="leg_right_1_link"/>
-        <exclude body1="torso_link" body2="leg_right_2_link"/>
-        <exclude body1="leg_left_1_link" body2="leg_right_1_link" />
-        <exclude body1="leg_left_1_link" body2="leg_left_3_link" />
-        <exclude body1="leg_left_2_link" body2="leg_left_3_link" />
-        <exclude body1="leg_left_2_link" body2="leg_left_1_link" />
-        <exclude body1="leg_left_3_link" body2="leg_left_4_link" />
-        <exclude body1="leg_left_3_link" body2="leg_left_5_link" />
-        <exclude body1="leg_left_3_link" body2="leg_left_knee_link" />
-        <exclude body1="leg_left_femur_link" body2="leg_left_3_link" />
-        <exclude body1="leg_left_femur_link" body2="leg_left_1_link" />
-        <exclude body1="leg_left_femur_link" body2="leg_left_knee_link" />
-        <exclude body1="leg_left_femur_link" body2="leg_left_4_link" />
-        <exclude body1="leg_left_femur_link" body2="leg_left_5_link" />
-        <exclude body1="leg_left_knee_link" body2="leg_left_4_link" />
-        <exclude body1="leg_left_knee_link" body2="leg_left_5_link" />
-        <exclude body1="leg_left_4_link" body2="leg_left_5_link" />
-        <exclude body1="leg_right_1_link" body2="leg_right_3_link" />
-        <exclude body1="leg_right_2_link" body2="leg_right_3_link" />
-        <exclude body1="leg_right_2_link" body2="leg_right_1_link" />
-        <exclude body1="leg_right_3_link" body2="leg_right_4_link" />
-        <exclude body1="leg_right_3_link" body2="leg_right_5_link" />
-        <exclude body1="leg_right_3_link" body2="leg_right_knee_link" />
-        <exclude body1="leg_right_femur_link" body2="leg_right_3_link" />
-        <exclude body1="leg_right_femur_link" body2="leg_right_1_link" />
-        <exclude body1="leg_right_femur_link" body2="leg_right_knee_link" />
-        <exclude body1="leg_right_femur_link" body2="leg_right_4_link" />
-        <exclude body1="leg_right_femur_link" body2="leg_right_5_link" />
-        <exclude body1="leg_right_knee_link" body2="leg_right_4_link" />
-        <exclude body1="leg_right_knee_link" body2="leg_right_5_link" />
-        <exclude body1="leg_right_4_link" body2="leg_right_5_link" />
+      <xacro:if value="${has_pelvis}">
+        <exclude body1="pelvis_base_link" body2="base_link" />
+        <exclude body1="pelvis_base_link" body2="back_handle" />
+        <exclude body1="pelvis_base_link" body2="leg_left_1_link" />
+        <exclude body1="pelvis_base_link" body2="leg_left_2_link" />
+        <exclude body1="pelvis_base_link" body2="leg_right_1_link" />
+        <exclude body1="pelvis_base_link" body2="leg_right_2_link" />
+        <exclude body1="pelvis_1_link" body2="base_link" />
+        <exclude body1="pelvis_1_link" body2="back_handle" />
+        <exclude body1="pelvis_1_link" body2="pelvis_base_link" />
+        <exclude body1="pelvis_1_link" body2="leg_left_1_link" />
+        <exclude body1="pelvis_1_link" body2="leg_left_2_link" />
+        <exclude body1="pelvis_1_link" body2="leg_right_1_link" />
+        <exclude body1="pelvis_1_link" body2="leg_right_2_link" />
+        <exclude body1="pelvis_2_link" body2="base_link" />
+        <exclude body1="pelvis_2_link" body2="back_handle" />
+        <exclude body1="pelvis_2_link" body2="pelvis_base_link" />
+        <exclude body1="pelvis_2_link" body2="pelvis_1_link" />
+        <exclude body1="pelvis_2_link" body2="leg_left_1_link" />
+        <exclude body1="pelvis_2_link" body2="leg_left_2_link" />
+        <exclude body1="pelvis_2_link" body2="leg_right_1_link" />
+        <exclude body1="pelvis_2_link" body2="leg_right_2_link" />
       </xacro:if>
+      <exclude body1="base_link" body2="back_handle" />
+      <exclude body1="base_link" body2="torso_link" />
+      <exclude body1="base_link" body2="leg_left_1_link" />
+      <exclude body1="base_link" body2="leg_left_2_link" />
+      <exclude body1="base_link" body2="leg_left_3_link" />
+      <exclude body1="base_link" body2="leg_right_1_link" />
+      <exclude body1="base_link" body2="leg_right_2_link" />
+      <exclude body1="base_link" body2="leg_right_3_link" />
+      <exclude body1="base_link" body2="leg_right_femur_link" />
+      <exclude body1="base_link" body2="leg_left_femur_link" />
+      <exclude body1="back_handle" body2="leg_left_1_link"/>
+      <exclude body1="back_handle" body2="leg_left_2_link"/>
+      <exclude body1="back_handle" body2="leg_right_1_link"/>
+      <exclude body1="back_handle" body2="leg_right_2_link"/>
+      <exclude body1="torso_link" body2="leg_left_1_link"/>
+      <exclude body1="torso_link" body2="leg_left_2_link"/>
+      <exclude body1="torso_link" body2="leg_right_1_link"/>
+      <exclude body1="torso_link" body2="leg_right_2_link"/>
+      <exclude body1="leg_left_1_link" body2="leg_right_1_link" />
+      <exclude body1="leg_left_1_link" body2="leg_left_3_link" />
+      <exclude body1="leg_left_2_link" body2="leg_left_3_link" />
+      <exclude body1="leg_left_2_link" body2="leg_left_1_link" />
+      <exclude body1="leg_left_3_link" body2="leg_left_4_link" />
+      <exclude body1="leg_left_3_link" body2="leg_left_5_link" />
+      <exclude body1="leg_left_3_link" body2="leg_left_knee_link" />
+      <exclude body1="leg_left_femur_link" body2="leg_left_3_link" />
+      <exclude body1="leg_left_femur_link" body2="leg_left_1_link" />
+      <exclude body1="leg_left_femur_link" body2="leg_left_knee_link" />
+      <exclude body1="leg_left_femur_link" body2="leg_left_4_link" />
+      <exclude body1="leg_left_femur_link" body2="leg_left_5_link" />
+      <exclude body1="leg_left_knee_link" body2="leg_left_4_link" />
+      <exclude body1="leg_left_knee_link" body2="leg_left_5_link" />
+      <exclude body1="leg_left_4_link" body2="leg_left_5_link" />
+      <exclude body1="leg_right_1_link" body2="leg_right_3_link" />
+      <exclude body1="leg_right_2_link" body2="leg_right_3_link" />
+      <exclude body1="leg_right_2_link" body2="leg_right_1_link" />
+      <exclude body1="leg_right_3_link" body2="leg_right_4_link" />
+      <exclude body1="leg_right_3_link" body2="leg_right_5_link" />
+      <exclude body1="leg_right_3_link" body2="leg_right_knee_link" />
+      <exclude body1="leg_right_femur_link" body2="leg_right_3_link" />
+      <exclude body1="leg_right_femur_link" body2="leg_right_1_link" />
+      <exclude body1="leg_right_femur_link" body2="leg_right_knee_link" />
+      <exclude body1="leg_right_femur_link" body2="leg_right_4_link" />
+      <exclude body1="leg_right_femur_link" body2="leg_right_5_link" />
+      <exclude body1="leg_right_knee_link" body2="leg_right_4_link" />
+      <exclude body1="leg_right_knee_link" body2="leg_right_5_link" />
+      <exclude body1="leg_right_4_link" body2="leg_right_5_link" />
     </xacro:macro>
     <!-- Actuators -->
@@ -152,5 +148,5 @@
           <motor joint="arm_right_7_joint" ctrllimited="true" ctrlrange="-43 43" name="arm_right_7_actuator_motor" />
         </xacro:if>
-        <xacro:if value="${mj_control == 'position' and legs_type != 'no-leg'}">
+        <xacro:if value="${mj_control == 'position'}">
           <position joint="leg_left_1_joint" kp="1000" ctrllimited="true" ctrlrange="-0.261799 0.698132" name="leg_left_1_actuator_position" />
           <position joint="leg_left_2_joint" kp="1000" ctrllimited="true" ctrlrange="-0.741765 0.741765" name="leg_left_2_actuator_position" />
@@ -166,5 +162,5 @@
           <position joint="leg_right_5_joint" kp="1000" ctrllimited="true" ctrlrange="-0.471239 0.471239" name="leg_right_5_actuator_position" />
         </xacro:if>
-        <xacro:if value="${mj_control == 'motor' and legs_type != 'no-leg'}">
+        <xacro:if value="${mj_control == 'motor'}">
           <motor joint="leg_left_1_joint" ctrllimited="true" ctrlrange="-80 80" name="leg_left_1_actuator_motor" />
           <motor joint="leg_left_2_joint" ctrllimited="true" ctrlrange="-230 230" name="leg_left_2_actuator_motor" />
@@ -246,30 +242,22 @@
     </xacro:if>
     <!-- legs positions -->
-    <xacro:unless value="${legs_type == 'no-leg'}">
-      <xacro:property name="leg_left_pose"
-        value="0 0.05 0
-              0.6
-              -0.07 0"/>
-      <!-- value="-0.012 0.054 0.04
-              0.6
-             -0.053 0" /> -->
-      <xacro:property name="leg_left_passive_pose"
-      value="0.9 1.8" />
-      <xacro:property name="leg_right_pose"
+    <xacro:property name="leg_left_pose"
       value="0 0.05 0
-              0.6
-              -0.07 0"/>
-      <!-- value="0.012 0.054 -0.04
-              0.6
-             -0.053 0" /> -->
-      <xacro:property name="leg_right_passive_pose"
-      value="0.9 1.8" />
-    </xacro:unless>
-    <xacro:if value="${legs_type == 'no-leg'}">
-      <xacro:property name="leg_left_pose" value="" />
-      <xacro:property name="leg_left_passive_pose" value="" />
-      <xacro:property name="leg_right_pose" value="" />
-      <xacro:property name="leg_right_passive_pose" value="" />
-    </xacro:if>
+            0.6
+            -0.07 0"/>
+    <!-- value="-0.012 0.054 0.04
+            0.6
+            -0.053 0" /> -->
+    <xacro:property name="leg_left_passive_pose"
+    value="0.9 1.8" />
+    <xacro:property name="leg_right_pose"
+    value="0 0.05 0
+            0.6
+            -0.07 0"/>
+    <!-- value="0.012 0.054 -0.04
+            0.6
+            -0.053 0" /> -->
+    <xacro:property name="leg_right_passive_pose"
+    value="0.9 1.8" />
     <!-- End effector pose -->
     <xacro:unless value="${end_effector_type in ['RH8D', 'gripper']}">

Commit message: Add end effectors sides on mujoco tags

File: kangaroo_description/mujoco/mj_tags.xacro (robot description, xacro)
@@ -260,16 +260,29 @@
     <xacro:property name="leg_right_passive_pose"
     value="0.9 1.8" />
-    <!-- End effector pose -->
-    <xacro:unless value="${end_effector_type in ['RH8D', 'gripper']}">
-      <xacro:property name="end_effector_actuator_pose" value="" />
-      <xacro:property name="end_effector_pose" value="" />
-    </xacro:unless>
-    <xacro:if value="${end_effector_type == 'RH8D'}">
-      <xacro:mj_hand_actuator_pose property_name="end_effector_actuator_pose"/>
-      <xacro:mj_hand_pose property_name="end_effector_pose"/>
-    </xacro:if>
-    <xacro:if value="${end_effector_type == 'gripper'}">
-      <xacro:mj_gripper_actuator_pose property_name="end_effector_actuator_pose"/>
-      <xacro:mj_gripper_pose property_name="end_effector_pose"/>
+    <!-- End effector pose right -->
+    <xacro:unless value="${end_effector_right in ['RH8D', 'gripper']}">
+      <xacro:property name="end_effector_right_actuator_pose" value="" />
+      <xacro:property name="end_effector_right_pose" value="" />
+    </xacro:unless>
+    <xacro:if value="${end_effector_right == 'RH8D'}">
+      <xacro:mj_hand_actuator_pose property_name="end_effector_right_actuator_pose"/>
+      <xacro:mj_hand_pose property_name="end_effector_right_pose"/>
+    </xacro:if>
+    <xacro:if value="${end_effector_right == 'gripper'}">
+      <xacro:mj_gripper_actuator_pose property_name="end_effector_right_actuator_pose"/>
+      <xacro:mj_gripper_pose property_name="end_effector_right_pose"/>
+    </xacro:if>
+    <!-- End effector pose left -->
+    <xacro:unless value="${end_effector_left in ['RH8D', 'gripper']}">
+      <xacro:property name="end_effector_left_actuator_pose" value="" />
+      <xacro:property name="end_effector_left_pose" value="" />
+    </xacro:unless>
+    <xacro:if value="${end_effector_left == 'RH8D'}">
+      <xacro:mj_hand_actuator_pose property_name="end_effector_left_actuator_pose"/>
+      <xacro:mj_hand_pose property_name="end_effector_left_pose"/>
+    </xacro:if>
+    <xacro:if value="${end_effector_left == 'gripper'}">
+      <xacro:mj_gripper_actuator_pose property_name="end_effector_left_actuator_pose"/>
+      <xacro:mj_gripper_pose property_name="end_effector_left_pose"/>
     </xacro:if>
     <!-- Keyframe Home using position actuators-->
@@ -283,13 +296,13 @@
             ${leg_left_pose}
             ${leg_right_pose}
-            ${end_effector_actuator_pose}
-            ${end_effector_actuator_pose}"
+            ${end_effector_right_actuator_pose}
+            ${end_effector_left_actuator_pose}"
           qpos="
             ${floating_base_pose}
             ${pelvis_pose}
             ${arm_left_pose}
-            ${end_effector_pose}
+            ${end_effector_left_pose}
             ${arm_right_pose}
-            ${end_effector_pose}
+            ${end_effector_right_pose}
             ${leg_left_pose}
             ${leg_left_passive_pose}
@@ -306,7 +319,7 @@
               ${pelvis_pose}
               ${arm_left_pose}
-              ${end_effector_pose}
+              ${end_effector_left_pose}
               ${arm_right_pose}
-              ${end_effector_pose}
+              ${end_effector_right_pose}
               ${leg_left_pose}
               ${leg_left_passive_pose}
