Commit message: (fix) correct torso position w.r.t. base link

File: kangaroo_description/urdf/torso/torso.urdf.xacro (robot description, xacro)
@@ -36,5 +36,5 @@
   </link>
   <joint name="torso_link" type="fixed">
-    <origin xyz="-0.0918000000000001 0 0.0175" rpy="0 0 0" />
+    <origin xyz="-0.0918000000000001 0 0.0075" rpy="0 0 0" />
     <parent link="${parent}" />
     <child link="torso_link" />

Commit message: add torso cameras

File: kangaroo_description/urdf/torso/torso.urdf.xacro (robot description, xacro)
@@ -11,5 +11,5 @@
   <!-- <xacro:include filename="$(find kangaroo_description)/urdf/deg_to_rad.xacro" />
   <xacro:include filename="$(find kangaroo_description)/urdf/collision.xacro" /> -->
-  <!-- <xacro:include filename="$(find realsense2_description)/urdf/_d435.urdf.xacro" /> -->
+  <xacro:include filename="$(find pal_urdf_utils)/urdf/camera/realsense_d435i.urdf.xacro"/>
   <xacro:macro name="kangaroo_torso" params="parent *origin">
   <link name="torso_link">
@@ -53,24 +53,18 @@
     <child link="torso_link" />
   </joint>
-  <!-- Torso front rgbd camera -->
-    <!-- <xacro:sensor_d435
-      name="torso_front_rgbd_camera"
-      parent="torso_link"
-      topics_ns="torso_front_rgbd_camera"
-      use_nominal_extrinsics="${simulation}">
-      <origin
-        xyz="0.1056 0 0.40767"
-        rpy="0 0.5236 0"/>
-    </xacro:sensor_d435> -->
-  <!-- Torso back rgbd camera -->
-    <!-- <xacro:sensor_d435
-      name="torso_back_rgbd_camera"
-      parent="torso_link"
-      topics_ns="torso_back_rgbd_camera"
-      use_nominal_extrinsics="${simulation}">
-      <origin
-        xyz="-0.1056 0 0.40767"
-        rpy="0 0.5236 ${180.0*deg_to_rad}"/>
-    </xacro:sensor_d435> -->
+  <!-- Torso front cameras -->
+  <xacro:realsense_d435i name="torso_front_roof_rgbd_camera"  parent="torso_link" use_nominal_extrinsics="false">
+      <origin xyz="0.1056 0 0.40767" rpy="0 0.5236 0"/>
+  </xacro:realsense_d435i>
+  <xacro:realsense_d435i name="torso_front_base_rgbd_camera"  parent="torso_link" use_nominal_extrinsics="false">
+    <origin xyz="0.095041 0 0.186487" rpy="0 1.0472 0"/>
+  </xacro:realsense_d435i>
+  <!-- Torso back cameras -->
+  <xacro:realsense_d435i name="torso_back_roof_rgbd_camera"  parent="torso_link" use_nominal_extrinsics="false">
+    <origin xyz="-0.1056 0 0.40767" rpy="0 0.5236 3.14159"/>
+  </xacro:realsense_d435i>
+  <xacro:realsense_d435i name="torso_back_base_rgbd_camera"  parent="torso_link" use_nominal_extrinsics="false">
+    <origin xyz="-0.095041 0 0.186487" rpy="0 1.0472 3.14159"/>
+  </xacro:realsense_d435i>
   </xacro:macro>
 </robot>

Commit message: added properties to make it compatible with last changes of pal_urdf_utils

File: kangaroo_description/urdf/torso/torso.urdf.xacro (robot description, xacro)
@@ -13,4 +13,6 @@
   <xacro:include filename="$(find pal_urdf_utils)/urdf/camera/realsense_d435i.urdf.xacro"/>
   <xacro:macro name="kangaroo_torso" params="parent *origin">
+  <xacro:property name="gazebo_version" value="classic"/>
+  <xacro:property name="namespace" value=""/>
   <link name="torso_link">
     <inertial>
@@ -53,5 +55,5 @@
     <child link="torso_link" />
   </joint>
-  <!-- Torso front cameras -->
+  <!-- Torso back cameras -->
   <xacro:realsense_d435i name="torso_front_roof_rgbd_camera"  parent="torso_link" use_nominal_extrinsics="false">
       <origin xyz="0.1056 0 0.40767" rpy="0 0.5236 0"/>

Commit message: Update torso link mass and inertial properties

File: kangaroo_description/urdf/torso/torso.urdf.xacro (robot description, xacro)
@@ -14,16 +14,8 @@
   <link name="torso_link">
     <inertial>
-      <origin
-        xyz="-0.01 -0.00074 0.22222"
-        rpy="0 0 0" />
-      <mass
-        value="13.33642" />
-      <inertia
-        ixx="0.28794"
-        ixy="-0.00047"
-        ixz="-0.00161"
-        iyy="0.26647"
-        iyz="0.00368"
-        izz="0.11215" />
+      <mass value="15.1027"/>
+      <origin xyz="-0.008953 0.001581 0.216619" rpy="0 0 0"/>
+      <inertia ixx="0.342263" ixy="-0.000525" ixz="-0.00056"
+        iyy="0.31113" iyz="0.002265" izz="0.128871"/>
     </inertial>
     <visual>
