Commit message: update pelvis_link mass and inertial parameters

File: kangaroo_description/urdf/pelvis/pelvis.urdf.xacro (robot description, xacro)
@@ -6,13 +6,8 @@
     <link name="${name}_base_link">
       <inertial>
-        <origin xyz="-0.020292 -0.000245 0.050005" rpy="0 0 0" />
-        <mass value="1.823847" />
-        <inertia
-          ixx="0.001676"
-          ixy="1.9E-05"
-          ixz="-0.000138"
-          iyy="0.007958"
-          iyz="-1.2E-05"
-          izz="0.00789" />
+        <mass value="1.610614"/>
+        <origin xyz="-0.019996 -0.000002 0.003623" rpy="0 0 0"/>
+        <inertia ixx="0.006767" ixy="0" ixz="-0.000146"
+          iyy="0.006367" iyz="0" izz="0.003838"/>
       </inertial>
       <visual>
@@ -82,13 +77,8 @@
     <link name="${name}_2_link">
       <inertial>
-        <origin xyz="0 0 -0.011136" rpy="0 0 0" />
-        <mass value="0.435922" />
-        <inertia
-          ixx="0.000633"
-          ixy="-1.1E-05"
-          ixz="0"
-          iyy="0.000672"
-          iyz="0"
-          izz="0.001275" />
+        <mass value="0.438705"/>
+        <origin xyz="0 0 -0.011237" rpy="0 0 0"/>
+        <inertia ixx="0.000637" ixy="0.000011" ixz="0"
+          iyy="0.000676" iyz="0" izz="0.001283"/>
       </inertial>
       <visual>

Commit message: Fix pelvis 1 axis

File: kangaroo_description/urdf/pelvis/pelvis.urdf.xacro (robot description, xacro)
@@ -68,5 +68,5 @@
       <parent link="${name}_base_link" />
       <child link="${name}_1_link" />
-      <axis xyz="0 0 -1" />
+      <axis xyz="0 0 1" />
       <limit
         lower="-0.3490658504"

Commit message: Fix the pelvis axis to maintain consistency with ROS 1

File: kangaroo_description/urdf/pelvis/pelvis.urdf.xacro (robot description, xacro)
@@ -68,5 +68,5 @@
       <parent link="${name}_base_link" />
       <child link="${name}_1_link" />
-      <axis xyz="0 0 1" />
+      <axis xyz="0 0 -1" />
       <limit
         lower="-0.3490658504"

File: kangaroo_description/urdf/pelvis/ros2_control.urdf.xacro (robot description, xacro)
@@ -23,5 +23,5 @@
       <xacro:kangaroo_pelvis_differential_transmission name="pelvis" number1="1" number2="2"
         act_reduction1="1.0" act_reduction2="1.0"
-        jnt_reduction1="1.0" jnt_reduction2="1.395348837" />
+        jnt_reduction1="-1.0" jnt_reduction2="1.395348837" />
     </xacro:if>
   </xacro:macro>
